File: PowerDistribution/timmi-powerdistribution/timmi-powerdistribution.kicad_sch (KiCad schematic)
At the start: 50 parts

Commit message: Removed Hall Sensors
Parts:
- removed C? (x2): 1000pF, powerDistribution:C0603, symbol powerDistribution-eagle-import:C-USC0603
- removed C? (x2): 0.1uF, powerDistribution:C0603, symbol powerDistribution-eagle-import:C-USC0603
- removed R? (x4): 39k, powerDistribution:R0603, symbol powerDistribution-eagle-import:R-US_R0603
- removed R? (x4): 20k, powerDistribution:R0603, symbol powerDistribution-eagle-import:R-US_R0603
- removed R? (x2): 100, powerDistribution:R0603, symbol powerDistribution-eagle-import:R-US_R0603
- removed U? (x2): CQ2065, powerDistribution:974-1092-1, symbol powerDistribution-eagle-import:CQ2065
- removed XF? (x2): 40A, powerDistribution:3550, symbol powerDistribution-eagle-import:3550(2)
Other:
- note removed: "0.1%"
- note removed: "Hall Effect Current Sensors"
