File: 500g/Therap-i/Schematic/Schematic.kicad_sch (KiCad schematic)
At the start: 1 part, among them U1 Teensy4.1

Commit message: STarted schematic
Parts:
- added TC78H653FTG1: ~, symbol Motordriver:Motordriver
Connections:
- new net +12V: TC78H653FTG1.14 (VM)
- new net GND: TC78H653FTG1.13 (GND)
Other:
- note added: "Motor Drivers"
- note added: "Teensy Microcontroller"
- moved on the sheet: U1
Changed lines of the file:
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@@
 (kicad_sch (version 20230121) (generator eeschema)
   (paper "A4")
-  (symbol (lib_id "teensy:Teensy4.1") (at 143.51 116.84 0) (unit 1)
+  (bus (pts (xy 95.25 154.94) (xy 95.25 104.14))
+    (stroke (width 0) (type default))
+  )
+  (bus (pts (xy 16.51 104.14) (xy 16.51 154.94))
+    (stroke (width 0) (type default))
+  )
+  (bus (pts (xy 96.52 16.51) (xy 177.8 16.51))
+    (stroke (width 0) (type default))
+  )
+  (wire (pts (xy 74.93 25.4) (xy 74.93 38.1))
+    (stroke (width 0) (type default))
+  )
+  (wire (pts (xy 55.88 29.21) (xy 55.88 22.86))
+    (stroke (width 0) (type default))
+  )
+  (wire (pts (xy 59.69 25.4) (xy 74.93 25.4))
+    (stroke (width 0) (type default))
+  )
+  (wire (pts (xy 59.69 29.21) (xy 59.69 25.4))
+    (stroke (width 0) (type default))
+  )
+  (bus (pts (xy 177.8 16.51) (xy 177.8 143.51))
+    (stroke (width 0) (type default))
+  )
+  (bus (pts (xy 95.25 17.78) (xy 95.25 101.6))
+    (stroke (width 0) (type default))
+  )
+  (bus (pts (xy 16.51 17.78) (xy 16.51 101.6))
+    (stroke (width 0) (type default))
+  )
+  (bus (pts (xy 95.25 17.78) (xy 16.51 17.78))
+    (stroke (width 0) (type default))
+  )
+  (bus (pts (xy 16.51 154.94) (xy 95.25 154.94))
+    (stroke (width 0) (type default))
+  )
+  (wire (pts (xy 55.88 22.86) (xy 67.31 22.86))
+    (stroke (width 0) (type default))
+  )
+  (bus (pts (xy 16.51 101.6) (xy 95.25 101.6))
+    (stroke (width 0) (type default))
+  )
+  (bus (pts (xy 177.8 143.51) (xy 96.52 143.51))
+    (stroke (width 0) (type default))
+  )
+  (bus (pts (xy 96.52 16.51) (xy 96.52 143.51))
+    (stroke (width 0) (type default))
+  )
+  (bus (pts (xy 16.51 104.14) (xy 95.25 104.14))
+    (stroke (width 0) (type default))
+  )
+  (text "Motor Drivers " (at 22.86 25.4 0)
+    (effects (font (size 2 2)) (justify left bottom))
+  )
+  (text "Teensy Microcontroller \n" (at 101.6 21.59 0)
+    (effects (font (size 1.27 1.27)) (justify left bottom))
+  )
+  (symbol (lib_id "power:GND") (at 74.93 38.1 0) (unit 1)
     (in_bom yes) (on_board yes) (dnp no) (fields_autoplaced)
-    (property "Reference" "U1" (at 143.51 50.8 0)
-      (effects (font (size 1.27 1.27)))
-    )
-    (property "Value" "Teensy4.1" (at 143.51 53.34 0)
-      (effects (font (size 1.27 1.27)))
-    )
-    (property "Footprint" "" (at 133.35 106.68 0)
-      (effects (font (size 1.27 1.27)) hide)
-    )
-    (property "Datasheet" "" (at 133.35 106.68 0)
+    (property "Reference" "#PWR02" (at 74.93 44.45 0)
+      (effects (font (size 1.27 1.27)) hide)
+    )
+    (property "Value" "GND" (at 74.93 43.18 0)
+      (effects (font (size 1.27 1.27)))
+    )
+    (property "Footprint" "" (at 74.93 38.1 0)
+      (effects (font (size 1.27 1.27)) hide)
+    )
+    (property "Datasheet" "" (at 74.93 38.1 0)
+      (effects (font (size 1.27 1.27)) hide)
+    )
+    (pin "1")
+    (instances
+      (project "Schematic"
+        (path "/91e90b3f-7b4c-476f-99fe-bef9ebae8203"
+          (reference "#PWR02") (unit 1)
+        )
+      )
+    )
+  )
+  (symbol (lib_id "teensy:Teensy4.1") (at 137.16 100.33 0) (unit 1)
+    (in_bom yes) (on_board yes) (dnp no) (fields_autoplaced)
+    (property "Reference" "U1" (at 137.16 34.29 0)
+      (effects (font (size 1.27 1.27)))
+    )
+    (property "Value" "Teensy4.1" (at 137.16 36.83 0)
+      (effects (font (size 1.27 1.27)))
+    )
+    (property "Footprint" "" (at 127 90.17 0)
+      (effects (font (size 1.27 1.27)) hide)
+    )
+    (property "Datasheet" "" (at 127 90.17 0)
       (effects (font (size 1.27 1.27)) hide)
     )
@@
         )
       )
+    )
+  )
+  (symbol (lib_id "power:+12V") (at 67.31 22.86 270) (unit 1)
+    (in_bom yes) (on_board yes) (dnp no) (fields_autoplaced)
+    (property "Reference" "#PWR01" (at 63.5 22.86 0)
+      (effects (font (size 1.27 1.27)) hide)
+    )
+    (property "Value" "+12V" (at 71.12 22.86 90)
+      (effects (font (size 1.27 1.27)) (justify left))
+    )
+    (property "Footprint" "" (at 67.31 22.86 0)
+      (effects (font (size 1.27 1.27)) hide)
+    )
+    (property "Datasheet" "" (at 67.31 22.86 0)
+      (effects (font (size 1.27 1.27)) hide)
+    )
+    (pin "1")
+    (instances
+      (project "Schematic"
+        (path "/91e90b3f-7b4c-476f-99fe-bef9ebae8203"
+          (reference "#PWR01") (unit 1)
+        )
+      )
+    )
+  )
+  (symbol (lib_id "Motordriver:Motordriver") (at 50.8 43.18 0) (unit 1)
+    (in_bom yes) (on_board yes) (dnp no)
+    (property "Reference" "TC78H653FTG1" (at 54.61 43.18 0)
+      (effects (font (size 1.27 1.27)))
+    )
+    (property "Value" "~" (at 50.8 43.18 0)
+      (effects (font (size 1.27 1.27)))
+    )
+    (property "Footprint" "" (at 50.8 43.18 0)
+      (effects (font (size 1.27 1.27)) hide)
+    )
+    (property "Datasheet" "" (at 50.8 43.18 0)
+      (effects (font (size 1.27 1.27)) hide)
+    )
+    (pin "1")
+    (pin "10")
+    (pin "11")
+    (pin "12")
+    (pin "13")
+    (pin "14")
+    (pin "15")
+    (pin "16")
+    (pin "2")
+    (pin "3")
+    (pin "4")
+    (pin "5")
+    (pin "6")
+    (pin "7")
+    (pin "8")
+    (pin "9")
+    (instances
+      (project "Schematic"
+        (path "/91e90b3f-7b4c-476f-99fe-bef9ebae8203"
+          (reference "TC78H653FTG1") (unit 1)
+        )
+      )

Commit message: more stuff on pcb
Parts:
- removed TC78H653FTG1: ~, symbol Motordriver:Motordriver
- added C1, C2: 0.1uF, symbol Device:C
- added IC1: TC78H653FTG,EL, QFN50P300X300X90-17N, symbol TC78H653FTG_EL:TC78H653FTG,EL
- added JS200XF1, JS200XF2, JS200XF3, JS200XF4: ~, symbol Sensor_Distance:JS200XF
- added ML2Line1, ML2Line2: ~, symbol Sensor_Distance:ML2_Line
Connections:
- net GND: now also C1.2, C2.2, IC1.15 (LARGE), IC1.16 (MODE), IC1.8 (GND_1), JS200XF1. (Signal), JS200XF2. (Signal), JS200XF3. (Signal), JS200XF4. (Signal), ML2Line1. (Sig2), ML2Line2. (Sig2)
- new net: C1.1, C2.1, IC1.14 (VM)
- new net +5V: JS200XF1. (Signal), JS200XF2. (Signal), JS200XF3. (Signal), JS200XF4. (Signal), ML2Line1. (Sig2), ML2Line2. (Sig2)
Other:
- note added: "IR Sensors"
- note added: "Line Sensors"

Commit message: i tried
Parts:
- removed ML2Line2: ~, symbol Sensor_Distance:ML2_Line
- added ML2Line3: ~, symbol Sensor_Distance:ML2_Line
- added U2, U3: IFX27001TFV50, Package_TO_SOT_SMD:TO-252-3_TabPin2, symbol Regulator_Linear:IFX27001TFV50
Connections:
- net +5V: now also ML2Line3. (Sig_NOR)
- net GND: now also ML2Line3. (Sig_NOR)
- net PIN6: now reaches ML2Line1. (Sig_NOR)
- net PIN6: now also U1.7 (5_IN2)
- net PIN3: now reaches JS200XF3. (Signal)
- net PIN3: now also U1.4 (2_OUT2)
- net PIN1: now reaches U1.2 (0_RX1_CRX2_CS1)
- net PIN1: now also JS200XF1. (Signal)
- net PIN2: now reaches U1.3 (1_TX1_CTX2_MISO1)
- net PIN2: now also JS200XF2. (Signal)
- net PIN4: now reaches U1.5 (3_LRCLK2)
- net PIN4: now also JS200XF4. (Signal)
- net PIN5: now reaches U1.6 (4_BCLK2)
- net PIN5: now also ML2Line3. (Sig_NOR)
Other:
- note added: "Voltage Regulators"

Commit message: Change names
Parts:
- removed JS200XF4: ~, symbol Sensor_Distance:JS200XF
- removed ML2Line1: ~, symbol Sensor_Distance:ML2_Line
- added JS1: JS15878, symbol Start_Module:JS15878
- added JS200XF5: ~, symbol Sensor_Distance:JS200XF
- added ML2Line2: ~, symbol Sensor_Distance:ML2_Line
Connections:
- net +5V: now also JS200XF5. (Signal), ML2Line2. (Sig_NOR)
- net GND: now also JS200XF5. (Signal), ML2Line2. (Sig_NOR)
- net PIN1: no longer JS200XF1. (Signal)
- net PIN2: no longer JS200XF2. (Signal)
- net PIN3: no longer JS200XF3. (Signal)
- net PIN5: now also ML2Line2. (Sig_NOR); no longer ML2Line3. (Sig_NOR)
- net PIN6: now also ML2Line3. (Sig_NOR)
- new net IR1: JS200XF5. (Signal)
- new net IR2: JS200XF1. (Signal)
- new net IR3: JS200XF2. (Signal)
- new net IR4: JS200XF3. (Signal)
Other:
- note added: "Start Module"
- moved on the sheet: U2, U3

Commit message: Yellow
Parts:
- JS15878: renamed from JS1; value JS15878 -> (none)
- JS200XF1, JS200XF2, JS200XF3, JS200XF5, ML2Line2, ML2Line3: value ~ -> (none)
Connections:
- net PIN1 is gone; now on net IR1: U1.2 (0_RX1_CRX2_CS1)
- net PIN2 is gone; now on net IR2: U1.3 (1_TX1_CTX2_MISO1)
- net PIN3 is gone; now on net IR3: U1.4 (2_OUT2)
- net PIN4 is gone; now on net IR4: U1.5 (3_LRCLK2)
- net PIN5 is gone; now on net LN1: ML2Line2. (Sig_NOR), U1.6 (4_BCLK2)
- net PIN6 is gone; now on net LN2: ML2Line3. (Sig_NOR), U1.7 (5_IN2)
- net LN1: now reaches ML2Line2. (Sig_NOR)
- net LN2: now reaches ML2Line3. (Sig_NOR)
Changed lines of the file:
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@@
     (effects (font (size 4 4)) (justify left bottom))
   )
-  (global_label "PIN3" (shape input) (at 104.14 53.34 180) (fields_autoplaced)
-    (effects (font (size 1.27 1.27)) (justify right))
-    (property "Intersheetrefs" "${INTERSHEET_REFS}" (at 96.74 53.34 0)
+  (global_label "IR3" (shape input) (at 104.14 53.34 180) (fields_autoplaced)
+    (effects (font (size 1.27 1.27)) (justify right))
+    (property "Intersheetrefs" "${INTERSHEET_REFS}" (at 98.0705 53.34 0)
       (effects (font (size 1.27 1.27)) (justify right) hide)
     )
@@
     )
   )
-  (global_label "PIN6" (shape input) (at 104.14 60.96 180) (fields_autoplaced)
-    (effects (font (size 1.27 1.27)) (justify right))
-    (property "Intersheetrefs" "${INTERSHEET_REFS}" (at 96.74 60.96 0)
-      (effects (font (size 1.27 1.27)) (justify right) hide)
-    )
-  )
-  (global_label "PIN4" (shape input) (at 104.14 55.88 180) (fields_autoplaced)
-    (effects (font (size 1.27 1.27)) (justify right))
-    (property "Intersheetrefs" "${INTERSHEET_REFS}" (at 96.74 55.88 0)
+  (global_label "LN2" (shape input) (at 104.14 60.96 180) (fields_autoplaced)
+    (effects (font (size 1.27 1.27)) (justify right))
+    (property "Intersheetrefs" "${INTERSHEET_REFS}" (at 97.5867 60.96 0)
+      (effects (font (size 1.27 1.27)) (justify right) hide)
+    )
+  )
+  (global_label "IR4" (shape input) (at 104.14 55.88 180) (fields_autoplaced)
+    (effects (font (size 1.27 1.27)) (justify right))
+    (property "Intersheetrefs" "${INTERSHEET_REFS}" (at 98.0705 55.88 0)
       (effects (font (size 1.27 1.27)) (justify right) hide)
     )
@@
     )
   )
-  (global_label "PIN5" (shape input) (at 33.02 135.89 270) (fields_autoplaced)
-    (effects (font (size 1.27 1.27)) (justify right))
-    (property "Intersheetrefs" "${INTERSHEET_REFS}" (at 33.02 143.29 90)
-      (effects (font (size 1.27 1.27)) (justify right) hide)
-    )
-  )
-  (global_label "PIN6" (shape input) (at 68.58 135.89 270) (fields_autoplaced)
-    (effects (font (size 1.27 1.27)) (justify right))
-    (property "Intersheetrefs" "${INTERSHEET_REFS}" (at 68.58 143.29 90)
-      (effects (font (size 1.27 1.27)) (justify right) hide)
-    )
-  )
-  (global_label "PIN1" (shape input) (at 104.14 48.26 180) (fields_autoplaced)
-    (effects (font (size 1.27 1.27)) (justify right))
-    (property "Intersheetrefs" "${INTERSHEET_REFS}" (at 96.74 48.26 0)
-      (effects (font (size 1.27 1.27)) (justify right) hide)
-    )
-  )
-  (global_label "PIN2" (shape input) (at 104.14 50.8 180) (fields_autoplaced)
-    (effects (font (size 1.27 1.27)) (justify right))
-    (property "Intersheetrefs" "${INTERSHEET_REFS}" (at 96.74 50.8 0)
-      (effects (font (size 1.27 1.27)) (justify right) hide)
-    )
-  )
-  (global_label "PIN5" (shape input) (at 104.14 58.42 180) (fields_autoplaced)
-    (effects (font (size 1.27 1.27)) (justify right))
-    (property "Intersheetrefs" "${INTERSHEET_REFS}" (at 96.74 58.42 0)
+  (global_label "LN1" (shape input) (at 33.02 135.89 270) (fields_autoplaced)
+    (effects (font (size 1.27 1.27)) (justify right))
+    (property "Intersheetrefs" "${INTERSHEET_REFS}" (at 33.02 142.4433 90)
+      (effects (font (size 1.27 1.27)) (justify right) hide)
+    )
+  )
+  (global_label "LN2" (shape input) (at 68.58 135.89 270) (fields_autoplaced)
+    (effects (font (size 1.27 1.27)) (justify right))
+    (property "Intersheetrefs" "${INTERSHEET_REFS}" (at 68.58 142.4433 90)
+      (effects (font (size 1.27 1.27)) (justify right) hide)
+    )
+  )
+  (global_label "IR1" (shape input) (at 104.14 48.26 180) (fields_autoplaced)
+    (effects (font (size 1.27 1.27)) (justify right))
+    (property "Intersheetrefs" "${INTERSHEET_REFS}" (at 98.0705 48.26 0)
+      (effects (font (size 1.27 1.27)) (justify right) hide)
+    )
+  )
+  (global_label "IR2" (shape input) (at 104.14 50.8 180) (fields_autoplaced)
+    (effects (font (size 1.27 1.27)) (justify right))
+    (property "Intersheetrefs" "${INTERSHEET_REFS}" (at 98.0705 50.8 0)
+      (effects (font (size 1.27 1.27)) (justify right) hide)
+    )
+  )
+  (global_label "LN1" (shape input) (at 104.14 58.42 180) (fields_autoplaced)
+    (effects (font (size 1.27 1.27)) (justify right))
+    (property "Intersheetrefs" "${INTERSHEET_REFS}" (at 97.5867 58.42 0)
       (effects (font (size 1.27 1.27)) (justify right) hide)
     )
@@
       (effects (font (size 1.27 1.27)) (justify left))
     )
-    (property "Value" "~" (at 35.56 125.73 0)
+    (property "Value" "" (at 35.56 125.73 0)
       (effects (font (size 1.27 1.27)))
     )
@@
       (effects (font (size 1.27 1.27)) (justify left))
     )
-    (property "Value" "~" (at 264.16 33.02 0)
-      (effects (font (size 1.27 1.27)))
+    (property "Value" "" (at 264.16 33.02 0)
+      (effects (font (size 1.27 1.27)) hide)
     )
     (property "Footprint" "" (at 264.16 33.02 0)
@@
     )
   )
-  (symbol (lib_name "JS200XF_1") (lib_id "Sensor_Distance:JS200XF") (at 238.76 33.02 0) (unit 1)
+  (symbol (lib_name "JS200XF_4") (lib_id "Sensor_Distance:JS200XF") (at 238.76 33.02 0) (unit 1)
     (in_bom yes) (on_board yes) (dnp no) (fields_autoplaced)
     (property "Reference" "JS200XF2" (at 246.38 33.655 0)
       (effects (font (size 1.27 1.27)) (justify left))
     )
-    (property "Value" "~" (at 238.76 33.02 0)
-      (effects (font (size 1.27 1.27)))
+    (property "Value" "" (at 238.76 33.02 0)
+      (effects (font (size 1.27 1.27)) hide)
     )
     (property "Footprint" "" (at 238.76 33.02 0)
@@
     )
   )
-  (symbol (lib_id "Sensor_Distance:ML2_Line") (at 71.12 127 0) (unit 1)
+  (symbol (lib_name "ML2_Line_1") (lib_id "Sensor_Distance:ML2_Line") (at 71.12 127 0) (unit 1)
     (in_bom yes) (on_board yes) (dnp no) (fields_autoplaced)
     (property "Reference" "ML2Line3" (at 81.28 125.095 0)
       (effects (font (size 1.27 1.27)) (justify left))
     )
-    (property "Value" "~" (at 71.12 127 0)
+    (property "Value" "" (at 71.12 127 0)
       (effects (font (size 1.27 1.27)))
     )
@@
     )
   )
-  (symbol (lib_name "JS200XF_1") (lib_id "Sensor_Distance:JS200XF") (at 213.36 33.02 0) (unit 1)
+  (symbol (lib_name "JS200XF_3") (lib_id "Sensor_Distance:JS200XF") (at 213.36 33.02 0) (unit 1)
     (in_bom yes) (on_board yes) (dnp no) (fields_autoplaced)
     (property "Reference" "JS200XF1" (at 220.98 33.655 0)
       (effects (font (size 1.27 1.27)) (justify left))
     )
-    (property "Value" "~" (at 213.36 33.02 0)
-      (effects (font (size 1.27 1.27)))
+    (property "Value" "" (at 213.36 33.02 0)
+      (effects (font (size 1.27 1.27)) hide)
     )
     (property "Footprint" "" (at 213.36 33.02 0)
@@
   (symbol (lib_id "Start_Module:JS15878") (at 31.75 167.64 0) (unit 1)
     (in_bom yes) (on_board yes) (dnp no) (fields_autoplaced)
-    (property "Reference" "JS1" (at 39.37 173.355 0)
-      (effects (font (size 1.27 1.27)) (justify left))
-    )
-    (property "Value" "JS15878" (at 39.37 175.895 0)
-      (effects (font (size 1.27 1.27)) (justify left))
+    (property "Reference" "JS15878" (at 39.37 173.355 0)
+      (effects (font (size 1.27 1.27)) (justify left))
+    )
+    (property "Value" "" (at 39.37 175.895 0)
+      (effects (font (size 1.27 1.27)) (justify left) hide)
     )
     (property "Footprint" "" (at 31.75 167.64 0)
@@
       (project "Schematic"
         (path "/91e90b3f-7b4c-476f-99fe-bef9ebae8203"
-          (reference "JS1") (unit 1)
-        )
-      )
-    )
-  )
-  (symbol (lib_name "JS200XF_1") (lib_id "Sensor_Distance:JS200XF") (at 189.23 33.02 0) (unit 1)
+          (reference "JS15878") (unit 1)
+        )
+      )
+    )
+  )
+  (symbol (lib_name "JS200XF_2") (lib_id "Sensor_Distance:JS200XF") (at 189.23 33.02 0) (unit 1)
     (in_bom yes) (on_board yes) (dnp no) (fields_autoplaced)
     (property "Reference" "JS200XF5" (at 196.85 33.655 0)
       (effects (font (size 1.27 1.27)) (justify left))
     )
-    (property "Value" "~" (at 189.23 33.02 0)
-      (effects (font (size 1.27 1.27)))
+    (property "Value" "" (at 208.28 38.1 0)
+      (effects (font (size 1.27 1.27)) hide)
     )
     (property "Footprint" "" (at 189.23 33.02 0)
