File: 500g/Therap-i/Schematic/Schematic.kicad_pcb (KiCad board)
At the start: 2 copper layers, 34 parts, among them J1 Screw_Terminal_01x03, J10 BDC1, J2 Screw_Terminal_01x03, J3 Screw_Terminal_01x03, J4 Screw_Terminal_01x03, J5 Screw_Terminal_01x03, J6 Screw_Terminal_01x03, J7 Screw_Terminal_01x04, J8 BAT, J9 BDC2, SW1 500SSP1S2M2QEA, U1 Teensy4.1, U2 IFX27001TFV, U3 A4950ELJTR-T, U4 A4950ELJTR-T

Commit message: layout work
Parts:
- moved J6 150.4 mm to (210.7, 51.5), turned to 90 degrees
- moved J5 145.9 mm to (210.7, 66.7), turned to 90 degrees
- moved J4 142.0 mm to (210.7, 82.9), turned to 90 degrees
- moved F1 118.4 mm to (55.9, 61.0), turned to 90 degrees
- moved SW1 116.3 mm to (74.4, 25.4), turned to 90 degrees
- moved C21 112.8 mm to (195.0, 55.9)
- moved C18 103.3 mm to (195.0, 71.1)
- moved C17 96.6 mm to (194.7, 87.9)
- moved C13 91.4 mm to (169.8, 45.7)
- moved C2 89.6 mm to (163.7, 58.4)
- moved J10 89.5 mm to (195.6, 17.8), turned to 90 degrees
- moved J2 85.8 mm to (137.4, 111.8)
- moved C16 82.1 mm to (131.7, 43.2)
- moved R1 81.6 mm to (171.9, 50.8)
- moved J1 79.0 mm to (123.2, 111.8)
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Routing:
- net ST1: track 0.00 -> 100.1 mm
- net GND: track 0.00 -> 97.8 mm
- net LN2: track 0.00 -> 96.9 mm
- net LN1: track 0.00 -> 94.9 mm
- net +12V: track 0.00 -> 93.9 mm
- net +3.3V: track 0.00 -> 91.3 mm
- net VOLT1: track 0.00 -> 53.2 mm
- net IR3: track 0.00 -> 52.1 mm
- net IR2: track 0.00 -> 39.8 mm
- net IR1: track 0.00 -> 35.0 mm
- net Net-(U4-LSS): track 0.00 -> 30.7 mm
- net Net-(U3-LSS): track 0.00 -> 25.4 mm
- net Net-(D1-K): track 0.00 -> 21.5 mm
- net Net-(C16-Pad2): track 0.00 -> 5.79 mm
- net Net-(C13-Pad2): track 0.00 -> 5.45 mm

Commit message: i d k
Parts:
- moved J9 55.4 mm to (126.9, 32.1)
- moved F1 43.8 mm to (99.1, 53.3)
- moved J10 40.8 mm to (157.4, 32.1)
- moved J8 37.8 mm to (96.5, 63.5)
- moved SW1 32.3 mm to (104.1, 38.1), turned to -90 degrees
- moved J7 17.0 mm to (147.3, 22.9)
- moved C16 13.8 mm to (135.9, 56.3), turned to 180 degrees
- moved R2 10.5 mm to (132.1, 58.4), turned to 180 degrees
- moved C4 7.72 mm to (80.6, 86.4)
- moved D1 7.72 mm to (91.2, 88.9)
- moved C3 7.72 mm to (84.5, 88.9)
- moved U2 7.72 mm to (96.5, 78.7)
- moved C5 5.68 mm to (107.8, 94.0)
Routing:
- net BDC12: track 0.00 -> 61.3 mm
- net BDC11: track 0.00 -> 44.5 mm
- net BDC22: track 0.00 -> 39.0 mm
- net BDC21: track 0.00 -> 35.4 mm
- net Net-(J10-Pin_2): track 0.00 -> 31.5 mm
- net Net-(J8-Pin_1): track 0.00 -> 27.1 mm
- net Net-(J9-Pin_2): track 0.00 -> 26.0 mm
- net Net-(J10-Pin_1): track 0.00 -> 21.6 mm
- net Net-(J9-Pin_1): track 0.00 -> 21.5 mm
- net +12V: track 93.9 -> 108.3 mm
- net Net-(U3-LSS): track 25.4 -> 18.0 mm
- net GND: track 97.8 -> 103.6 mm
- net Net-(C16-Pad2): track 5.79 -> 3.45 mm
- net VOLT1: track 53.2 -> 53.9 mm

Commit message: didn't realize it wasnt a screw terminal
Parts:
- J1, J2, J3, J4, J5, J6: footprint Therapi:screw3 -> THERAPI:SCREWTERM3
- moved J6 183.2 mm to (28.4, 33.0), turned to 0 degrees
- moved J5 159.0 mm to (55.5, 32.3), turned to 180 degrees
- moved J4 156.5 mm to (62.5, 32.5), turned to 0 degrees
- moved C18 151.8 mm to (50.1, 26.0), turned to 180 degrees
- moved C17 141.0 mm to (68.0, 26.0), turned to 180 degrees
- moved C21 138.8 mm to (60.9, 20.0)
- moved J1 104.6 mm to (28.4, 67.5)
- moved J2 100.8 mm to (46.9, 67.5)
- moved C5 100.4 mm to (33.9, 26.0), turned to 180 degrees
- moved J3 98.3 mm to (64.0, 67.5)
- moved C19 96.7 mm to (42.6, 65.8), turned to 90 degrees
- moved C9 93.0 mm to (60.5, 65.9), turned to -90 degrees
- moved C10 92.8 mm to (77.9, 65.9), turned to 90 degrees
- moved C13 90.7 mm to (83.1, 19.0)
- moved U1 85.9 mm to (57.5, 50.4)
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Routing:
- net +12V: track 108.3 -> 2.09 mm
- net ST1: track 100.1 -> 0.00 mm
- net LN2: track 96.9 -> 0.00 mm
- net LN1: track 94.9 -> 0.00 mm
- net +3.3V: track 91.3 -> 15.8 mm
- net GND: track 103.6 -> 28.5 mm
- net BDC12: track 61.3 -> 1.83 mm
- net VOLT1: track 53.9 -> 0.00 mm
- net IR3: track 52.1 -> 0.00 mm
- net BDC11: track 44.5 -> 0.47 mm
- net IR2: track 39.8 -> 0.00 mm
- net BDC22: track 39.0 -> 1.47 mm
- net IR1: track 35.0 -> 0.00 mm
- net BDC21: track 35.4 -> 0.47 mm
- net Net-(J10-Pin_2): track 31.5 -> 0.80 mm
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
Commit message: Layout work
Parts:
- C1, C14: footprint Therapi:0.22uF -> THERAPI:0.22uF
- C10, C17, C18, C19, C21, C3, C4, C9: footprint Therapi:100nf -> THERAPI:100NF
- C13, C16: footprint Therapi:1uF -> THERAPI:1uF
- C15, C2, C5: footprint Therapi:100uF -> THERAPI:100uF
- D1: footprint Therapi:diode -> THERAPI:DIODE
- J10, J9: footprint Therapi:screw2 -> THERAPI:SCREW2
- J7: footprint Therapi:4Screwterminal -> THERAPI:SCREWTHIS4; moved to B.Cu
- J8: footprint Therapi:JST -> THERAPI:JSTT
- R1, R2: footprint resistor:RESC1608X55N -> THERAPI:0.25OH
- SW1: footprint Therapi:switch -> THERAPI:SWITCH
- U3, U4: footprint Motordriver:SOIC-8_ALM -> THERAPI:A495; moved to B.Cu
- moved R1 80.5 mm to (91.4, 47.4), turned to -90 degrees
- moved U4 78.8 mm to (81.3, 47.6), turned to 0 degrees
- moved C2 73.5 mm to (90.3, 53.3), turned to 180 degrees
- moved C3 66.1 mm to (81.7, 22.9)
- moved C1 62.9 mm to (91.6, 40.6)
- moved U2 60.3 mm to (43.6, 107.7)
- moved J6 49.2 mm to (77.6, 32.8), turned to 180 degrees
- moved C16 44.7 mm to (91.4, 60.5), turned to 90 degrees
- moved U3 43.3 mm to (81.3, 53.3), turned to 0 degrees
- moved R2 40.7 mm to (91.4, 56.7), turned to 90 degrees
- moved C15 36.6 mm to (90.0, 38.1)
- moved C14 35.4 mm to (91.9, 51.0)
- moved J4 32.0 mm to (30.5, 33.0)
- moved C4 31.2 mm to (73.3, 17.3)
- moved C21 29.0 mm to (32.6, 26.2), turned to 180 degrees
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Connections:
- J7 pad 3: BDC21 -> BDC22
- J7 pad 4: BDC22 -> BDC21
- U1 pad 11: BDC21 -> BDC22
- U1 pad 12: BDC22 -> BDC21
Routing:
- net ST1: track 0.00 -> 37.1 mm
- net BDC11: track 0.47 -> 34.6 mm
- net IR3: track 0.00 -> 33.4 mm
- net +3.3V: track 15.8 -> 47.2 mm
- net BDC12: track 1.83 -> 32.4 mm
- net LN2: track 0.00 -> 28.2 mm
- net LN1: track 0.00 -> 27.9 mm
- net BDC22: track 1.47 -> 27.7 mm
- net BDC21: track 0.47 -> 23.7 mm
- net GND: track 28.5 -> 46.6 mm
- net IR2: track 0.00 -> 17.5 mm
- net +12V: track 2.09 -> 19.3 mm, vias 0 -> 2
- net Net-(J10-Pin_2): track 0.80 -> 16.7 mm
- net Net-(J10-Pin_1): track 0.47 -> 15.7 mm
- net Net-(J9-Pin_1): track 0.47 -> 15.4 mm
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
Commit message: more layout work
Parts:
- C5: value 100µF -> 100nF; footprint THERAPI:100uF -> THERAPI:100NF
- moved U2 77.6 mm to (35.6, 30.5), turned to 180 degrees
- moved C3 62.3 mm to (94.4, 83.8)
- moved C4 58.6 mm to (121.5, 50.8)
- moved SW1 36.2 mm to (82.0, 66.0)
- moved J4 34.5 mm to (64.9, 33.0), turned to 180 degrees
- moved C21 30.5 mm to (63.0, 26.2), turned to 0 degrees
- moved C17 28.1 mm to (103.7, 27.9), turned to -90 degrees
- moved C18 23.0 mm to (78.3, 26.0)
- moved J5 22.9 mm to (81.3, 33.0)
- moved J6 21.6 mm to (99.1, 30.5)
- moved C5 20.8 mm to (30.0, 40.6), turned to 0 degrees
- moved D1 15.5 mm to (81.3, 71.1), turned to 0 degrees
- moved J8 14.8 mm to (101.1, 66.0)
- moved J3 2.54 mm to (63.5, 66.0)
- moved C10 2.54 mm to (70.7, 73.7)
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Routing:
- net ST1: track 37.1 -> 56.4 mm
- net LN2: track 28.2 -> 38.3 mm
- net +12V: track 19.3 -> 24.5 mm
- net LN1: track 27.9 -> 30.7 mm
- net VOLT1: track 0.00 -> 2.70 mm
- net IR3: track 33.4 -> 30.9 mm
- net +3.3V: track 47.2 -> 49.2 mm
- net IR2: track 17.5 -> 16.3 mm
- net GND: track 46.6 -> 45.8 mm

Commit message: layouut5
Parts:
- U2: moved to B.Cu
- moved C4 91.6 mm to (36.0, 17.8)
- moved F1 91.1 mm to (50.8, 32.1)
- moved C3 80.3 mm to (48.7, 17.8)
- moved SW1 60.6 mm to (33.0, 30.5)
- moved J8 59.7 mm to (48.3, 38.1)
- moved D1 58.5 mm to (33.0, 38.1), turned to 90 degrees
- moved U2 18.2 mm to (34.5, 48.7), turned to -90 degrees
Routing:
- net Net-(J8-Pin_1): track 0.00 -> 14.8 mm
- net Net-(D1-K): track 0.00 -> 6.84 mm, vias 0 -> 1
- net +12V: track 24.5 -> 25.8 mm

Commit message: clutched up finish on the pcb
Parts:
- added H1: MountingHole, MountingHole:MountingHole_3mm, F.Cu at (101.0, 70.5)
- added H2: MountingHole, MountingHole:MountingHole_3mm, F.Cu at (28.5, 30.0)
- moved C17 38.8 mm to (96.5, 66.0)
- moved J6 37.8 mm to (91.7, 67.5)
- moved U2 24.0 mm to (55.5, 37.0), turned to 0 degrees
- moved C4 23.7 mm to (45.5, 39.5), turned to 180 degrees
- moved C3 20.0 mm to (45.5, 37.5), turned to 180 degrees
- moved J4 19.1 mm to (84.0, 31.8)
- moved J5 19.1 mm to (100.3, 31.8)
- moved C18 19.1 mm to (97.3, 26.0)
- moved C21 19.0 mm to (82.0, 26.0)
- moved J8 15.9 mm to (62.0, 30.0), turned to 180 degrees
- moved D1 13.3 mm to (46.1, 35.5), turned to 180 degrees
- moved F1 5.50 mm to (55.6, 29.5), turned to 180 degrees
- moved SW1 4.81 mm to (37.6, 29.0)
- moved C5 2.64 mm to (30.0, 38.0)
- moved J3 1.96 mm to (63.5, 68.0)
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Connections:
- SW1 pad 2: unconnected-(SW1-Pad2) -> Net-(J8-Pin_1)
- SW1 pad 3: Net-(J8-Pin_1) -> unconnected-(SW1-Pad3)
Routing:
- net +3.3V: track 49.2 -> 185.7 mm, vias 0 -> 4
- net +12V: track 25.8 -> 104.4 mm
- net VOLT1: track 2.70 -> 35.4 mm, vias 0 -> 1
- net LN2: track 38.3 -> 58.1 mm
- net ST1: track 56.4 -> 39.3 mm
- net LN1: track 30.7 -> 45.5 mm
- net Net-(J8-Pin_1): track 14.8 -> 23.4 mm
- net GND: track 45.8 -> 48.4 mm, vias 0 -> 1
- net BDC12: track 32.4 -> 30.8 mm
- net IR3: track 30.9 -> 31.8 mm
- net Net-(D1-K): track 6.84 -> 6.19 mm
- added copper zone on B.Cu, net GND
- added copper zone on F.Cu, net GND
Other:
- board outline added: 80 x 50 mm
