File: 500g/Frosti/Frosti.kicad_pcb (KiCad board)
At the start: 2 copper layers, 32 parts, among them SW1 SW_SPDT, SW2 SW_SPDT, SW3 SW_SPDT, U10 DRV8871DDA, U12 DRV8871DDA, U14 DEV-16771, U4 DRV8871DDA

Commit message: pcb layout done
Parts:
- removed U16: ~, Package_SO:Zetex_SM8
- added C10: 22uF, Capacitor_SMD:C_0201_0603Metric, F.Cu at (105.1, 53.3)
- added L1: 4.7uH, Inductor_SMD:L_0201_0603Metric, F.Cu at (113.3, 49.5)
- added U17: AP63205WU, Package_TO_SOT_SMD:TSOT-23-6, F.Cu at (113.5, 44.8)
- R1, R2, R3: footprint Resistor_SMD:R_0603_1608Metric -> Resistor_SMD:R_0201_0603Metric
- moved U5 199.6 mm to (176.5, 118.1), turned to 90 degrees
- moved U4 198.3 mm to (168.0, 117.5)
- moved U3 183.7 mm to (177.2, 82.0), turned to -90 degrees
- moved U1 183.4 mm to (165.7, 82.0), turned to -90 degrees
- moved U2 183.3 mm to (171.4, 82.0), turned to -90 degrees
- moved R1 182.2 mm to (164.5, 124.8), turned to -90 degrees
- moved C6 177.5 mm to (173.4, 124.8), turned to -90 degrees
- moved C5 176.3 mm to (168.9, 124.8), turned to -90 degrees
- moved U6 175.1 mm to (176.5, 74.9), turned to 90 degrees
- moved U7 167.0 mm to (170.8, 74.9), turned to 90 degrees
- moved U14 163.2 mm to (139.7, 83.8), turned to 90 degrees
- moved U13 160.9 mm to (120.0, 117.4), turned to 90 degrees
- moved U8 159.0 mm to (165.1, 74.9), turned to 90 degrees
- moved U12 157.7 mm to (109.8, 116.8)
- moved U9 155.1 mm to (105.4, 95.7), turned to 90 degrees
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Connections:
- SW1 pad 3: SPDT 3.3V Source -> +3V3
- SW2 pad 3: SPDT 3.3V Source -> +3V3
- SW3 pad 3: SPDT 3.3V Source -> +3V3
- U1 pad 1: Distance Sensor 1 3.3V Power -> +3V3
- U14 pad 26: SPDT 1 Data -> unconnected-(U14-A12-Pad26)
- U14 pad 27: SPDT 2 Data -> unconnected-(U14-A13-Pad27)
- U14 pad 3.3V_1: SPDT 3.3V Source -> +3V3
- U14 pad 3.3V_2: SPDT 3.3V Source -> +3V3
- U14 pad 3.3V_3: SPDT 3.3V Source -> +3V3
- U14 pad 32: unconnected-(U14-OUT1B-Pad32) -> Line Sensor 1 Data
- U14 pad 35: Line Sensor 1 Data -> unconnected-(U14-TX8-Pad35)
- U14 pad 39: unconnected-(U14-A15-Pad39) -> SPDT 2 Data
- U14 pad 40: unconnected-(U14-A16-Pad40) -> SPDT 1 Data
- U14 pad 5V: MPU-6050 5V Power -> unconnected-(U14-Pad5V)
- U14 pad GND1: GNDREF -> Net-(U14-GND-PadGND1)
- U14 pad GND2: GNDREF -> Net-(U14-GND-PadGND1)
- U14 pad GND3: GNDREF -> Net-(U14-GND-PadGND1)
- U14 pad GND4: GNDREF -> Net-(U14-GND-PadGND1)
- U14 pad GND5: GNDREF -> Net-(U14-GND-PadGND1)
- U14 pad VIN: Distance Sensor 1 3.3V Power -> MPU-6050 5V Power
- U15 pad 1: Distance Sensor 1 3.3V Power -> +3V3
- U2 pad 1: Distance Sensor 1 3.3V Power -> +3V3
- U3 pad 1: Distance Sensor 1 3.3V Power -> +3V3
- U6 pad 1: Distance Sensor 1 3.3V Power -> +3V3
- U7 pad 1: Distance Sensor 1 3.3V Power -> +3V3
- U8 pad 1: Distance Sensor 1 3.3V Power -> +3V3
Routing:
- net GNDREF: track 0.00 -> 425.0 mm, vias 0 -> 4
- net 11.1V Converter Source: track 0.00 -> 282.2 mm, vias 0 -> 4
- net MPU-6050 5V Power: track 0.00 -> 266.9 mm
- net +3V3: track 0.00 -> 153.8 mm
- net Motor Driver 1 PWM High: track 0.00 -> 79.3 mm
- net Motor Driver 3 PWM High: track 0.00 -> 74.0 mm
- net Net-(U14-GND-PadGND1): track 0.00 -> 73.8 mm, vias 0 -> 1
- net Motor Driver 3 PWM Low: track 0.00 -> 70.8 mm
- net Motor Driver 1 PWM Low: track 0.00 -> 62.4 mm
- net Distance Sensor Data 3: track 0.00 -> 49.3 mm
- net Distance Sensor Data 2: track 0.00 -> 42.6 mm
- net Motor Driver 2 PWM Low: track 0.00 -> 41.4 mm, vias 0 -> 1
- net Line Sensor 1 Data: track 0.00 -> 36.7 mm
- net Motor Driver 2 PWM High: track 0.00 -> 36.6 mm, vias 0 -> 1
- net Distance Sensor Data 1: track 0.00 -> 36.5 mm
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Other:
- board text added: "FROSTI CONTROL BOARD"
- board text added: "Rudra Goel Spring 2024"

Commit message: pcb layout done
Parts:
- removed C5: .47 uF, Capacitor_SMD:C_0201_0603Metric
- removed C6: .1 uF, Capacitor_SMD:C_0201_0603Metric
- removed R3: 30k, Resistor_SMD:R_0201_0603Metric
- removed SW2, SW3: SW_SPDT, Connector_PinHeader_1.00mm:PinHeader_1x03_P1.00mm_Vertical
- removed U12: DRV8871DDA, Package_SO:Texas_HTSOP-8-1EP_3.9x4.9mm_P1.27mm_EP2.95x4.9mm_Mask2.4x3.1mm_ThermalVias
- removed U13: ~, Connector_JST:JST_EH_B2B-EH-A_1x02_P2.50mm_Vertical
- C1, C10, C2, C3, C4: footprint Capacitor_SMD:C_0201_0603Metric -> Capacitor_SMD:C_0805_2012Metric
- C7: value 100nF -> 10uF; footprint Capacitor_SMD:C_0201_0603Metric -> Capacitor_SMD:C_0805_2012Metric
- C8: value 10pF -> .1 uF; footprint Capacitor_SMD:C_0201_0603Metric -> Capacitor_SMD:C_0805_2012Metric
- C9: value 1uF -> 22uF; footprint Capacitor_SMD:C_0201_0603Metric -> Capacitor_SMD:C_0805_2012Metric
- L1: footprint Inductor_SMD:L_0201_0603Metric -> Inductor_SMD:L_Bourns_SRP1038C_10.0x10.0mm
- R1, R2: footprint Resistor_SMD:R_0201_0603Metric -> Resistor_SMD:R_0805_2012Metric
- SW1: footprint Connector_PinHeader_1.00mm:PinHeader_1x03_P1.00mm_Vertical -> footprints:3 Pheonix
- U1, U2, U3, U6, U7, U8: footprint Connector_JST:JST_EH_B3B-EH-A_1x03_P2.50mm_Vertical -> footprints:3 Pheonix
- U11, U5: footprint Connector_JST:JST_EH_B2B-EH-A_1x02_P2.50mm_Vertical -> footprints:2 Pheonis
- U15: footprint Connector_JST:JST_EH_B3B-EH-A_1x03_P2.50mm_Vertical -> Connector_PinSocket_2.00mm:PinSocket_1x03_P2.00mm_Vertical
- moved C3 93.6 mm to (163.2, 128.0), turned to 90 degrees
- moved C4 93.4 mm to (166.8, 128.0), turned to 90 degrees
- moved U11 91.9 mm to (116.2, 129.0)
- moved C9 83.5 mm to (177.8, 86.7), turned to -90 degrees
- moved R2 82.0 mm to (126.4, 128.9), turned to 0 degrees
- moved U10 79.4 mm to (130.2, 123.8)
- moved C10 76.6 mm to (175.9, 82.5), turned to 0 degrees
- moved U9 72.4 mm to (177.8, 94.7), turned to -90 degrees
- moved L1 67.3 mm to (175.9, 74.3), turned to -90 degrees
- moved C8 64.3 mm to (167.0, 66.7), turned to 90 degrees
- moved C7 60.9 mm to (160.7, 66.7)
- moved U17 59.9 mm to (170.0, 64.8)
- moved SW1 54.5 mm to (155.6, 93.3), turned to 180 degrees
- moved U1 53.9 mm to (113.7, 67.9), turned to 0 degrees
- moved U8 51.9 mm to (113.7, 81.9), turned to 0 degrees
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Connections:
- C8 pad 1: Distance Sensor 1 3.3V Power -> Net-(U17-BST)
- C8 pad 2: Net-(U16-SPG) -> Net-(U17-SW)
- C9 pad 1: Distance Sensor 1 3.3V Power -> Net-(C10-Pad2)
- U14 pad 0: unconnected-(U14-RX1-Pad0) -> Start Module Signal
- U14 pad 11: Motor Driver 3 PWM Low -> unconnected-(U14-MOSI-Pad11)
- U14 pad 12: Motor Driver 3 PWM High -> unconnected-(U14-MISO-Pad12)
- U14 pad 13: Distance Sensor Data 1 -> unconnected-(U14-SCK-Pad13)
- U14 pad 14: Distance Sensor Data 2 -> unconnected-(U14-A0-Pad14)
- U14 pad 15: Distance Sensor Data 3 -> unconnected-(U14-A1-Pad15)
- U14 pad 18: unconnected-(U14-A4-Pad18) -> Motor Driver 1 PWM High
- U14 pad 19: unconnected-(U14-A5-Pad19) -> Motor Driver 1 PWM Low
- U14 pad 24: Motor Driver 2 PWM Low -> unconnected-(U14-A10-Pad24)
- U14 pad 25: Motor Driver 2 PWM High -> unconnected-(U14-A11-Pad25)
- U14 pad 26: unconnected-(U14-A12-Pad26) -> SPDT 1 Data
- U14 pad 27: unconnected-(U14-A13-Pad27) -> Line Sensor 1 Data
- U14 pad 28: unconnected-(U14-RX7-Pad28) -> Distance Sensor Data 3
- U14 pad 29: Motor Driver 1 PWM Low -> Distance Sensor Data 2
- U14 pad 30: Line Sensor 2 Data -> Line Sensor 3 Data
- U14 pad 31: Line Sensor 3 Data -> Distance Sensor Data 1
- U14 pad 32: Line Sensor 1 Data -> Line Sensor 2 Data
- U14 pad 34: Motor Driver 1 PWM High -> unconnected-(U14-RX8-Pad34)
- U14 pad 36: unconnected-(U14-CS2-Pad36) -> Motor Driver 2 PWM High
- U14 pad 37: unconnected-(U14-CS3-Pad37) -> Motor Driver 2 PWM Low
- U14 pad 38: SPDT 3 Data -> unconnected-(U14-A14-Pad38)
- U14 pad 39: SPDT 2 Data -> unconnected-(U14-A15-Pad39)
- U14 pad 40: SPDT 1 Data -> unconnected-(U14-A16-Pad40)
- U14 pad 41: Start Module Signal -> unconnected-(U14-A17-Pad41)
- U14 pad GND1: Net-(U14-GND-PadGND1) -> GNDREF
- U14 pad GND2: Net-(U14-GND-PadGND1) -> GNDREF
- U14 pad GND3: Net-(U14-GND-PadGND1) -> GNDREF
- U14 pad GND4: Net-(U14-GND-PadGND1) -> GNDREF
- U14 pad GND5: Net-(U14-GND-PadGND1) -> GNDREF
Routing:
- net MPU-6050 5V Power: track 266.9 -> 68.7 mm
- net 11.1V Converter Source: track 282.2 -> 140.3 mm, vias 4 -> 1
- net Motor Driver 3 PWM High: track 74.0 -> 0.00 mm
- net Net-(U14-GND-PadGND1): track 73.8 -> 0.00 mm, vias 1 -> 0
- net Motor Driver 3 PWM Low: track 70.8 -> 0.00 mm
- net Motor Driver 1 PWM High: track 79.3 -> 11.6 mm
- net GNDREF: track 425.0 -> 363.0 mm, vias 4 -> 0
- net Motor Driver 1 PWM Low: track 62.4 -> 10.9 mm
- net Net-(U10-OUT2): track 7.47 -> 47.8 mm
- net Motor Driver 2 PWM Low: track 41.4 -> 8.29 mm, vias 1 -> 0
- net +3V3: track 153.8 -> 182.5 mm, vias 0 -> 1
- net SPDT 3 Data: track 27.8 -> 0.00 mm
- net SPDT 2 Data: track 27.3 -> 0.00 mm
- net Motor Driver 2 PWM High: track 36.6 -> 10.6 mm, vias 1 -> 0
- net Net-(U4-OUT1): track 0.00 -> 18.1 mm
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Other:
- board outline added: 71.1 x 71.1 mm
- board text added: "Designed by Rudra Goel"
- board text added: "Distance Sensors"
- board text added: "Interntial Measurement Unit"
- board text added: "Line Sensors"
- board text added: "Robowrestling - Spring 2024"
- board text removed: "Rudra Goel Spring 2024"

Commit message: parts list and schemaitc reviewed'
Parts:
- removed SW1: SW_SPDT, footprints:3 Pheonix
- added C11: .1 uF, Capacitor_SMD:C_0805_2012Metric, F.Cu at (100.7, 81.0)
- added C12: .1 uF, Capacitor_SMD:C_0805_2012Metric, F.Cu at (103.7, 81.0)
- added C13: .1 uF, Capacitor_SMD:C_0805_2012Metric, F.Cu at (106.7, 81.0)
- added C14: .1 uF, Capacitor_SMD:C_0805_2012Metric, F.Cu at (135.6, 58.4)
- added C15: .1 uF, Capacitor_SMD:C_0805_2012Metric, F.Cu at (138.6, 58.4)
- added C16: .1 uF, Capacitor_SMD:C_0805_2012Metric, F.Cu at (141.6, 58.4)
- added C17: .1 uF, Capacitor_SMD:C_0805_2012Metric, F.Cu at (84.8, 81.4)
- added C18: .1 uF, Capacitor_SMD:C_0805_2012Metric, F.Cu at (84.8, 84.5)
- added C5: 10uF, Capacitor_SMD:C_0805_2012Metric, F.Cu at (80.3, 72.4)
- added C6: .1 uF, Capacitor_SMD:C_0805_2012Metric, F.Cu at (80.3, 75.4)
- added D1: LED, LED_SMD:LED_0603_1608Metric, F.Cu at (189.2, 64.4)
- added F1: 2A, Fuse:Fuse_0805_2012Metric_Pad1.15x1.40mm_HandSolder, F.Cu at (81.3, 93.3)
- added R3: 300ohm, Resistor_SMD:R_0805_2012Metric, F.Cu at (182.1, 64.4)
- added R4: 200ohm, Resistor_SMD:R_0805_2012Metric, F.Cu at (185.4, 64.4)
- added SW2: SW_SPST, footprints:500SSP1_EWI, F.Cu at (186.1, 71.5)
- U10: footprint Package_SO:Texas_HTSOP-8-1EP_3.9x4.9mm_P1.27mm_EP2.95x4.9mm_Mask2.4x3.1mm_ThermalVias -> footprints:DDA0008H_N
- U4: footprint Package_SO:Texas_HTSOP-8-1EP_3.9x4.9mm_P1.27mm_EP2.95x4.9mm_Mask2.4x3.1mm_ThermalVias -> footprints:DDA0008H_L
- U9: footprint Connector_JST:JST_EH_B8B-EH-A_1x08_P2.50mm_Vertical -> Connector_PinSocket_2.00mm:PinSocket_1x04_P2.00mm_Vertical
- moved U9 14.9 mm to (190.7, 102.2)
Connections:
- C10 pad 1: MPU-6050 5V Power -> Teensy 5V Source
- GND1 pad 2: 11.1V Converter Source -> Net-(GND1-Pin_2)
- L1 pad 2: MPU-6050 5V Power -> Teensy 5V Source
- U14 pad 26: SPDT 1 Data -> unconnected-(U14-A12-Pad26)
- U14 pad VIN: MPU-6050 5V Power -> Teensy 5V Source
- U17 pad 1: MPU-6050 5V Power -> Teensy 5V Source
- U9 pad 1: MPU-6050 5V Power -> +3V3
Routing:
- net Teensy 5V Source: track 0.00 -> 68.7 mm
- net MPU-6050 5V Power: track 68.7 -> 0.00 mm
- net +3V3: track 182.5 -> 155.7 mm
- net SPDT 1 Data: track 26.6 -> 0.00 mm
- net unconnected-(U14-A12-Pad26): track 0.00 -> 14.4 mm
- net Net-(U14-USB_GND-PadUSB_GND1): track 2.54 -> 0.00 mm
Other:
- board size 71.1 x 71.1 mm -> 80 x 80 mm
- board text removed: "Designed by Rudra Goel"
- board text removed: "FROSTI CONTROL BOARD"
- board text removed: "Robowrestling - Spring 2024"

Commit message: pcb layout done
Parts:
- removed U15: ~, Connector_PinSocket_2.00mm:PinSocket_1x03_P2.00mm_Vertical
- removed U9: ~, Connector_PinSocket_2.00mm:PinSocket_1x04_P2.00mm_Vertical
- added C19: .1 uF, Capacitor_SMD:C_0805_2012Metric, F.Cu at (140.0, 62.2)
- added IMU: ~, Connector_PinSocket_2.00mm:PinSocket_1x04_P2.00mm_Vertical, F.Cu at (137.8, 87.6)
- added Servo Motor: Motor_Servo_Robbe, Connector_PinHeader_2.54mm:PinHeader_1x03_P2.54mm_Vertical, F.Cu at (144.1, 65.4)
- added Start Module: ~, Connector_PinSocket_2.00mm:PinSocket_1x03_P2.00mm_Vertical, F.Cu at (151.6, 98.0)
- U10, U4: value DRV8871DDA -> Motor Driver
- moved F1 86.0 mm to (163.4, 68.1), turned to 180 degrees
- moved C5 83.2 mm to (163.5, 71.9)
- moved C6 83.2 mm to (163.5, 75.7), turned to 180 degrees
- moved C17 70.0 mm to (152.1, 100.5)
- moved C4 52.0 mm to (114.9, 131.8)
- moved C18 50.6 mm to (135.3, 88.2), turned to -90 degrees
- moved C3 44.6 mm to (118.7, 131.8)
- moved C14 40.5 mm to (132.1, 98.7), turned to -90 degrees
- moved U6 39.1 mm to (108.6, 68.7), turned to 90 degrees
- moved U3 38.2 mm to (125.1, 100.3), turned to 90 degrees
- moved R4 30.2 mm to (160.7, 81.6)
- moved C16 26.2 mm to (132.1, 82.9), turned to -90 degrees
- moved D1 25.7 mm to (168.9, 80.2)
- moved R3 24.6 mm to (164.5, 81.6), turned to -90 degrees
- moved U7 21.1 mm to (108.6, 84.6), turned to 90 degrees
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Connections:
- net Teensy 5V Source renamed Servo 5V Source
- U10 pad 9: (no net) -> GNDREF
- U14 pad 16: IMU Clock -> unconnected-(U14-A2-Pad16)
- U14 pad 17: IMU Data -> unconnected-(U14-A3-Pad17)
- U14 pad 18: Motor Driver 1 PWM High -> unconnected-(U14-A4-Pad18)
- U14 pad 19: Motor Driver 1 PWM Low -> unconnected-(U14-A5-Pad19)
- U14 pad 21: unconnected-(U14-A7-Pad21) -> Motor Driver 1 PWM High
- U14 pad 22: unconnected-(U14-A8-Pad22) -> Motor Driver 1 PWM Low
- U14 pad 24: unconnected-(U14-A10-Pad24) -> IMU Clock
- U14 pad 25: unconnected-(U14-A11-Pad25) -> IMU Data
- U14 pad 27: Line Sensor 1 Data -> Distance Sensor Data 3
- U14 pad 28: Distance Sensor Data 3 -> Distance Sensor Data 1
- U14 pad 30: Line Sensor 3 Data -> Line Sensor 2 Data
- U14 pad 31: Distance Sensor Data 1 -> Line Sensor 3 Data
- U14 pad 32: Line Sensor 2 Data -> Line Sensor 1 Data
- U14 pad 6: unconnected-(U14-OUT1D-Pad6) -> Servo PWM Signal
- U4 pad 9: (no net) -> GNDREF
Routing:
- net GNDREF: track 363.0 -> 10.0 mm
- net 11.1V Converter Source: track 140.3 -> 197.0 mm
- net Servo PWM Signal: track 0.00 -> 43.0 mm
- net Servo 5V Source: track 68.7 -> 109.7 mm
- net Distance Sensor Data 3: track 58.3 -> 19.8 mm
- net +3V3: track 155.7 -> 184.5 mm, vias 1 -> 0
- net Net-(GND1-Pin_2): track 0.00 -> 25.0 mm
- net Net-(U10-OUT2): track 47.8 -> 23.2 mm
- net IMU Clock: track 38.2 -> 23.3 mm
- net unconnected-(U14-A12-Pad26): track 14.4 -> 0.00 mm
- net IMU Data: track 35.4 -> 23.9 mm
- net Distance Sensor Data 2: track 49.8 -> 60.0 mm
- net Net-(U4-OUT2): track 17.1 -> 7.05 mm
- net Net-(U10-OUT1): track 23.3 -> 15.1 mm
- net Line Sensor 2 Data: track 26.5 -> 20.2 mm
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- added copper zone on B.Cu, net GNDREF
- added copper zone on F.Cu, net GNDREF
Other:
- board size 80 x 80 mm -> 71.8 x 80.6 mm
- board text added: "C12"
- board text added: "Designed by Rudra Goel"
- board text added: "Distance Sensor"
- board text added: "FROSTIII Control Board"
- board text added: "Line Sensor"
- board text added: "Spring 2024"
- board text removed: "Distance Sensors"
- board text removed: "Interntial Measurement Unit"
- board text removed: "Line Sensors"

Commit message: pcb finished
Parts:
- moved U11 0.12 mm to (110.0, 130.8)
Changed lines of the file:
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@@
       (outputformat 1)
       (mirror false)
-      (drillshape 1)
+      (drillshape 0)
       (scaleselection 1)
-      (outputdirectory "")
+      (outputdirectory "../Gerber Files/")
     )
   )
@@
     (fp_line (start 1 0.625) (end -1 0.625)
       (stroke (width 0.1) (type solid)) (layer "F.Fab"))
-    (pad "1" smd roundrect (at -0.9125 0 270) (size 1.025 1.4) (layers "F.Cu" "F.Paste" "F.Mask") (roundrect_rratio 0.243902)
+    (pad "1" smd roundrect (at -0.9125 0 270) (size 1.025 1.4) (layers "F.Cu" "F.Paste" "F.Mask") (roundrect_rratio 0.243902439)
       (net 8 "Net-(U10-ILIM)") (pintype "passive"))
-    (pad "2" smd roundrect (at 0.9125 0 270) (size 1.025 1.4) (layers "F.Cu" "F.Paste" "F.Mask") (roundrect_rratio 0.243902)
+    (pad "2" smd roundrect (at 0.9125 0 270) (size 1.025 1.4) (layers "F.Cu" "F.Paste" "F.Mask") (roundrect_rratio 0.243902439)
       (net 2 "GNDREF") (pintype "passive"))
     (model "${KICAD6_3DMODEL_DIR}/Resistor_SMD.3dshapes/R_0805_2012Metric.wrl"
@@
   )
   (footprint "footprints:2 Pheonis" (layer "F.Cu")
-    (at 109.9801 130.934999 180)
+    (at 109.9801 130.81 180)
     (tags "1890963 ")
     (property "Sheetfile" "Frosti.kicad_sch")
@@
     (fp_line (start 1 0.6) (end -1 0.6)
       (stroke (width 0.1) (type solid)) (layer "F.Fab"))
-    (pad "1" smd roundrect (at -1.025 0 180) (size 1.15 1.4) (layers "F.Cu" "F.Paste" "F.Mask") (roundrect_rratio 0.217391)
+    (pad "1" smd roundrect (at -1.025 0 180) (size 1.15 1.4) (layers "F.Cu" "F.Paste" "F.Mask") (roundrect_rratio 0.2173913043)
       (net 68 "Net-(SW2-B)") (pintype "passive"))
-    (pad "2" smd roundrect (at 1.025 0 180) (size 1.15 1.4) (layers "F.Cu" "F.Paste" "F.Mask") (roundrect_rratio 0.217391)
+    (pad "2" smd roundrect (at 1.025 0 180) (size 1.15 1.4) (layers "F.Cu" "F.Paste" "F.Mask") (roundrect_rratio 0.2173913043)
       (net 67 "Net-(GND1-Pin_2)") (pintype "passive"))
     (model "${KICAD6_3DMODEL_DIR}/Fuse.3dshapes/Fuse_0805_2012Metric.wrl"
@@
     (fp_line (start 1 0.625) (end -1 0.625)
       (stroke (width 0.1) (type solid)) (layer "F.Fab"))
-    (pad "1" smd roundrect (at -0.9125 0 90) (size 1.025 1.4) (layers "F.Cu" "F.Paste" "F.Mask") (roundrect_rratio 0.243902)
+    (pad "1" smd roundrect (at -0.9125 0 90) (size 1.025 1.4) (layers "F.Cu" "F.Paste" "F.Mask") (roundrect_rratio 0.243902439)
       (net 70 "Net-(R3-Pad2)") (pintype "passive"))
-    (pad "2" smd roundrect (at 0.9125 0 90) (size 1.025 1.4) (layers "F.Cu" "F.Paste" "F.Mask") (roundrect_rratio 0.243902)
+    (pad "2" smd roundrect (at 0.9125 0 90) (size 1.025 1.4) (layers "F.Cu" "F.Paste" "F.Mask") (roundrect_rratio 0.243902439)
       (net 2 "GNDREF") (pintype "passive"))
     (model "${KICAD6_3DMODEL_DIR}/Resistor_SMD.3dshapes/R_0805_2012Metric.wrl"
@@
     (fp_line (start 1 0.625) (end -1 0.625)
       (stroke (width 0.1) (type solid)) (layer "F.Fab"))
-    (pad "1" smd roundrect (at -0.9125 0 270) (size 1.025 1.4) (layers "F.Cu" "F.Paste" "F.Mask") (roundrect_rratio 0.243902)
+    (pad "1" smd roundrect (at -0.9125 0 270) (size 1.025 1.4) (layers "F.Cu" "F.Paste" "F.Mask") (roundrect_rratio 0.243902439)
       (net 7 "Net-(U4-ILIM)") (pintype "passive"))
-    (pad "2" smd roundrect (at 0.9125 0 270) (size 1.025 1.4) (layers "F.Cu" "F.Paste" "F.Mask") (roundrect_rratio 0.243902)
+    (pad "2" smd roundrect (at 0.9125 0 270) (size 1.025 1.4) (layers "F.Cu" "F.Paste" "F.Mask") (roundrect_rratio 0.243902439)
       (net 2 "GNDREF") (pintype "passive"))
     (model "${KICAD6_3DMODEL_DIR}/Resistor_SMD.3dshapes/R_0805_2012Metric.wrl"
@@
     (property "ki_keywords" "cap capacitor")
     (attr smd)
-    (fp_text reference "C4" (at 0 -1.68 90) (layer "F.SilkS")
+    (fp_text reference "C4" (at 2.855 0 90) (layer "F.SilkS")
         (effects (font (size 1 1) (thickness 0.15)))
     )
@@
     (fp_line (start 1 0.625) (end -1 0.625)
       (stroke (width 0.1) (type solid)) (layer "F.Fab"))
-    (pad "1" smd roundrect (at -0.9125 0 270) (size 1.025 1.4) (layers "F.Cu" "F.Paste" "F.Mask") (roundrect_rratio 0.243902)
+    (pad "1" smd roundrect (at -0.9125 0 270) (size 1.025 1.4) (layers "F.Cu" "F.Paste" "F.Mask") (roundrect_rratio 0.243902439)
       (net 69 "Net-(D1-K)") (pintype "passive"))
-    (pad "2" smd roundrect (at 0.9125 0 270) (size 1.025 1.4) (layers "F.Cu" "F.Paste" "F.Mask") (roundrect_rratio 0.243902)
+    (pad "2" smd roundrect (at 0.9125 0 270) (size 1.025 1.4) (layers "F.Cu" "F.Paste" "F.Mask") (roundrect_rratio 0.243902439)
       (net 70 "Net-(R3-Pad2)") (pintype "passive"))
     (model "${KICAD6_3DMODEL_DIR}/Resistor_SMD.3dshapes/R_0805_2012Metric.wrl"
