File: 500g/Frosti/Frosti.kicad_sch (KiCad schematic)
At the start: 32 parts, among them SW1 SW_SPDT, SW2 SW_SPDT, SW3 SW_SPDT, U10 DRV8871DDA, U12 DRV8871DDA, U14 DEV-16771, U4 DRV8871DDA

Commit message: pcb layout done
Parts:
- removed U16: ~, Package_SO:Zetex_SM8, symbol FROSTI Parts:ZLDO330_3.3_volt_ultra_low_dropout_regulator_datasheet
- added C10: 22uF, Capacitor_SMD:C_0201_0603Metric, symbol Device:C
- added L1: 4.7uH, Inductor_SMD:L_0201_0603Metric, symbol Device:L
- added U17: AP63205WU, Package_TO_SOT_SMD:TSOT-23-6, symbol Regulator_Switching:AP63205WU
- C7: value 100nF -> 10uF
- C8: value 10pF -> 100nF
- C9: value 1uF -> 22uF
- R1, R2, R3: footprint Resistor_SMD:R_0603_1608Metric -> Resistor_SMD:R_0201_0603Metric
Connections:
- net SPDT 3.3V Source is gone; now on net +3V3: SW1.3 (C), SW2.3 (C), SW3.3 (C), U14.3.3V_1 (3.3V), U14.3.3V_2 (3.3V), U14.3.3V_3 (3.3V)
- net 11.1V Converter Source: now also U17.2 (EN), U17.3 (IN)
- net GNDREF: now also U17.4 (GND); no longer U14.GND1 (GND), U14.GND2 (GND), U14.GND3 (GND), U14.GND4 (GND), U14.GND5 (GND)
- net Line Sensor 1 Data: now also U14.32 (OUT1B); no longer U14.35 (TX8)
- net MPU-6050 5V Power: now also U14.VIN, C10.1, L1.2, U17.1 (FB); no longer U14.5V
- net SPDT 1 Data: now also U14.40 (A16); no longer U14.26 (A12)
- net SPDT 2 Data: now also U14.39 (A15); no longer U14.27 (A13)
- net at C8.2: now also L1.1, U17.5 (SW)
- net Distance Sensor 1 3.3V Power renamed +3V3
- net +3V3: no longer C8.1, C9.1, U14.VIN
- new net: C8.1, U17.6 (BST)
- new net: C10.2, C9.1
- new net: U14.GND1 (GND), U14.GND2 (GND), U14.GND3 (GND), U14.GND4 (GND), U14.GND5 (GND)

Commit message: pcb layout done
Parts:
- removed C5: .47 uF, Capacitor_SMD:C_0201_0603Metric, symbol Device:C
- removed C6: .1 uF, Capacitor_SMD:C_0201_0603Metric, symbol Device:C
- removed R3: 30k, Resistor_SMD:R_0201_0603Metric, symbol Device:R_US
- removed SW2, SW3: SW_SPDT, Connector_PinHeader_1.00mm:PinHeader_1x03_P1.00mm_Vertical, symbol Switch:SW_SPDT
- removed U12: DRV8871DDA, Package_SO:Texas_HTSOP-8-1EP_3.9x4.9mm_P1.27mm_EP2.95x4.9mm_Mask2.4x3.1mm_ThermalVias, symbol Driver_Motor:DRV8871DDA
- removed U13: ~, Connector_JST:JST_EH_B2B-EH-A_1x02_P2.50mm_Vertical, symbol FROSTI Parts:MP12_Micro_Gear_Motor_6V
- C1, C10, C2, C3, C4, C7, C9: footprint Capacitor_SMD:C_0201_0603Metric -> Capacitor_SMD:C_0805_2012Metric
- C8: value 100nF -> .1 uF; footprint Capacitor_SMD:C_0201_0603Metric -> Capacitor_SMD:C_0805_2012Metric
- L1: footprint Inductor_SMD:L_0201_0603Metric -> Inductor_SMD:L_Bourns_SRP1038C_10.0x10.0mm
- R1, R2: footprint Resistor_SMD:R_0201_0603Metric -> Resistor_SMD:R_0805_2012Metric
- SW1: footprint Connector_PinHeader_1.00mm:PinHeader_1x03_P1.00mm_Vertical -> footprints:3 Pheonix
- U1, U2, U3, U6, U7, U8: footprint Connector_JST:JST_EH_B3B-EH-A_1x03_P2.50mm_Vertical -> footprints:3 Pheonix
- U11, U5: footprint Connector_JST:JST_EH_B2B-EH-A_1x02_P2.50mm_Vertical -> footprints:2 Pheonis
- U15: footprint Connector_JST:JST_EH_B3B-EH-A_1x03_P2.50mm_Vertical -> Connector_PinSocket_2.00mm:PinSocket_1x03_P2.00mm_Vertical
Connections:
- net Distance Sensor Data 1: now also U14.31 (CTX3); no longer U14.13 (SCK)
- net Distance Sensor Data 2: now also U14.29 (TX7); no longer U14.14 (A0)
- net Distance Sensor Data 3: now also U14.28 (RX7); no longer U14.15 (A1)
- net GNDREF: now also U14.GND1 (GND), U14.GND2 (GND), U14.GND3 (GND), U14.GND4 (GND), U14.GND5 (GND)
- net Line Sensor 1 Data: now also U14.27 (A13); no longer U14.32 (OUT1B)
- net Line Sensor 2 Data: now also U14.32 (OUT1B); no longer U14.30 (CRX3)
- net Line Sensor 3 Data: now also U14.30 (CRX3); no longer U14.31 (CTX3)
- net Motor Driver 1 PWM High: now also U14.18 (A4); no longer U14.34 (RX8)
- net Motor Driver 1 PWM Low: now also U14.19 (A5); no longer U14.29 (TX7)
- net Motor Driver 2 PWM High: now also U14.36 (CS2); no longer U14.25 (A11)
- net Motor Driver 2 PWM Low: now also U14.37 (CS3); no longer U14.24 (A10)
- net SPDT 1 Data: now also U14.26 (A12); no longer U14.40 (A16)
- net Start Module Signal: now also U14.0 (RX1); no longer U14.41 (A17)
- net Motor Driver 3 PWM High: no longer names the net of U14.12 (MISO)
- net Motor Driver 3 PWM Low: no longer names the net of U14.11 (MOSI)
- net SPDT 2 Data: no longer names the net of U14.39 (A15)
- net SPDT 3 Data: no longer names the net of U14.38 (A14)
Other:
- note added: "11.1V to 5V Converter"
- note removed: "11.1V to 3.3V Converter"
- moved on the sheet: C3, C4, R2, U10, U11

Commit message: parts list and schemaitc reviewed'
Parts:
- removed SW1: SW_SPDT, footprints:3 Pheonix, symbol Switch:SW_SPDT
- added C11, C12, C13, C14, C15, C16, C17, C18, C6: .1 uF, Capacitor_SMD:C_0805_2012Metric, symbol Device:C
- added C5: 10uF, Capacitor_SMD:C_0805_2012Metric, symbol Device:C
- added D1: LED, LED_SMD:LED_0603_1608Metric, symbol Device:LED
- added F1: 2A, Fuse:Fuse_0805_2012Metric_Pad1.15x1.40mm_HandSolder, symbol Device:Fuse
- added R3: 300ohm, Resistor_SMD:R_0805_2012Metric, symbol Device:R
- added R4: 200ohm, Resistor_SMD:R_0805_2012Metric, symbol Device:R
- added SW2: SW_SPST, footprints:500SSP1_EWI, symbol Switch:SW_SPST
- U10: footprint Package_SO:Texas_HTSOP-8-1EP_3.9x4.9mm_P1.27mm_EP2.95x4.9mm_Mask2.4x3.1mm_ThermalVias -> footprints:DDA0008H_N
- U4: footprint Package_SO:Texas_HTSOP-8-1EP_3.9x4.9mm_P1.27mm_EP2.95x4.9mm_Mask2.4x3.1mm_ThermalVias -> footprints:DDA0008H_L
- U9: footprint Connector_JST:JST_EH_B8B-EH-A_1x08_P2.50mm_Vertical -> Connector_PinSocket_2.00mm:PinSocket_1x04_P2.00mm_Vertical
Connections:
- net +3V3: now also U9.1 (VCC), C11.2, C12.2, C13.2, C14.2, C15.2, C16.2, C17.1, C18.1
- net 11.1V Converter Source: now also C5.2, C6.1, SW2.1 (A); no longer GND1.2 (Pin_2)
- net GNDREF: now also C11.1, C12.1, C13.1, C14.1, C15.1, C16.1, C17.2, C18.2, C5.1, C6.2, R4.2
- net MPU-6050 5V Power renamed Teensy 5V Source
- net Teensy 5V Source: now also D1.2 (A); no longer U9.1 (VCC)
- net SPDT 1 Data: no longer names the net of U14.26 (A12)
- new net: R3.2, R4.1
- new net: D1.1 (K), R3.1
- new net: F1.1, SW2.2 (B)
- new net: F1.2, GND1.2 (Pin_2)
Other:
- note added: "Add ground planes to pcb"
- note removed: "SPDT Collision Switches"
- moved on the sheet: GND1

Commit message: pcb layout done
Parts:
- added C19: .1 uF, Capacitor_SMD:C_0805_2012Metric, symbol Device:C
- added M1: Motor_Servo_Robbe, Connector_PinHeader_2.54mm:PinHeader_1x03_P2.54mm_Vertical, symbol Motor:Motor_Servo_Robbe
Connections:
- net Distance Sensor Data 1: now also U14.28 (RX7); no longer U14.31 (CTX3)
- net Distance Sensor Data 3: now also U14.27 (A13); no longer U14.28 (RX7)
- net GNDREF: now also C19.1, M1.3 (-)
- net IMU Clock: now also U14.24 (A10); no longer U14.16 (A2)
- net IMU Data: now also U14.25 (A11); no longer U14.17 (A3)
- net Line Sensor 1 Data: now also U14.32 (OUT1B); no longer U14.27 (A13)
- net Line Sensor 2 Data: now also U14.30 (CRX3); no longer U14.32 (OUT1B)
- net Line Sensor 3 Data: now also U14.31 (CTX3); no longer U14.30 (CRX3)
- net Motor Driver 1 PWM High: now also U14.21 (A7); no longer U14.18 (A4)
- net Motor Driver 1 PWM Low: now also U14.22 (A8); no longer U14.19 (A5)
- net Servo PWM Signal: now reaches U14.6 (OUT1D)
- net Servo PWM Signal: now also M1.1 (PWM)
- net Teensy 5V Source renamed Servo 5V Source
- net Servo 5V Source: now also C19.2, M1.2 (+)
Other:
- note added: "Servo Module"
- note added: "Start Module"

Commit message: pcb finished
Other:
- note removed: "Add ground planes to pcb"
Changed lines of the file:
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@@
     (effects (font (size 3 3) (thickness 0.6) bold (color 132 0 0 1)) (justify left bottom))
-  )
-  (text "Add ground planes to pcb\n" (at 141.097 220.218 0)
-    (effects (font (size 1.27 1.27)) (justify left bottom))
   )
   (text "MPU-6050 IMU \n(GY-521 Breakout Board)" (at 13.843 67.691 0)
