File: ControlBoard/Timmi/rwTimmiCB/rwTimmiCB/rwTimmiCB.kicad_pcb (KiCad board)
At the start: 2 copper layers, 2 parts, among them J1 75869-130LF, U1 DEV-16771

Commit message: Timmi cb
Parts:
- added J10: T4040034041-000, timmi footprints:TE_T4040034041-000, F.Cu at (243.8, 66.9)
- added J2: 75869-130LF, timmi footprints:FCI_75869-130LF, F.Cu at (261.6, 22.9)
- added J3: 75869-130LF, timmi footprints:FCI_75869-130LF, F.Cu at (246.3, 22.9)
- added J4: 75869-130LF, timmi footprints:FCI_75869-130LF, F.Cu at (246.3, 33.9)
- added J5: 75869-130LF, timmi footprints:FCI_75869-130LF, F.Cu at (261.6, 33.9)
- added J6: T4040034041-000, timmi footprints:TE_T4040034041-000, F.Cu at (243.8, 81.3)
- added J7: T4040034041-000, timmi footprints:TE_T4040034041-000, F.Cu at (225.1, 81.3)
- added J8: T4040034041-000, timmi footprints:TE_T4040034041-000, F.Cu at (262.6, 66.9)
- added J9: T4040034041-000, timmi footprints:TE_T4040034041-000, F.Cu at (225.1, 66.9)
Connections:
- U1 pad 15: unconnected-(U1-Pad15) -> Line RF
- U1 pad 16: unconnected-(U1-Pad16) -> Line LF
- U1 pad 17: unconnected-(U1-Pad17) -> Line RB
- U1 pad 18: unconnected-(U1-Pad18) -> Line LB
- U1 pad GND1: Net-(U1-PadGND1) -> unconnected-(U1-PadGND1)
- U1 pad GND2: Net-(U1-PadGND1) -> unconnected-(U1-PadGND2)
- U1 pad GND3: Net-(U1-PadGND1) -> unconnected-(U1-PadGND3)
- U1 pad GND4: Net-(U1-PadGND1) -> unconnected-(U1-PadGND4)
- U1 pad GND5: Net-(U1-PadGND1) -> unconnected-(U1-PadGND5)
- U1 pad USB_GND1: Net-(U1-PadUSB_GND1) -> unconnected-(U1-PadUSB_GND1)
- U1 pad USB_GND2: Net-(U1-PadUSB_GND1) -> unconnected-(U1-PadUSB_GND2)
