File: ControlBoard/Timmi/rwTimmiCB/rwTimmiCB.kicad_sch (KiCad schematic)
At the start: 18 parts, among them U1 DEV-16771

Commit message: Timmi cb
Parts:
- added C1, C2, C3, C4, C5, C6: 0.1uf, symbol Device:C
- added J?: Battery, symbol Connector_Generic:Conn_01x02
- added U4: LTV-827S, Package_DIP:SMDIP-8_W9.53mm, symbol Isolator:LTV-827S
- J1, J10, J11, J2, J3, J4, J5, J6, J7, J8, J9: renamed from J?; footprint CONN3_B3B-EH-ALFSN_JST -> 3pos screw terminal:CUI_TB002-500-03BE
- S1, S2: footprint CONN3_B3B-EH-ALFSN_JST -> 3pos screw terminal:CUI_TB002-500-03BE
- U1: footprint teensy footprint:MODULE_DEV-16771 -> timmi footprints:MODULE_DEV-16771
- gave numbers to parts that had none: 2
Connections:
- net +12V: now also C1.1, C2.1, C3.1, C4.1, C5.1, C6.1, J?.1 (Pin_1)
- net +3.3V: now also U2.6, U2.8, U3.6, U3.8, U4.6, U4.8
- net GND: now also U2.2, U2.4, U3.2, U3.4, C1.2, C2.2, C3.2, C4.2, C5.2, C6.2, J?.2 (Pin_2), U4.2, U4.4
- net oct5: now also U4.1
- net oct6: now also U4.3
- net ir3: now reaches U3.7
- net ir3: now also U1.21 (A7)
- net ir4: now reaches U3.5
- net ir4: now also U1.22 (A8)
- net ir2: now reaches U2.5
- net ir2: now also U1.20 (A6)
- net ir1: now reaches U2.7
- net ir1: now also U1.19 (A5)
- net ir5: now reaches U1.23 (A9)
- net ir5: now also U4.7
- net ir6: now reaches U1.24 (A10)
- net ir6: now also U4.5
- no-connect marks 0 -> 2
Other:
- note added: "Optocoupler"
- moved on the sheet: S1, S2, U2A, U2B, U3A, U3B

Commit message: Added battery connection stuff and chose BMI323 as IMU
Parts:
- added C7: 1uF, symbol Device:C_Small
- added C8: 10uF, symbol Device:C_Small
- added F1: Fuse, symbol Device:Fuse
- added SW1: SW_SPST, symbol Switch:SW_SPST
- added U5: BMI323, BMI323_BOS, symbol 2024-02-18_20-15-12:BMI323
Connections:
- net +12V: now also C7.1, C8.1, F1.1; no longer J?.1 (Pin_1)
- net GND: now also C7.2, C8.2
- new net: J?.1 (Pin_1), SW1.2 (B)
- new net: F1.2, SW1.1 (A)
Other:
- note added: "/channel current limit = 20A why? i said so we really should have been limiting this the whole time"
- note added: "Battery Connection"
- moved on the sheet: J?

Commit message: added voltage regulators to timmi cb
Parts:
- added C10, C12: 2.2uF, symbol Device:C_Small
- added C11, C14, C15: 22uH, symbol Device:C_Small
- added C13, C9: 0.1uF, symbol Device:C_Small
- added D1, D2, D3, D4: LED, symbol Device:LED
- added L1: 68uH, symbol Device:L
- added L2: 33uH, symbol Device:L
- added R1, R2, R3, R4: R_US, symbol Device:R_US
- added R5: 309k, symbol Device:R_US
- added R6, R8: 22.1k, symbol Device:R_US
- added R7: 118k, symbol Device:R_US
- added U6, U7: PLMR51610XDBVR, DBV0006A-IPC_A, symbol 2024-02-23_01-12-42:PLMR51610XDBVR
Connections:
- net +12V: now also C10.1, C11.1, C12.1, C14.1, D3.2 (A), D4.2 (A), L1.2, R5.2, U6.4 (EN), U6.5 (VIN), U7.4 (EN), U7.5 (VIN)
- net +3.3V: now also D1.2 (A)
- net GND: now also C10.2, C11.2, C12.2, C14.2, C15.2, R1.2, R2.2, R3.2, R4.2, R6.1, R8.1, U6.2 (GND), U7.2 (GND)
- new net: C9.2, L1.1, U6.6 (SW)
- new net: D3.1 (K), R3.1
- new net: R7.1, R8.2, U7.3 (FB)
- new net: D2.1 (K), R2.1
- new net: C13.2, L2.1, U7.6 (SW)
- new net: R5.1, R6.2, U6.3 (FB)
- new net: D1.1 (K), R1.1
- new net: C9.1, U6.1 (CB)
- new net: D4.1 (K), R4.1
- new net: C13.1, U7.1 (CB)
- new net +5V: C15.1, D2.2 (A), L2.2, R7.2
Other:
- note added: "Indicator LEDs"
- note added: "Voltage Regulator"
- moved on the sheet: S1, S2, U5

Commit message: added power switch circuit
Parts:
- removed C1, C2, C3, C4, C5, C6: 0.1uf, symbol Device:C
- removed C7: 1uF, symbol Device:C_Small
- removed C8: 10uF, symbol Device:C_Small
- removed F1: Fuse, symbol Device:Fuse
- removed J?: Battery, symbol Connector_Generic:Conn_01x02
- removed SW1: SW_SPST, symbol Switch:SW_SPST
- added C1, C2, C3, C4, C5, C6: 0.1uF, symbol Device:C_Small
- added C16: 10uF, symbol Device:C_Small
- added C17, C18: 1uF, symbol Device:C_Small
- added F2: Fuse, symbol Device:Fuse
- added J12: Battery, symbol Connector_Generic:Conn_01x02
- added Q1: SQM40P10-40L_GE3, SQM40P1040L_GE3, symbol SQM40P10-40L_GE3:SQM40P10-40L_GE3
- added Q2: SQ2318AES-T1_BE3, SOT95P237X112-3N, symbol TimmiCtrlBoard:SQ2318AES-T1_BE3
- added R10, R11, R12, R9: R_Small_US, symbol Device:R_Small_US
- added SW2: SW_SPST, symbol Switch:SW_SPST
Connections:
- net +12V: now also C1.1, C16.1, C17.1, C18.1, C2.1, C3.1, C4.1, C5.1, C6.1, Q1.2 (D)
- net GND: now also C1.2, C16.2, C17.2, C2.2, C3.2, C4.2, C5.2, C6.2, J12.2 (Pin_2), Q2.2 (S), R11.2
- new net: C18.2, Q1.1 (G), R10.1, R9.1
- new net: F2.1, Q1.3 (S), R10.2, SW2.2 (B)
- new net: F2.2, J12.1 (Pin_1)
- new net: R12.2, SW2.1 (A)
- new net: Q2.1 (G), R11.1, R12.1
- new net: Q2.3 (D), R9.2
Other:
- note added: "Battery Connection & Power Switch"
- note removed: "Battery Connection"
- moved on the sheet: D1, D2, D3, D4, J10, J11, J6, J7, J8, J9, R1, R2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

Commit message: wired imu and added ir indicators
Parts:
- added C19, C20, C21: 0.1uF, symbol Device:C_Small
- added C7, C8: 100nF, symbol Device:C_Small
- added D10, D5, D6, D7, D8, D9: LED, symbol Device:LED
- added R13, R14: 4.7k, symbol Device:R_Small_US
- added R15, R16, R17, R18, R19, R20: 500, symbol Device:R_US
Connections:
- net +3.3V: now also U5.5 (VDDIO), U5.8 (VDD), C19.1, C21.1, C7.1, C8.1, R13.1, R14.1
- net +5V: now also U1.5V, U1.VIN, C20.1
- net GND: now also U1.GND1, U1.GND2 (GND), U1.GND3 (GND), U1.GND4 (GND), U1.GND5 (GND), U1.USB_GND1 (USB_GND), U1.USB_GND2 (USB_GND), U5.1 (SDO), U5.12 (CSB), U5.6 (GNDIO), U5.7 (GND), C19.2, C20.2, C21.2, C7.2, C8.2
- net ir6: now also U1.26 (A12); no longer U1.24 (A10)
- net oct1: now also D5.2 (A); no longer U2.1
- net oct2: now also D6.2 (A); no longer U2.3
- net oct3: now also D7.2 (A); no longer U3.1
- net oct4: now also D8.2 (A); no longer U3.3
- net oct5: now also D9.2 (A); no longer U4.1
- net oct6: now also D10.2 (A); no longer U4.3
- net 3V3_IMU_SCL: now reaches U5.13 (SCX)
- net 3V3_IMU_SCL: now also U1.24 (A10), R14.2
- net 3V3_IMU_SDA: now reaches U5.14 (SDX)
- net 3V3_IMU_SDA: now also U1.25 (A11), R13.2
- net IMU_INT1: now reaches U5.4 (INT1)
- net IMU_INT2: now reaches U5.9 (INT2)
- new net: R19.2, U3.1
- new net: R18.2, U2.3
- new net: D9.1 (K), R15.1
- new net: R16.2, U3.3
- new net: D10.1 (K), R20.1
- new net: D6.1 (K), R18.1
- new net: D7.1 (K), R19.1
- new net: D5.1 (K), R17.1
- new net: D8.1 (K), R16.1
- new net: R17.2, U2.1
- new net: R20.2, U4.3
- new net: R15.2, U4.1
- no-connect marks 2 -> 40
Other:
- note added: "IMU"
- moved on the sheet: C1, C10, C11, C12, C13, C14, C15, C16, C17, C18, C2, C3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

Commit message: added load switch values
Parts:
- R10, R11, R12: value R_Small_US -> 10k
- R9: value R_Small_US -> 15k
Changed lines of the file:
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@@
       (effects (font (size 1.27 1.27)))
     )
-    (property "Value" "R_Small_US" (at 351.409 109.982 90)
+    (property "Value" "10k" (at 351.409 109.982 90)
       (effects (font (size 1.27 1.27)))
     )
@@
       (effects (font (size 1.27 1.27)))
     )
-    (property "Value" "R_Small_US" (at 360.299 129.667 90)
+    (property "Value" "10k" (at 360.299 129.667 90)
       (effects (font (size 1.27 1.27)))
     )
@@
       (effects (font (size 1.27 1.27)) (justify left))
     )
-    (property "Value" "R_Small_US" (at 348.869 119.507 0)
+    (property "Value" "15k" (at 348.869 119.507 0)
       (effects (font (size 1.27 1.27)) (justify left))
     )
@@
       (effects (font (size 1.27 1.27)) (justify left))
     )
-    (property "Value" "R_Small_US" (at 358.394 138.557 0)
-      (effects (font (size 1.27 1.27)) (justify left))
-    )
+    (property "Value" "10k" (at 358.394 138.557 0)
+      (effects (font (size 1.27 1.27)) (justify left))
+    )
