File: Skibidi/Skibid-i/Skibid-i.kicad_sch (KiCad schematic)
At the start: 75 parts, among them IC1 TEENSY_4.1, J1 XT60-M, J10 Screw_Terminal_01x04, J11 Screw_Terminal_01x04, J12 Screw_Terminal_01x03, J13 Screw_Terminal_01x03, J14 XT60-M, J15 Conn_01x03_Pin, J16 BDC2, J17 BDC1, J18 XT60-M, J19 XT60-M, J2 XT60-M, J20 Screw_Terminal_01x04, J21 Motor1, J22 Motor2, J3 Screw_Terminal_01x03, J4 Screw_Terminal_01x03, J5 Screw_Terminal_01x03, J6 Screw_Terminal_01x03, J7 Screw_Terminal_01x03, J8 Screw_Terminal_01x03, J9 Screw_Terminal_01x03, Q1 2N2219, Q2 2N2219, Q3 2N2219, Q4 2N2219, Q5 2N2219, Q6 2N2219, Q7 2N2219, Q8 2N2219, SW1 500SSP1S2M2QEA, U1 LTV-827S, U2 LTV-827S, U3 LTV-827S, U4 LTV-827S, U5 LTV-827S, U6 LTV-827S, U7 LTV-827S

Commit message: joe
Parts:
- removed D10, D11, D12, D13, D14, D15, D8, D9: D, symbol Device:D
- removed J16: BDC2, symbol Connector:Screw_Terminal_01x02
- removed J17: BDC1, symbol Connector:Screw_Terminal_01x02
- removed Q1, Q2, Q3, Q4, Q5, Q6, Q7, Q8: 2N2219, Package_TO_SOT_THT:TO-39-3, symbol Transistor_BJT:2N2219
Other:
- note removed: "H-Bridge?"

Commit message: schematic is pretty muchdone
Parts:
- removed D1, D2, D3, D4, D5, D6, D7: BLUE, symbol Device:D
- removed J20: Screw_Terminal_01x04, symbol Connector:Screw_Terminal_01x04
- added C14: 0.1uF, symbol Device:C
- added D1: LED, symbol Device:LED
- added J16: XT60-M, XT60-M:AMASS_XT60-M, symbol XT60-M:XT60-M
- added R8: 500ohm, symbol Device:R_US
- J18: value XT60-M -> Sparkin
- J19: value XT60-M -> Sparkout
Connections:
- net +24V: now also R8.2
- net +3.3V: now also C14.1
- net BDC1: now also IC1.18 (A4); no longer IC1.11 (MOSI)
- net BDC11: now also IC1.19 (A5); no longer IC1.12 (MISO)
- net BDC2: now also IC1.22 (A8)
- net BDC22: now also IC1.23 (A9)
- net GND: now also C14.2, D1.1 (K), J16.N (NEG)
- net LN5: now also IC1.20 (A6); no longer IC1.18 (A4)
- net LN6: now also IC1.21 (A7); no longer IC1.19 (A5)
- net Start: now also IC1.11 (MOSI)
- net at U2.1: now also R2.2
- net at R1.2: now also U1.1
- net at U7.1: now also R4.2
- net at R3.2: now also U5.1
- net at U4.1: now also R6.2
- net at U6.1: now also R7.2
- net at U3.1: now also R5.2
- net 68V renamed +48V
- net +48V: now also J16.P (POS)
- new net: D1.2 (A), R8.1
- no-connect marks 39 -> 37
Other:
- note added: "LEDs"
- note added: "Motor Driver Connectors"
- moved on the sheet: C2, J1, J14, J15, J18, J19, J2, J21, J22, R1, R2, R3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

Commit message: added foortprints
Parts:
- removed IC1: TEENSY_4.1, TEENSY41, symbol TEENSY_4_1:TEENSY_4.1
- added C15: 0.1uF, Skibidi-feet:C_0805_2012Metric, symbol Device:C
- added J17: Conn_01x08_Pin, Connector_PinHeader_2.54mm:PinHeader_1x08_P2.54mm_Vertical, symbol Connector:Conn_01x08_Pin
- added U8: DEV-16771, Skibidi-feet:TEENSY, symbol Teensy4.1:DEV-16771
- C10, C11, C12, C13, C14, C3, C4, C5, C6, C7, C8, C9: footprint (none) -> Skibidi-feet:C_0805_2012Metric
- D1: footprint (none) -> Skibidi-feet:LED
- J1, J14, J16, J18, J19, J2: footprint XT60-M:AMASS_XT60-M -> Skibidi-feet:XT60
- J12, J13, J3, J4, J5, J6, J7, J8, J9: footprint (none) -> Skibidi-feet:ScrewTerminal3
- J15: footprint (none) -> Connector_PinHeader_2.54mm:PinHeader_1x03_P2.54mm_Vertical
- PS1: footprint P78E05-1000:CONV_P78E05-1000 -> Skibidi-feet:5vConvertor
- R1, R2, R3, R4, R5, R6, R7, R8: footprint (none) -> Resistor_SMD:R_0805_2012Metric
- SW1: footprint THERAPI:SWITCH -> Skibidi-feet:SWitch
- U1, U2, U3, U4, U5, U6, U7: footprint Package_DIP:SMDIP-8_W9.53mm -> Skibidi-feet:Optocoupler
Connections:
- net +24V: no longer J14.P (POS), J2.N (NEG), R8.2
- net +3.3V: now also C15.2, J17.1 (Pin_1), U8.3.3V_1 (3.3V), U8.3.3V_2 (3.3V), U8.3.3V_3 (3.3V)
- net +48V: now also R8.2
- net +5V: now also U8.VIN
- net BDC1: now also U8.11 (MOSI)
- net BDC11: now also U8.12 (MISO)
- net BDC2: now also U8.9 (OUT1C)
- net BDC22: now also U8.10 (CS1), U8.41 (A17)
- net Dis1: now also U8.2 (OUT2)
- net Dis2: now also U8.3 (LRCLK2)
- net Dis3: now also U8.4 (BCLK2)
- net Dis4: now also U8.5 (IN2)
- net Dis5: now also U8.6 (OUT1D)
- net Dis6: now also U8.7 (RX2)
- net Dis7: now also U8.8 (TX2)
- net GND: now also C15.1, J17.2 (Pin_2), U8.GND1 (GND), U8.GND2 (GND), U8.GND3 (GND), U8.GND4 (GND), U8.GND5 (GND), U8.USB_GND1 (USB_GND), U8.USB_GND2 (USB_GND)
- net LN1: now also U8.14 (A0)
- net LN2: now also U8.15 (A1)
- net LN3: now also U8.16 (A2)
- net LN4: now also U8.17 (A3)
- net LN5: now also U8.20 (A6)
- net LN6: now also U8.21 (A7)
- new net: J14.P (POS), J2.N (NEG)
- new net SCL: J17.3 (Pin_3), U8.40 (A16)
- new net SDA: J17.4 (Pin_4), U8.18 (A4), U8.19 (A5), U8.39 (A15)
Other:
- note added: "IMU"
- moved on the sheet: D1, J1, J14, J18, J19, J2, R8, SW1

Commit message: finished fooorptinrt
Parts:
- C1, C2: footprint (none) -> Capacitor_SMD:C_0805_2012Metric
- J10, J11: footprint (none) -> Skibidi-feet:Screwterminal4
- J21, J22: footprint (none) -> Skibidi-feet:Screwterminal2
- U1, U2, U3, U4, U5, U6, U7: footprint Skibidi-feet:Optocoupler -> Skibidi-feet:RealOPtocoupler
- U8: footprint Skibidi-feet:TEENSY -> Skibidi-feet:Teensy4.1
Connections:
- net +24V: now also J1.P (POS), J18.P (POS)
Changed lines of the file:
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@@
 	)
 	(junction
+		(at 180.34 157.48)
+		(diameter 0)
+		(color 0 0 0 0)
+	)
+	(junction
 		(at 92.71 52.07)
 		(diameter 0)
@@
 			)
 		)
-		(property "Footprint" ""
+		(property "Footprint" "Skibidi-feet:Screwterminal2"
 			(at 256.54 72.39 0)
 			(effects
@@
 			)
 		)
-		(property "Footprint" ""
+		(property "Footprint" "Skibidi-feet:Screwterminal4"
 			(at 26.67 179.07 0)
 			(effects
@@
 	)
 	(symbol
+		(lib_id "power:+24V")
+		(at 180.34 157.48 180)
+		(unit 1)
+		(exclude_from_sim no)
+		(in_bom yes)
+		(on_board yes)
+		(dnp no)
+		(property "Reference" "#PWR069"
+			(at 180.34 153.67 0)
+			(effects
+				(font
+					(size 1.27 1.27)
+				)
+				(hide yes)
+			)
+		)
+		(property "Value" "+24V"
+			(at 182.88 161.29 0)
+			(effects
+				(font
+					(size 1.27 1.27)
+				)
+				(justify left)
+			)
+		)
+		(property "Footprint" ""
+			(at 180.34 157.48 0)
+			(effects
+				(font
+					(size 1.27 1.27)
+				)
+				(hide yes)
+			)
+		)
+		(property "Datasheet" ""
+			(at 180.34 157.48 0)
+			(effects
+				(font
+					(size 1.27 1.27)
+				)
+				(hide yes)
+			)
+		)
+		(property "Description" ""
+			(at 180.34 157.48 0)
+			(effects
+				(font
+					(size 1.27 1.27)
+				)
+				(hide yes)
+			)
+		)
+		(pin "1"
+		)
+		(instances
+			(project "Skibid-i"
+				(path "/bfc511a5-2c92-46fd-9868-0fe25107d7eb"
+					(reference "#PWR069")
+					(unit 1)
+				)
+			)
+		)
+	)
+	(symbol
 		(lib_id "Connector:Screw_Terminal_01x02")
 		(at 265.43 72.39 90)
@@
 			)
 		)
-		(property "Footprint" ""
+		(property "Footprint" "Skibidi-feet:Screwterminal2"
 			(at 265.43 72.39 0)
 			(effects
@@
 			)
 		)
-		(property "Footprint" "Skibidi-feet:Optocoupler"
+		(property "Footprint" "Skibidi-feet:RealOPtocoupler"
 			(at 96.52 143.51 0)
 			(effects
@@
 			)
 		)
-		(property "Footprint" "Skibidi-feet:Optocoupler"
+		(property "Footprint" "Skibidi-feet:RealOPtocoupler"
 			(at 46.99 111.76 0)
 			(effects
@@
 			)
 		)
-		(property "Footprint" ""
+		(property "Footprint" "Skibidi-feet:Screwterminal4"
 			(at 57.15 179.07 0)
 			(effects
@@
 			)
 		)
-		(property "Footprint" "Skibidi-feet:Optocoupler"
+		(property "Footprint" "Skibidi-feet:RealOPtocoupler"
 			(at 96.52 113.03 0)
 			(effects
@@
 			)
 		)
-		(property "Footprint" "Skibidi-feet:Optocoupler"
+		(property "Footprint" "Skibidi-feet:RealOPtocoupler"
 			(at 96.52 128.27 0)
 			(effects
@@
 			)
 		)
-		(property "Footprint" "Skibidi-feet:Optocoupler"
+		(property "Footprint" "Skibidi-feet:RealOPtocoupler"
 			(at 46.99 127 0)
 			(effects
@@
 			)
 		)
-		(property "Footprint" ""
+		(property "Footprint" "Capacitor_SMD:C_0805_2012Metric"
 			(at 274.0152 35.56 0)
 			(effects
@@
 			)
 		)
-		(property "Footprint" "Skibidi-feet:Optocoupler"
+		(property "Footprint" "Skibidi-feet:RealOPtocoupler"
 			(at 46.99 143.51 0)
 			(effects
@@
 			)
 		)
-		(property "Footprint" "Skibidi-feet:Optocoupler"
+		(property "Footprint" "Skibidi-feet:RealOPtocoupler"
 			(at 46.99 160.02 0)
 			(effects
@@
 			)
 		)
-		(property "Footprint" ""
+		(property "Footprint" "Capacitor_SMD:C_0805_2012Metric"
 			(at 227.6348 35.56 0)
 			(effects
@@
 			)
 		)
-		(property "Footprint" "Skibidi-feet:TEENSY"
+		(property "Footprint" "Skibidi-feet:Teensy4.1"
 			(at 165.1 77.47 0)
 			(effects

Commit message: progress on layout
Parts:
- removed J2: XT60-M, Skibidi-feet:XT60, symbol XT60-M:XT60-M
Connections:
- net +24V: no longer J1.P (POS), J18.P (POS)
- net at J14.P (POS): now also J1.N (NEG)
- new net: J1.P (POS), J18.P (POS)
Other:
- moved on the sheet: C15, D1, J14, J17, R8

Commit message: Layout progress
Connections:
- net +24V: now also J1.N (NEG), J14.P (POS)
Changed lines of the file:
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@@
 	)
 	(junction
+		(at 198.12 154.94)
+		(diameter 0)
+		(color 0 0 0 0)
+	)
+	(junction
 		(at 143.51 162.56)
 		(diameter 0)
@@
 					(unit 1)
 				)
+			)
+		)
+	)
+	(symbol
+		(lib_name "+24V_1")
+		(lib_id "power:+24V")
+		(at 198.12 154.94 180)
+		(unit 1)
+		(exclude_from_sim no)
+		(in_bom yes)
+		(on_board yes)
+		(dnp no)
+		(fields_autoplaced yes)
+		(property "Reference" "#PWR069"
+			(at 198.12 151.13 0)
+			(effects
+				(font
+					(size 1.27 1.27)
+				)
+				(hide yes)
+			)
+		)
+		(property "Value" "+24V"
+			(at 198.12 160.02 0)
+			(effects
+				(font
+					(size 1.27 1.27)
+				)
+			)
+		)
+		(property "Footprint" ""
+			(at 198.12 154.94 0)
+			(effects
+				(font
+					(size 1.27 1.27)
+				)
+				(hide yes)
+			)
+		)
+		(property "Datasheet" ""
+			(at 198.12 154.94 0)
+			(effects
+				(font
+					(size 1.27 1.27)
+				)
+				(hide yes)
+			)
+		)
+		(property "Description" "Power symbol creates a global label with name \"+24V\""
+			(at 198.12 154.94 0)
+			(effects
+				(font
+					(size 1.27 1.27)
+				)
+				(hide yes)
+			)
+		)
+		(pin "1"
+		)
+		(instances
+			(project ""
+				(path "/bfc511a5-2c92-46fd-9868-0fe25107d7eb"
+					(reference "#PWR069")
+					(unit 1)
+				)

Commit message: mode select
Parts:
- added SW2, SW3: 500SSP1S2M2QEA, Skibidi-feet:SWitch, symbol Connector_Audio:500SSP1S2M2QEA
Connections:
- net +3.3V: now also SW2.1, SW3.1
- net SelA: now reaches U8.36 (CS2)
- net SelA: now also SW2.2
- net SelB: now reaches U8.37 (CS3)
- net SelB: now also SW3.2
Other:
- moved on the sheet: C15, D1, J17, R8

Commit message: joe
Parts:
- added D2: D, symbol Device:D
Connections:
- net +24V: now also D2.1 (K); no longer J1.N (NEG), J14.P (POS)
- net SelA: now also SW2.3; no longer SW2.2
- net SelB: now also SW3.3; no longer SW3.2
- new net: D2.2 (A), J1.N (NEG), J14.P (POS)
Other:
- moved on the sheet: J1, J14, J16, J21, J22
