File: Skibidi/Skibid-i/Skibid-i.kicad_pcb (KiCad board)
At the start: 2 copper layers, 140 x 104.8 mm, 62 parts, among them IC1 TEENSY_4.1, J1 Conn_01x02_Pin, J10 Screw_Terminal_01x04, J11 Screw_Terminal_01x04, J12 Screw_Terminal_01x03, J13 P78E05-1000, J14 Conn_01x02_Pin, J15 Conn_01x03_Pin, J16 Conn_01x02_Pin, J17 Conn_01x08_Pin, J18 Conn_01x02_Pin, J19 Conn_01x02_Pin, J2 Screw_Terminal_01x03, J21 Motor1, J22 Motor2, J3 Screw_Terminal_01x03, J4 Screw_Terminal_01x03, J5 Screw_Terminal_01x03, J6 Screw_Terminal_01x03, J7 Screw_Terminal_01x03, J8 Screw_Terminal_01x03, J9 Screw_Terminal_01x03, Q1 WL-OCPT_SERIES_357, Q2 WL-OCPT_SERIES_357, Q3 WL-OCPT_SERIES_357, Q4 WL-OCPT_SERIES_357, Q5 WL-OCPT_SERIES_357, Q6 WL-OCPT_SERIES_357, Q7 WL-OCPT_SERIES_357, SW2 210-4MS, U10 TXB0108PWR

Commit message: layout
Parts:
- removed J11: Screw_Terminal_01x04, askibidi:Screwterimal4
- removed U10: TXB0108PWR, askibidi:levelshifter
- added J20: Screw_Terminal_01x03, askibidi:Screwterimanl3, F.Cu at (144.8, 35.7)
- J10: value Screw_Terminal_01x04 -> Screw_Terminal_01x03; footprint askibidi:Screwterimal4 -> askibidi:Screwterimanl3
- moved J10 12.1 mm to (267.1, 37.2), turned to 180 degrees
- moved C10 5.82 mm to (263.0, 43.6), turned to 180 degrees
- moved C11 1.91 mm to (148.8, 42.8), turned to 0 degrees
Connections:
- C10 pad 2: +5V -> +3.3V
- C11 pad 2: +5V -> +3.3V
- IC1 pad 14: LN1A -> LN1
- IC1 pad 15: LN2A -> LN2
- IC1 pad 16: LN3A -> LN3
- IC1 pad 17: LN4A -> LN4
- IC1 pad 18: LN5 -> unconnected-(IC1-A4-Pad18)
- IC1 pad 19: LN6 -> unconnected-(IC1-A5-Pad19)
- J10 pad 2: +5V -> +3.3V
- J12 pad 3: LN5 -> LN3
- J2 pad 3: LN6 -> LN4
Routing:
- net +5V: track 215.1 -> 34.3 mm
- net LN5: track 85.9 -> 0.00 mm
- net LN3: track 0.00 -> 85.9 mm
- net LN6: track 85.5 -> 0.00 mm
- net LN4: track 0.00 -> 85.5 mm
- net +3.3V: track 217.2 -> 230.8 mm

Commit message: Finished Layout Draft
Routing:
- net +3.3V: track 230.8 -> 403.2 mm
- net Start: track 0.00 -> 72.2 mm, vias 0 -> 1
- net LN2: track 0.00 -> 69.2 mm
- net LN1: track 0.00 -> 68.4 mm
- added copper zone on F.Cu, net GND

Commit message: layout done
Parts:
- removed C17: 22uF, Capacitor_SMD:C_0805_2012Metric
- added C18: 100uF, Capacitor_SMD:CP_Elec_6.3x5.4, F.Cu at (235.3, 109.8)
- C1: footprint Capacitor_SMD:C_0805_2012Metric -> askibidi:10uF
- C16: value 10uF -> 22uF; footprint Capacitor_SMD:C_0805_2012Metric -> askibidi:Ecap
- C2: footprint Capacitor_SMD:C_0805_2012Metric -> askibidi:Ecap
- moved C14 51.4 mm to (169.7, 85.8), turned to -90 degrees
- moved C1 19.2 mm to (251.2, 88.1), turned to 0 degrees
- moved C16 15.7 mm to (249.1, 109.5), turned to 0 degrees
- moved C2 2.62 mm to (226.2, 87.0)
Connections:
- C16 pad 1: GND -> +12V
- C16 pad 2: +48V -> GND
Routing:
- net +3.3V: track 403.2 -> 488.2 mm, vias 0 -> 2
- net +12V: track 215.7 -> 279.0 mm
- net LN4: track 85.5 -> 90.6 mm
- net LN3: track 85.9 -> 80.9 mm
- net +5V: track 34.3 -> 35.5 mm

Commit message: layout
Parts:
- moved D1 63.2 mm to (314.4, 63.4)
- moved R8 63.2 mm to (307.9, 63.3)
- moved J17 35.9 mm to (142.5, 78.6), turned to 90 degrees
- moved C14 31.2 mm to (138.4, 85.8)
- moved C13 28.5 mm to (271.0, 89.5), turned to -90 degrees
- moved C18 27.2 mm to (218.4, 88.5), turned to 180 degrees
- moved C15 24.6 mm to (142.5, 94.1)
- moved J1 24.6 mm to (179.3, 102.2)
- moved J12 24.6 mm to (140.5, 101.1)
- moved J14 24.6 mm to (162.4, 95.1)
- moved J18 24.6 mm to (193.2, 102.2)
- moved J21 24.6 mm to (212.5, 100.5)
- moved J22 24.6 mm to (226.1, 100.6)
- moved J2 24.5 mm to (270.7, 101.5)
- moved J19 23.8 mm to (245.1, 103.7), turned to 180 degrees
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Routing:
- net +3.3V: track 488.2 -> 307.2 mm
- net LN4: track 90.6 -> 42.5 mm
- net BDC22: track 61.0 -> 35.6 mm
- net BDC2: track 62.0 -> 36.9 mm
- net BDC1: track 83.1 -> 58.5 mm
- net BDC11: track 82.1 -> 59.1 mm
- net SDA: track 21.7 -> 0.00 mm
- net SCL: track 17.3 -> 0.00 mm
- net LN3: track 80.9 -> 73.2 mm
- net Net-(J18-Pin_2): track 18.5 -> 11.0 mm
- net Net-(D1-A): track 6.40 -> 0.00 mm
- net +5V: track 35.5 -> 29.6 mm
- net +12V: track 279.0 -> 275.0 mm
- net Net-(J1-Pin_2): track 8.40 -> 11.9 mm
- net Start: track 72.2 -> 69.7 mm
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Other:
- board size 140 x 104.8 mm -> 140 x 78.5 mm

Commit message: ig im done
Parts:
- removed J1: Conn_01x02_Pin, Connector_AMASS:AMASS_XT60-F_1x02_P7.20mm_Vertical
- moved R8 49.5 mm to (259.0, 71.1), turned to 180 degrees
- moved D1 48.0 mm to (267.1, 71.8), turned to 180 degrees
- moved J16 38.5 mm to (224.2, 82.8)
- moved J19 38.4 mm to (212.8, 82.8), turned to -90 degrees
- moved J22 26.3 mm to (202.9, 88.3)
- moved C14 24.8 mm to (150.9, 64.4)
- moved J18 24.6 mm to (177.4, 83.2), turned to -90 degrees
- moved J21 24.2 mm to (191.5, 88.4)
- moved R7 22.9 mm to (160.2, 56.8), turned to 90 degrees
- moved Q5 19.1 mm to (167.9, 55.7), turned to 0 degrees
- moved C1 17.1 mm to (241.4, 71.7), turned to 180 degrees
- moved F1 17.0 mm to (171.8, 96.3)
- moved C18 16.6 mm to (234.7, 91.7)
- moved C15 15.1 mm to (152.5, 82.8), turned to -90 degrees
- moved J17 14.5 mm to (146.1, 64.6), turned to 0 degrees
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Connections:
- F1 pad 2: Net-(J1-Pin_2) -> Net-(J14-Pin_2)
- J14 pad 2: Net-(J1-Pin_1) -> Net-(J14-Pin_2)
- J15 pad 2: +3.3V -> GND
- J15 pad 3: GND -> +3.3V
Routing:
- net SDA: track 0.00 -> 48.5 mm
- net SCL: track 0.00 -> 46.2 mm
- net +3.3V: track 307.2 -> 340.7 mm, vias 2 -> 1
- net BDC1: track 58.5 -> 33.8 mm
- net BDC11: track 59.1 -> 34.9 mm
- net +48V: track 58.9 -> 37.5 mm
- net BDC2: track 36.9 -> 15.9 mm
- net Dis7: track 58.1 -> 37.2 mm
- net BDC22: track 35.6 -> 14.9 mm
- net Net-(J1-Pin_1): track 17.0 -> 0.00 mm
- net LN4: track 42.5 -> 58.1 mm
- net Net-(J1-Pin_2): track 11.9 -> 0.00 mm
- net +5V: track 29.6 -> 41.4 mm
- net LN3: track 73.2 -> 61.7 mm
- net Net-(J14-Pin_2): track 0.00 -> 7.64 mm
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Other:
- board size 140 x 78.5 mm -> 128.7 x 68 mm

Commit message: erm what the sigma
Other:
- board size 128.7 x 68 mm -> 128.7 x 66.8 mm
Changed lines of the file:
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@@
 		(at 243.8625 81.75)
 		(property "Reference" "PS1"
-			(at 0 0 360)
+			(at 0 0 0)
 			(layer "F.SilkS")
 			(effects
@@
 		)
 		(property "Value" "RSO-4812S_H2"
-			(at -0.355 5.665 360)
+			(at -0.355 5.665 0)
 			(layer "F.Fab")
 			(effects
@@
 		)
 		(property "Footprint" "askibidi:12vConvertor"
-			(at 0 0 360)
+			(at 0 0 0)
 			(layer "F.Fab")
 			(hide yes)
@@
 		)
 		(property "Datasheet" ""
-			(at 0 0 360)
+			(at 0 0 0)
 			(layer "F.Fab")
 			(hide yes)
@@
 		)
 		(property "Description" ""
-			(at 0 0 360)
+			(at 0 0 0)
 			(layer "F.Fab")
 			(hide yes)
@@
 		(tags "Through hole pin header THT 1x03 2.54mm single row")
 		(property "Reference" "J15"
-			(at 0 -2.33 360)
+			(at 0 -2.33 0)
 			(layer "F.SilkS")
 			(effects
@@
 		)
 		(property "Value" "Conn_01x03_Pin"
-			(at 0 7.41 360)
+			(at 0 7.41 0)
 			(layer "F.Fab")
 			(effects
@@
 		(tags "capacitor")
 		(property "Reference" "C13"
-			(at 0 -1.68 360)
+			(at 0 -1.68 0)
 			(layer "F.SilkS")
 			(effects
@@
 		)
 		(property "Value" "0.1uF"
-			(at 0 1.68 360)
+			(at 0 1.68 0)
 			(layer "F.Fab")
 			(effects
@@
 		)
 		(fp_text user "${REFERENCE}"
-			(at 0 0 360)
+			(at 0 0 0)
 			(layer "F.Fab")
 			(effects
@@
 		(tags "capacitor")
 		(property "Reference" "R8"
-			(at 0 -1.85 360)
+			(at 0 -1.85 0)
 			(layer "F.SilkS")
 			(effects
@@
 		)
 		(property "Value" "500ohm"
-			(at 0 1.85 360)
+			(at 0 1.85 0)
 			(layer "F.Fab")
 			(effects
@@
 		)
 		(fp_text user "${REFERENCE}"
-			(at 0 0 360)
+			(at 0 0 0)
 			(layer "F.Fab")
 			(effects
@@
 		)
 		(property "Footprint" "askibidi:5vregulator"
-			(at 0 0 360)
+			(at 0 0 0)
 			(layer "F.Fab")
 			(hide yes)
@@
 		)
 		(property "Datasheet" "P78E05-1000"
-			(at 0 0 360)
+			(at 0 0 0)
 			(layer "F.Fab")
 			(hide yes)
@@
 		)
 		(property "Description" ""
-			(at 0 0 360)
+			(at 0 0 0)
 			(layer "F.Fab")
 			(hide yes)
@@
 		)
 		(property "Footprint" "askibidi:LED"
-			(at 0 0 360)
+			(at 0 0 0)
 			(layer "F.Fab")
 			(hide yes)
@@
 		)
 		(property "Datasheet" ""
-			(at 0 0 360)
+			(at 0 0 0)
 			(layer "F.Fab")
 			(hide yes)
@@
 		)
 		(property "Description" "Light emitting diode"
-			(at 0 0 360)
+			(at 0 0 0)
 			(layer "F.Fab")
 			(hide yes)
@@
 		(tags "capacitor electrolytic")
 		(property "Reference" "C18"
-			(at 0 -4.35 360)
+			(at 0 -4.35 0)
 			(layer "F.SilkS")
 			(effects
@@
 		)
 		(property "Value" "100uF"
-			(at 0 4.35 360)
+			(at 0 4.35 0)
 			(layer "F.Fab")
 			(effects
@@
 		)
 		(fp_text user "${REFERENCE}"
-			(at 0 0 360)
+			(at 0 0 0)
 			(layer "F.Fab")
 			(effects
@@
 		(descr "<b> WL-OCPT Optocoupler Phototransistor</b><br>Size : SOP4, SMT, 4pins")
 		(property "Reference" "Q5"
-			(at 0 -3.235 360)
+			(at 0 -3.235 0)
 			(layer "F.SilkS")
 			(effects
@@
 		)
 		(property "Value" "WL-OCPT_SERIES_357"
-			(at 0.05 -4.8899 360)
+			(at 0.05 -4.8899 0)
 			(layer "F.Fab")
 			(effects
@@
 		)
 		(property "Footprint" "askibidi:optopt"
-			(at 0 0 360)
+			(at 0 0 0)
 			(layer "F.Fab")
 			(hide yes)
@@
 		)
 		(property "Datasheet" ""
-			(at 0 0 360)
+			(at 0 0 0)
 			(layer "F.Fab")
 			(hide yes)
@@
 		)
 		(property "Description" ""
-			(at 0 0 360)
+			(at 0 0 0)
 			(layer "F.Fab")
 			(hide yes)
@@
 		(descr "<B>WCAP-ASLI</B><BR> Aluminium Electrolytic Capacitors,4X5.5X1(DiameterXLengthXPitch)")
 		(property "Reference" "C1"
-			(at -0.3 -3.5064 360)
+			(at -0.3 -3.5064 0)
 			(layer "F.SilkS")
 			(effects
@@
 		)
 		(property "Value" "10uF"
-			(at -0.5 3.4936 360)
+			(at -0.5 3.4936 0)
 			(layer "F.Fab")
 			(effects
@@
 		)
 		(property "Footprint" "askibidi:10uF"
-			(at 0 0 360)
+			(at 0 0 0)
 			(layer "F.Fab")
 			(hide yes)
@@
 		)
 		(property "Datasheet" ""
-			(at 0 0 360)
+			(at 0 0 0)
 			(layer "F.Fab")
 			(hide yes)
@@
 		)
 		(property "Description" "Unpolarized capacitor"
-			(at 0 0 360)
+			(at 0 0 0)
 			(layer "F.Fab")
 			(hide yes)
@@
 		)
 		(fp_text user "+"
-			(at 2.9 2.1 360)
+			(at 2.9 2.1 0)
 			(layer "F.SilkS")
 			(effects
@@
 		(tags "capacitor")
 		(property "Reference" "C12"
-			(at 0 -1.68 360)
+			(at 0 -1.68 0)
 			(layer "F.SilkS")
 			(effects
@@
 		)
 		(property "Value" "0.1uF"
-			(at 0 1.68 360)
+			(at 0 1.68 0)
 			(layer "F.Fab")
 			(effects
@@
 		)
 		(fp_text user "${REFERENCE}"
-			(at 0 0 360)
+			(at 0 0 0)
 			(layer "F.Fab")
 			(effects
@@
 		(tags "fuse")
 		(property "Reference" "F1"
-			(at 0 -1.82 360)
+			(at 0 -1.82 0)
 			(layer "F.SilkS")
 			(effects
@@
 		)
 		(property "Value" "Fuse"
-			(at 0 1.82 360)
+			(at 0 1.82 0)
 			(layer "F.Fab")
 			(effects
@@
 		)
 		(fp_text user "${REFERENCE}"
-			(at 0 0 360)
+			(at 0 0 0)
 			(layer "F.Fab")
 			(effects
@@
 		(tags "Through hole pin header THT 1x08 2.54mm single row")
 		(property "Reference" "J17"
-			(at 0 -2.33 360)
+			(at 0 -2.33 0)
 			(layer "F.SilkS")
 			(effects
@@
 		)
 		(property "Value" "Conn_01x08_Pin"
-			(at -0.08 23.06 360)
+			(at -0.08 23.06 0)
 			(layer "F.Fab")
 			(effects
@@
 		(at 250.95 71.7)
 		(property "Reference" "C2"
-			(at 0.475 -4.685 360)
+			(at 0.475 -4.685 0)
 			(layer "F.SilkS")
 			(effects
@@
 		)
 		(property "Value" "22uF"
-			(at 0.35 2.05 360)
+			(at 0.35 2.05 0)
 			(layer "F.Fab")
 			(effects
@@
 		)
 		(property "Footprint" "askibidi:Ecap"
-			(at 0 0 360)
+			(at 0 0 0)
 			(layer "F.Fab")
 			(hide yes)
@@
 		)
 		(property "Datasheet" ""
-			(at 0 0 360)
+			(at 0 0 0)
 			(layer "F.Fab")
 			(hide yes)
@@
 		)
 		(property "Description" "Unpolarized capacitor"
-			(at 0 0 360)
+			(at 0 0 0)
 			(layer "F.Fab")
 			(hide yes)
@@
 		(at 250.2125 91.95)
 		(property "Reference" "C16"
-			(at 0.475 -4.685 360)
+			(at 0.475 -4.685 0)
 			(layer "F.SilkS")
 			(effects
@@
 		)
 		(property "Value" "22uF"
-			(at 4.1 -4.85 360)
+			(at 4.1 -4.85 0)
 			(layer "F.Fab")
 			(effects
@@
 		)
 		(property "Footprint" "askibidi:Ecap"
-			(at 0 0 360)
+			(at 0 0 0)
 			(layer "F.Fab")
 			(hide yes)
@@
 		)
 		(property "Datasheet" ""
-			(at 0 0 360)
+			(at 0 0 0)
 			(layer "F.Fab")
 			(hide yes)
@@
 		)
 		(property "Description" "Polarized capacitor, US symbol"
-			(at 0 0 360)
+			(at 0 0 0)
 			(layer "F.Fab")
 			(hide yes)
@@
 	)
 	(gr_rect
-		(start 143.75 29.5)
+		(start 143.75 30.8)
 		(end 272.496 97.55)
 		(stroke
@@
 	)
 	(segment
-		(start 211.654899 51.794899)
-		(end 219.31 59.45)
+		(start 211.654899 50.57)
+		(end 211.654899 51.154899)
 		(width 0.25)
 		(layer "F.Cu")
@@
 	)
 	(segment
-		(start 211.654899 50.57)
-		(end 211.654899 51.794899)
+		(start 211.654899 51.154899)
+		(end 219.31 58.81)
 		(width 0.25)
 		(layer "F.Cu")
@@
 	)
 	(segment
+		(start 219.31 58.81)
+		(end 219.31 59.45)
+		(width 0.25)
+		(layer "F.Cu")
+		(net 46)
+	)
+	(segment
 		(start 250.645101 60.445101)
 		(end 257.43 60.445101)
@@
 	)
 	(segment
-		(start 210.52 53.2)
-		(end 216.77 59.45)
+		(start 193.954899 50.77)
+		(end 196.384899 53.2)
+		(width 0.25)
+		(layer "F.Cu")
+		(net 59)
+	)
+	(segment
+		(start 210.4 53.2)
+		(end 216.65 59.45)
 		(width 0.25)
 		(layer "F.Cu")
@@
 	(segment
 		(start 196.384899 53.2)
-		(end 210.52 53.2)
+		(end 210.4 53.2)
 		(width 0.25)
 		(layer "F.Cu")
@@
 	)
 	(segment
-		(start 193.954899 50.77)
-		(end 196.384899 53.2)
+		(start 216.65 59.45)
+		(end 216.77 59.45)
 		(width 0.25)
 		(layer "F.Cu")
@@
 		(polygon
 			(pts
-				(xy 144.05 29.725) (xy 143.7 97.625) (xy 272.304 97.470101) (xy 272.654 29.570101)
+				(xy 143.823 30.875) (xy 143.7 97.625) (xy 272.304 97.470101) (xy 272.427 30.720101)
 			)
 		)

Commit message: sigma moves
Parts:
- removed F1: Fuse, Fuse:Fuse_1206_3216Metric
- added F2: 3587, askibidi:Fusemount, F.Cu at (174.3, 87.0)
- J14: value Conn_01x02_Pin -> Battery
- J18: value Conn_01x02_Pin -> SparkIN
- J19: value Conn_01x02_Pin -> SparkOUT
- moved J18 9.92 mm to (184.0, 90.7), turned to 90 degrees
- moved Q1 8.28 mm to (262.7, 50.0), turned to 180 degrees
- moved J21 5.73 mm to (197.1, 89.8)
- moved J22 5.46 mm to (208.2, 89.7)
- moved R1 5.45 mm to (269.7, 50.1), turned to 90 degrees
- moved J19 3.96 mm to (216.8, 83.0)
- moved C18 2.87 mm to (237.6, 92.0), turned to -90 degrees
- moved J16 2.55 mm to (226.8, 82.9)
- moved J14 1.90 mm to (164.6, 83.6)
- moved R8 0.75 mm to (259.0, 71.8)
- moved J12 0.42 mm to (147.1, 89.5)
- moved C15 0.30 mm to (152.2, 82.9)
Routing:
- net +48V: track 37.5 -> 30.1 mm
- net Net-(J14-Pin_2): track 7.64 -> 14.2 mm
- net BDC1: track 33.8 -> 39.2 mm
- net BDC22: track 14.9 -> 18.6 mm
- net BDC2: track 15.9 -> 19.6 mm
- net BDC11: track 34.9 -> 38.4 mm
- net Dis1: track 34.4 -> 37.8 mm
- net OM1: track 5.58 -> 6.88 mm

Commit message: sigma moves
Routing:
- net +12V: track 280.9 -> 287.4 mm
Other:
- board text added: "A16"
- board text added: "A17"
- board text added: "Erm What the Skibidi..."
- board text added: "Pin10"
- board text added: "Pin2"
- board text added: "Pin3"
- board text added: "Pin4"
- board text added: "Pin5"
- board text added: "Pin6"
- board text added: "Pin9"
