File: Skibidi/Skibid-i/Skibidi-Motordriver/Skibidi-Motordriver.kicad_pcb (KiCad board)
At the start: 2 copper layers, 21 parts, among them J1 XT90, J2 XT90, J3 Screw_Terminal_01x02, J5 XT90, J6 Screw_Terminal_01x03, Q1 IGBT, Q2 IGBT, Q3 IGBT, Q4 IGBT, Q5 IGBT, Q6 IGBT, Q7 IGBT, Q8 IGBT, U3 SFH617A-1, U4 SFH617A-1, U5 SFH617A-1, U6 SFH617A-1

Commit message: finished motordriver layout
Parts:
- removed J3: Screw_Terminal_01x02, Skibidi-feet:Screwterminal2
- removed J6: Screw_Terminal_01x03, Skibidi-feet:ScrewTerminal3
- removed R1, R2, R3, R4: 10kΩ, Resistor_SMD:R_1206_3216Metric
- removed U3, U4, U5, U6: SFH617A-1, Skibidi-feet:Optocoupler
- added J7: Screw_Terminal_01x02, Skibidi-feet:Screwterminal2, F.Cu at (133.9, 119.5)
- added J8: Screw_Terminal_01x02, Skibidi-feet:Screwterminal2, F.Cu at (174.5, 119.0)
- moved J5 17.5 mm to (152.5, 117.0)
- moved Q5 1.56 mm to (144.0, 87.8)
- moved Q7 1.50 mm to (144.0, 69.9)
- moved Q4 1.07 mm to (160.5, 69.9)
- moved Q1 1.00 mm to (177.5, 87.3)
- moved Q2 1.00 mm to (177.5, 69.5)
- moved Q3 1.00 mm to (160.5, 87.3)
- moved J1 0.95 mm to (165.5, 55.5)
- moved Q6 0.61 mm to (127.0, 88.0)
Connections:
- J5 pad N: Bat- -> GND
- Q2 pad 2: Bat- -> GND
- Q4 pad 2: Bat- -> GND
- Q7 pad 2: Bat- -> GND
- Q8 pad 2: Bat- -> GND
Routing:
- net Bat-: track 88.6 -> 0.00 mm
- net BDC1: track 0.00 -> 60.7 mm
- net BDC11: track 0.00 -> 60.7 mm, vias 0 -> 2
- net BDC2: track 0.00 -> 60.4 mm, vias 0 -> 2
- net BDC22: track 23.8 -> 61.5 mm
- net +48V: track 44.3 -> 59.7 mm
- net Net-(J1-POS): track 51.0 -> 37.0 mm
- net Net-(J2-NEG): track 50.3 -> 38.5 mm
- net Net-(J1-NEG): track 56.5 -> 60.2 mm
- net Net-(J2-POS): track 58.7 -> 60.2 mm
- net Motor1A: track 1.00 -> 0.00 mm
- net Net-(R3-Pad2): track 0.71 -> 0.00 mm
- added copper zone on B.Cu, net GND
Other:
- board outline added: 65.5 x 94 mm

Commit message: progress on layout
Changed lines of the file:
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@@
 		)
 		(property "Footprint" "Skibidi-feet:Screwterminal2"
-			(at 0 0 360)
+			(at 0 0 0)
 			(layer "F.Fab")
 			(hide yes)
@@
 		)
 		(property "Datasheet" ""
-			(at 0 0 360)
+			(at 0 0 0)
 			(layer "F.Fab")
 			(hide yes)
@@
 		)
 		(property "Description" "Generic screw terminal, single row, 01x02, script generated (kicad-library-utils/schlib/autogen/connector/)"
-			(at 0 0 360)
+			(at 0 0 0)
 			(layer "F.Fab")
 			(hide yes)
@@
 		)
 		(property "Footprint" "Skibidi-feet:Screwterminal2"
-			(at 0 0 360)
+			(at 0 0 0)
 			(layer "F.Fab")
 			(hide yes)
@@
 		)
 		(property "Datasheet" ""
-			(at 0 0 360)
+			(at 0 0 0)
 			(layer "F.Fab")
 			(hide yes)
@@
 		)
 		(property "Description" "Generic screw terminal, single row, 01x02, script generated (kicad-library-utils/schlib/autogen/connector/)"
-			(at 0 0 360)
+			(at 0 0 0)
 			(layer "F.Fab")
 			(hide yes)
@@
 	)
 	(segment
-		(start 138.5 82)
-		(end 134.5 78)
+		(start 137 81.5)
+		(end 133.75 78.25)
 		(width 0.2)
 		(layer "F.Cu")
@@
 	)
 	(via
-		(at 134.5 78)
+		(at 137 81.5)
 		(size 0.6)
 		(drill 0.3)
@@
 	)
 	(via
-		(at 138.5 82)
+		(at 133.75 78.25)
 		(size 0.6)
 		(drill 0.3)
@@
 	)
 	(segment
-		(start 133.8951 97.9313)
-		(end 144 87.8264)
+		(start 127 71.5)
+		(end 133.75 78.25)
 		(width 0.2)
 		(layer "B.Cu")
@@
 	)
 	(segment
-		(start 133.8951 119.499999)
-		(end 133.8951 97.9313)
+		(start 133.8951 97.9313)
+		(end 144 87.8264)
 		(width 0.2)
 		(layer "B.Cu")
@@
 	)
 	(segment
-		(start 134.5 77.5142)
-		(end 127 70.0142)
+		(start 144 87.8264)
+		(end 143.3264 87.8264)
 		(width 0.2)
 		(layer "B.Cu")
@@
 	)
 	(segment
-		(start 144 87.8264)
-		(end 138.5 82.3264)
+		(start 143.3264 87.8264)
+		(end 137 81.5)
 		(width 0.2)
 		(layer "B.Cu")
@@
 	)
 	(segment
-		(start 134.5 78)
-		(end 134.5 77.5142)
+		(start 133.8951 119.499999)
+		(end 133.8951 97.9313)
 		(width 0.2)
 		(layer "B.Cu")
@@
 	)
 	(segment
-		(start 138.5 82.3264)
-		(end 138.5 82)
+		(start 127 70.0142)
+		(end 127 71.5)
 		(width 0.2)
 		(layer "B.Cu")

Commit message: finish motor driver
Parts:
- removed J1: XT90, Skibidi-feet:xt90Female
- removed Q1, Q2, Q3, Q4: IGBT, Skibidi-feet:IGBT
- added D1: D_Schottky_AKA, Skibidi-feet:SchottkyDiode, F.Cu at (162.7, 74.4)
- added D2: D_Schottky_AKA, Skibidi-feet:SchottkyDiode, F.Cu at (162.5, 93.0)
- added D3: D_Schottky_AKA, Skibidi-feet:SchottkyDiode, F.Cu at (134.3, 93.6)
- added D4: D_Schottky_AKA, Skibidi-feet:SchottkyDiode, F.Cu at (134.1, 74.4)
- added D5: D_Schottky_AKA, Skibidi-feet:SchottkyDiode, F.Cu at (176.4, 73.3)
- added D6: D_Schottky_AKA, Skibidi-feet:SchottkyDiode, F.Cu at (177.3, 94.4)
- added D7: D_Schottky_AKA, Skibidi-feet:SchottkyDiode, F.Cu at (204.6, 72.7)
- added D8: D_Schottky_AKA, Skibidi-feet:SchottkyDiode, F.Cu at (204.2, 94.5)
- added J3: XT90, Skibidi-feet:xt90Female, F.Cu at (195.7, 50.7)
- added Q10: IGBT, Skibidi-feet:IGBT, F.Cu at (185.4, 102.8)
- added Q11: IGBT, Skibidi-feet:IGBT, F.Cu at (196.9, 81.0)
- added Q12: IGBT, Skibidi-feet:IGBT, F.Cu at (196.8, 103.3)
- added Q9: IGBT, Skibidi-feet:IGBT, F.Cu at (185.5, 80.7)
- moved J5 68.8 mm to (171.6, 51.0), turned to 180 degrees
- moved Q8 42.3 mm to (154.7, 102.0), turned to 90 degrees
- moved Q7 32.0 mm to (143.2, 102.0), turned to 90 degrees
- moved Q6 28.1 mm to (154.6, 82.6), turned to 90 degrees
- moved J8 20.2 mm to (193.6, 112.4)
- moved J7 18.5 mm to (151.3, 113.2)
- moved J2 8.95 mm to (145.5, 51.2), turned to 180 degrees
- moved Q5 5.57 mm to (143.3, 82.3), turned to 90 degrees
Routing:
- net Net-(J1-NEG): track 60.2 -> 0.00 mm
- net Net-(D8-K): track 0.00 -> 59.4 mm
- net Net-(D6-K): track 0.00 -> 57.4 mm
- net Net-(J1-POS): track 37.0 -> 0.00 mm
- net +48V: track 59.7 -> 96.2 mm
- net BDC11: track 61.1 -> 37.0 mm, vias 2 -> 1
- net BDC1: track 60.7 -> 37.7 mm, vias 0 -> 1
- net Net-(D3-K): track 38.5 -> 60.0 mm
- net BDC22: track 61.5 -> 72.8 mm
- net BDC2: track 60.4 -> 71.2 mm, vias 2 -> 0
- net Net-(D2-K): track 60.2 -> 53.7 mm
Other:
- board outline removed

Commit message: Layout progress
Changed lines of the file:
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@@
 		(at 171.6 50.95 180)
 		(property "Reference" "J5"
-			(at -7.475 -15.005 360)
+			(at -7.475 -15.005 0)
 			(layer "F.SilkS")
 			(effects
@@
 		)
 		(property "Value" "XT90"
-			(at -1.76 -13.445 360)
+			(at -1.76 -13.445 0)
 			(layer "F.Fab")
 			(effects
@@
 		)
 		(property "Footprint" "Skibidi-feet:xt90Female"
-			(at 0 0 360)
+			(at 0 0 0)
 			(layer "F.Fab")
 			(hide yes)
@@
 		)
 		(property "Datasheet" ""
-			(at 0 0 360)
+			(at 0 0 0)
 			(layer "F.Fab")
 			(hide yes)
@@
 		)
 		(property "Description" ""
-			(at 0 0 360)
+			(at 0 0 0)
 			(layer "F.Fab")
 			(hide yes)
@@
 		(at 145.5 51.25 180)
 		(property "Reference" "J2"
-			(at -7.475 -15.005 360)
+			(at -7.475 -15.005 0)
 			(layer "F.SilkS")
 			(effects
@@
 		)
 		(property "Value" "XT90"
-			(at -1.76 -13.445 360)
+			(at -1.76 -13.445 0)
 			(layer "F.Fab")
 			(effects
@@
 		)
 		(property "Footprint" "Skibidi-feet:xt90Female"
-			(at 0 0 360)
+			(at 0 0 0)
 			(layer "F.Fab")
 			(hide yes)
@@
 		)
 		(property "Datasheet" ""
-			(at 0 0 360)
+			(at 0 0 0)
 			(layer "F.Fab")
 			(hide yes)
@@
 		)
 		(property "Description" ""
-			(at 0 0 360)
+			(at 0 0 0)
 			(layer "F.Fab")
 			(hide yes)
@@
 		(at 195.7 50.7 180)
 		(property "Reference" "J3"
-			(at -7.475 -15.005 360)
+			(at -7.475 -15.005 0)
 			(layer "F.SilkS")
 			(effects
@@
 		)
 		(property "Value" "XT90"
-			(at -1.76 -13.445 360)
+			(at -1.76 -13.445 0)
 			(layer "F.Fab")
 			(effects
@@
 		)
 		(property "Footprint" "Skibidi-feet:xt90Female"
-			(at 0 0 360)
+			(at 0 0 0)
 			(layer "F.Fab")
 			(hide yes)
@@
 		)
 		(property "Datasheet" ""
-			(at 0 0 360)
+			(at 0 0 0)
 			(layer "F.Fab")
 			(hide yes)
@@
 		)
 		(property "Description" ""
-			(at 0 0 360)
+			(at 0 0 0)
 			(layer "F.Fab")
 			(hide yes)
@@
 		)
 		(property "Footprint" "Skibidi-feet:Screwterminal2"
-			(at 0 0 360)
+			(at 0 0 0)
 			(layer "F.Fab")
 			(hide yes)
@@
 		)
 		(property "Datasheet" ""
-			(at 0 0 360)
+			(at 0 0 0)
 			(layer "F.Fab")
 			(hide yes)
@@
 		)
 		(property "Description" "Generic screw terminal, single row, 01x02, script generated (kicad-library-utils/schlib/autogen/connector/)"
-			(at 0 0 360)
+			(at 0 0 0)
 			(layer "F.Fab")
 			(hide yes)
@@
 		)
 		(property "Footprint" "Skibidi-feet:Screwterminal2"
-			(at 0 0 360)
+			(at 0 0 0)
 			(layer "F.Fab")
 			(hide yes)
@@
 		)
 		(property "Datasheet" ""
-			(at 0 0 360)
+			(at 0 0 0)
 			(layer "F.Fab")
 			(hide yes)
@@
 		)
 		(property "Description" "Generic screw terminal, single row, 01x02, script generated (kicad-library-utils/schlib/autogen/connector/)"
-			(at 0 0 360)
+			(at 0 0 0)
 			(layer "F.Fab")
 			(hide yes)
@@
 		)
 	)
+	(gr_rect
+		(start 130 34)
+		(end 213 119.5)
+		(stroke
+			(width 0.2)
+			(type default)
+		)
+		(fill none)
+		(layer "F.Cu")
+	)
 	(segment
 		(start 151.67325 79.93705)
@@
 		(start 176.4 75.851)
 		(end 179.1974 75.851)
-		(width 0.2)
+		(width 1.3)
 		(layer "F.Cu")
 		(net 3)
@@
 		(polygon
 			(pts
-				(xy 129.2 34.3) (xy 213.8 34.1) (xy 213.1 119.1) (xy 129.2 119.9)
+				(xy 130 34) (xy 213 34) (xy 213 119.5) (xy 130 119.5)
 			)
 		)

Commit message: joe
Parts:
- moved D3 22.9 mm to (111.4, 93.6)
- moved D4 22.9 mm to (111.2, 74.4)
- moved Q5 22.9 mm to (120.4, 82.3)
- moved Q7 22.9 mm to (120.3, 102.0)
Routing:
- net +48V: track 96.2 -> 66.3 mm
- net BDC11: track 37.0 -> 14.9 mm
- net Net-(D3-K): track 60.0 -> 40.3 mm
- net BDC22: track 72.8 -> 60.2 mm
Changed lines of the file:
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@@
 	(footprint "Skibidi-feet:SchottkyDiode"
 		(layer "F.Cu")
-		(at 134.07325 74.35965 -90)
+		(at 111.1513 74.35965 -90)
 		(tags "STPS20H100CT ")
 		(property "Reference" "D4"
@@
 	(footprint "Skibidi-feet:SchottkyDiode"
 		(layer "F.Cu")
-		(at 134.27325 93.59965 -90)
+		(at 111.3513 93.59965 -90)
 		(tags "STPS20H100CT ")
 		(property "Reference" "D3"
@@
 	(footprint "Skibidi-feet:IGBT"
 		(layer "F.Cu")
-		(at 143.27325 82.29965 90)
+		(at 120.3513 82.29965 90)
 		(tags "FGH75T65SHD-F155 ")
 		(property "Reference" "Q5"
@@
 	(footprint "Skibidi-feet:IGBT"
 		(layer "F.Cu")
-		(at 143.17325 101.96225 90)
+		(at 120.2513 101.96225 90)
 		(tags "FGH75T65SHD-F155 ")
 		(property "Reference" "Q7"
@@
 	)
 	(gr_rect
-		(start 130 34)
+		(start 105 34)
 		(end 213 119.5)
 		(stroke
@@
 	)
 	(segment
-		(start 158.6477 67.4)
-		(end 171.8 67.4)
-		(width 1.3)
-		(layer "F.Cu")
-		(net 3)
-	)
-	(segment
 		(start 177.05 62.15)
 		(end 177.05 60.35)
@@
 	)
 	(segment
-		(start 137.54805 76.89965)
-		(end 143.27325 71.17445)
+		(start 114.6261 76.89965)
+		(end 120.3513 71.17445)
 		(width 1.3)
 		(layer "F.Cu")
@@
 	)
 	(segment
-		(start 154.57325 71.47445)
-		(end 158.6477 67.4)
-		(width 1.3)
-		(layer "F.Cu")
-		(net 3)
-	)
-	(segment
-		(start 143.27325 71.17445)
-		(end 154.27325 71.17445)
-		(width 1.3)
-		(layer "F.Cu")
-		(net 3)
-	)
-	(segment
 		(start 185.5 69.5484)
 		(end 185.5 68.8)
@@
 	)
 	(segment
-		(start 134.07325 76.89965)
-		(end 137.54805 76.89965)
+		(start 111.1513 76.89965)
+		(end 114.6261 76.89965)
 		(width 1.3)
 		(layer "F.Cu")
@@
 		(net 7)
 	)
-	(segment
-		(start 154.67325 109.79965)
-		(end 151.27325 113.19965)
-		(width 1)
-		(layer "F.Cu")
-		(net 7)
-	)
-	(segment
-		(start 154.67325 101.96225)
-		(end 154.67325 109.79965)
-		(width 1)
-		(layer "F.Cu")
-		(net 7)
-	)
 	(via
 		(at 149.97325 97.19965)
@@
 	)
 	(segment
-		(start 149.97325 88.99965)
-		(end 143.27325 82.29965)
-		(width 1)
-		(layer "B.Cu")
-		(net 7)
-	)
-	(segment
 		(start 149.97325 97.19965)
 		(end 149.97325 88.99965)
@@
 	)
 	(segment
-		(start 143.17325 101.96225)
-		(end 143.17325 110.09965)
-		(width 1)
-		(layer "F.Cu")
-		(net 8)
-	)
-	(segment
-		(start 143.17325 110.09965)
-		(end 146.27325 113.19965)
-		(width 1)
-		(layer "F.Cu")
-		(net 8)
-	)
-	(segment
 		(start 163.37325 82.59965)
 		(end 154.57325 82.59965)
@@
 	)
 	(segment
-		(start 146.47325 87.53705)
-		(end 143.17325 90.83705)
+		(start 123.5513 87.53705)
+		(end 120.2513 90.83705)
 		(width 1.3)
 		(layer "F.Cu")
@@
 	)
 	(segment
-		(start 137.87065 96.13965)
-		(end 143.17325 90.83705)
+		(start 114.9487 96.13965)
+		(end 120.2513 90.83705)
 		(width 1.3)
 		(layer "F.Cu")
@@
 	)
 	(segment
-		(start 143.27325 76.73705)
-		(end 146.47325 79.93705)
+		(start 120.3513 76.73705)
+		(end 123.5513 79.93705)
 		(width 1.3)
 		(layer "F.Cu")
@@
 	)
 	(segment
-		(start 140.57065 79.43965)
-		(end 143.27325 76.73705)
+		(start 117.6487 79.43965)
+		(end 120.3513 76.73705)
 		(width 1.3)
 		(layer "F.Cu")
@@
 	)
 	(segment
-		(start 134.07325 79.43965)
-		(end 140.57065 79.43965)
+		(start 111.1513 79.43965)
+		(end 117.6487 79.43965)
 		(width 1.3)
 		(layer "F.Cu")
@@
 	)
 	(segment
-		(start 134.27325 96.13965)
-		(end 137.87065 96.13965)
+		(start 111.3513 96.13965)
+		(end 114.9487 96.13965)
 		(width 1.3)
 		(layer "F.Cu")
@@
 	)
 	(segment
-		(start 146.47325 79.93705)
-		(end 146.47325 87.53705)
+		(start 123.5513 79.93705)
+		(end 123.5513 87.53705)
 		(width 1.3)
 		(layer "F.Cu")
@@
 	)
 	(segment
-		(start 147.1 72.9103)
-		(end 147.1 65.6)
-		(width 1.3)
-		(layer "B.Cu")
-		(net 10)
-	)
-	(segment
 		(start 142.15 60.65)
 		(end 140.05 60.65)
 		(width 1.3)
 		(layer "B.Cu")
-		(net 10)
-	)
-	(segment
-		(start 143.27325 76.73705)
-		(end 147.1 72.9103)
-		(width 1.3)
-		(layer "B.Cu")
-		(net 10)
-	)
-	(segment
-		(start 147.1 65.6)
-		(end 142.15 60.65)
-		(width 1.3)
-		(layer "B.Cu")

Commit message: joe
Parts:
- moved D3 16.2 mm to (127.5, 92.9)
- moved D4 15.4 mm to (126.5, 73.5)
- moved J2 12.5 mm to (133.0, 51.5)
- moved Q10 11.0 mm to (174.4, 103.6)
- moved Q9 11.0 mm to (174.5, 81.5)
- moved J5 8.72 mm to (163.0, 49.5)
- moved D1 7.67 mm to (155.1, 74.4)
- moved D2 7.67 mm to (154.8, 93.0)
- moved J7 7.67 mm to (143.6, 113.2)
- moved Q6 7.67 mm to (146.9, 82.6)
- moved Q8 7.67 mm to (147.0, 102.0)
- moved D5 5.11 mm to (181.5, 72.9)
- moved D7 3.74 mm to (208.3, 72.7)
- moved D8 3.74 mm to (208.0, 94.5)
- moved Q11 3.74 mm to (200.6, 81.0)
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Routing:
- net +48V: track 66.3 -> 140.7 mm
- net BDC11: track 14.9 -> 47.5 mm, vias 1 -> 0
- net GND: track 0.00 -> 31.6 mm
- net BDC22: track 60.2 -> 83.3 mm
- net Net-(D3-K): track 40.3 -> 59.0 mm
- net BDC1: track 37.7 -> 47.1 mm, vias 1 -> 0
- net BDC2: track 71.2 -> 79.7 mm
- net Net-(D6-K): track 57.4 -> 53.3 mm
- net Net-(D8-K): track 59.4 -> 56.3 mm
- net Net-(D2-K): track 53.7 -> 54.9 mm

Commit message: added bigass capcacitor
Parts:
- removed J5: XT90, Skibidi-feet:xt90Female
- added C1: 440uF, ZSKIBIDI:BIGASSCAP, F.Cu at (212.2, 42.5)
- added C2: 440uF, ZSKIBIDI:BIGASSCAP, F.Cu at (212.0, 57.5)
- added C3: 440uF, ZSKIBIDI:BIGASSCAP, F.Cu at (111.2, 43.5)
- added C4: 440uF, ZSKIBIDI:BIGASSCAP, F.Cu at (111.7, 56.5)
- added J1: Conn_01x02_Pin, Connector_AMASS:AMASS_XT60-F_1x02_P7.20mm_Vertical, F.Cu at (159.8, 50.5)
- D1, D2, D3, D4, D5, D6, D7, D8: footprint Skibidi-feet:SchottkyDiode -> ZSKIBIDI:schottky
- J2, J3: value XT90 -> Conn_01x02_Pin; footprint Skibidi-feet:xt90Female -> Connector_AMASS:AMASS_XT60-F_1x02_P7.20mm_Vertical
- moved J3 5.45 mm to (190.3, 50.0), turned to 0 degrees
- moved J2 3.09 mm to (130.3, 50.0), turned to 0 degrees
Routing:
- net +48V: track 140.7 -> 211.7 mm
- net Net-(D8-K): track 56.3 -> 67.9 mm
- net Net-(D2-K): track 54.9 -> 66.2 mm
- net Net-(D6-K): track 53.3 -> 63.4 mm
- net Net-(D3-K): track 59.0 -> 66.3 mm
Other:
- board outline added: 117.5 x 83.5 mm

Commit message: motor driver shhrinking
Parts:
- moved C1 40.5 mm to (174.8, 58.0)
- moved C3 38.5 mm to (145.8, 60.4)
- moved J2 12.2 mm to (129.9, 62.1)
- moved J3 10.1 mm to (188.1, 59.8)
- moved J7 8.82 mm to (136.5, 108.0)
- moved J1 8.77 mm to (159.2, 59.2)
- moved C2 8.11 mm to (204.3, 60.0)
- moved C4 6.62 mm to (116.6, 61.0)
- moved J8 4.67 mm to (192.3, 107.9)
Routing:
- net Net-(D3-K): track 66.3 -> 47.3 mm
- net +48V: track 211.7 -> 224.1 mm
- net Net-(D8-K): track 67.9 -> 55.6 mm
- net Net-(D2-K): track 66.2 -> 54.2 mm
- net Net-(D6-K): track 63.4 -> 52.7 mm
- net BDC2: track 79.7 -> 74.5 mm
- net BDC22: track 83.3 -> 78.4 mm
- net BDC1: track 47.1 -> 46.4 mm
Other:
- board size 117.5 x 83.5 mm -> 103.1 x 62.5 mm
