File: 3kg/Monki/team2 try 2/team2 try 2.kicad_pcb (KiCad board)
At the start: 2 copper layers, 109 parts, among them J1 Conn_01x03_MountingPin, J10 Conn_01x03_MountingPin, J11 Conn_01x03_MountingPin, J12 Conn_01x03_MountingPin, J13 Conn_01x03_MountingPin, J14 XT60-M, J15 Conn_01x03_Pin, J16 Conn_01x08_Pin, J17 XT60-M, J18 XT60-M, J19 Conn_01x03_MountingPin, J2 Conn_01x03_MountingPin, J22 Conn_01x03_MountingPin, J3 Conn_01x03_MountingPin, J4 Conn_01x03_MountingPin, J5 Conn_01x03_MountingPin, J6 Conn_01x03_MountingPin, J7 Conn_01x03_MountingPin, J8 Conn_01x03_MountingPin, J9 Conn_01x03_MountingPin, Q1 SQM40P10-40L_GE3, Q2 SQ2318AES-T1_BE3, SW1 SW_SPST, U1 S-1142DA0I-E6T1U, U2 Teensy4.1, U3 TQL850CSV50_RLG

Commit message: added some footprints
Parts:
- added C23: C, Capacitor_SMD:C_0603_1608Metric_Pad1.08x0.95mm_HandSolder, F.Cu at (150.8, 35.7)
- added R45: 8k, Resistor_SMD:R_0805_2012Metric_Pad1.20x1.40mm_HandSolder, F.Cu at (151.0, 33.0)
- C15: value 10uF -> C; footprint Capacitor_SMD:C_0805_2012Metric_Pad1.18x1.45mm_HandSolder -> Capacitor_SMD:C_0603_1608Metric_Pad1.08x0.95mm_HandSolder
- C16, C17: value 1uF -> C; footprint Capacitor_SMD:C_0805_2012Metric_Pad1.18x1.45mm_HandSolder -> Capacitor_SMD:C_0603_1608Metric_Pad1.08x0.95mm_HandSolder
- C18: value C -> 10uF; footprint Capacitor_SMD:C_0603_1608Metric_Pad1.08x0.95mm_HandSolder -> Capacitor_SMD:C_0805_2012Metric_Pad1.18x1.45mm_HandSolder
- C20, C21: value C -> 1uF; footprint Capacitor_SMD:C_0603_1608Metric_Pad1.08x0.95mm_HandSolder -> Capacitor_SMD:C_0805_2012Metric_Pad1.18x1.45mm_HandSolder
- J1: value Conn_01x03_MountingPin -> Conn_01x08_Pin; footprint Jst Xh 2.5-3 Pin:JST_B3B-XH-A_LF__SN_ -> Connector_PinHeader_2.54mm:PinHeader_1x06_P2.54mm_Vertical
- J2: value Conn_01x03_MountingPin -> Conn_01x03_Pin; footprint Jst Xh 2.5-3 Pin:JST_B3B-XH-A_LF__SN_ -> Connector:FanPinHeader_1x03_P2.54mm_Vertical
- R27: value 15k -> R; footprint Resistor_SMD:R_0805_2012Metric_Pad1.20x1.40mm_HandSolder -> Resistor_SMD:R_0603_1608Metric_Pad0.98x0.95mm_HandSolder
- R28: value 10k -> R; footprint Resistor_SMD:R_0805_2012Metric_Pad1.20x1.40mm_HandSolder -> Resistor_SMD:R_0603_1608Metric_Pad0.98x0.95mm_HandSolder
- R29: value 1k -> R; footprint Resistor_SMD:R_0805_2012Metric_Pad1.20x1.40mm_HandSolder -> Resistor_SMD:R_0603_1608Metric_Pad0.98x0.95mm_HandSolder
- R30: value 8k -> R; footprint Resistor_SMD:R_0805_2012Metric_Pad1.20x1.40mm_HandSolder -> Resistor_SMD:R_0603_1608Metric_Pad0.98x0.95mm_HandSolder
- R40: footprint Resistor_SMD:R_0603_1608Metric_Pad0.98x0.95mm_HandSolder -> Resistor_SMD:R_1206_3216Metric_Pad1.30x1.75mm_HandSolder
- R42: value R -> 15k; footprint Resistor_SMD:R_0603_1608Metric_Pad0.98x0.95mm_HandSolder -> Resistor_SMD:R_0805_2012Metric_Pad1.20x1.40mm_HandSolder
- R43: value R -> 10k; footprint Resistor_SMD:R_0603_1608Metric_Pad0.98x0.95mm_HandSolder -> Resistor_SMD:R_0805_2012Metric_Pad1.20x1.40mm_HandSolder
- R44: value R -> 1k; footprint Resistor_SMD:R_0603_1608Metric_Pad0.98x0.95mm_HandSolder -> Resistor_SMD:R_0805_2012Metric_Pad1.20x1.40mm_HandSolder
- moved U2 26.4 mm to (169.7, 89.5)
Connections:
- C1 pad 1: (no net) -> +5V
- C1 pad 2: (no net) -> GND1
- C10 pad 1: (no net) -> +12V
- C10 pad 2: (no net) -> GND1
- C11 pad 1: (no net) -> +5V
- C11 pad 2: (no net) -> GND1
- C12 pad 1: (no net) -> +12V
- C12 pad 2: (no net) -> GND1
- C13 pad 1: (no net) -> +12V
- C13 pad 2: (no net) -> GND1
- C14 pad 1: (no net) -> +12V
- C14 pad 2: (no net) -> GND1
- C15 pad 1: (no net) -> +12V
- C15 pad 2: (no net) -> GND1
- C16 pad 1: (no net) -> +12V
- C16 pad 2: (no net) -> GND1
- C17 pad 1: (no net) -> 44.4v
- C17 pad 2: (no net) -> GND1
- C18 pad 1: (no net) -> 44.4V
- C18 pad 2: (no net) -> GND1
- C19 pad 1: (no net) -> 12v
- C19 pad 2: (no net) -> GND1
- C2 pad 1: (no net) -> +5V
- C2 pad 2: (no net) -> GND1
- C20 pad 1: (no net) -> 44.4V
- C20 pad 2: (no net) -> GND1
- C21 pad 1: (no net) -> 44.4V
- C21 pad 2: (no net) -> Net-(Q1-G)
- C22 pad 1: (no net) -> 44.4v
- C22 pad 2: (no net) -> GND1
- C3 pad 1: (no net) -> GND1
- C3 pad 2: (no net) -> +3.3V
- C4 pad 1: (no net) -> +5V
- C4 pad 2: (no net) -> GND1
- C5 pad 1: (no net) -> +5V
- C5 pad 2: (no net) -> GND1
- C6 pad 1: (no net) -> +12V
- C6 pad 2: (no net) -> GND1
- C7 pad 1: (no net) -> +5V
- C7 pad 2: (no net) -> GND1
- C8 pad 1: (no net) -> +12V
- C8 pad 2: (no net) -> GND1
- C9 pad 1: (no net) -> +12V
- C9 pad 2: (no net) -> GND1
- D1 pad 1: (no net) -> GND1
- D1 pad 2: (no net) -> Net-(D1-A)
- D10 pad 1: (no net) -> GND1
- D10 pad 2: (no net) -> Net-(D10-A)
- D11 pad 1: (no net) -> GND1
- D11 pad 2: (no net) -> Net-(D11-A)
- D12 pad 1: (no net) -> GND1
- D12 pad 2: (no net) -> Net-(D12-A)
- D13 pad 1: (no net) -> GND1
- D13 pad 2: (no net) -> Net-(D13-A)
- D14 pad 1: (no net) -> GND1
- D14 pad 2: (no net) -> Net-(D14-A)
- D15 pad 1: (no net) -> GND1
- D15 pad 2: (no net) -> Net-(D15-A)
- D2 pad 1: (no net) -> GND1
- D2 pad 2: (no net) -> Net-(D2-A)
- D3 pad 1: (no net) -> GND1
- D3 pad 2: (no net) -> Net-(D3-A)
- D4 pad 1: (no net) -> GND1
- D4 pad 2: (no net) -> Net-(D4-A)
- D5 pad 1: (no net) -> GND1
- D5 pad 2: (no net) -> Net-(D5-A)
- D6 pad 1: (no net) -> GND1
- D6 pad 2: (no net) -> Net-(D6-A)
- D7 pad 1: (no net) -> GND1
- D7 pad 2: (no net) -> Net-(D7-A)
- D8 pad 1: (no net) -> GND1
- D8 pad 2: (no net) -> Net-(D8-A)
- D9 pad 1: (no net) -> GND1
- D9 pad 2: (no net) -> Net-(D9-A)
- J1 pad 1: (no net) -> +5V
- J1 pad 2: (no net) -> GND1
- J1 pad 3: (no net) -> SCL
- J10 pad 1: (no net) -> Distance Sensor 1 12V
- J10 pad 2: (no net) -> +12V
- J10 pad 3: (no net) -> GND1
- J11 pad 1: (no net) -> Distance Sensor 2 12V
- J11 pad 2: (no net) -> +12V
- J11 pad 3: (no net) -> GND1
- J12 pad 1: (no net) -> Distance Sensor 3 12V
- J12 pad 2: (no net) -> +12V
- J12 pad 3: (no net) -> GND1
- J13 pad 1: (no net) -> Distance Sensor 4 12V
- J13 pad 2: (no net) -> +12V
- J13 pad 3: (no net) -> GND1
- J2 pad 1: (no net) -> Signal Start Module
- J2 pad 2: (no net) -> GND1
- J2 pad 3: (no net) -> +3.3V
- J4 pad 1: (no net) -> Direction MD1
- J4 pad 2: (no net) -> PWM MD1
- J4 pad 3: (no net) -> GND1
- J5 pad 1: (no net) -> Direction MD2
- J5 pad 2: (no net) -> PWM MD2
- J5 pad 3: (no net) -> GND1
- J6 pad 1: (no net) -> Line Sensor 1 5v
- J6 pad 2: (no net) -> +5V
- J6 pad 3: (no net) -> GND1
- J7 pad 1: (no net) -> Line Sensor 2 5v
- J7 pad 2: (no net) -> +5V
- J7 pad 3: (no net) -> GND1
- J8 pad 1: (no net) -> Line Sensor 3 5v
- J8 pad 2: (no net) -> +5V
- J8 pad 3: (no net) -> GND1
- J9 pad 1: (no net) -> Line Sensor 4 5v
- J9 pad 2: (no net) -> +5V
- J9 pad 3: (no net) -> GND1
- Q1 pad 1: (no net) -> Net-(Q1-G)
- Q1 pad 2: (no net) -> 44.4V
- Q1 pad 3: (no net) -> Net-(Q1-S)
- Q2 pad 1: (no net) -> Net-(Q2-G)
- Q2 pad 2: (no net) -> GND1
- Q2 pad 3: (no net) -> Net-(Q2-D)
- R1 pad 1: (no net) -> Line Sensor 1 5v
- R1 pad 2: (no net) -> Line Sensor 1 3.3V
- R10 pad 1: (no net) -> Distance Sensor 7 12V
- R10 pad 2: (no net) -> Distance Sensor 7 3.3V
- R11 pad 1: (no net) -> Distance Sensor 3 12V
- R11 pad 2: (no net) -> Distance Sensor 3 3.3V
- R12 pad 1: (no net) -> Distance Sensor 9 12V
- R12 pad 2: (no net) -> Distance Sensor 9 3.3V
- R13 pad 1: (no net) -> Distance Sensor 5 12V
- R13 pad 2: (no net) -> Distance Sensor 5 3.3V
- R14 pad 1: (no net) -> Line Sensor 1 3.3V
- R14 pad 2: (no net) -> GND1
- R15 pad 1: (no net) -> Line Sensor 3 3.3V
- R15 pad 2: (no net) -> GND1
- R16 pad 1: (no net) -> Line Sensor 2 3.3V
- R16 pad 2: (no net) -> GND1
- R17 pad 1: (no net) -> Line Sensor 4 3.3V
- R17 pad 2: (no net) -> GND1
- R18 pad 1: (no net) -> Distance Sensor 1 3.3V
- R18 pad 2: (no net) -> GND1
- R19 pad 1: (no net) -> Distance Sensor 8 3.3V
- R19 pad 2: (no net) -> GND1
- R2 pad 1: (no net) -> Line Sensor 3 5v
- R2 pad 2: (no net) -> Line Sensor 3 3.3V
- R20 pad 1: (no net) -> Distance Sensor 2 3.3V
- R20 pad 2: (no net) -> GND1
- R21 pad 1: (no net) -> Distance Sensor 4 3.3V
- R21 pad 2: (no net) -> GND1
- R22 pad 1: (no net) -> Distance Sensor 6 3.3V
- R22 pad 2: (no net) -> GND1
- R23 pad 1: (no net) -> Distance Sensor 7 3.3V
- R23 pad 2: (no net) -> GND1
- R24 pad 1: (no net) -> Distance Sensor 3 3.3V
- R24 pad 2: (no net) -> GND1
- R25 pad 1: (no net) -> Distance Sensor 9 3.3V
- R25 pad 2: (no net) -> GND1
- R26 pad 1: (no net) -> Distance Sensor 5 3.3V
- R26 pad 2: (no net) -> GND1
- R27 pad 1: (no net) -> Line Sensor 1 3.3V
- R27 pad 2: (no net) -> Net-(D1-A)
- R28 pad 1: (no net) -> Line Sensor 2 3.3V
- R28 pad 2: (no net) -> Net-(D2-A)
- R29 pad 1: (no net) -> Line Sensor 3 3.3V
- R29 pad 2: (no net) -> Net-(D3-A)
- R3 pad 1: (no net) -> Line Sensor 2 5v
- R3 pad 2: (no net) -> Line Sensor 2 3.3V
- R30 pad 1: (no net) -> Line Sensor 4 3.3V
- R30 pad 2: (no net) -> Net-(D4-A)
- R31 pad 1: (no net) -> Distance Sensor 1 3.3V
- R31 pad 2: (no net) -> Net-(D5-A)
- R32 pad 1: (no net) -> Distance Sensor 2 3.3V
- R32 pad 2: (no net) -> Net-(D6-A)
- R33 pad 1: (no net) -> Distance Sensor 4 3.3V
- R33 pad 2: (no net) -> Net-(D7-A)
- R34 pad 1: (no net) -> Distance Sensor 3 3.3V
- R34 pad 2: (no net) -> Net-(D8-A)
- R35 pad 1: (no net) -> Distance Sensor 8 3.3V
- R35 pad 2: (no net) -> Net-(D9-A)
- R36 pad 1: (no net) -> Distance Sensor 6 3.3V
- R36 pad 2: (no net) -> Net-(D10-A)
- R37 pad 1: (no net) -> Distance Sensor 7 3.3V
- R37 pad 2: (no net) -> Net-(D11-A)
- R38 pad 1: (no net) -> Distance Sensor 9 3.3V
- R38 pad 2: (no net) -> Net-(D12-A)
- R39 pad 1: (no net) -> Distance Sensor 5 3.3V
- R39 pad 2: (no net) -> Net-(D13-A)
- R4 pad 1: (no net) -> Line Sensor 4 5v
- R4 pad 2: (no net) -> Line Sensor 4 3.3V
- R40 pad 1: (no net) -> 5v
- R40 pad 2: (no net) -> Net-(D14-A)
- R41 pad 1: (no net) -> 12v
- R41 pad 2: (no net) -> Net-(D15-A)
- R42 pad 1: (no net) -> Net-(Q1-G)
- R42 pad 2: (no net) -> Net-(Q2-D)
- R43 pad 1: (no net) -> Net-(Q1-G)
- R43 pad 2: (no net) -> Net-(Q1-S)
- R44 pad 1: (no net) -> Net-(Q2-G)
- R44 pad 2: (no net) -> GND1
- R5 pad 1: (no net) -> Distance Sensor 1 12V
- R5 pad 2: (no net) -> Distance Sensor 1 3.3V
- R6 pad 1: (no net) -> Distance Sensor 8 12V
- R6 pad 2: (no net) -> Distance Sensor 8 3.3V
- R7 pad 1: (no net) -> Distance Sensor 2 12V
- R7 pad 2: (no net) -> Distance Sensor 2 3.3V
- R8 pad 1: (no net) -> Distance Sensor 4 12V
- R8 pad 2: (no net) -> Distance Sensor 4 3.3V
- R9 pad 1: (no net) -> Distance Sensor 6 12V
- R9 pad 2: (no net) -> Distance Sensor 6 3.3V
- SW1 pad 1: (no net) -> Net-(SW1-A)
- SW1 pad 2: (no net) -> Net-(Q1-S)
- U3 pad 1: (no net) -> 44.4v
- U3 pad 2: (no net) -> 44.4v
- U3 pad 3: (no net) -> unconnected-(U3-RO/WDO-Pad3)
- U3 pad 4: (no net) -> GND1
- U3 pad 5: (no net) -> GND1
- U3 pad 6: (no net) -> GND1
- U3 pad 7: (no net) -> unconnected-(U3-NC-Pad7)
- U3 pad 8: (no net) -> 5v
- U3 pad 9: (no net) -> unconnected-(U3-EXP-Pad9)
