File: 3kg/Monki/team2 try 2/team2 try 2.kicad_sch (KiCad schematic)
At the start: 110 parts, among them J1 Conn_01x08_Pin, J10 Conn_01x03_MountingPin, J11 Conn_01x03_MountingPin, J12 Conn_01x03_MountingPin, J13 Conn_01x03_MountingPin, J14 Conn_01x03_MountingPin, J15 Conn_01x03_MountingPin, J16 Conn_01x03_MountingPin, J17 Conn_01x03_MountingPin, J18 Conn_01x03_MountingPin, J19 XT60-M, J2 Conn_01x03_Pin, J20 XT60-M, J3 XT60-M, J4 Conn_01x03_MountingPin, J5 Conn_01x03_MountingPin, J6 Conn_01x03_MountingPin, J7 Conn_01x03_MountingPin, J8 Conn_01x03_MountingPin, J9 Conn_01x03_MountingPin, Q1 SQM40P10-40L_GE3, Q2 SQ2318AES-T1_BE3, SW1 SW_SPST, U1 Teensy4.1, U2 S-1142DA0I-E6T1U, U3 TQL850CSV50_RLG

Commit message: added some footprints
Parts:
- J10, J11, J12, J13, J14, J15, J16, J17, J18, J4, J5, J6, J7, J8, J9: footprint Jst Xh 2.5-3 Pin:JST_B3B-XH-A_LF__SN_ -> Connector_JST:JST_XH_B3B-XH-A_1x03_P2.50mm_Vertical
- J19, J20, J3: footprint XT60-M:AMASS_XT60-M -> Connector_AMASS:AMASS_XT60-F_1x02_P7.20mm_Vertical
Changed lines of the file:
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@@
 			)
 		)
-		(property "Footprint" "Jst Xh 2.5-3 Pin:JST_B3B-XH-A_LF__SN_"
+		(property "Footprint" "Connector_JST:JST_XH_B3B-XH-A_1x03_P2.50mm_Vertical"
 			(at 198.12 81.28 0)
 			(effects
@@
 			)
 		)
-		(property "Footprint" "Jst Xh 2.5-3 Pin:JST_B3B-XH-A_LF__SN_"
+		(property "Footprint" "Connector_JST:JST_XH_B3B-XH-A_1x03_P2.50mm_Vertical"
 			(at 198.12 171.45 0)
 			(effects
@@
 			)
 		)
-		(property "Footprint" "Jst Xh 2.5-3 Pin:JST_B3B-XH-A_LF__SN_"
+		(property "Footprint" "Connector_JST:JST_XH_B3B-XH-A_1x03_P2.50mm_Vertical"
 			(at 198.12 114.3 0)
 			(effects
@@
 			)
 		)
-		(property "Footprint" "Jst Xh 2.5-3 Pin:JST_B3B-XH-A_LF__SN_"
+		(property "Footprint" "Connector_JST:JST_XH_B3B-XH-A_1x03_P2.50mm_Vertical"
 			(at 198.12 34.29 0)
 			(effects
@@
 			)
 		)
-		(property "Footprint" "Jst Xh 2.5-3 Pin:JST_B3B-XH-A_LF__SN_"
+		(property "Footprint" "Connector_JST:JST_XH_B3B-XH-A_1x03_P2.50mm_Vertical"
 			(at 142.24 34.29 0)
 			(effects
@@
 			)
 		)
-		(property "Footprint" "Jst Xh 2.5-3 Pin:JST_B3B-XH-A_LF__SN_"
+		(property "Footprint" "Connector_JST:JST_XH_B3B-XH-A_1x03_P2.50mm_Vertical"
 			(at 198.12 50.8 0)
 			(effects
@@
 			)
 		)
-		(property "Footprint" "Jst Xh 2.5-3 Pin:JST_B3B-XH-A_LF__SN_"
+		(property "Footprint" "Connector_JST:JST_XH_B3B-XH-A_1x03_P2.50mm_Vertical"
 			(at 198.12 213.36 0)
 			(effects
@@
 			)
 		)
-		(property "Footprint" "XT60-M:AMASS_XT60-M"
+		(property "Footprint" "Connector_AMASS:AMASS_XT60-F_1x02_P7.20mm_Vertical"
 			(at 551.18 52.07 0)
 			(effects
@@
 			)
 		)
-		(property "Footprint" "XT60-M:AMASS_XT60-M"
+		(property "Footprint" "Connector_AMASS:AMASS_XT60-F_1x02_P7.20mm_Vertical"
 			(at 139.7 69.85 0)
 			(effects
@@
 			)
 		)
-		(property "Footprint" "Jst Xh 2.5-3 Pin:JST_B3B-XH-A_LF__SN_"
+		(property "Footprint" "Connector_JST:JST_XH_B3B-XH-A_1x03_P2.50mm_Vertical"
 			(at 198.12 254 0)
 			(effects
@@
 			)
 		)
-		(property "Footprint" "Jst Xh 2.5-3 Pin:JST_B3B-XH-A_LF__SN_"
+		(property "Footprint" "Connector_JST:JST_XH_B3B-XH-A_1x03_P2.50mm_Vertical"
 			(at 198.12 152.4 0)
 			(effects
@@
 			)
 		)
-		(property "Footprint" "XT60-M:AMASS_XT60-M"
+		(property "Footprint" "Connector_AMASS:AMASS_XT60-F_1x02_P7.20mm_Vertical"
 			(at 551.18 41.91 0)
 			(effects
@@
 			)
 		)
-		(property "Footprint" "Jst Xh 2.5-3 Pin:JST_B3B-XH-A_LF__SN_"
+		(property "Footprint" "Connector_JST:JST_XH_B3B-XH-A_1x03_P2.50mm_Vertical"
 			(at 198.12 66.04 0)
 			(effects
@@
 			)
 		)
-		(property "Footprint" "Jst Xh 2.5-3 Pin:JST_B3B-XH-A_LF__SN_"
+		(property "Footprint" "Connector_JST:JST_XH_B3B-XH-A_1x03_P2.50mm_Vertical"
 			(at 198.12 191.77 0)
 			(effects
@@
 			)
 		)
-		(property "Footprint" "Jst Xh 2.5-3 Pin:JST_B3B-XH-A_LF__SN_"
+		(property "Footprint" "Connector_JST:JST_XH_B3B-XH-A_1x03_P2.50mm_Vertical"
 			(at 198.12 233.68 0)
 			(effects
@@
 			)
 		)
-		(property "Footprint" "Jst Xh 2.5-3 Pin:JST_B3B-XH-A_LF__SN_"
+		(property "Footprint" "Connector_JST:JST_XH_B3B-XH-A_1x03_P2.50mm_Vertical"
 			(at 142.24 46.99 0)
 			(effects
@@
 			)
 		)
-		(property "Footprint" "Jst Xh 2.5-3 Pin:JST_B3B-XH-A_LF__SN_"
+		(property "Footprint" "Connector_JST:JST_XH_B3B-XH-A_1x03_P2.50mm_Vertical"
 			(at 199.39 274.32 0)
 			(effects
@@
 			)
 		)
-		(property "Footprint" "Jst Xh 2.5-3 Pin:JST_B3B-XH-A_LF__SN_"
+		(property "Footprint" "Connector_JST:JST_XH_B3B-XH-A_1x03_P2.50mm_Vertical"
 			(at 198.12 133.35 0)
 			(effects
