File: Skibidi/Skibid-i/Skibidi-Power/Skibidipower.kicad_pcb (KiCad board)
At the start: 2 copper layers, 49.8 x 49.2 mm, 19 parts, among them J1 SparkOut, J2 Bat2, J3 Bat1, J5 Sparkout 48V, J6 Sparkin, Q1 SQM40P10-40L_GE3, Q2 SQ2318AES-T1_BE3

Commit message: joe skibidi deez nus
Parts:
- removed C4: 100uF, Capacitor_SMD:CP_Elec_6.3x5.4
- removed C5: 22uF, Capacitor_SMD:C_2220_5750Metric
- removed J1: SparkOut, Connector_AMASS:AMASS_XT30U-F_1x02_P5.0mm_Vertical
- removed PS1: RSO-4812S_H2, askibidi:12vConvertor
- moved J3 2.74 mm to (204.2, 80.3)
- moved J2 1.19 mm to (192.4, 87.5)
- moved J6 1.19 mm to (179.8, 87.5)
- moved J5 0.46 mm to (218.0, 79.8)
Routing:
- net +12V: track 57.0 -> 0.14 mm, vias 1 -> 0
- net +48V: track 43.7 -> 15.4 mm, vias 1 -> 0
- net Net-(J5-Pin_2): track 12.3 -> 7.04 mm
- net Net-(J2-Pin_2): track 13.7 -> 11.8 mm
Other:
- board size 49.8 x 49.2 mm -> 49.8 x 42.8 mm

Commit message: sigma fanum
Parts:
- moved J3 2.74 mm to (206.8, 79.3)
- moved J2 1.19 mm to (193.1, 86.5)
- moved J6 1.19 mm to (180.4, 86.5)
- moved J5 0.46 mm to (218.1, 79.3)
Routing:
- net Net-(J5-Pin_2): track 7.04 -> 12.3 mm
- net Net-(J2-Pin_2): track 11.8 -> 13.7 mm
Other:
- board size 49.8 x 42.8 mm -> 49.8 x 43.6 mm
Changed lines of the file:
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@@
 	(footprint "Connector_AMASS:AMASS_XT60-F_1x02_P7.20mm_Vertical"
 		(layer "F.Cu")
-		(at 179.8 87.5 90)
+		(at 180.45 86.5 90)
 		(descr "AMASS female XT60, through hole, vertical, https://www.tme.eu/Document/2d152ced3b7a446066e6c419d84bb460/XT60%20SPEC.pdf")
 		(tags "XT60 female vertical")
@@
 	(footprint "Connector_AMASS:AMASS_XT60-F_1x02_P7.20mm_Vertical"
 		(layer "F.Cu")
-		(at 192.4 87.5 90)
+		(at 193.05 86.5 90)
 		(descr "AMASS female XT60, through hole, vertical, https://www.tme.eu/Document/2d152ced3b7a446066e6c419d84bb460/XT60%20SPEC.pdf")
 		(tags "XT60 female vertical")
@@
 	(footprint "Connector_AMASS:AMASS_XT60-F_1x02_P7.20mm_Vertical"
 		(layer "F.Cu")
-		(at 218 79.75 -90)
+		(at 218.1 79.3 -90)
 		(descr "AMASS female XT60, through hole, vertical, https://www.tme.eu/Document/2d152ced3b7a446066e6c419d84bb460/XT60%20SPEC.pdf")
 		(tags "XT60 female vertical")
@@
 	(footprint "Connector_AMASS:AMASS_XT60-F_1x02_P7.20mm_Vertical"
 		(layer "F.Cu")
-		(at 204.2 80.3 -90)
+		(at 206.75 79.3 -90)
 		(descr "AMASS female XT60, through hole, vertical, https://www.tme.eu/Document/2d152ced3b7a446066e6c419d84bb460/XT60%20SPEC.pdf")
 		(tags "XT60 female vertical")
@@
 	)
 	(gr_rect
-		(start 173.75 75.1)
+		(start 173.75 74.25)
 		(end 223.55 117.85)
 		(stroke
@@
 	)
 	(segment
+		(start 214.39 90.21)
+		(end 218.1 86.5)
+		(width 1.5)
+		(layer "F.Cu")
+		(net 5)
+	)
+	(segment
 		(start 201.015 110.035)
 		(end 198.85 112.2)
@@
 	)
 	(segment
-		(start 176.35 106.75)
-		(end 176.35 103.65)
+		(start 201.015 106.525)
+		(end 201.015 108.765)
 		(width 1.3)
 		(layer "F.Cu")
@@
 	(segment
 		(start 201.015 106.525)
-		(end 201.015 108.765)
+		(end 201.015 110.035)
 		(width 1.3)
 		(layer "F.Cu")
@@
 	)
 	(segment
-		(start 203.85 116.45)
-		(end 186.05 116.45)
+		(start 176.35 103.65)
+		(end 179.85 100.15)
 		(width 1.3)
 		(layer "F.Cu")
@@
 	)
 	(segment
-		(start 201.015 106.525)
-		(end 201.015 110.035)
+		(start 176.35 106.75)
+		(end 176.35 103.65)
+		(width 1.3)
+		(layer "F.Cu")
+		(net 6)
+	)
+	(segment
+		(start 212.09 112.1)
+		(end 208.2 112.1)
 		(width 1.3)
 		(layer "F.Cu")
@@
 	(segment
 		(start 208.2 112.1)
-		(end 203.85 116.45)
+		(end 203.8 116.5)
 		(width 1.3)
 		(layer "F.Cu")
@@
 	)
 	(segment
-		(start 186.05 116.45)
+		(start 186.1 116.5)
 		(end 176.35 106.75)
 		(width 1.3)
@@
 	)
 	(segment
-		(start 176.35 103.65)
-		(end 179.85 100.15)
-		(width 1.3)
-		(layer "F.Cu")
-		(net 6)
-	)
-	(segment
 		(start 212.09 112.1)
 		(end 213.48 110.71)
@@
 	)
 	(segment
-		(start 212.09 112.1)
-		(end 208.2 112.1)
+		(start 203.8 116.5)
+		(end 186.1 116.5)
 		(width 1.3)
 		(layer "F.Cu")
@@
 	)
 	(segment
-		(start 192.4 87.5)
-		(end 179.8 87.5)
+		(start 193.05 86.5)
+		(end 180.45 86.5)
 		(width 3)
 		(layer "F.Cu")
@@
 	)
 	(segment
-		(start 192.4 80.3)
-		(end 204.2 80.3)
-		(width 2)
+		(start 193.05 79.3)
+		(end 206.75 79.3)
+		(width 3)
 		(layer "F.Cu")
 		(net 8)
@@
 		(polygon
 			(pts
-				(xy 173.85 75.1) (xy 223.65 75.1) (xy 223.65 117.85) (xy 173.85 117.85)
+				(xy 173.75 74.25) (xy 223.55 74.25) (xy 223.65 117.85) (xy 173.85 117.85)
 			)
 		)

Commit message: i thiknk its done
Parts:
- moved C3 11.1 mm to (208.6, 95.0), turned to 0 degrees
- moved C1 8.51 mm to (208.9, 104.5)
- moved C2 2.97 mm to (208.6, 99.0)
Routing:
- net Net-(Q1-G): track 41.7 -> 60.6 mm
- net Net-(Q1-S): track 72.9 -> 74.2 mm
- net +48V: track 15.4 -> 16.2 mm
Changed lines of the file:
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@@
 	(footprint "Capacitor_SMD:C_0805_2012Metric"
 		(layer "F.Cu")
-		(at 207.8 106 -90)
+		(at 208.55 94.95)
 		(descr "Capacitor SMD 0805 (2012 Metric), square (rectangular) end terminal, IPC_7351 nominal, (Body size source: IPC-SM-782 page 76, https://www.pcb-3d.com/wordpress/wp-content/uploads/ipc-sm-782a_amendment_1_and_2.pdf, https://docs.google.com/spreadsheets/d/1BsfQQcO9C6DZCsRaXUlFlo91Tg2WpOkGARC1WS5S8t0/edit?usp=sharing), generated with kicad-footprint-generator")
 		(tags "capacitor")
 		(property "Reference" "C3"
-			(at 0 -1.68 90)
+			(at 0 -1.68 360)
 			(layer "F.SilkS")
 			(effects
@@
 		)
 		(property "Value" "1uF"
-			(at 0 1.68 90)
+			(at 0 1.68 360)
 			(layer "F.Fab")
 			(effects
@@
 		)
 		(property "Footprint" "Capacitor_SMD:C_0805_2012Metric"
-			(at 0 0 -90)
+			(at 0 0 0)
 			(unlocked yes)
 			(layer "F.Fab")
@@
 		)
 		(property "Datasheet" ""
-			(at 0 0 -90)
+			(at 0 0 0)
 			(unlocked yes)
 			(layer "F.Fab")
@@
 		)
 		(property "Description" ""
-			(at 0 0 -90)
+			(at 0 0 0)
 			(unlocked yes)
 			(layer "F.Fab")
@@
 		(attr smd)
 		(fp_line
+			(start -0.261252 -0.735)
+			(end 0.261252 -0.735)
+			(stroke
+				(width 0.12)
+				(type solid)
+			)
+			(layer "F.SilkS")
+		)
+		(fp_line
 			(start -0.261252 0.735)
 			(end 0.261252 0.735)
@@
 		)
 		(fp_line
-			(start -0.261252 -0.735)
-			(end 0.261252 -0.735)
-			(stroke
-				(width 0.12)
-				(type solid)
-			)
-			(layer "F.SilkS")
+			(start -1.7 -0.98)
+			(end 1.7 -0.98)
+			(stroke
+				(width 0.05)
+				(type solid)
+			)
+			(layer "F.CrtYd")
 		)
 		(fp_line
@@
 		)
 		(fp_line
+			(start 1.7 -0.98)
+			(end 1.7 0.98)
+			(stroke
+				(width 0.05)
+				(type solid)
+			)
+			(layer "F.CrtYd")
+		)
+		(fp_line
 			(start 1.7 0.98)
 			(end -1.7 0.98)
@@
 		)
 		(fp_line
-			(start -1.7 -0.98)
-			(end 1.7 -0.98)
-			(stroke
-				(width 0.05)
-				(type solid)
-			)
-			(layer "F.CrtYd")
-		)
-		(fp_line
-			(start 1.7 -0.98)
-			(end 1.7 0.98)
-			(stroke
-				(width 0.05)
-				(type solid)
-			)
-			(layer "F.CrtYd")
+			(start -1 -0.625)
+			(end 1 -0.625)
+			(stroke
+				(width 0.1)
+				(type solid)
+			)
+			(layer "F.Fab")
 		)
 		(fp_line
@@
 		)
 		(fp_line
+			(start 1 -0.625)
+			(end 1 0.625)
+			(stroke
+				(width 0.1)
+				(type solid)
+			)
+			(layer "F.Fab")
+		)
+		(fp_line
 			(start 1 0.625)
 			(end -1 0.625)
@@
 			(layer "F.Fab")
 		)
-		(fp_line
-			(start -1 -0.625)
-			(end 1 -0.625)
-			(stroke
-				(width 0.1)
-				(type solid)
-			)
-			(layer "F.Fab")
-		)
-		(fp_line
-			(start 1 -0.625)
-			(end 1 0.625)
-			(stroke
-				(width 0.1)
-				(type solid)
-			)
-			(layer "F.Fab")
-		)
 		(fp_text user "${REFERENCE}"
-			(at 0 0 90)
+			(at 0 0 360)
 			(layer "F.Fab")
 			(effects
@@
 		)
 		(pad "1" smd roundrect
-			(at -0.95 0 270)
+			(at -0.95 0)
 			(size 1 1.45)
 			(layers "F.Cu" "F.Paste" "F.Mask")
@@
 		)
 		(pad "2" smd roundrect
-			(at 0.95 0 270)
+			(at 0.95 0)
 			(size 1 1.45)
 			(layers "F.Cu" "F.Paste" "F.Mask")
@@
 	(footprint "Capacitor_SMD:C_0805_2012Metric"
 		(layer "F.Cu")
-		(at 207.7 101.85)
+		(at 208.55 99)
 		(descr "Capacitor SMD 0805 (2012 Metric), square (rectangular) end terminal, IPC_7351 nominal, (Body size source: IPC-SM-782 page 76, https://www.pcb-3d.com/wordpress/wp-content/uploads/ipc-sm-782a_amendment_1_and_2.pdf, https://docs.google.com/spreadsheets/d/1BsfQQcO9C6DZCsRaXUlFlo91Tg2WpOkGARC1WS5S8t0/edit?usp=sharing), generated with kicad-footprint-generator")
 		(tags "capacitor")
@@
 	(footprint "askibidi:10uF"
 		(layer "F.Cu")
-		(at 208.5 96.05 180)
+		(at 208.9 104.55 180)
 		(descr "<B>WCAP-ASLI</B><BR> Aluminium Electrolytic Capacitors,4X5.5X1(DiameterXLengthXPitch)")
 		(property "Reference" "C1"
@@
 	)
 	(segment
-		(start 206.75 104)
-		(end 207.8 105.05)
+		(start 207.05 104.5)
+		(end 207.1 104.55)
 		(width 1)
 		(layer "F.Cu")
@@
 	)
 	(segment
-		(start 206.7 96.05)
-		(end 206.7 101.8)
+		(start 201.25 94.95)
+		(end 207.6 94.95)
 		(width 1)
 		(layer "F.Cu")
@@
 	)
 	(segment
-		(start 205.6 94.95)
-		(end 206.7 96.05)
+		(start 207.6 94.95)
+		(end 207.6 99)
 		(width 1)
 		(layer "F.Cu")
@@
 	)
 	(segment
-		(start 206.7 101.8)
-		(end 206.75 101.85)
-		(width 0.5)
+		(start 207.05 99.55)
+		(end 207.05 104.5)
+		(width 1)
 		(layer "F.Cu")
 		(net 2)
 	)
 	(segment
-		(start 206.75 101.85)
-		(end 206.75 104)
+		(start 207.6 99)
+		(end 207.05 99.55)
 		(width 1)
 		(layer "F.Cu")
@@
 	)
 	(segment
-		(start 201.25 94.95)
-		(end 205.6 94.95)
+		(start 214.05 106.35)
+		(end 214.05 101.47457)
 		(width 1)
 		(layer "F.Cu")
-		(net 2)
+		(net 3)
+	)
+	(segment
+		(start 214.05 101.47457)
+		(end 211.25 98.67457)
+		(width 1)
+		(layer "F.Cu")
+		(net 3)
 	)
 	(segment
@@
 	)
 	(segment
+		(start 211.25 98.67457)
+		(end 211.25 96.7)
+		(width 1)
+		(layer "F.Cu")
+		(net 3)
+	)
+	(segment
 		(start 190.8375 96.2625)
 		(end 190.8 96.3)
@@
 	)
 	(segment
+		(start 206.9 109.35)
+		(end 211.05 109.35)
+		(width 1)
+		(layer "F.Cu")
+		(net 3)
+	)
+	(segment
 		(start 195.925 110.65)
 		(end 195.925 109.4)
@@
 	)
 	(segment
-		(start 207.8 108.45)
-		(end 207.8 106.95)
+		(start 211.25 96.7)
+		(end 209.5 94.95)
 		(width 1)
 		(layer "F.Cu")
@@
 	)
 	(segment
-		(start 206.9 109.35)
-		(end 207.8 108.45)
+		(start 211.05 109.35)
+		(end 214.05 106.35)
 		(width 1)
 		(layer "F.Cu")
@@
 	)
 	(segment
+		(start 208.2 112.1)
+		(end 203.8 116.5)
+		(width 1.3)
+		(layer "F.Cu")
+		(net 6)
+	)
+	(segment
 		(start 201.015 110.035)
 		(end 198.85 112.2)
@@
 	)
 	(segment
+		(start 203.8 116.5)
+		(end 183.8 116.5)
+		(width 1.3)
+		(layer "F.Cu")
+		(net 6)
+	)
+	(segment
+		(start 183.8 116.5)
+		(end 176.35 109.05)
+		(width 1.3)
+		(layer "F.Cu")
+		(net 6)
+	)
+	(segment
 		(start 176.35 103.65)
 		(end 179.85 100.15)
@@
 	)
 	(segment
-		(start 176.35 106.75)
-		(end 176.35 103.65)
+		(start 204.35 112.1)
+		(end 212.09 112.1)
+		(width 1.3)
+		(layer "F.Cu")
+		(net 6)
+	)
+	(segment
+		(start 201.015 108.765)
+		(end 204.35 112.1)
 		(width 1.3)
 		(layer "F.Cu")
@@
 	)
 	(segment
-		(start 208.2 112.1)
-		(end 203.8 116.5)
-		(width 1.3)
-		(layer "F.Cu")
-		(net 6)
-	)
-	(segment
-		(start 186.1 116.5)
-		(end 176.35 106.75)
-		(width 1.3)
-		(layer "F.Cu")
-		(net 6)
-	)
-	(segment
-		(start 204.35 112.1)
-		(end 212.09 112.1)
-		(width 1.3)
-		(layer "F.Cu")
-		(net 6)
-	)
-	(segment
-		(start 201.015 108.765)
-		(end 204.35 112.1)
+		(start 176.35 109.05)
+		(end 176.35 103.65)
 		(width 1.3)
 		(layer "F.Cu")
@@
 		(width 1.3)
 		(layer "F.Cu")
-		(net 6)
-	)
-	(segment
-		(start 203.8 116.5)
-		(end 186.1 116.5)
-		(width 1.3)
-		(layer "F.Cu")
