File: Skibidi/Skibid-i/Skibidi-Power/Skibidipower.kicad_sch (KiCad schematic)
At the start: 19 parts, among them J1 SparkOut, J2 Bat2, J3 Bat1, J5 Sparkout 48V, J6 Sparkin, Q1 SQM40P10-40L_GE3, Q2 SQ2318AES-T1_BE3

Commit message: pushsuskibnbiid
Other:
- note added: "Switch"
- moved on the sheet: C1, C2, C3, F2, J5, Q1, Q2, R1, R2, R3, R4, S1

Commit message: joe skibidi deez nus
Parts:
- removed C4: 100uF, Capacitor_SMD:CP_Elec_6.3x5.4, symbol Device:C_Polarized_US
- removed C5: 22uF, Capacitor_SMD:C_2220_5750Metric, symbol Device:C_Polarized_US
- removed J1: SparkOut, Connector_AMASS:AMASS_XT30U-F_1x02_P5.0mm_Vertical, symbol Connector_Generic:Conn_01x02
- removed PS1: RSO-4812S_H2, askibidi:12vConvertor, symbol 76to5:RSO-4812S_H2
Connections:
- no-connect marks 4 -> 1

Commit message: i thiknk its done
Other:
- moved on the sheet: J2, J3, J6

Commit message: fff
Other:
- moved on the sheet: F2, J5, J6
Changed lines of the file:
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@@
 	(paper "A4")
+	(junction
+		(at 101.6 118.11)
+		(diameter 0)
+		(color 0 0 0 0)
+	)
 	(junction
 		(at 151.13 95.25)
@@
 	)
 	(junction
-		(at 101.6 118.745)
-		(diameter 0)
-		(color 0 0 0 0)
-	)
-	(junction
 		(at 55.245 118.11)
 		(diameter 0)
@@
 	(wire
 		(pts
-			(xy 101.6 118.745) (xy 101.6 118.11)
-		)
-		(stroke
-			(width 0)
-			(type default)
-		)
-	)
-	(wire
-		(pts
 			(xy 66.675 118.11) (xy 66.675 119.38)
 		)
@@
 	(wire
 		(pts
-			(xy 101.6 118.745) (xy 107.95 118.745)
+			(xy 101.6 118.11) (xy 106.68 118.11)
 		)
 		(stroke
@@
 	(wire
 		(pts
-			(xy 97.155 146.05) (xy 101.6 146.05)
+			(xy 97.155 146.05) (xy 104.14 146.05)
 		)
 		(stroke
@@
 	(wire
 		(pts
+			(xy 101.6 118.11) (xy 101.6 125.095)
+		)
+		(stroke
+			(width 0)
+			(type default)
+		)
+	)
+	(wire
+		(pts
 			(xy 55.245 128.27) (xy 55.245 128.905)
 		)
@@
 	(wire
 		(pts
-			(xy 123.19 121.285) (xy 123.19 118.745)
-		)
-		(stroke
-			(width 0)
-			(type default)
-		)
-	)
-	(wire
-		(pts
-			(xy 127 117.475) (xy 127 118.745)
+			(xy 125.73 114.3) (xy 125.73 115.57)
 		)
 		(stroke
@@
 	(wire
 		(pts
-			(xy 72.39 73.66) (xy 72.39 77.47)
+			(xy 72.39 74.93) (xy 72.39 77.47)
 		)
 		(stroke
@@
 	(wire
 		(pts
-			(xy 101.6 125.095) (xy 101.6 118.745)
-		)
-		(stroke
-			(width 0)
-			(type default)
-		)
-	)
-	(wire
-		(pts
-			(xy 101.6 146.05) (xy 101.6 140.335)
+			(xy 104.14 146.05) (xy 104.14 140.335)
 		)
 		(stroke
@@
 		)
 	)
-	(wire
-		(pts
-			(xy 101.6 140.335) (xy 104.14 140.335)
-		)
-		(stroke
-			(width 0)
-			(type default)
-		)
-	)
 	(bus
 		(pts
@@
 	(wire
 		(pts
-			(xy 127 121.285) (xy 123.19 121.285)
+			(xy 125.73 118.11) (xy 121.92 118.11)
 		)
 		(stroke
@@
 	(symbol
 		(lib_id "fuse mount:3587")
-		(at 115.57 118.745 0)
+		(at 114.3 118.11 0)
 		(unit 1)
 		(exclude_from_sim no)
@@
 		(fields_autoplaced yes)
 		(property "Reference" "F2"
-			(at 115.57 112.395 0)
+			(at 114.3 111.76 0)
 			(effects
 				(font
@@
 		)
 		(property "Value" "Fusemount"
-			(at 115.57 114.935 0)
+			(at 114.3 114.3 0)
 			(effects
 				(font
@@
 		)
 		(property "Footprint" "askibidi:Fusemount"
-			(at 115.57 118.745 0)
+			(at 114.3 118.11 0)
 			(effects
 				(font
@@
 		)
 		(property "Datasheet" ""
-			(at 115.57 118.745 0)
+			(at 114.3 118.11 0)
 			(effects
 				(font
@@
 		)
 		(property "Description" ""
-			(at 115.57 118.745 0)
+			(at 114.3 118.11 0)
 			(effects
 				(font
@@
 		)
 		(property "PARTREV" "D"
-			(at 115.57 118.745 0)
+			(at 114.3 118.11 0)
 			(effects
 				(font
@@
 		)
 		(property "STANDARD" "Manufacturer Recommendation"
-			(at 115.57 118.745 0)
+			(at 114.3 118.11 0)
 			(effects
 				(font
@@
 		)
 		(property "SNAPEDA_PN" "3587"
-			(at 115.57 118.745 0)
+			(at 114.3 118.11 0)
 			(effects
 				(font
@@
 		)
 		(property "MAXIMUM_PACKAGE_HEIGHT" "8.37mm"
-			(at 115.57 118.745 0)
+			(at 114.3 118.11 0)
 			(effects
 				(font
@@
 		)
 		(property "MANUFACTURER" "Keystone"
-			(at 115.57 118.745 0)
+			(at 114.3 118.11 0)
 			(effects
 				(font
@@
 	(symbol
 		(lib_id "power:GND")
-		(at 74.93 73.66 90)
+		(at 74.93 74.93 90)
 		(unit 1)
 		(exclude_from_sim no)
@@
 		(fields_autoplaced yes)
 		(property "Reference" "#PWR03"
-			(at 81.28 73.66 0)
+			(at 81.28 74.93 0)
 			(effects
 				(font
@@
 		)
 		(property "Value" "GND"
-			(at 78.74 73.66 90)
+			(at 78.74 74.93 90)
 			(effects
 				(font
@@
 		)
 		(property "Footprint" ""
-			(at 74.93 73.66 0)
+			(at 74.93 74.93 0)
 			(effects
 				(font
@@
 		)
 		(property "Datasheet" ""
-			(at 74.93 73.66 0)
+			(at 74.93 74.93 0)
 			(effects
 				(font
@@
 		)
 		(property "Description" ""
-			(at 74.93 73.66 0)
+			(at 74.93 74.93 0)
 			(effects
 				(font
@@
 		(lib_name "GND_1")
 		(lib_id "power:GND")
-		(at 127 117.475 180)
+		(at 125.73 114.3 180)
 		(unit 1)
 		(exclude_from_sim no)
@@
 		(fields_autoplaced yes)
 		(property "Reference" "#PWR08"
-			(at 127 111.125 0)
+			(at 125.73 107.95 0)
 			(effects
 				(font
@@
 		)
 		(property "Value" "GND"
-			(at 127 112.395 0)
+			(at 125.73 109.22 0)
 			(effects
 				(font
@@
 		)
 		(property "Footprint" ""
-			(at 127 117.475 0)
+			(at 125.73 114.3 0)
 			(effects
 				(font
@@
 		)
 		(property "Datasheet" ""
-			(at 127 117.475 0)
+			(at 125.73 114.3 0)
 			(effects
 				(font
@@
 		)
 		(property "Description" ""
-			(at 127 117.475 0)
+			(at 125.73 114.3 0)
 			(effects
 				(font
@@
 	(symbol
 		(lib_id "Connector_Generic:Conn_01x02")
-		(at 72.39 68.58 90)
+		(at 72.39 69.85 90)
 		(unit 1)
 		(exclude_from_sim no)
@@
 		(fields_autoplaced yes)
 		(property "Reference" "J6"
-			(at 77.47 67.3099 90)
+			(at 77.47 68.5799 90)
 			(effects
 				(font
@@
 		)
 		(property "Value" "Sparkin"
-			(at 77.47 69.8499 90)
+			(at 77.47 71.1199 90)
 			(effects
 				(font
@@
 		)
 		(property "Footprint" "Connector_AMASS:AMASS_XT60-F_1x02_P7.20mm_Vertical"
-			(at 72.39 68.58 0)
+			(at 72.39 69.85 0)
 			(effects
 				(font
@@
 		)
 		(property "Datasheet" "~"
-			(at 72.39 68.58 0)
+			(at 72.39 69.85 0)
 			(effects
 				(font
@@
 		)
 		(property "Description" ""
-			(at 72.39 68.58 0)
+			(at 72.39 69.85 0)
 			(effects
 				(font
@@
 	(symbol
 		(lib_id "Connector_Generic:Conn_01x02")
-		(at 132.08 118.745 0)
+		(at 130.81 115.57 0)
 		(unit 1)
 		(exclude_from_sim no)
@@
 		(fields_autoplaced yes)
 		(property "Reference" "J5"
-			(at 134.62 118.7449 0)
+			(at 133.35 115.5699 0)
 			(effects
 				(font
@@
 		)
 		(property "Value" "Sparkout 48V"
-			(at 134.62 121.2849 0)
+			(at 133.35 118.1099 0)
 			(effects
 				(font
@@
 		)
 		(property "Footprint" "Connector_AMASS:AMASS_XT60-F_1x02_P7.20mm_Vertical"
-			(at 132.08 118.745 0)
+			(at 130.81 115.57 0)
 			(effects
 				(font
@@
 		)
 		(property "Datasheet" "~"
-			(at 132.08 118.745 0)
+			(at 130.81 115.57 0)
 			(effects
 				(font
@@
 		)
 		(property "Description" ""
-			(at 132.08 118.745 0)
-			(effects
-				(font
+			(at 130.81 115.57 0)
+			(effects
+				(font
