File: Skibidi/Skibid-i/Skibidi-ControlBoard/Skibid-i.kicad_pcb (KiCad board)
At the start: 2 copper layers, 128.7 x 66.8 mm, 60 parts, among them IC1 TEENSY_4.1, J10 Screw_Terminal_01x03, J12 Screw_Terminal_01x03, J13 P78E05-1000, J14 Battery, J15 Conn_01x03_Pin, J16 Conn_01x02_Pin, J17 Conn_01x08_Pin, J18 SparkIN, J19 SparkOUT, J2 Screw_Terminal_01x03, J20 Screw_Terminal_01x03, J21 Motor1, J22 Motor2, J3 Screw_Terminal_01x03, J4 Screw_Terminal_01x03, J5 Screw_Terminal_01x03, J6 Screw_Terminal_01x03, J7 Screw_Terminal_01x03, J8 Screw_Terminal_01x03, J9 Screw_Terminal_01x03, Q1 WL-OCPT_SERIES_357, Q2 WL-OCPT_SERIES_357, Q3 WL-OCPT_SERIES_357, Q4 WL-OCPT_SERIES_357, Q5 WL-OCPT_SERIES_357, Q6 WL-OCPT_SERIES_357, Q7 WL-OCPT_SERIES_357, SW2 210-4MS

Commit message: erm
Parts:
- removed C16: 22uF, askibidi:Ecap
- removed C18: 100uF, Capacitor_SMD:CP_Elec_6.3x5.4
- removed F2: 3587, askibidi:Fusemount
- removed J14: Battery, Connector_AMASS:AMASS_XT60-F_1x02_P7.20mm_Vertical
- removed J16: Conn_01x02_Pin, Connector_AMASS:AMASS_XT60-F_1x02_P7.20mm_Vertical
- removed J18: SparkIN, Connector_AMASS:AMASS_XT60-F_1x02_P7.20mm_Vertical
- removed PS1: RSO-4812S_H2, askibidi:12vConvertor
- J19: value SparkOUT -> 12V; footprint Connector_AMASS:AMASS_XT60-F_1x02_P7.20mm_Vertical -> Connector_AMASS:AMASS_XT30U-F_1x02_P5.0mm_Vertical
- moved J2 40.0 mm to (228.5, 83.6)
- moved J12 34.2 mm to (180.5, 82.6)
- moved C13 30.5 mm to (233.3, 83.7), turned to -90 degrees
- moved J15 26.6 mm to (243.3, 86.9), turned to 90 degrees
- moved C15 23.3 mm to (175.4, 84.0)
- moved J19 21.5 mm to (238.1, 80.5)
- moved C12 16.1 mm to (248.6, 81.4), turned to -90 degrees
- moved D1 11.6 mm to (257.1, 77.5), turned to 90 degrees
- moved J17 10.8 mm to (155.5, 69.8)
- moved J21 8.09 mm to (201.6, 83.1)
- moved J22 7.85 mm to (212.6, 83.2)
- moved C4 7.56 mm to (260.9, 72.3), turned to -90 degrees
- moved J3 7.05 mm to (258.8, 66.3)
- moved R1 4.55 mm to (266.2, 53.0)
- moved C14 4.54 mm to (155.3, 65.5)
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Connections:
- J19 pad 2: +48V -> +12V
Routing:
- net LN4: track 58.1 -> 11.8 mm
- net LN3: track 62.0 -> 21.9 mm
- net +48V: track 30.1 -> 0.00 mm
- net +12V: track 287.4 -> 263.0 mm
- net Start: track 70.8 -> 50.1 mm
- net Net-(J14-Pin_2): track 14.2 -> 0.00 mm
- net SCL: track 46.2 -> 34.7 mm
- net SDA: track 48.5 -> 37.2 mm
- net +5V: track 41.1 -> 32.3 mm
- net Net-(J18-Pin_2): track 7.85 -> 0.00 mm
- net +3.3V: track 340.9 -> 347.7 mm
- net Dis1: track 37.8 -> 33.7 mm
- net BDC22: track 18.6 -> 16.3 mm
- net Net-(Q1-Pad1): track 5.19 -> 3.61 mm
- net OM1: track 6.88 -> 8.17 mm
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Other:
- board size 128.7 x 66.8 mm -> 121.1 x 59.4 mm

Commit message: fanum taxed
fixed connection issue + added label
Parts:
- moved R2 1.36 mm to (239.0, 45.4)
Connections:
- IC1 pad 48: unconnected-(IC1-GND_2-Pad48) -> GND
- IC1 pad 49: unconnected-(IC1-GND_3-Pad49) -> GND
- IC1 pad 69: unconnected-(IC1-GND_4-Pad69) -> GND
- IC1 pad 70: unconnected-(IC1-GND_5-Pad70) -> GND
- IC1 pad 71: unconnected-(IC1-GND_6-Pad71) -> GND
Routing:
- net Start: track 50.1 -> 51.8 mm
- net OM2: track 7.00 -> 8.36 mm
- net Net-(Q2-Pad1): track 4.63 -> 3.27 mm
- net Dis1: track 33.7 -> 33.8 mm, vias 0 -> 2
- net +3.3V: vias 1 -> 7
- net DIP1: vias 0 -> 2
- net Dis3: vias 0 -> 2
- net Dis2: vias 0 -> 2
Other:
- board text added: "+"
- board text added: "gnd"
- board text added: "p2"
- board text added: "p3"
- board text added: "p4"
- board text added: "p5"
- board text removed: "Pin2"

Commit message: push tuah
finished labeling control board
Other:
- board text added: "p10"
- board text added: "p14"
- board text added: "p15"
- board text added: "p16"
- board text added: "p17"
- board text added: "p6"
- board text added: "p9"

Commit message: sigma fanum
Parts:
- added J1: Motor3, askibidi:Screwterminal2, F.Cu at (261.9, 83.6)
- moved J17 5.80 mm to (149.7, 70.0)
- moved D1 2.41 mm to (255.5, 75.7), turned to 0 degrees
- moved C10 2.40 mm to (261.9, 45.5)
- moved C7 1.61 mm to (231.1, 45.4), turned to 0 degrees
- moved C12 1.38 mm to (249.1, 82.7)
- moved C11 1.30 mm to (149.5, 44.0)
- moved C5 1.28 mm to (246.6, 45.4), turned to 180 degrees
- moved R2 1.26 mm to (239.0, 44.1)
- moved R6 1.25 mm to (168.1, 44.5)
- moved C3 1.12 mm to (177.7, 44.5), turned to 0 degrees
- moved C13 0.95 mm to (233.3, 84.6)
- moved J15 0.58 mm to (243.9, 86.8)
Routing:
- net +3.3V: track 347.7 -> 365.4 mm
- net SCL: track 34.7 -> 40.5 mm
- net SDA: track 37.2 -> 42.9 mm
- net +12V: track 263.0 -> 268.6 mm
- net OM2: track 8.36 -> 7.10 mm
- net Net-(Q2-Pad1): track 3.27 -> 4.53 mm
- net OM6: track 6.52 -> 7.77 mm
- net Net-(Q6-Pad1): track 4.55 -> 3.37 mm
Other:
- board size 121.1 x 59.4 mm -> 121.3 x 59.4 mm
- board text added: "+3.3V"
- board text added: "-"
- board text added: "Designed by: Joe Sung Cody Gee Elliot Anders"
- board text added: "GND"
- board text added: "XXX"
- board text added: "p13"
- board text removed: "A16"
- board text removed: "A17"
- board text removed: "Pin10"
- board text removed: "Pin3"
- board text removed: "Pin4"
- board text removed: "Pin5"
- board text removed: "Pin6"
- board text removed: "Pin9"

Commit message: done with contrl board
Parts:
- C2: footprint askibidi:Ecap -> Capacitor_SMD:C_2220_5750Metric
- D1: footprint askibidi:LED -> LED_SMD:LED_1206_3216Metric
- moved C15 12.4 mm to (163.7, 80.0), turned to 0 degrees
- moved D1 5.47 mm to (260.9, 76.2), turned to 180 degrees
- moved J17 0.90 mm to (148.8, 70.0)
Routing:
- net +3.3V: track 365.4 -> 360.1 mm
- net Net-(D1-A): track 4.22 -> 6.47 mm
- net SCL: track 40.5 -> 41.4 mm
- net SDA: track 42.9 -> 43.8 mm

Commit message: fff
Changed lines of the file:
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@@
 		(tags "LED")
 		(property "Reference" "D1"
-			(at 0 -1.82 360)
+			(at 0 -1.82 0)
 			(layer "F.SilkS")
 			(effects
@@
 		)
 		(property "Value" "LED"
-			(at 0 1.82 360)
+			(at 0 1.82 0)
 			(layer "F.Fab")
 			(effects
@@
 		)
 		(fp_text user "${REFERENCE}"
-			(at 0 0 360)
+			(at 0 0 0)
 			(layer "F.Fab")
 			(effects
@@
 		(tags "capacitor")
 		(property "Reference" "C15"
-			(at 0 -1.68 360)
+			(at 0 -1.68 0)
 			(layer "F.SilkS")
 			(effects
@@
 		)
 		(property "Value" "0.1uF"
-			(at 0 1.68 360)
+			(at 0 1.68 0)
 			(layer "F.Fab")
 			(effects
@@
 		)
 		(fp_text user "${REFERENCE}"
-			(at 0 0 360)
+			(at 0 0 0)
 			(layer "F.Fab")
 			(effects
@@
 		(tags "Through hole pin header THT 1x08 2.54mm single row")
 		(property "Reference" "J17"
-			(at 0 -2.33 360)
+			(at 0 -2.33 0)
 			(layer "F.SilkS")
 			(effects
@@
 		)
 		(property "Value" "Conn_01x08_Pin"
-			(at 28.37 22.81 360)
+			(at 28.37 22.81 0)
 			(layer "F.Fab")
 			(effects
@@
 		)
 	)
-	(gr_text "Designed by: \n  Joe Sung\n  Cody Gee \n  Elliot Anders"
-		(at 166.4 86.45 0)
+	(gr_text " Designed by: \n  Joe Sung\n  Cody Gee \n Elliot Anders"
+		(at 166.1 87.1 0)
 		(layer "F.SilkS")
 		(effects
 			(font
-				(size 1 1)
+				(size 1.2 1)
 				(thickness 0.25)
 				(bold yes)
@@
 	)
 	(segment
-		(start 188.87 67.03)
+		(start 187.8 68.1)
 		(end 184.9 71)
 		(width 0.25)
@@
 	)
 	(segment
-		(start 188.87 67)
-		(end 188.87 67.03)
+		(start 184.9 71)
+		(end 171.1 71)
 		(width 0.25)
 		(layer "F.Cu")
@@
 		(net 32)
 	)
-	(segment
-		(start 171.1 71)
-		(end 184.9 71)
-		(width 0.25)
-		(layer "F.Cu")
-		(net 32)
-	)
 	(via
 		(at 193.38 62.52)
@@
 	)
 	(via
-		(at 188.87 67)
+		(at 187.8 68.1)
 		(size 0.8)
 		(drill 0.4)
@@
 	)
 	(segment
-		(start 188.9 67)
-		(end 188.87 67)
-		(width 0.25)
-		(layer "B.Cu")
-		(net 32)
-	)
-	(segment
-		(start 193.38 62.52)
-		(end 188.9 67)
+		(start 187.8 68.1)
+		(end 193.38 62.52)
 		(width 0.25)
 		(layer "B.Cu")
@@
 	)
 	(segment
-		(start 254.07 48.93)
-		(end 256.3 48.93)
+		(start 229.65 56.73)
+		(end 226.93 59.45)
 		(width 0.25)
 		(layer "F.Cu")
@@
 	)
 	(segment
-		(start 233.2 55.3)
+		(start 235.7 55.3)
 		(end 247.7 55.3)
 		(width 0.25)
@@
 	)
 	(segment
-		(start 229.65 56.73)
-		(end 226.93 59.45)
+		(start 247.7 55.3)
+		(end 254.07 48.93)
 		(width 0.25)
 		(layer "F.Cu")
@@
 	)
 	(segment
-		(start 247.7 55.3)
-		(end 254.07 48.93)
+		(start 254.07 48.93)
+		(end 256.3 48.93)
 		(width 0.25)
 		(layer "F.Cu")
@@
 	)
 	(via
-		(at 233.2 55.3)
+		(at 235.7 55.3)
 		(size 0.8)
 		(drill 0.4)
@@
 	)
 	(segment
-		(start 229.73 56.73)
-		(end 231.16 55.3)
+		(start 231.16 55.3)
+		(end 229.73 56.73)
 		(width 0.25)
 		(layer "B.Cu")
@@
 	)
 	(segment
-		(start 231.16 55.3)
-		(end 233.2 55.3)
+		(start 235.7 55.3)
+		(end 231.16 55.3)
 		(width 0.25)
 		(layer "B.Cu")
@@
 	)
 	(segment
-		(start 227.945 55.895)
-		(end 224.39 59.45)
+		(start 246.754899 52.245101)
+		(end 246.754899 51.22)
 		(width 0.25)
 		(layer "F.Cu")
@@
 	)
 	(segment
-		(start 246.754899 52.245101)
-		(end 246.754899 51.22)
+		(start 237.5 53.4)
+		(end 245.6 53.4)
 		(width 0.25)
 		(layer "F.Cu")
@@
 	)
 	(segment
-		(start 235.87 53.4)
-		(end 245.6 53.4)
+		(start 227.945 55.895)
+		(end 224.39 59.45)
 		(width 0.25)
 		(layer "F.Cu")
@@
 	)
 	(via
-		(at 235.87 53.4)
+		(at 237.5 53.4)
 		(size 0.8)
 		(drill 0.4)
@@
 	)
 	(segment
-		(start 227.945 55.895)
-		(end 230.44 53.4)
+		(start 230.44 53.4)
+		(end 227.945 55.895)
 		(width 0.25)
 		(layer "B.Cu")
@@
 	)
 	(segment
-		(start 230.44 53.4)
-		(end 235.87 53.4)
+		(start 237.5 53.4)
+		(end 230.44 53.4)
 		(width 0.25)
 		(layer "B.Cu")

Commit message: Added Logo
Parts:
- added G***: LOGO, SkibidiLogos:skibidi_logo, F.Cu at (155.6, 79.9)

Commit message: joehjoe
Parts:
- added G***: LOGO, SkibidiLogos:skibidi_logo, F.Cu at (193.5, 66.5)
- added G***: LOGO, SkibidiLogos:skibidi_logo, F.Cu at (156.8, 80.3)
- added G***: LOGO, SkibidiLogos:skibidi_logo, F.Cu at (179.5, 66.6)
- added G***: LOGO, SkibidiLogos:skibidi_logo, F.Cu at (186.5, 66.5)
- moved G*** 109.2 mm to (264.7, 83.6)
- moved J1 3.42 mm to (258.5, 84.0)
- moved C12 1.10 mm to (248.1, 82.2)
- moved J15 0.81 mm to (243.1, 86.8)
Routing:
- net +3.3V: track 360.1 -> 357.2 mm
- net Start: track 51.9 -> 49.9 mm
Other:
- board text added: "Joe Alex Cody Eilliot"
- board text added: "Skibidi Toliet"
- board text added: "Skibidi Toliet Ohio Rizz"
- board text removed: "Erm What the Skibidi..."
