File: Skibidi/Skibid-i/Skibidi-ControlBoard/Skibid-i.kicad_sch (KiCad schematic)
At the start: 53 parts, among them IC1 TEENSY_4.1, J10 Screw_Terminal_01x03, J12 Screw_Terminal_01x03, J13 P78E05-1000, J15 Conn_01x03_Pin, J17 Conn_01x08_Pin, J19 12V, J2 Screw_Terminal_01x03, J20 Screw_Terminal_01x03, J21 Motor1, J22 Motor2, J3 Screw_Terminal_01x03, J4 Screw_Terminal_01x03, J5 Screw_Terminal_01x03, J6 Screw_Terminal_01x03, J7 Screw_Terminal_01x03, J8 Screw_Terminal_01x03, J9 Screw_Terminal_01x03, Q1 WL-OCPT_SERIES_357, Q2 WL-OCPT_SERIES_357, Q3 WL-OCPT_SERIES_357, Q4 WL-OCPT_SERIES_357, Q5 WL-OCPT_SERIES_357, Q6 WL-OCPT_SERIES_357, Q7 WL-OCPT_SERIES_357, SW2 210-4MS

Commit message: fanum taxed
fixed connection issue + added label
Connections:
- net GND: now also IC1.45 (GND_1), IC1.48 (GND_2), IC1.49 (GND_3), IC1.69 (GND_4), IC1.70 (GND_5), IC1.71 (GND_6)
- no-connect marks 41 -> 35

Commit message: sigma fanum
Parts:
- added J1: Motor3, askibidi:Screwterminal2, symbol Connector:Screw_Terminal_01x02
Connections:
- net +3.3V: now also J1.2 (Pin_2)
- net GND: now also J1.1 (Pin_1)
Changed lines of the file:
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@@
 	)
 	(symbol
+		(lib_id "Connector:Screw_Terminal_01x02")
+		(at 190.5 92.71 270)
+		(unit 1)
+		(exclude_from_sim no)
+		(in_bom yes)
+		(on_board yes)
+		(dnp no)
+		(property "Reference" "J1"
+			(at 191.77 99.06 90)
+			(effects
+				(font
+					(size 1.27 1.27)
+				)
+				(justify right)
+			)
+		)
+		(property "Value" "Motor3"
+			(at 191.77 96.52 90)
+			(effects
+				(font
+					(size 1.27 1.27)
+				)
+				(justify right)
+			)
+		)
+		(property "Footprint" "askibidi:Screwterminal2"
+			(at 190.5 92.71 0)
+			(effects
+				(font
+					(size 1.27 1.27)
+				)
+				(hide yes)
+			)
+		)
+		(property "Datasheet" "~"
+			(at 190.5 92.71 0)
+			(effects
+				(font
+					(size 1.27 1.27)
+				)
+				(hide yes)
+			)
+		)
+		(property "Description" ""
+			(at 190.5 92.71 0)
+			(effects
+				(font
+					(size 1.27 1.27)
+				)
+				(hide yes)
+			)
+		)
+		(pin "1"
+		)
+		(pin "2"
+		)
+		(instances
+			(project "Skibid-i"
+				(path "/bfc511a5-2c92-46fd-9868-0fe25107d7eb"
+					(reference "J1")
+					(unit 1)
+				)
+			)
+		)
+	)
+	(symbol
 		(lib_id "Connector:Screw_Terminal_01x03")
 		(at 57.15 48.26 180)
@@
 	)
 	(symbol
+		(lib_name "+3.3V_1")
+		(lib_id "power:+3.3V")
+		(at 187.96 87.63 0)
+		(unit 1)
+		(exclude_from_sim no)
+		(in_bom yes)
+		(on_board yes)
+		(dnp no)
+		(fields_autoplaced yes)
+		(property "Reference" "#PWR059"
+			(at 187.96 91.44 0)
+			(effects
+				(font
+					(size 1.27 1.27)
+				)
+				(hide yes)
+			)
+		)
+		(property "Value" "+3.3V"
+			(at 187.96 82.55 0)
+			(effects
+				(font
+					(size 1.27 1.27)
+				)
+			)
+		)
+		(property "Footprint" ""
+			(at 187.96 87.63 0)
+			(effects
+				(font
+					(size 1.27 1.27)
+				)
+				(hide yes)
+			)
+		)
+		(property "Datasheet" ""
+			(at 187.96 87.63 0)
+			(effects
+				(font
+					(size 1.27 1.27)
+				)
+				(hide yes)
+			)
+		)
+		(property "Description" "Power symbol creates a global label with name \"+3.3V\""
+			(at 187.96 87.63 0)
+			(effects
+				(font
+					(size 1.27 1.27)
+				)
+				(hide yes)
+			)
+		)
+		(pin "1"
+		)
+		(instances
+			(project ""
+				(path "/bfc511a5-2c92-46fd-9868-0fe25107d7eb"
+					(reference "#PWR059")
+					(unit 1)
+				)
+			)
+		)
+	)
+	(symbol
 		(lib_id "Device:C")
 		(at 63.5 30.48 0)
@@
 					(unit 1)
 				)
+			)
+		)
+	)
+	(symbol
+		(lib_name "GND_2")
+		(lib_id "power:GND")
+		(at 190.5 87.63 180)
+		(unit 1)
+		(exclude_from_sim no)
+		(in_bom yes)
+		(on_board yes)
+		(dnp no)
+		(fields_autoplaced yes)
+		(property "Reference" "#PWR061"
+			(at 190.5 81.28 0)
+			(effects
+				(font
+					(size 1.27 1.27)
+				)
+				(hide yes)
+			)
+		)
+		(property "Value" "GND"
+			(at 190.5 82.55 0)
+			(effects
+				(font
+					(size 1.27 1.27)
+				)
+			)
+		)
+		(property "Footprint" ""
+			(at 190.5 87.63 0)
+			(effects
+				(font
+					(size 1.27 1.27)
+				)
+				(hide yes)
+			)
+		)
+		(property "Datasheet" ""
+			(at 190.5 87.63 0)
+			(effects
+				(font
+					(size 1.27 1.27)
+				)
+				(hide yes)
+			)
+		)
+		(property "Description" "Power symbol creates a global label with name \"GND\" , ground"
+			(at 190.5 87.63 0)
+			(effects
+				(font
+					(size 1.27 1.27)
+				)
+				(hide yes)
+			)
+		)
+		(pin "1"
+		)
+		(instances
+			(project ""
+				(path "/bfc511a5-2c92-46fd-9868-0fe25107d7eb"
+					(reference "#PWR061")
+					(unit 1)
+				)

Commit message: done with contrl board
Parts:
- C2: footprint askibidi:Ecap -> Capacitor_SMD:C_2220_5750Metric
- D1: footprint askibidi:LED -> LED_SMD:LED_1206_3216Metric
Changed lines of the file:
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@@
 			)
 		)
-		(property "Footprint" "askibidi:Ecap"
+		(property "Footprint" "Capacitor_SMD:C_2220_5750Metric"
 			(at 246.6848 34.29 0)
 			(effects
@@
 			)
 		)
-		(property "Footprint" "askibidi:LED"
+		(property "Footprint" "LED_SMD:LED_1206_3216Metric"
 			(at 227.33 63.5 0)
 			(effects

Commit message: done
Parts:
- removed J1: Motor3, askibidi:Screwterminal2, symbol Connector:Screw_Terminal_01x02
- removed J21: Motor1, askibidi:Screwterminal2, symbol Connector:Screw_Terminal_01x02
- removed J22: Motor2, askibidi:Screwterminal2, symbol Connector:Screw_Terminal_01x02
- added F1: Fuse, Fuse:Fuse_1206_3216Metric, symbol Device:Fuse
- added H1, H2, H3, H4, H5: MountingHole, MountingHole:MountingHole_2.5mm, symbol Mechanical:MountingHole
- added J1: Conn_02x05_Odd_Even, Connector_PinSocket_2.54mm:PinSocket_2x05_P2.54mm_Vertical, symbol Connector_Generic:Conn_02x05_Odd_Even
- added SW1: SW_Nidec_CAS-120A1, askibidi:swotcslide, symbol Switch:SW_Nidec_CAS-120A1
Connections:
- net +12V: now also F1.1; no longer J19.2 (Pin_2)
- net +5V: now also J1.9 (Pin_9)
- net BDC1: now also J1.5 (Pin_5)
- net BDC11: now also J1.3 (Pin_3)
- net BDC2: now also J1.4 (Pin_4)
- net BDC22: now also J1.6 (Pin_6)
- net GND: now also J1.1 (Pin_1)
- new net: F1.2, SW1.1 (C)
- new net: J19.2 (Pin_2), SW1.2 (B)
- no-connect marks 35 -> 40
Other:
- moved on the sheet: J19

Commit message: think its done
Parts:
- C1: footprint askibidi:10uF -> Capacitor_SMD:C_0805_2012Metric
- C2: value 22uF -> 10uF; footprint Capacitor_SMD:C_2220_5750Metric -> Capacitor_SMD:C_0805_2012Metric
Changed lines of the file:
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@@
 			)
 		)
-		(property "Value" "22uF"
+		(property "Value" "10uF"
 			(at 244.602 36.83 0)
 			(effects
@@
 			)
 		)
-		(property "Footprint" "Capacitor_SMD:C_2220_5750Metric"
+		(property "Footprint" "Capacitor_SMD:C_0805_2012Metric"
 			(at 246.6848 34.29 0)
 			(effects
@@
 			)
 		)
-		(property "Footprint" "askibidi:10uF"
+		(property "Footprint" "Capacitor_SMD:C_0805_2012Metric"
 			(at 246.6848 46.99 0)
 			(effects

Commit message: some final changese
Parts:
- added D2, D3, D4, D5, D6, D7, D8: LED, LED_SMD:LED_1206_3216Metric, symbol Device:LED
- added J11: Conn_01x02_Pin, Connector_PinHeader_2.54mm:PinHeader_1x02_P2.54mm_Vertical, symbol Connector:Conn_01x02_Pin
- R1, R2, R3, R4, R5, R6, R7, R8: footprint Capacitor_SMD:C_1206_3216Metric -> Resistor_SMD:R_0805_2012Metric
Connections:
- net +5V: now also J11.1 (Pin_1); no longer J1.9 (Pin_9)
- net at R1.2: now also D2.2 (A); no longer Q1.1
- net at Q4.1: now also D5.1 (K); no longer R4.2
- net at Q6.1: now also D7.1 (K); no longer R6.2
- net at R3.2: now also D4.2 (A); no longer Q3.1
- net at Q2.1: now also D3.1 (K); no longer R2.2
- net at Q5.1: now also D6.1 (K); no longer R7.2
- net at Q7.1: now also D8.1 (K); no longer R5.2
- new net: J1.9 (Pin_9), J11.2 (Pin_2)
- new net: D5.2 (A), R4.2
- new net: D2.1 (K), Q1.1
- new net: D8.2 (A), R5.2
- new net: D6.2 (A), R7.2
- new net: D4.1 (K), Q3.1
- new net: D3.2 (A), R2.2
- new net: D7.2 (A), R6.2
Other:
- moved on the sheet: Q5, Q6, Q7, R1, R2, R3, R4, R5, R6, R7
