File: Jongmyeong-I/Jongmyeong-i/Jongmyeong-i.kicad_pcb (KiCad board)
At the start: 2 copper layers, 44 parts, among them J1 Screw3, J10 Screw3, J11 Screw3, J12 xt30, J2 Screw3, J3 Screw3, J4 Screw3, J5 Screw3, J6 Conn_01x03_Pin, J7 Conn_01x08_Pin, J8 Conn_01x03_Pin, J9 Screw3, SW2 SW_DPDT_x2

Commit message: finished layout
Parts:
- removed C13: 0.1uF, Capacitor_SMD:C_0805_2012Metric
- removed J10: Screw3, Connector_JST:JST_EH_B3B-EH-A_1x03_P2.50mm_Vertical
- added DRV1: ~, ZSKIBIDI:drvmotordriver, F.Cu at (185.4, 106.9)
- added DRV3: ~, ZSKIBIDI:drvmotordriver, F.Cu at (117.3, 107.2)
- added J13: Screw_Terminal_01x02, Connector_PinHeader_2.54mm:PinHeader_1x02_P2.54mm_Vertical, F.Cu at (157.8, 112.8)
- added J14: Screw_Terminal_01x02, Connector_PinHeader_2.54mm:PinHeader_1x02_P2.54mm_Vertical, F.Cu at (147.7, 113.0)
- moved J12 72.3 mm to (111.9, 96.2), turned to 90 degrees
- moved J6 57.1 mm to (116.7, 66.5), turned to -90 degrees
- moved D1 56.8 mm to (112.2, 79.5), turned to 90 degrees
- moved C8 51.3 mm to (174.6, 112.2), turned to 90 degrees
- moved C1 49.8 mm to (111.5, 72.0), turned to -90 degrees
- moved D6 49.5 mm to (119.7, 96.4), turned to 90 degrees
- moved C6 47.6 mm to (124.2, 83.2), turned to -90 degrees
- moved C11 44.1 mm to (128.3, 76.2)
- moved D4 44.0 mm to (127.1, 66.3)
- moved J8 43.0 mm to (165.7, 113.2), turned to 90 degrees
- moved C9 42.8 mm to (191.8, 97.0), turned to 90 degrees
- moved R1 41.6 mm to (117.2, 71.5), turned to 180 degrees
- moved R6 39.2 mm to (119.7, 89.2), turned to -90 degrees
- moved C5 39.1 mm to (152.4, 106.7), turned to 180 degrees
- moved J5 37.8 mm to (185.7, 77.0), turned to -90 degrees
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Connections:
- J11 pad 1: S1 -> LN2
- J7 pad 3: SDA -> SCL
- J9 pad 1: S1 -> LN1
- TB1 pad 15: unconnected-(TB1-D12/MISO-Pad15) -> ST
Routing:
- net +5V: track 0.00 -> 182.1 mm, vias 0 -> 1
- net +12V: track 0.00 -> 141.5 mm
- net +3.3V: track 0.00 -> 128.4 mm, vias 0 -> 3
- net S4: track 0.00 -> 48.5 mm
- net MOTOR1B: track 0.00 -> 45.1 mm
- net LN2: track 0.00 -> 43.0 mm
- net 5v: track 0.00 -> 42.9 mm, vias 0 -> 2
- net MOTOR1A: track 0.00 -> 42.6 mm
- net MOTOR2A: track 0.00 -> 38.9 mm
- net Net-(DRV1-Out1): track 0.00 -> 37.4 mm
- net MOTOR2B: track 0.00 -> 33.1 mm
- net Net-(DRV1-Out2): track 0.00 -> 31.5 mm
- net LN1: track 0.00 -> 31.3 mm
- net Net-(DRV3-Out2): track 0.00 -> 30.8 mm
- net S5: track 0.00 -> 27.1 mm
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- added copper zone on F.Cu, net GND
Other:
- board outline added: 88 x 56.4 mm
- board text added: "${REFERENCE}"

Commit message: jong
Routing:
- net Servo: track 0.00 -> 56.1 mm, vias 0 -> 1
Changed lines of the file:
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@@
 		)
 		(fp_text user "${REFERENCE}"
-			(at 0 8.89 360)
+			(at 0 8.89 0)
 			(layer "F.Fab")
 			(effects
@@
 		)
 		(fp_text user "${REFERENCE}"
-			(at 0 1.27 360)
+			(at 0 1.27 0)
 			(layer "F.Fab")
 			(effects
@@
 		)
 		(fp_text user "${REFERENCE}"
-			(at 0 2.54 360)
+			(at 0 2.54 0)
 			(layer "F.Fab")
 			(effects
@@
 		(tags "LED")
 		(property "Reference" "D4"
-			(at 0 -1.82 360)
+			(at 0 -1.82 0)
 			(layer "F.SilkS")
 			(effects
@@
 		)
 		(property "Value" "LED"
-			(at 0 1.82 360)
+			(at 0 1.82 0)
 			(layer "F.Fab")
 			(effects
@@
 		)
 		(fp_text user "${REFERENCE}"
-			(at 0 0 360)
+			(at 0 0 0)
 			(layer "F.Fab")
 			(effects
@@
 		(tags "capacitor")
 		(property "Reference" "C5"
-			(at 0 -1.68 360)
+			(at 0 -1.68 0)
 			(layer "F.SilkS")
 			(effects
@@
 		)
 		(property "Value" "0.1uF"
-			(at 0 1.68 360)
+			(at 0 1.68 0)
 			(layer "F.Fab")
 			(effects
@@
 		)
 		(fp_text user "${REFERENCE}"
-			(at 0 0 360)
+			(at 0 0 0)
 			(layer "F.Fab")
 			(effects
@@
 		(tags "resistor")
 		(property "Reference" "R1"
-			(at 0 -1.65 360)
+			(at 0 -1.65 0)
 			(layer "F.SilkS")
 			(effects
@@
 		)
 		(property "Value" "180"
-			(at 0 1.65 360)
+			(at 0 1.65 0)
 			(layer "F.Fab")
 			(effects
@@
 		)
 		(fp_text user "${REFERENCE}"
-			(at 0 0 360)
+			(at 0 0 0)
 			(layer "F.Fab")
 			(effects
@@
 		)
 		(fp_text user "${REFERENCE}"
-			(at 0 1.27 360)
+			(at 0 1.27 0)
 			(layer "F.Fab")
 			(effects
@@
 		(tags "LED")
 		(property "Reference" "D2"
-			(at 0 -1.82 360)
+			(at 0 -1.82 0)
 			(layer "F.SilkS")
 			(effects
@@
 		)
 		(property "Value" "LED"
-			(at 0 1.82 360)
+			(at 0 1.82 0)
 			(layer "F.Fab")
 			(effects
@@
 		)
 		(fp_text user "${REFERENCE}"
-			(at 0 0 360)
+			(at 0 0 0)
 			(layer "F.Fab")
 			(effects
@@
 		(at 132.7 111.15 180)
 		(property "Reference" "SW2"
-			(at -3.175 -4.445 360)
+			(at -3.175 -4.445 0)
 			(layer "F.SilkS")
 			(hide yes)
@@
 		)
 		(property "Value" "SW_DPDT_x2"
-			(at 3.175 4.445 360)
+			(at 3.175 4.445 0)
 			(layer "F.Fab")
 			(effects
@@
 		)
 		(property "Footprint" "ZSKIBIDI:switch"
-			(at 0 0 360)
+			(at 0 0 0)
 			(layer "F.Fab")
 			(hide yes)
@@
 		)
 		(property "Datasheet" ""
-			(at 0 0 360)
+			(at 0 0 0)
 			(layer "F.Fab")
 			(hide yes)
@@
 		)
 		(property "Description" "Switch, dual pole double throw, separate symbols"
-			(at 0 0 360)
+			(at 0 0 0)
 			(layer "F.Fab")
 			(hide yes)
@@
 		(tags "LED")
 		(property "Reference" "D3"
-			(at 0 -1.82 360)
+			(at 0 -1.82 0)
 			(layer "F.SilkS")
 			(effects
@@
 		)
 		(property "Value" "LED"
-			(at 0 1.82 360)
+			(at 0 1.82 0)
 			(layer "F.Fab")
 			(effects
@@
 		)
 		(fp_text user "${REFERENCE}"
-			(at 0 0 360)
+			(at 0 0 0)
 			(layer "F.Fab")
 			(effects
@@
 		(tags "fuse")
 		(property "Reference" "F1"
-			(at 0 -1.82 360)
+			(at 0 -1.82 0)
 			(layer "F.SilkS")
 			(effects
@@
 		)
 		(property "Value" "Fuse"
-			(at 0 1.82 360)
+			(at 0 1.82 0)
 			(layer "F.Fab")
 			(effects
@@
 		)
 		(fp_text user "${REFERENCE}"
-			(at 0 0 360)
+			(at 0 0 0)
 			(layer "F.Fab")
 			(effects
@@
 		(tags "resistor")
 		(property "Reference" "R2"
-			(at 0 -1.65 360)
+			(at 0 -1.65 0)
 			(layer "F.SilkS")
 			(effects
@@
 		)
 		(property "Value" "180"
-			(at 0 1.65 360)
+			(at 0 1.65 0)
 			(layer "F.Fab")
 			(effects
@@
 		)
 		(fp_text user "${REFERENCE}"
-			(at 0 0 360)
+			(at 0 0 0)
 			(layer "F.Fab")
 			(effects
@@
 		(tags "resistor")
 		(property "Reference" "R3"
-			(at 0 -1.65 360)
+			(at 0 -1.65 0)
 			(layer "F.SilkS")
 			(effects
@@
 		)
 		(property "Value" "180"
-			(at 0 1.65 360)
+			(at 0 1.65 0)
 			(layer "F.Fab")
 			(effects
@@
 		)
 		(fp_text user "${REFERENCE}"
-			(at 0 0 360)
+			(at 0 0 0)
 			(layer "F.Fab")
 			(effects
@@
 		)
 		(fp_text user "${REFERENCE}"
-			(at 0 2.54 360)
+			(at 0 2.54 0)
 			(layer "F.Fab")
 			(effects
@@
 		(tags "resistor")
 		(property "Reference" "R4"
-			(at 0 -1.65 360)
+			(at 0 -1.65 0)
 			(layer "F.SilkS")
 			(effects
@@
 		)
 		(property "Value" "180"
-			(at 0 1.65 360)
+			(at 0 1.65 0)
 			(layer "F.Fab")
 			(effects
@@
 		)
 		(fp_text user "${REFERENCE}"
-			(at 0 0 360)
+			(at 0 0 0)
 			(layer "F.Fab")
 			(effects
@@
 	)
 	(segment
-		(start 171.76 97.15)
-		(end 177 97.15)
+		(start 146.55 104.05)
+		(end 159.4 104.05)
 		(width 0.2)
 		(layer "F.Cu")
@@
 	)
 	(segment
-		(start 177 107.8)
+		(start 171.76 97.15)
 		(end 177 97.15)
 		(width 0.2)
@@
 	)
 	(segment
-		(start 191.8 97.9)
-		(end 187.5 97.9)
+		(start 159.4 104.05)
+		(end 168.88 94.57)
 		(width 0.2)
 		(layer "F.Cu")
@@
 	)
 	(segment
-		(start 187.5 97.9)
-		(end 185.35 95.75)
+		(start 177 107.8)
+		(end 177 97.15)
 		(width 0.2)
 		(layer "F.Cu")
@@
 	)
 	(segment
-		(start 168.43 94.57)
-		(end 169.18 94.57)
+		(start 191.8 97.9)
+		(end 187.5 97.9)
 		(width 0.2)
 		(layer "F.Cu")
@@
 	)
 	(segment
-		(start 146.55 104.05)
-		(end 158.95 104.05)
+		(start 187.5 97.9)
+		(end 185.35 95.75)
 		(width 0.2)
 		(layer "F.Cu")
@@
 	)
 	(segment
-		(start 183.4 97.15)
-		(end 184.8 95.75)
+		(start 168.88 94.57)
+		(end 169.18 94.57)
 		(width 0.2)
 		(layer "F.Cu")
@@
 	)
 	(segment
-		(start 158.95 104.05)
-		(end 168.43 94.57)
+		(start 183.4 97.15)
+		(end 184.8 95.75)
 		(width 0.2)
 		(layer "F.Cu")
@@
 	)
 	(segment
+		(start 142.58 96.82)
+		(end 142.55 96.85)
+		(width 0.2)
+		(layer "F.Cu")
+		(net 24)
+	)
+	(segment
+		(start 142.58 80.67)
+		(end 142.58 96.82)
+		(width 0.2)
+		(layer "F.Cu")
+		(net 24)
+	)
+	(segment
+		(start 141.24 79.33)
+		(end 142.58 80.67)
+		(width 0.2)
+		(layer "F.Cu")
+		(net 24)
+	)
+	(via
+		(at 142.55 96.85)
+		(size 0.6)
+		(drill 0.3)
+		(layers "F.Cu" "B.Cu")
+		(net 24)
+	)
+	(segment
+		(start 161.75 113.15)
+		(end 165.66 113.15)
+		(width 0.2)
+		(layer "B.Cu")
+		(net 24)
+	)
+	(segment
+		(start 139.45 99.95)
+		(end 139.45 103.2)
+		(width 0.2)
+		(layer "B.Cu")
+		(net 24)
+	)
+	(segment
+		(start 139.45 103.2)
+		(end 143.6 107.35)
+		(width 0.2)
+		(layer "B.Cu")
+		(net 24)
+	)
+	(segment
+		(start 142.55 96.85)
+		(end 139.45 99.95)
+		(width 0.2)
+		(layer "B.Cu")
+		(net 24)
+	)
+	(segment
+		(start 143.6 107.35)
+		(end 155.95 107.35)
+		(width 0.2)
+		(layer "B.Cu")
+		(net 24)
+	)
+	(segment
+		(start 155.95 107.35)
+		(end 161.75 113.15)
+		(width 0.2)
+		(layer "B.Cu")
+		(net 24)
+	)
+	(segment

Commit message: mom
Parts:
- removed C11, C12: 0.1uF, Capacitor_SMD:C_0805_2012Metric
- J12: footprint Connector_AMASS:AMASS_XT30U-F_1x02_P5.0mm_Vertical -> Connector_AMASS:AMASS_XT30PW-F_1x02_P2.50mm_Horizontal
- moved D6 16.3 mm to (135.3, 100.8), turned to 180 degrees
- moved R6 15.5 mm to (129.9, 100.8), turned to 0 degrees
- moved J12 10.8 mm to (122.7, 95.4)
- moved D3 1.00 mm to (151.5, 66.8)
- moved R3 0.91 mm to (146.7, 66.8)
Connections:
- J6 pad 2: GND -> +5V
- J6 pad 3: +5V -> GND
Routing:
- net +5V: track 182.1 -> 217.7 mm
- net Net-(J12-Pin_1): track 27.0 -> 19.9 mm
- net +3.3V: track 128.4 -> 122.7 mm
- net Net-(D6-A): track 4.83 -> 3.12 mm
- net S2: track 15.5 -> 16.5 mm
- net Net-(DRV1-Out1): track 37.4 -> 38.0 mm
- net Net-(DRV1-Out2): track 31.5 -> 32.1 mm
- net +12V: track 141.5 -> 142.0 mm, vias 0 -> 2
Other:
- board size 88 x 56.4 mm -> 87.8 x 55.3 mm
- board text removed: "${REFERENCE}"

Commit message: pooki done
Parts:
- removed C1, C5: 0.1uF, Capacitor_SMD:C_0805_2012Metric
- J12: footprint Connector_AMASS:AMASS_XT30PW-F_1x02_P2.50mm_Horizontal -> Connector_AMASS:AMASS_XT30U-F_1x02_P5.0mm_Vertical
- moved J14 14.1 mm to (133.6, 114.6)
- moved J12 11.9 mm to (112.2, 89.7), turned to 0 degrees
- moved J13 11.6 mm to (169.3, 114.6)
- moved J8 9.36 mm to (174.9, 111.7), turned to 180 degrees
- moved C8 9.31 mm to (174.9, 102.9)
- moved DRV3 8.71 mm to (116.9, 98.5)
- moved R2 7.85 mm to (169.7, 66.7)
- moved PS1 7.00 mm to (180.6, 88.1), turned to 180 degrees
- moved C9 5.39 mm to (190.4, 91.8), turned to 0 degrees
- moved SW2 4.61 mm to (132.4, 106.5)
- moved R8 4.50 mm to (174.9, 96.9), turned to 90 degrees
- moved DRV1 3.55 mm to (185.6, 103.3)
- moved F1 3.31 mm to (148.4, 104.3)
- moved C10 1.65 mm to (190.5, 88.2), turned to 0 degrees
- moved D1 0.60 mm to (112.8, 79.5)
Connections:
- J11 pad 2: +3.3V -> +5V
- J12 pad 1: Net-(J12-Pin_1) -> GND
- J12 pad 2: GND -> Net-(J12-Pin_2)
- J9 pad 2: +3.3V -> +5V
- S1 pad 1A: +3.3V -> +5V
- S1 pad 2A: +3.3V -> +5V
- SW2 pad 2: Net-(J12-Pin_1) -> Net-(J12-Pin_2)
Routing:
- net +3.3V: track 122.7 -> 0.00 mm, vias 3 -> 0
- net Net-(J12-Pin_2): track 0.00 -> 24.3 mm
- net 5v: track 42.9 -> 66.5 mm, vias 2 -> 0
- net Net-(J12-Pin_1): track 19.9 -> 0.00 mm
- net Net-(DRV3-Out1): track 24.8 -> 9.92 mm
- net Net-(DRV3-Out2): track 30.8 -> 16.7 mm
- net Net-(DRV1-Out2): track 32.1 -> 19.6 mm
- net Net-(DRV1-Out1): track 38.0 -> 26.2 mm
- net Servo: track 56.1 -> 64.7 mm
- net Net-(D2-A): track 11.8 -> 4.27 mm
- net MOTOR2B: track 33.4 -> 26.4 mm
- net +12V: track 142.0 -> 148.6 mm, vias 2 -> 0
- net S1: track 13.4 -> 19.7 mm
- net MOTOR2A: track 38.9 -> 35.8 mm
- net MOTOR1B: track 45.1 -> 42.4 mm
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Other:
- board text added: "Andrew Li"
- board text added: "Joe Sung"
- board text added: "Jonathon Jia"
- board text added: "Pooki"

Commit message: done with pooki
Parts:
- added J10: Conn_01x03_Pin, Connector_PinHeader_2.54mm:PinHeader_1x03_P2.54mm_Vertical, F.Cu at (114.5, 65.5)
- moved R4 7.13 mm to (128.8, 66.3)
- moved R2 5.65 mm to (175.3, 66.7)
- moved D2 4.95 mm to (180.8, 66.6)
- moved J12 4.88 mm to (111.3, 84.8), turned to -90 degrees
- moved D4 4.40 mm to (122.7, 66.3)
- moved J6 3.69 mm to (114.5, 69.4)
- moved F1 2.95 mm to (151.4, 104.3)
- moved D1 2.89 mm to (111.3, 77.0)
- moved D5 2.32 mm to (191.4, 77.4)
- moved C7 1.57 mm to (178.6, 80.4)
- moved R1 1.20 mm to (117.2, 72.7)
- moved D6 0.85 mm to (135.2, 100.0)
- moved R6 0.85 mm to (129.8, 100.0)
- moved DRV1 0.76 mm to (185.8, 104.1)
- moved D3 0.65 mm to (152.2, 66.8)
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Connections:
- TB1 pad 13: S5 -> ST
- TB1 pad 15: ST -> S5
- TB1 pad 29: unconnected-(TB1-COM/GND-Pad29)_1 -> GND
- TB1 pad 4: unconnected-(TB1-COM/GND-Pad29) -> GND
Routing:
- net +5V: track 217.9 -> 240.2 mm
- net ST: track 25.9 -> 36.6 mm
- net Net-(J12-Pin_2): track 24.3 -> 31.3 mm
- net S5: track 27.1 -> 20.9 mm
- net S3: track 18.3 -> 24.5 mm
- net S1: track 19.7 -> 25.4 mm
- net +12V: track 148.6 -> 145.3 mm
- net Net-(SW2A-A): track 10.8 -> 13.8 mm
- net Net-(D4-A): track 6.63 -> 3.80 mm
- net Net-(D2-A): track 4.27 -> 3.17 mm
- net 5v: track 66.5 -> 65.5 mm
- net Net-(D1-A): track 8.04 -> 7.24 mm
- net Net-(D5-A): track 7.74 -> 7.04 mm
- net Net-(D3-A): track 2.47 -> 3.10 mm
- net Net-(DRV3-Out2): track 16.7 -> 17.3 mm
Other:
- board text added: "+"
- board text added: "+5V"
- board text added: "-"
- board text added: "-Pooki"
- board text added: "A0"
- board text added: "A1"
- board text added: "D12"
- board text added: "D2"
- board text added: "D4"
- board text added: "D7"
- board text added: "D8"
- board text added: "Gnd"
- board text added: "IMU"
- board text added: "LED"
- board text added: "R4"
- board text added: "Sig"

Commit message: nond
Parts:
- removed R7, R8: 1k, Resistor_SMD:R_0805_2012Metric
- removed S1: DIP, ZSKIBIDI:DIp
- added R10: 1k, Resistor_SMD:R_0805_2012Metric, F.Cu at (172.8, 97.9)
- added R9: 1k, Resistor_SMD:R_0805_2012Metric, F.Cu at (161.6, 105.9)
- added SW1: SW_DIP_x04, ZSKIBIDI:DIP8_210-4_CTS[1], F.Cu at (166.5, 109.3)
- moved C8 36.5 mm to (191.5, 70.3)
- moved J8 25.2 mm to (190.3, 91.7)
- moved C9 17.0 mm to (176.1, 82.7), turned to 180 degrees
- moved C10 6.48 mm to (191.5, 81.8), turned to 90 degrees
- moved J14 2.50 mm to (136.1, 114.7)
- moved C7 1.46 mm to (178.4, 79.0)
- moved J7 0.75 mm to (160.8, 98.8)
- moved D5 0.70 mm to (191.5, 76.7)
- moved J13 0.18 mm to (169.1, 114.6)
Connections:
- DRV1 pad 7: unconnected-(DRV1-VM-Pad7) -> +5V
- DRV3 pad 7: unconnected-(DRV3-VM-Pad7) -> +5V
- J8 pad 2: GND -> 5v
- J8 pad 3: 5v -> GND
Routing:
- net +5V: track 240.2 -> 281.4 mm, vias 1 -> 0
- net Servo: track 64.7 -> 92.0 mm
- net 5v: track 65.5 -> 40.6 mm
- net Net-(DRV3-Out2): track 17.3 -> 20.3 mm
- net Net-(DRV3-Out1): track 10.2 -> 13.2 mm
- net DIP2: track 20.8 -> 18.2 mm
- net +12V: track 145.3 -> 146.6 mm, vias 0 -> 1
- net DIP1: track 20.6 -> 21.7 mm
- net SDA: track 5.71 -> 4.96 mm
- net SCL: track 5.71 -> 4.96 mm
- net GND: track 0.74 -> 0.00 mm
- net Net-(D5-A): track 7.04 -> 6.36 mm
Other:
- board text added: "B"
- board text added: "O"
- board text added: "R"

Commit message: grhrsggfsfsgn
Parts:
- added H1: MountingHole, MountingHole:MountingHole_2.1mm, F.Cu at (127.8, 113.1)
- added H2: MountingHole, MountingHole:MountingHole_2.1mm, F.Cu at (109.9, 74.4)
- added H3: MountingHole, MountingHole:MountingHole_2.1mm, F.Cu at (192.1, 65.6)
- added H4: MountingHole, MountingHole:MountingHole_2.1mm, F.Cu at (174.5, 113.3)
- moved D1 2.39 mm to (112.5, 79.1)
- moved D2 1.40 mm to (179.4, 66.6)
- moved R2 0.95 mm to (174.4, 66.7)
- moved C8 0.73 mm to (191.7, 71.0)
Connections:
- DRV1 pad 7: +5V -> unconnected-(DRV1-VM-Pad7)
- DRV3 pad 7: +5V -> unconnected-(DRV3-VM-Pad7)
Routing:
- net +5V: track 281.4 -> 232.1 mm
- net S1: track 25.4 -> 24.4 mm
- net 5v: track 40.6 -> 39.8 mm
- net Net-(D1-A): track 7.24 -> 6.56 mm
Other:
- board text added: "Alex Peng is Cool"
