File: Jongmyeong-I/Jongmyeong-i/Jongmyeong-i.kicad_sch (KiCad schematic)
At the start: 20 parts, among them J1 Screw3, J2 Screw3, J3 Screw3, J4 Screw3, J5 Screw3, J6 Conn_01x03_Pin, J7 Conn_01x08_Pin, J8 Conn_01x03_Pin

Commit message: almostdone
Parts:
- added C11, C12, C13: 0.1uF, Capacitor_SMD:C_0805_2012Metric, symbol Device:C
- added D1, D2, D3, D4, D5, D6: LED, LED_SMD:LED_1206_3216Metric, symbol Device:LED
- added F1: Fuse, Fuse:Fuse_1206_3216Metric, symbol Device:Fuse
- added J10, J11, J9: Screw3, Connector_JST:JST_EH_B3B-EH-A_1x03_P2.50mm_Vertical, symbol Connector:Screw_Terminal_01x03
- added J12: xt30, Connector_AMASS:AMASS_XT30U-F_1x02_P5.0mm_Vertical, symbol Connector:Conn_01x02_Pin
- added R1, R2, R3, R4, R5, R6: 180, Resistor_SMD:R_0805_2012Metric, symbol Device:R_US
- added R7, R8: 1k, Resistor_SMD:R_0805_2012Metric, symbol Device:R_US
- added S1: DIP, ZSKIBIDI:DIp, symbol Dip:219-2MSTR
- added SW2: SW_DPDT_x2, ZSKIBIDI:switch, symbol Switch:SW_DPDT_x2
- C1, C10, C2, C3, C4, C5, C6, C7, C8, C9: footprint (none) -> Capacitor_SMD:C_0805_2012Metric
- J1, J2, J3, J4, J5: footprint (none) -> Connector_JST:JST_EH_B3B-EH-A_1x03_P2.50mm_Vertical
- J6, J8: footprint (none) -> Connector_PinHeader_2.54mm:PinHeader_1x03_P2.54mm_Vertical
- J7: footprint (none) -> Connector_PinHeader_2.54mm:PinHeader_1x08_P2.54mm_Vertical
- PS1: footprint P78E05-1000:CONV_P78E05-1000 -> ZSKIBIDI:5vCOnv
- TB1: footprint ARDUINO_NANO:SHIELD_ARDUINO_NANO -> ZSKIBIDI:SHIELD_ARDUINO_NANO[1]
Connections:
- net +12V: now also F1.2
- net +3.3V: now also C11.1, C12.1, C13.1, J10.2 (Pin_2), J11.2 (Pin_2), J9.2 (Pin_2), S1.1A, S1.2A
- net +5V: now also R6.1
- net 5v: now also C10.1
- net GND: now also C11.2, C12.2, C13.2, D1.1 (K), D2.1 (K), D3.1 (K), D4.1 (K), D5.1 (K), D6.1 (K), J10.3 (Pin_3), J11.3 (Pin_3), J12.2 (Pin_2), J9.3 (Pin_3), R7.1, R8.2
- net MOTOR2B: now also TB1.14 (D11/MOSI); no longer TB1.12 (D9)
- net S1: now also TB1.5 (D2), J10.1 (Pin_1), J11.1 (Pin_1), J9.1 (Pin_1), R2.1; no longer TB1.2 (D0/RX)
- net S2: now also TB1.7 (D4), R3.1; no longer TB1.5 (D2)
- net S3: now also TB1.10 (D7), R4.1; no longer TB1.7 (D4)
- net S4: now also TB1.11 (D8), R5.1; no longer TB1.10 (D7)
- net S5: now also TB1.13 (D10), R1.1; no longer TB1.11 (D8)
- net Servo: now also TB1.12 (D9); no longer TB1.13 (D10)
- net DIP1: now reaches TB1.25 (A6)
- net DIP1: now also R7.2, S1.1B
- net DIP2: now reaches TB1.26 (A7)
- net DIP2: now also R8.1, S1.2B
- new net: D6.2 (A), R6.2
- new net: D2.2 (A), R2.2
- new net: D3.2 (A), R3.2
- new net: D4.2 (A), R4.2
- new net: F1.1, SW2.1 (A)
- new net: D1.2 (A), R1.2
- new net: D5.2 (A), R5.2
- new net: J12.1 (Pin_1), SW2.2 (B)
- no-connect marks 11 -> 14
Other:
- note added: "Dipswitch"
- note added: "LEDs"
- note added: "Line Sensors"
- note added: "Power"
- note removed: "5V Convertor"
- moved on the sheet: C10, C8, C9, J8, PS1

Commit message: joe
Parts:
- added DRV1, DRV3: ~, symbol Custom:drvmotor
- added J13, J14: Screw_Terminal_01x02, symbol Connector:Screw_Terminal_01x02
Connections:
- net +12V: now also DRV1.5 (Pow), DRV3.5 (Pow)
- net GND: now also DRV1.6 (GND), DRV1.8 (GND), DRV3.6 (GND), DRV3.8 (GND)
- net MOTOR1A: now also DRV1.3 (PWM1)
- net MOTOR1B: now also DRV1.4 (PWM2)
- net MOTOR2A: now also DRV3.3 (PWM1)
- net MOTOR2B: now also DRV3.4 (PWM2)
- new net: DRV3.1 (Out1), J14.2 (Pin_2)
- new net: DRV3.2 (Out2), J14.1 (Pin_1)
- new net: DRV1.2 (Out2), J13.1 (Pin_1)
- new net: DRV1.1 (Out1), J13.2 (Pin_2)

Commit message: finished layout
Parts:
- removed C12: 0.1uF, Capacitor_SMD:C_0805_2012Metric, symbol Device:C
- removed J10: Screw3, Connector_JST:JST_EH_B3B-EH-A_1x03_P2.50mm_Vertical, symbol Connector:Screw_Terminal_01x03
- DRV1, DRV3: footprint (none) -> ZSKIBIDI:drvmotordriver
- J13, J14: footprint (none) -> Connector_PinHeader_2.54mm:PinHeader_1x02_P2.54mm_Vertical
Connections:
- net LN1: now also J9.1 (Pin_1)
- net LN2: now also J11.1 (Pin_1)
- net S1: no longer J11.1 (Pin_1), J9.1 (Pin_1)
- net SCL: now also J7.3 (Pin_3)
- net SDA: no longer J7.3 (Pin_3)
- net ST: now also TB1.15 (D12/MISO)
- no-connect marks 14 -> 13

Commit message: mom
Parts:
- removed C11, C13, C6: 0.1uF, Capacitor_SMD:C_0805_2012Metric, symbol Device:C
- J12: footprint Connector_AMASS:AMASS_XT30U-F_1x02_P5.0mm_Vertical -> Connector_AMASS:AMASS_XT30PW-F_1x02_P2.50mm_Horizontal
Connections:
- net +5V: now also J6.2 (Pin_2); no longer J6.3 (Pin_3)
- net GND: now also J6.3 (Pin_3); no longer J6.2 (Pin_2)

Commit message: pooki done
Parts:
- removed C7: 0.1uF, Capacitor_SMD:C_0805_2012Metric, symbol Device:C
- J12: footprint Connector_AMASS:AMASS_XT30PW-F_1x02_P2.50mm_Horizontal -> Connector_AMASS:AMASS_XT30U-F_1x02_P5.0mm_Vertical
Connections:
- net +12V: no longer DRV3.5 (Pow)
- net +3.3V: no longer J11.2 (Pin_2), J9.2 (Pin_2), S1.1A, S1.2A
- net +5V: now also J11.2 (Pin_2), J9.2 (Pin_2), S1.1A
- net GND: now also J12.1 (Pin_1); no longer DRV3.6 (GND), DRV3.8 (GND), J12.2 (Pin_2)
- net MOTOR2A: no longer DRV3.3 (PWM1)
- net MOTOR2B: no longer DRV3.4 (PWM2)
- net at DRV3.1 (Out1): no longer J14.2 (Pin_2)
- net at DRV3.2 (Out2): no longer J14.1 (Pin_1)
- net at SW2.2 (B): now also J12.2 (Pin_2); no longer J12.1 (Pin_1)
Other:
- moved on the sheet: DRV3, J12

Commit message: done with pooki
Parts:
- added C6: 0.1uF, Capacitor_SMD:C_0805_2012Metric, symbol Device:C
- added J10: Conn_01x03_Pin, Connector_PinHeader_2.54mm:PinHeader_1x03_P2.54mm_Vertical, symbol Connector:Conn_01x03_Pin
Connections:
- net +12V: now also DRV3.5 (Pow), C6.1
- net +5V: now also S1.2A, J10.3 (Pin_3)
- net GND: now also DRV3.6 (GND), DRV3.8 (GND), TB1.29 (COM/GND), TB1.4 (COM/GND), C6.2, J10.2 (Pin_2)
- net MOTOR2A: now also DRV3.3 (PWM1)
- net MOTOR2B: now also DRV3.4 (PWM2)
- net S5: now also TB1.15 (D12/MISO); no longer TB1.13 (D10)
- net ST: now also TB1.13 (D10), J10.1 (Pin_1); no longer TB1.15 (D12/MISO)
- net at DRV3.1 (Out1): now also J14.2 (Pin_2)
- net at DRV3.2 (Out2): now also J14.1 (Pin_1)
- no-connect marks 13 -> 14
Other:
- moved on the sheet: DRV3

Commit message: nond
Parts:
- removed C8: 0.1uF, Capacitor_SMD:C_0805_2012Metric, symbol Device:C
- removed R7, R8: 1k, Resistor_SMD:R_0805_2012Metric, symbol Device:R_US
- removed S1: DIP, ZSKIBIDI:DIp, symbol Dip:219-2MSTR
- added C7: 0.1uF, Capacitor_SMD:C_0805_2012Metric, symbol Device:C
- added R10, R9: 1k, Resistor_SMD:R_0805_2012Metric, symbol Device:R_US
- added SW1: SW_DIP_x04, ZSKIBIDI:DIP8_210-4_CTS[1], symbol Switch:SW_DIP_x04
Connections:
- net +5V: now also DRV1.7 (VM), DRV3.7 (VM), SW1.1, SW1.2
- net 5v: now also J8.2 (Pin_2), C7.1; no longer J8.3 (Pin_3)
- net DIP1: now also R9.2, SW1.8
- net DIP2: now also R10.2, SW1.7
- net GND: now also J8.3 (Pin_3), C7.2, R10.1, R9.1; no longer J8.2 (Pin_2)
- no-connect marks 14 -> 16

Commit message: grhrsggfsfsgn
Parts:
- added H1, H2, H3, H4: MountingHole, MountingHole:MountingHole_2.1mm, symbol Mechanical:MountingHole
Connections:
- net +5V: no longer DRV1.7 (VM), DRV3.7 (VM)
- no-connect marks 16 -> 18
