File: 3kg/Monki/Team2(EvenNewer9_19) copy/_autosave-Team2(EvenNewer9_19).kicad_pcb (KiCad board)
At the start: 2 copper layers, 109 parts, among them J1 Conn_01x03_MountingPin, J10 Conn_01x03_MountingPin, J11 Conn_01x03_MountingPin, J12 Conn_01x03_MountingPin, J13 Conn_01x03_MountingPin, J14 XT60-M, J15 Conn_01x03_Pin, J16 Conn_01x08_Pin, J17 XT60-M, J18 XT60-M, J19 Conn_01x03_MountingPin, J2 Conn_01x03_MountingPin, J22 Conn_01x03_MountingPin, J3 Conn_01x03_MountingPin, J4 Conn_01x03_MountingPin, J5 Conn_01x03_MountingPin, J6 Conn_01x03_MountingPin, J7 Conn_01x03_MountingPin, J8 Conn_01x03_MountingPin, J9 Conn_01x03_MountingPin, Q1 SQM40P10-40L_GE3, Q2 SQ2318AES-T1_BE3, SW1 SW_SPST, U1 S-1142DA0I-E6T1U, U2 Teensy4.1, U3 TQL850CSV50_RLG

Commit message: 10/13_Isabelli
Parts:
- moved J14 122.9 mm to (147.0, 113.5), turned to 180 degrees
- moved J19 112.1 mm to (127.0, 134.0), turned to -90 degrees
- moved C3 111.1 mm to (142.5, 75.0)
- moved C1 111.1 mm to (142.5, 69.9)
- moved C10 111.1 mm to (142.5, 92.5)
- moved C11 111.1 mm to (146.9, 69.9)
- moved C12 111.1 mm to (146.9, 72.4)
- moved C13 111.1 mm to (146.9, 74.9)
- moved C14 111.1 mm to (146.9, 77.5)
- moved C18 111.1 mm to (146.9, 80.0)
- moved C19 111.1 mm to (146.9, 82.5)
- moved C2 111.1 mm to (142.5, 72.4)
- moved C20 111.1 mm to (146.9, 85.0)
- moved C21 111.1 mm to (146.9, 87.5)
- moved C22 111.1 mm to (146.9, 90.0)
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