File: 3kg/Monki/Team2(10-27)/Team2(10-27)/Team2(10-27).kicad_pcb (KiCad board)
At the start: 2 copper layers, 110.9 x 54.1 mm, 112 parts, among them J1 Conn_01x03_MountingPin, J10 Conn_01x03_MountingPin, J11 Conn_01x03_MountingPin, J12 Conn_01x03_MountingPin, J13 Conn_01x03_MountingPin, J14 XT60-M, J15 Conn_01x03_Pin, J16 Conn_01x08_Pin, J17 XT60-M, J18 XT60-M, J19 Conn_01x03_MountingPin, J2 Conn_01x03_MountingPin, J22 Conn_01x03_MountingPin, J3 Conn_01x03_MountingPin, J4 Conn_01x03_MountingPin, J5 Conn_01x03_MountingPin, J6 Conn_01x03_MountingPin, J7 Conn_01x03_MountingPin, J8 Conn_01x03_MountingPin, J9 Conn_01x03_MountingPin, Q1 SQM40P10-40L_GE3, Q2 SQ2318AES-T1_BE3, SW1 SW_SPST, U1 S-1142DA0I-E6T1U, U2 Teensy4.1, U3 TQL850CSV50_RLG, U4 TMCS1126A1AQDVGRQ1

Commit message: Isabelli_10-29
Parts:
- moved C20 3.76 mm to (45.5, 36.5), turned to 180 degrees
- moved C15 3.32 mm to (68.0, 59.5), turned to 0 degrees
- moved R28 3.26 mm to (68.0, 66.0), turned to 0 degrees
- moved C17 1.65 mm to (68.0, 63.5), turned to 0 degrees
- moved C16 1.11 mm to (68.0, 61.5), turned to 0 degrees
- moved R29 0.88 mm to (55.5, 65.0)
- moved Q2 0.83 mm to (61.4, 64.0), turned to -90 degrees
- moved C13 0.41 mm to (145.0, 67.1)
- moved F3 0.27 mm to (45.5, 35.0)
- turned Q1 to 0 degrees
Connections:
- C1 pad 1: +5V -> 5v
- C10 pad 1: +12V -> 12v
- C11 pad 1: +12V -> 12v
- C12 pad 1: +12V -> 12v
- C13 pad 1: +5V -> 5v
- C18 pad 1: 44.4v -> 44.4V
- C2 pad 1: +5V -> 5v
- C20 pad 1: 44.4v -> 44.4V
- C22 pad 1: +5V -> 5v
- C24 pad 1: +5V -> 5v
- C3 pad 1: +5V -> 5v
- C4 pad 1: +12V -> 12v
- C5 pad 1: +12V -> 12v
- C6 pad 1: +12V -> 12v
- C7 pad 1: +12V -> 12v
- C8 pad 1: +12V -> 12v
- C9 pad 1: +12V -> 12v
- F2 pad 1: 44.4v -> 44.4V
- F3 pad 1: 44.4v -> 44.4V
- J10 pad 2: +12V -> 12v
- J11 pad 2: +12V -> 12v
- J12 pad 2: +12V -> 12v
- J13 pad 2: +12V -> 12v
- J16 pad 1: +5V -> 5v
- J19 pad 2: +5V -> 5v
- J2 pad 2: +5V -> 5v
- J3 pad 2: +5V -> 5v
- J4 pad 2: +5V -> 5v
- J5 pad 2: +12V -> 12v
- J6 pad 2: +12V -> 12v
- J7 pad 2: +12V -> 12v
- J8 pad 2: +12V -> 12v
- J9 pad 2: +12V -> 12v
- U2 pad 48: +5V -> 5v
Routing:
- net GND1: track 0.32 -> 384.2 mm, vias 0 -> 14
- net 12v: track 4.26 -> 114.0 mm
- net 5v: track 0.00 -> 90.0 mm
- net +3.3V: track 4.01 -> 93.5 mm, vias 0 -> 1
- net 44.4V: track 13.0 -> 61.4 mm
- net +12V: track 42.8 -> 0.00 mm
- net Net-(J17-POS): track 3.03 -> 36.9 mm, vias 0 -> 2
- net +5V: track 26.6 -> 0.00 mm
- net Signal Start Module: track 0.00 -> 22.0 mm, vias 0 -> 2
- net Net-(Q1-G): track 1.38 -> 16.2 mm
- net Vout Current Sensor: track 0.00 -> 12.7 mm
- net Vref Current Sensor: track 0.00 -> 10.4 mm
- net Interupt: track 0.00 -> 8.10 mm
- net Distance Sensor 1 3.3V: track 23.9 -> 31.4 mm
- net Line Sensor 4 5v: track 0.12 -> 6.98 mm
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