File: 3kg/Monki/Team2(10-27)/Team2(10-27)/Team2(10-27).kicad_sch (KiCad schematic)
At the start: 112 parts, among them J1 Conn_01x03_MountingPin, J10 Conn_01x03_MountingPin, J11 Conn_01x03_MountingPin, J12 Conn_01x03_MountingPin, J13 Conn_01x03_MountingPin, J14 XT60-M, J15 Conn_01x03_Pin, J16 Conn_01x08_Pin, J17 XT60-M, J18 XT60-M, J19 Conn_01x03_MountingPin, J2 Conn_01x03_MountingPin, J22 Conn_01x03_MountingPin, J3 Conn_01x03_MountingPin, J4 Conn_01x03_MountingPin, J5 Conn_01x03_MountingPin, J6 Conn_01x03_MountingPin, J7 Conn_01x03_MountingPin, J8 Conn_01x03_MountingPin, J9 Conn_01x03_MountingPin, Q1 SQM40P10-40L_GE3, Q2 SQ2318AES-T1_BE3, SW1 SW_SPST, U1 S-1142DA0I-E6T1U, U2 Teensy4.1, U3 TQL850CSV50_RLG, U4 TMCS1126A1AQDVGRQ1

Commit message: Isabelli_10-29
Connections:
- net +12V is gone; now on net 12v: C10.1, C11.1, C12.1, C4.1, C5.1, C6.1, C7.1, C8.1, C9.1, J10.2 (Pin_2), J11.2 (Pin_2), J12.2 (Pin_2), J13.2 (Pin_2), J5.2 (Pin_2), J6.2 (Pin_2), J7.2 (Pin_2), J8.2 (Pin_2), J9.2 (Pin_2)
- net +5V is gone; now on net 5v: C1.1, C13.1, C2.1, C22.1, C24.1, C3.1, J16.1 (Pin_1), J19.2 (Pin_2), J2.2 (Pin_2), J3.2 (Pin_2), J4.2 (Pin_2), U2.48 (VIN)
- net 44.4v is gone; now on net 44.4V: C18.1, C20.1, F2.1, F3.1
