File: 500g/Rata2i/Schematic/Schematic.kicad_pcb (KiCad board)
At the start: 2 copper layers, 90 x 59.5 mm, 42 parts, among them J1 Screw_Terminal_01x03, J10 Conn_01x03_Pin, J2 Screw_Terminal_01x03, J3 Screw_Terminal_01x03, J4 Screw_Terminal_01x03, J5 Screw_Terminal_01x03, J6 Screw_Terminal_01x03, J7 Battery, J8 Screw_Terminal_01x02, J9 Screw_Terminal_01x02, SW1 SW_SPDT, U1 DEV-16771, U2 TB6612FNG, U3 R-78K5.0-0.5, U4 R-78K5.0-0.5

Commit message: PCB extravaganza
pcb update
Parts:
- removed U2: TB6612FNG, Package_SO:SSOP-24_5.3x8.2mm_P0.65mm
- added J11: Screw_Terminal_01x02, TerminalBlock:TerminalBlock_Xinya_XY308-2.54-2P_1x02_P2.54mm_Horizontal, F.Cu at (2.04, 3.62)
- added J12: Screw_Terminal_01x02, TerminalBlock:TerminalBlock_Xinya_XY308-2.54-2P_1x02_P2.54mm_Horizontal, F.Cu at (9.69, 3.62)
- added U5: ROB-14450, robowrestling:MOTOR_DRIVER, F.Cu at (82.1, 33.4)
- J1, J2, J3, J4, J5, J6: footprint Connector_PinHeader_2.54mm:PinHeader_1x03_P2.54mm_Vertical -> TerminalBlock:TerminalBlock_Xinya_XY308-2.54-3P_1x03_P2.54mm_Horizontal
- J8, J9: footprint robowrestling:Screw Terminal -> TerminalBlock:TerminalBlock_Xinya_XY308-2.54-2P_1x02_P2.54mm_Horizontal
- moved D3 39.0 mm to (127.5, 37.5)
- moved R3 39.0 mm to (120.5, 37.5)
- moved J3 38.0 mm to (121.1, 43.7), turned to 0 degrees
- moved J2 29.7 mm to (114.8, 72.2), turned to 180 degrees
- moved J5 28.1 mm to (131.6, 43.7), turned to 0 degrees
- moved D2 27.4 mm to (117.0, 77.5), turned to 180 degrees
- moved R2 23.4 mm to (109.6, 77.7)
- moved J6 21.9 mm to (126.7, 72.2), turned to 180 degrees
- moved J4 21.0 mm to (142.1, 43.7), turned to 0 degrees
- moved R4 20.2 mm to (146.6, 37.0)
- moved D4 19.5 mm to (140.9, 37.0)
- moved U1 17.1 mm to (119.0, 57.5)
- moved J1 12.5 mm to (138.2, 72.2), turned to 180 degrees
- moved R5 10.6 mm to (130.5, 78.5), turned to 0 degrees
- moved D6 9.86 mm to (138.2, 78.5)
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Routing:
- net +5V: track 104.5 -> 0.00 mm
- net s3: track 32.2 -> 49.7 mm
- net L1: track 11.7 -> 19.0 mm
- net s4: track 55.4 -> 61.4 mm
- net s2: track 17.0 -> 21.1 mm
- net Net-(D6-A): track 7.81 -> 5.25 mm
- net +12V: track 23.1 -> 20.6 mm
- net GND: track 1.15 -> 0.00 mm
- net unconnected-(U1-RX1-Pad0): track 0.00 -> 0.79 mm
