File: 500g/Rata2i/Schematic/Schematic.kicad_sch (KiCad schematic)
At the start: 7 parts, among them J1 Screw_Terminal_01x03, J2 Screw_Terminal_01x03, J3 Screw_Terminal_01x03, J4 Screw_Terminal_01x03, J5 Screw_Terminal_01x03, J7 Screw_Terminal_01x03, U1 DEV-16771

Commit message: Updated Rata2i schematic
Now with more stuff! And 1 (one) LED
Parts:
- added C1: C_Small, symbol Device:C_Small
- added C2, C3: C, symbol Device:C
- added D1: LED, symbol Device:LED
- added F1: Fuse, symbol Device:Fuse
- added H1, H2: MountingHole, symbol Mechanical:MountingHole
- added J10: Conn_01x03_Pin, symbol Connector:Conn_01x03_Pin
- added J7: Battery, symbol Connector_Generic:Conn_01x02
- added J8, J9: Screw_Terminal_01x02, symbol Connector:Screw_Terminal_01x02
- added R1: R_US, symbol Device:R_US
- added SW2: SW_SPST, symbol Switch:SW_SPST
- added U2: TB6612FNG, Package_SO:SSOP-24_5.3x8.2mm_P0.65mm, symbol Driver_Motor:TB6612FNG
- added U3: R-78K5.0-0.5, SIP3_R-78K-0.5_RCP, symbol 2024-11-08_01-03-56:R-78K5.0-0.5
- renumbered J7 to J6
Connections:
- net +3.3V: now also J6.2 (Pin_2), U1.3.3V_1 (3.3V), U1.3.3V_2 (3.3V), U1.3.3V_3 (3.3V), J10.3 (Pin_3), U2.19 (STBY), U2.20 (VCC)
- net GND: now also J6.1 (Pin_1), U1.GND1 (GND), U1.GND2 (GND), U1.GND3 (GND), U1.GND4 (GND), U1.GND5 (GND), U1.USB_GND1 (USB_GND), U1.USB_GND2 (USB_GND), C1.2, C2.2, C3.1, D1.1 (K), J10.2 (Pin_2), J7.2 (Pin_2), U2.10 (PGND2), U2.18 (GND), U2.3 (PGND1), U2.4 (PGND1), U2.9 (PGND2), U3.2 (GND)
- net s1: now also U1.5 (IN2)
- net s2: now also U1.2 (OUT2)
- net s3: now also U1.3 (LRCLK2)
- net s4: now also U1.4 (BCLK2)
- net L2: now reaches J6.3 (Pin_3)
- net L2: now also U1.15 (A1)
- net L1: now reaches U1.14 (A0)
- net L1: now also J5.3 (Pin_3)
- net start: now reaches U1.17 (A3)
- net start: now also J10.1 (Pin_1)
- net md1: now reaches U1.19 (A5)
- net md2: now reaches U1.20 (A6)
- net md3: now reaches U1.21 (A7)
- net md4: now reaches U1.22 (A8)
- net md8: now reaches U1.23 (A9)
- net md7: now reaches U1.24 (A10)
- net md6: now reaches U1.25 (A11)
- net md5: now reaches U1.26 (A12)
- net motorapwm: now reaches U1.6 (OUT1D)
- net motorapwm: now also U2.23 (PWMA)
- net motorbpwm: now reaches U1.9 (OUT1C)
- net motorbpwm: now also U2.15 (PWMB)
- net +5V: now reaches U1.VIN
- net +5V: now also C2.1, C3.2, U3.3 (+VOUT)
- new net: D1.2 (A), R1.2
- new net: J9.1 (Pin_1), U2.11 (BO1), U2.12 (BO1)
- new net: J9.2 (Pin_2), U2.7 (BO2), U2.8 (BO2)
- new net: J8.1 (Pin_1), U2.1 (AO1), U2.2 (AO1)
- new net: J8.2 (Pin_2), U2.5 (AO2), U2.6 (AO2)
- new net: J7.1 (Pin_1), SW2.1 (A)
- new net +12V: C1.1, F1.1, R1.1, SW2.2 (B), U2.13 (VM2), U2.14 (VM3), U2.24 (VM1), U3.1 (+VIN)
- new net mdr1: U2.21 (AIN1)
- new net mdr2: U2.22 (AIN2)
- new net mdr3: U2.17 (BIN1)
- new net mdr4: U2.16 (BIN2)
- no-connect marks 2 -> 35
Other:
- note added: "7 leds total: 1 for each distance sensor, 1 for on/off,1 for each motor"
- note added: "leds"
- note added: "motor driver"
- note added: "power and decoupling"
- note added: "voltage regulator"
- moved on the sheet: J1, J2, J3, J4, J6, U1

Commit message: Updated Rata2i (thrilling sequel)
Parts:
- added D2, D3, D4, D5, D6, D7, D8: LED, symbol Device:LED
Connections:
- net GND: now also D2.1 (K), D3.1 (K), D4.1 (K), D5.1 (K), D6.1 (K), D7.1 (K), D8.1 (K)
- net L1: now also D6.2 (A)
- net L2: now also D7.2 (A)
- net s1: now also D2.2 (A)
- net s2: now also D3.2 (A)
- net s3: now also D4.2 (A)
- net s4: now also D5.2 (A)
- net start: now also D8.2 (A)
Other:
- note added: "led (just 1 lmao)"
- note removed: "leds"
- moved on the sheet: C1, C2, D1, F1, H1, H2, J1, J10, J2, J3, J4, J5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

Commit message: Cool Schematic, Some Footprints
thanks kyle and joe
Parts:
- removed D6, D7, D8: LED, symbol Device:LED
- removed SW2: SW_SPST, symbol Switch:SW_SPST
- added C1: 10uF, Capacitor_SMD:C_0805_2012Metric, symbol Device:C_Small
- added C5: 10uF, Capacitor_SMD:C_0805_2012Metric, symbol Device:C
- added R2, R3, R4, R5: R_US, Resistor_SMD:R_0805_2012Metric, symbol Device:R_US
- added SW1: SW_SPDT, symbol Switch:SW_SPDT
- added U4: R-78K5.0-0.5, footprints:SIP3_R-78K-0.5_RCP, symbol 2024-11-08_01-03-56:R-78K5.0-0.5
- C2: value C -> 10 uF; footprint (none) -> Capacitor_SMD:C_0805_2012Metric
- C3: value C -> 0.1uF; footprint (none) -> Capacitor_SMD:C_0805_2012Metric
- C4: renamed from C1; value C_Small -> 10uF; footprint (none) -> Capacitor_SMD:C_0805_2012Metric
- D1, D2, D3, D4, D5: footprint (none) -> Capacitor_SMD:C_1206_3216Metric
- R1: footprint (none) -> Resistor_SMD:R_0805_2012Metric
- U3: footprint SIP3_R-78K-0.5_RCP -> footprints:SIP3_R-78K-0.5_RCP
Connections:
- net +12V: now also C1.1, SW1.1 (A), U4.1 (+VIN); no longer R1.1
- net +3.3V: now also C5.1, U4.3 (+VOUT); no longer J6.2 (Pin_2)
- net +5V: now also R1.1
- net GND: now also D2.2 (A), J6.2 (Pin_2), C1.2, C5.2, R2.2, U4.2 (GND)
- net s1: now also R2.1; no longer D2.2 (A)
- net s2: now also R3.1; no longer J2.3 (Pin_3)
- net s3: now also R4.1; no longer J3.3 (Pin_3)
- net s4: now also R5.1; no longer J4.3 (Pin_3)
- net at J7.1 (Pin_1): now also SW1.2 (B)
- net md5: no longer names the net of U1.26 (A12)
- net md6: no longer names the net of U1.25 (A11)
- net md7: no longer names the net of U1.24 (A10)
- net md8: no longer names the net of U1.23 (A9)
- new net: J3.3 (Pin_3), R4.2
- new net: J4.3 (Pin_3), R5.2
- new net: J2.3 (Pin_3), R3.2
- no-connect marks 35 -> 40
Other:
- moved on the sheet: C2, C4, D2, J8, U3

Commit message: rata2i
complete schematic yippee!! pcb not so complete
Parts:
- removed D5: LED, Capacitor_SMD:C_1206_3216Metric, symbol Device:LED
- added D6: LED, LED_SMD:LED_1206_3216Metric_ReverseMount_Hole1.8x2.4mm, symbol Device:LED
- D1, D2, D3, D4: footprint Capacitor_SMD:C_1206_3216Metric -> LED_SMD:LED_1206_3216Metric_ReverseMount_Hole1.8x2.4mm
- F1: footprint (none) -> Fuse:Fuse_1206_3216Metric
- H1, H2: footprint (none) -> MountingHole:MountingHole_2.5mm
- J1, J10, J2, J3, J4, J5, J6: footprint (none) -> Connector_PinHeader_2.54mm:PinHeader_1x03_P2.54mm_Vertical
- J7: footprint (none) -> Connector_AMASS:AMASS_XT30U-F_1x02_P5.0mm_Vertical
- J8, J9: footprint (none) -> robowrestling:Screw Terminal
- SW1: footprint (none) -> robowrestling:Switch
Connections:
- net GND: now also J7.1 (Pin_1), D6.1 (K); no longer D2.2 (A), J7.2 (Pin_2), R2.2
- net s1: now also R5.1; no longer R2.1
- net s2: now also J2.3 (Pin_3), R2.1; no longer D3.2 (A), R3.1
- net s3: now also J3.3 (Pin_3), R3.1; no longer D4.2 (A), R4.1
- net s4: now also J4.3 (Pin_3), R4.1; no longer R5.1
- net at R4.2: now also D4.2 (A); no longer J3.3 (Pin_3)
- net at R5.2: now also D6.2 (A); no longer J4.3 (Pin_3)
- net at R3.2: now also D3.2 (A); no longer J2.3 (Pin_3)
- net at SW1.2 (B): now also J7.2 (Pin_2); no longer J7.1 (Pin_1)
- new net: D2.2 (A), R2.2
Other:
- note removed: "7 leds total: 1 for each distance sensor, 1 for on/off,1 for each motor"

Commit message: PCB extravaganza
pcb update
Parts:
- removed J8, J9: Screw_Terminal_01x02, robowrestling:Screw Terminal, symbol Connector:Screw_Terminal_01x02
- removed U2: TB6612FNG, Package_SO:SSOP-24_5.3x8.2mm_P0.65mm, symbol Driver_Motor:TB6612FNG
- added J11, J12: Screw_Terminal_01x02, TerminalBlock:TerminalBlock_Xinya_XY308-2.54-2P_1x02_P2.54mm_Horizontal, symbol Connector:Screw_Terminal_01x02
- added U5: ROB-14450, robowrestling:MOTOR_DRIVER, symbol motor driver:ROB-14450
- J1, J2, J3, J4, J5, J6: footprint Connector_PinHeader_2.54mm:PinHeader_1x03_P2.54mm_Vertical -> TerminalBlock:TerminalBlock_Xinya_XY308-2.54-3P_1x03_P2.54mm_Horizontal
Connections:
- net +12V: now also U5.1 (VM)
- net +3.3V: now also U5.2 (VCC)
- net +5V: now also U5.13 (STBY)
- net GND: now also U5.3 (GND), U5.8 (GND), U5.9 (GND)
- net mdr1: now also U5.14 (AI1)
- net mdr2: now also U5.15 (AI2)
- net mdr3: now also U5.12 (BI1)
- net mdr4: now also U5.11 (BI2)
- net motorapwm: now also U5.16 (PWMA)
- net motorbpwm: now also U5.10 (PWMB)
- new net: J11.1 (Pin_1), U5.4 (A01)
- new net: J11.2 (Pin_2), U5.5 (A02)
- new net: J12.2 (Pin_2), U5.6 (B02)
- new net: J12.1 (Pin_1), U5.7 (B01)
