File: 500g/Rata2i2.0/pcbn't/Schematic/Schematic.kicad_sch (KiCad schematic)
At the start: 33 parts, among them J1 Screw_Terminal_01x03, J10 Conn_01x03_Pin, J11 Screw_Terminal_01x02, J12 Screw_Terminal_01x02, J2 Screw_Terminal_01x03, J3 Screw_Terminal_01x03, J4 Screw_Terminal_01x03, J5 Screw_Terminal_01x03, J6 Screw_Terminal_01x03, J7 Battery, SW1 SW_SPDT, U1 DEV-16771, U3 R-78K5.0-0.5, U4 R-78K5.0-0.5, U5 ROB-14450

Commit message: new thingy
Connections:
- net md1 is gone; now on net mdr1: U1.19 (A5)
- net md2 is gone; now on net mdr2: U1.20 (A6)
- net md3 is gone; now on net mdr3: U1.21 (A7)
- net md4 is gone; now on net mdr4: U1.22 (A8)
- net +12V: now also F1.2; no longer F1.1, SW1.1 (A)
- net +3.3V: now also J6.2 (Pin_2)
- net GND: no longer J6.2 (Pin_2)
- new net: F1.1, SW1.1 (A)
Changed lines of the file:
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@@
 	)
 	(junction
-		(at 68.58 184.15)
-		(diameter 0)
-		(color 0 0 0 0)
-	)
-	(junction
 		(at 140.97 173.99)
 		(diameter 0)
@@
 	(wire
 		(pts
-			(xy 74.93 184.15) (xy 68.58 184.15)
-		)
-		(stroke
-			(width 0)
-			(type default)
-		)
-	)
-	(wire
-		(pts
 			(xy 242.57 123.19) (xy 242.57 124.46)
 		)
@@
 	(wire
 		(pts
+			(xy 74.93 184.15) (xy 76.2 184.15)
+		)
+		(stroke
+			(width 0)
+			(type default)
+		)
+	)
+	(wire
+		(pts
 			(xy 148.59 173.99) (xy 148.59 176.53)
 		)
@@
 		)
 	)
-	(global_label "md3"
+	(global_label "mdr3"
 		(shape input)
 		(at 60.96 118.11 180)
@@
 		)
 	)
-	(global_label "md1"
+	(global_label "mdr1"
 		(shape input)
 		(at 60.96 113.03 180)
@@
 		)
 	)
-	(global_label "md2"
+	(global_label "mdr2"
 		(shape input)
 		(at 60.96 115.57 180)
@@
 		)
 	)
-	(global_label "md4"
+	(global_label "mdr4"
 		(shape input)
 		(at 60.96 120.65 180)
@@
 	)
 	(symbol
-		(lib_id "power:GND")
-		(at 19.05 83.82 0)
+		(lib_id "power:+3.3V")
+		(at 223.52 50.8 180)
 		(unit 1)
 		(exclude_from_sim no)
@@
 		(on_board yes)
 		(dnp no)
-		(fields_autoplaced yes)
-		(property "Reference" "#PWR035"
-			(at 19.05 90.17 0)
+		(property "Reference" "#PWR011"
+			(at 223.52 46.99 0)
 			(effects
 				(font
@@
 			)
 		)
-		(property "Value" "GND"
-			(at 19.05 88.9 0)
+		(property "Value" "+3.3V"
+			(at 223.774 56.134 0)
 			(effects
 				(font
@@
 		)
 		(property "Footprint" ""
-			(at 19.05 83.82 0)
+			(at 223.52 50.8 0)
 			(effects
 				(font
@@
 		)
 		(property "Datasheet" ""
-			(at 19.05 83.82 0)
+			(at 223.52 50.8 0)
 			(effects
 				(font
@@
 			)
 		)
-		(property "Description" "Power symbol creates a global label with name \"GND\" , ground"
-			(at 19.05 83.82 0)
+		(property "Description" "Power symbol creates a global label with name \"+3.3V\""
+			(at 223.52 50.8 0)
 			(effects
 				(font
@@
 			(project "Schematic"
 				(path "/68c7ddae-445d-49f5-81ac-f496a7c86e74"
-					(reference "#PWR035")
+					(reference "#PWR011")
 					(unit 1)
 				)
@@
 	(symbol
 		(lib_id "power:GND")
-		(at 223.52 50.8 0)
+		(at 19.05 83.82 0)
 		(unit 1)
 		(exclude_from_sim no)
@@
 		(dnp no)
 		(fields_autoplaced yes)
-		(property "Reference" "#PWR011"
-			(at 223.52 57.15 0)
+		(property "Reference" "#PWR035"
+			(at 19.05 90.17 0)
 			(effects
 				(font
@@
 		)
 		(property "Value" "GND"
-			(at 223.52 55.88 0)
+			(at 19.05 88.9 0)
 			(effects
 				(font
@@
 		)
 		(property "Footprint" ""
-			(at 223.52 50.8 0)
+			(at 19.05 83.82 0)
 			(effects
 				(font
@@
 		)
 		(property "Datasheet" ""
-			(at 223.52 50.8 0)
+			(at 19.05 83.82 0)
 			(effects
 				(font
@@
 		)
 		(property "Description" "Power symbol creates a global label with name \"GND\" , ground"
-			(at 223.52 50.8 0)
+			(at 19.05 83.82 0)
 			(effects
 				(font
@@
 		)
 		(instances
-			(project ""
+			(project "Schematic"
 				(path "/68c7ddae-445d-49f5-81ac-f496a7c86e74"
-					(reference "#PWR011")
+					(reference "#PWR035")
 					(unit 1)
 				)

Commit message: pcb??
did we do it guys
Parts:
- added J8: Conn_01x08_Pin, Connector_PinHeader_2.54mm:PinHeader_1x08_P2.54mm_Vertical, symbol Connector:Conn_01x08_Pin
Connections:
- net +3.3V: now also J8.1 (Pin_1)
- net GND: now also J8.2 (Pin_2)
- net sda: now reaches U1.40 (A16)
- net sda: now also J8.4 (Pin_4)
- net scl: now reaches U1.41 (A17)
- net scl: now also J8.3 (Pin_3)
- no-connect marks 40 -> 42
Other:
- note added: "imu"
- moved on the sheet: C1, C2, C4, D1, F1, H1, H2, J1, J10, J11, J12, J2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

Commit message: PCB!!!!!
dont worry about the 2 errors its done
Parts:
- D1, D2, D3, D4, D6: footprint LED_SMD:LED_1206_3216Metric_ReverseMount_Hole1.8x2.4mm -> LED_SMD:LED_1206_3216Metric
Connections:
- net int: now reaches U1.39 (A15)
- net int: now also J8.8 (Pin_8)
- no-connect marks 42 -> 40
Changed lines of the file:
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@@
 	)
 	(no_connect
-		(at 135.89 95.25)
-	)
-	(no_connect
-		(at 101.6 105.41)
-	)
-	(no_connect
 		(at 135.89 87.63)
 	)
@@
 		)
 	)
+	(global_label "int"
+		(shape input)
+		(at 135.89 95.25 0)
+		(fields_autoplaced yes)
+		(effects
+			(font
+				(size 1.27 1.27)
+			)
+			(justify left)
+		)
+		(property "Intersheetrefs" "${INTERSHEET_REFS}"
+			(at 141.3547 95.25 0)
+			(effects
+				(font
+					(size 1.27 1.27)
+				)
+				(justify left)
+				(hide yes)
+			)
+		)
+	)
 	(global_label "motorapwm"
 		(shape input)
@@
 		)
 	)
+	(global_label "int"
+		(shape input)
+		(at 101.6 105.41 0)
+		(fields_autoplaced yes)
+		(effects
+			(font
+				(size 1.27 1.27)
+			)
+			(justify left)
+		)
+		(property "Intersheetrefs" "${INTERSHEET_REFS}"
+			(at 107.0647 105.41 0)
+			(effects
+				(font
+					(size 1.27 1.27)
+				)
+				(justify left)
+				(hide yes)
+			)
+		)
+	)
 	(global_label "mdr4"
 		(shape input)
@@
 			)
 		)
-		(property "Footprint" "LED_SMD:LED_1206_3216Metric_ReverseMount_Hole1.8x2.4mm"
+		(property "Footprint" "LED_SMD:LED_1206_3216Metric"
 			(at 38.1 34.29 0)
 			(effects
@@
 			)
 		)
-		(property "Footprint" "LED_SMD:LED_1206_3216Metric_ReverseMount_Hole1.8x2.4mm"
+		(property "Footprint" "LED_SMD:LED_1206_3216Metric"
 			(at 19.05 72.39 0)
 			(effects
@@
 			)
 		)
-		(property "Footprint" "LED_SMD:LED_1206_3216Metric_ReverseMount_Hole1.8x2.4mm"
+		(property "Footprint" "LED_SMD:LED_1206_3216Metric"
 			(at 20.32 34.29 0)
 			(effects
@@
 			)
 		)
-		(property "Footprint" "LED_SMD:LED_1206_3216Metric_ReverseMount_Hole1.8x2.4mm"
+		(property "Footprint" "LED_SMD:LED_1206_3216Metric"
 			(at 25.4 121.92 0)
 			(effects
@@
 			)
 		)
-		(property "Footprint" "LED_SMD:LED_1206_3216Metric_ReverseMount_Hole1.8x2.4mm"
+		(property "Footprint" "LED_SMD:LED_1206_3216Metric"
 			(at 38.1 72.39 0)
 			(effects
