File: 500g/Rata2i2.0/pcbn't/Schematic/Schematic.kicad_pcb (KiCad board)
At the start: 2 copper layers, 90 x 59.5 mm, 33 parts, among them J1 Screw_Terminal_01x03, J10 Conn_01x03_Pin, J11 Screw_Terminal_01x02, J12 Screw_Terminal_01x02, J2 Screw_Terminal_01x03, J3 Screw_Terminal_01x03, J4 Screw_Terminal_01x03, J5 Screw_Terminal_01x03, J6 Screw_Terminal_01x03, J7 Battery, SW1 SW_SPDT, U1 DEV-16771, U3 R-78K5.0-0.5, U4 R-78K5.0-0.5, U5 ROB-14450

Commit message: new thingy
Parts:
- moved F1 78.9 mm to (154.6, 65.0), turned to -90 degrees
- moved J10 29.1 mm to (126.5, 29.0)
- moved U5 23.6 mm to (105.5, 36.6), turned to -90 degrees
- moved J12 11.6 mm to (105.0, 71.5), turned to 180 degrees
- moved J11 9.91 mm to (95.3, 71.0)
- moved SW1 6.70 mm to (154.5, 54.0)
- moved U3 2.93 mm to (154.8, 74.0)
- moved U4 2.75 mm to (145.0, 74.0)
Connections:
- F1 pad 1: +12V -> Net-(SW1-A)
- F1 pad 2: unconnected-(F1-Pad2) -> +12V
- J6 pad 2: GND -> +3.3V
- SW1 pad 1: +12V -> Net-(SW1-A)
- U1 pad 19: md1 -> mdr1
- U1 pad 20: md2 -> mdr2
- U1 pad 21: md3 -> mdr3
- U1 pad 22: md4 -> mdr4
Routing:
- net +3.3V: track 0.00 -> 106.0 mm
- net Net-(J11-Pin_1): track 0.00 -> 79.9 mm
- net +12V: track 20.6 -> 99.5 mm
- net Net-(J11-Pin_2): track 0.00 -> 74.4 mm
- net Net-(J12-Pin_2): track 0.00 -> 71.5 mm
- net Net-(J12-Pin_1): track 0.00 -> 67.5 mm
- net motorbpwm: track 0.00 -> 39.4 mm
- net start: track 0.00 -> 29.0 mm, vias 0 -> 2
- net motorapwm: track 0.00 -> 24.1 mm
- net mdr2: track 0.00 -> 9.14 mm
- net mdr3: track 0.00 -> 6.33 mm
- net mdr1: track 0.00 -> 6.33 mm
- net mdr4: track 0.00 -> 6.33 mm
- net Net-(SW1-A): track 0.00 -> 4.94 mm
- net Net-(J7-Pin_2): track 16.9 -> 14.9 mm
- added copper zone on F.Cu, net GND
Other:
- board size 90 x 59.5 mm -> 83.5 x 59.5 mm

Commit message: cleaning up for you guys
Parts:
- moved H1 115.2 mm to (170.2, 32.8)
- moved C2 90.9 mm to (165.2, 74.8)
- moved C1 88.6 mm to (162.9, 72.4)
- moved C5 75.4 mm to (148.6, 86.0)
- moved C4 67.7 mm to (141.9, 86.8)
- moved H2 46.9 mm to (66.0, 81.8)
- moved C3 46.7 mm to (121.2, 90.9)
- moved R1 33.8 mm to (86.3, 88.5)
- moved D1 31.5 mm to (85.8, 84.6)
Routing:
- net +12V: track 99.5 -> 106.5 mm
- net motorbpwm: track 39.4 -> 44.4 mm
- net s4: track 61.4 -> 63.5 mm
Changed lines of the file:
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@@
 		(tags "THT Terminal Block Xinya XY308-2.54-2P pitch 2.54mm size 5.58x6.5mm^2 drill 1.2mm pad 2mm")
 		(property "Reference" "J12"
-			(at 1.27 -4.22 360)
+			(at 1.27 -4.22 0)
 			(layer "F.SilkS")
 			(effects
@@
 		)
 		(property "Value" "Screw_Terminal_01x02"
-			(at 1.71 4.52 360)
+			(at 1.71 4.52 0)
 			(layer "F.Fab")
 			(effects
@@
 		)
 		(property "Footprint" "TerminalBlock:TerminalBlock_Xinya_XY308-2.54-2P_1x02_P2.54mm_Horizontal"
-			(at 0 0 360)
+			(at 0 0 0)
 			(layer "F.Fab")
 			(hide yes)
@@
 		)
 		(property "Datasheet" ""
-			(at 0 0 360)
+			(at 0 0 0)
 			(layer "F.Fab")
 			(hide yes)
@@
 		)
 		(property "Description" "Generic screw terminal, single row, 01x02, script generated (kicad-library-utils/schlib/autogen/connector/)"
-			(at 0 0 360)
+			(at 0 0 0)
 			(layer "F.Fab")
 			(hide yes)
@@
 		)
 		(fp_text user "${REFERENCE}"
-			(at 1.27 2.15 360)
+			(at 1.27 2.15 0)
 			(layer "F.Fab")
 			(effects
@@
 	(footprint "Capacitor_SMD:C_0805_2012Metric"
 		(layer "F.Cu")
-		(at 84.57 119.79)
+		(at 121.25 90.9)
 		(descr "Capacitor SMD 0805 (2012 Metric), square (rectangular) end terminal, IPC_7351 nominal, (Body size source: IPC-SM-782 page 76, https://www.pcb-3d.com/wordpress/wp-content/uploads/ipc-sm-782a_amendment_1_and_2.pdf, https://docs.google.com/spreadsheets/d/1BsfQQcO9C6DZCsRaXUlFlo91Tg2WpOkGARC1WS5S8t0/edit?usp=sharing), generated with kicad-footprint-generator")
 		(tags "capacitor")
@@
 	(footprint "LED_SMD:LED_1206_3216Metric_ReverseMount_Hole1.8x2.4mm"
 		(layer "F.Cu")
-		(at 96.19 114.285)
+		(at 85.8 84.6)
 		(descr "LED SMD 1206 (3216 Metric), reverse mount, square (rectangular) end terminal, IPC_7351 nominal, (Body size source: http://www.tortai-tech.com/upload/download/2011102023233369053.pdf), generated with kicad-footprint-generator")
 		(tags "diode reverse")
@@
 	(footprint "Capacitor_SMD:C_0805_2012Metric"
 		(layer "F.Cu")
-		(at 84.57 116.78)
+		(at 165.2 74.75)
 		(descr "Capacitor SMD 0805 (2012 Metric), square (rectangular) end terminal, IPC_7351 nominal, (Body size source: IPC-SM-782 page 76, https://www.pcb-3d.com/wordpress/wp-content/uploads/ipc-sm-782a_amendment_1_and_2.pdf, https://docs.google.com/spreadsheets/d/1BsfQQcO9C6DZCsRaXUlFlo91Tg2WpOkGARC1WS5S8t0/edit?usp=sharing), generated with kicad-footprint-generator")
 		(tags "capacitor")
@@
 	(footprint "MountingHole:MountingHole_2.5mm"
 		(layer "F.Cu")
-		(at 90.07 122.09)
+		(at 66 81.8)
 		(descr "Mounting Hole 2.5mm, no annular")
 		(tags "mounting hole 2.5mm no annular")
@@
 	(footprint "MountingHole:MountingHole_2.5mm"
 		(layer "F.Cu")
-		(at 90.07 115.54)
+		(at 170.2 32.75)
 		(descr "Mounting Hole 2.5mm, no annular")
 		(tags "mounting hole 2.5mm no annular")
@@
 	(footprint "Resistor_SMD:R_0805_2012Metric"
 		(layer "F.Cu")
-		(at 95.55 121.07)
+		(at 86.2875 88.55)
 		(descr "Resistor SMD 0805 (2012 Metric), square (rectangular) end terminal, IPC_7351 nominal, (Body size source: IPC-SM-782 page 72, https://www.pcb-3d.com/wordpress/wp-content/uploads/ipc-sm-782a_amendment_1_and_2.pdf), generated with kicad-footprint-generator")
 		(tags "resistor")
 		(property "Reference" "R1"
-			(at 58.45 -54.6 0)
+			(at 0 0 0)
 			(layer "F.SilkS")
 			(effects
@@
 	(footprint "Capacitor_SMD:C_0805_2012Metric"
 		(layer "F.Cu")
-		(at 84.57 122.8)
+		(at 141.95 86.85)
 		(descr "Capacitor SMD 0805 (2012 Metric), square (rectangular) end terminal, IPC_7351 nominal, (Body size source: IPC-SM-782 page 76, https://www.pcb-3d.com/wordpress/wp-content/uploads/ipc-sm-782a_amendment_1_and_2.pdf, https://docs.google.com/spreadsheets/d/1BsfQQcO9C6DZCsRaXUlFlo91Tg2WpOkGARC1WS5S8t0/edit?usp=sharing), generated with kicad-footprint-generator")
 		(tags "capacitor")
@@
 	(footprint "Capacitor_SMD:C_0805_2012Metric"
 		(layer "F.Cu")
-		(at 84.57 113.77)
+		(at 162.95 72.4)
 		(descr "Capacitor SMD 0805 (2012 Metric), square (rectangular) end terminal, IPC_7351 nominal, (Body size source: IPC-SM-782 page 76, https://www.pcb-3d.com/wordpress/wp-content/uploads/ipc-sm-782a_amendment_1_and_2.pdf, https://docs.google.com/spreadsheets/d/1BsfQQcO9C6DZCsRaXUlFlo91Tg2WpOkGARC1WS5S8t0/edit?usp=sharing), generated with kicad-footprint-generator")
 		(tags "capacitor")
@@
 	(footprint "Capacitor_SMD:C_0805_2012Metric"
 		(layer "F.Cu")
-		(at 84.57 125.81)
+		(at 148.55 85.95)
 		(descr "Capacitor SMD 0805 (2012 Metric), square (rectangular) end terminal, IPC_7351 nominal, (Body size source: IPC-SM-782 page 76, https://www.pcb-3d.com/wordpress/wp-content/uploads/ipc-sm-782a_amendment_1_and_2.pdf, https://docs.google.com/spreadsheets/d/1BsfQQcO9C6DZCsRaXUlFlo91Tg2WpOkGARC1WS5S8t0/edit?usp=sharing), generated with kicad-footprint-generator")
 		(tags "capacitor")
@@
 	)
 	(segment
-		(start 155 26.5)
-		(end 159 30.5)
+		(start 153.839 71.46)
+		(end 143.935 71.46)
 		(width 0.2)
 		(layer "F.Cu")
@@
 	)
 	(segment
-		(start 153.225 71.46)
-		(end 143.935 71.46)
+		(start 154.6 66.4)
+		(end 154.6 70.699)
+		(width 0.2)
+		(layer "F.Cu")
+		(net 1)
+	)
+	(segment
+		(start 153 71.42)
+		(end 153.879 71.42)
 		(width 0.2)
 		(layer "F.Cu")
@@
 	(segment
 		(start 159 30.5)
-		(end 159 63.5)
+		(end 155 26.5)
 		(width 0.2)
 		(layer "F.Cu")
@@
 	)
 	(segment
-		(start 154.6 70.085)
-		(end 153.225 71.46)
+		(start 116.92 26.5)
+		(end 114.39 29.03)
 		(width 0.2)
 		(layer "F.Cu")
@@
 	)
 	(segment
-		(start 157.4 65)
-		(end 160.4 68)
+		(start 154.6 70.699)
+		(end 153.839 71.46)
 		(width 0.2)
 		(layer "F.Cu")
@@
 	)
 	(segment
-		(start 116.92 26.5)
-		(end 155 26.5)
+		(start 153.879 71.42)
+		(end 159 66.299)
 		(width 0.2)
 		(layer "F.Cu")
@@
 	)
 	(segment
-		(start 114.39 29.03)
-		(end 116.92 26.5)
+		(start 159 66.299)
+		(end 159 30.5)
 		(width 0.2)
 		(layer "F.Cu")
@@
 	)
 	(segment
-		(start 154.6 66.4)
-		(end 154.6 70.085)
+		(start 155 26.5)
+		(end 116.92 26.5)
 		(width 0.2)
 		(layer "F.Cu")
@@
 	)
 	(segment
-		(start 126.21 42.21)
-		(end 125.5 41.5)
-		(width 0.2)
-		(layer "F.Cu")
-		(net 7)
-	)
-	(segment
 		(start 101.21 60.766195)
 		(end 99.95 62.026195)
@@
 	)
 	(segment
-		(start 125.5 41.5)
-		(end 123.5875 41.5)
+		(start 126.21 41.66)
+		(end 125.15 40.6)
 		(width 0.2)
 		(layer "F.Cu")
@@
 	)
 	(segment
-		(start 119.5875 37.5)
-		(end 113.52084 37.5)
+		(start 125.15 40.6)
+		(end 122.6875 40.6)
 		(width 0.2)
 		(layer "F.Cu")
@@
 	(segment
 		(start 119.5875 37.5)
-		(end 123.5875 41.5)
+		(end 113.52084 37.5)
 		(width 0.2)
 		(layer "F.Cu")
@@
 	)
 	(segment
-		(start 126.21 43.7)
-		(end 126.21 42.21)
+		(start 122.6875 40.6)
+		(end 119.5875 37.5)
 		(width 0.2)
 		(layer "F.Cu")
@@
 	)
 	(segment
+		(start 126.21 43.7)
+		(end 126.21 41.66)
+		(width 0.2)
+		(layer "F.Cu")
+		(net 7)
+	)
+	(segment
 		(start 113.51042 37.51042)
 		(end 101.21 49.81084)
@@
 	)
 	(segment
-		(start 147.21 43.7)
-		(end 141.984 48.926)
+		(start 102.49 65.12)
+		(end 104.11 63.5)
+		(width 0.2)
+		(layer "F.Cu")
+		(net 8)
+	)
+	(segment
+		(start 144.5 46.41)
+		(end 147.21 43.7)
 		(width 0.2)
 		(layer "F.Cu")
@@
 	(segment
 		(start 104.11 63.5)
-		(end 102.49 65.12)
+		(end 121 63.5)
 		(width 0.2)
 		(layer "F.Cu")
@@
 	(segment
 		(start 121 63.5)
-		(end 104.11 63.5)
+		(end 133.2 51.3)
 		(width 0.2)
 		(layer "F.Cu")
@@
 	)
 	(segment
-		(start 135.11484 48.926)
-		(end 134 50.04084)
+		(start 133.2 51.3)
+		(end 143.6 51.3)
 		(width 0.2)
 		(layer "F.Cu")
@@
 	)
 	(segment
-		(start 134 50.04084)
-		(end 134 50.5)
+		(start 143.6 51.3)
+		(end 144.5 50.4)
 		(width 0.2)
 		(layer "F.Cu")
@@
 	)
 	(segment
-		(start 141.984 48.926)
-		(end 135.11484 48.926)
+		(start 144.5 50.4)
+		(end 144.5 46.41)
 		(width 0.2)
 		(layer "F.Cu")
@@
 	)
 	(segment
-		(start 134 50.5)
-		(end 121 63.5)
-		(width 0.2)
-		(layer "F.Cu")
-		(net 8)
-	)
-	(segment
 		(start 147.21 37.29)
 		(end 147.5 37)
@@
 	)
 	(segment
-		(start 98.996 60.440195)
-		(end 99.609 61.053195)
+		(start 96.15 53.65)
+		(end 94.75 55.05)
 		(width 0.2)
 		(layer "B.Cu")
@@
 	)
 	(segment
-		(start 99.074 66.074)
-		(end 114.236 66.074)
+		(start 94.75 63.01884)
+		(end 96.15 64.41884)
 		(width 0.2)
 		(layer "B.Cu")
@@
 	)
 	(segment
-		(start 99.609 61.053195)
-		(end 99.609 63.891)
+		(start 96.15 65.7)
+		(end 96.85 66.4)
 		(width 0.2)
 		(layer "B.Cu")
@@
 	)
 	(segment
-		(start 98.996 44.424)
-		(end 98.996 60.440195)
+		(start 96.15 64.41884)
+		(end 96.15 65.7)
 		(width 0.2)
 		(layer "B.Cu")
@@
 	)
 	(segment
-		(start 98.996 64.504)
-		(end 98.996 65.996)
+		(start 113.91 66.4)
+		(end 115.19 65.12)
 		(width 0.2)
 		(layer "B.Cu")
@@
 	)
 	(segment
-		(start 114.236 66.074)
-		(end 115.19 65.12)
+		(start 94.75 55.05)
+		(end 94.75 63.01884)
 		(width 0.2)
 		(layer "B.Cu")
@@
 	)
 	(segment
+		(start 96.15 47.27)
+		(end 96.15 53.65)
+		(width 0.2)
+		(layer "B.Cu")
+		(net 19)
+	)
+	(segment
 		(start 99.23 44.27)
 		(end 99.5 44)
@@
 	)
 	(segment
-		(start 98.996 65.996)
-		(end 99.074 66.074)
+		(start 99.15 44.27)
+		(end 96.15 47.27)
 		(width 0.2)
 		(layer "B.Cu")
@@
 	)
 	(segment
-		(start 99.609 63.891)
-		(end 98.996 64.504)
+		(start 96.85 66.4)
+		(end 113.91 66.4)
 		(width 0.2)
 		(layer "B.Cu")
@@
 		(polygon
 			(pts
-				(xy 78 22) (xy 160.5 22.5) (xy 161 81) (xy 77.5 81.5) (xy 77.5 22.5) (xy 79.5 22.5)
+				(xy 77.5 22) (xy 161 22) (xy 161 81.5) (xy 77.5 81.5)
 			)
 		)

Commit message: pcb??
did we do it guys
Parts:
- added J8: Conn_01x08_Pin, Connector_PinHeader_2.54mm:PinHeader_1x08_P2.54mm_Vertical, F.Cu at (132.0, 31.0)
- moved H2 57.2 mm to (72.5, 25.0)
- moved C3 56.1 mm to (89.0, 45.0)
- moved C4 29.0 mm to (158.5, 63.0), turned to 90 degrees
- moved C5 15.4 mm to (135.1, 78.5), turned to 180 degrees
- moved C1 13.4 mm to (151.5, 65.5), turned to 90 degrees
- moved D6 10.2 mm to (128.1, 78.0)
- moved H1 9.06 mm to (165.5, 25.0)
- moved R5 7.11 mm to (123.4, 78.0)
- moved C2 5.88 mm to (160.0, 77.5), turned to -90 degrees
Connections:
- U1 pad 40: unconnected-(U1-A16-Pad40) -> sda
- U1 pad 41: unconnected-(U1-A17-Pad41) -> scl
Routing:
- net scl: track 0.00 -> 28.0 mm
- net sda: track 0.00 -> 27.7 mm
- net +3.3V: track 106.0 -> 128.9 mm
- net +5V: track 0.00 -> 12.0 mm
- net +12V: track 106.5 -> 118.0 mm
- net s1: track 41.0 -> 44.1 mm
- net Net-(D6-A): track 5.25 -> 2.17 mm
- net GND: track 0.00 -> 1.21 mm

Commit message: PCB!!!!!
dont worry about the 2 errors its done
Parts:
- removed D1: LED, LED_SMD:LED_1206_3216Metric_ReverseMount_Hole1.8x2.4mm
- removed R1: R_US, Resistor_SMD:R_0805_2012Metric
- D2, D3, D4, D6: footprint LED_SMD:LED_1206_3216Metric_ReverseMount_Hole1.8x2.4mm -> LED_SMD:LED_1206_3216Metric
- moved C4 17.6 mm to (159.0, 45.5)
- moved C2 14.1 mm to (158.5, 63.5), turned to 90 degrees
- moved H2 9.06 mm to (81.5, 26.0)
- moved H1 7.50 mm to (158.0, 25.0)
Connections:
- J8 pad 8: unconnected-(J8-Pin_8-Pad8) -> int
- U1 pad 39: unconnected-(U1-A15-Pad39) -> int
Routing:
- net GND: track 1.21 -> 139.8 mm
- net +5V: track 12.0 -> 109.4 mm, vias 0 -> 5
- net +3.3V: track 128.9 -> 189.5 mm
- net int: track 0.00 -> 29.5 mm
- net s3: track 50.0 -> 51.4 mm
- net +12V: track 118.0 -> 116.9 mm
- net L1: track 19.0 -> 19.1 mm, vias 0 -> 1

Commit message: Surprise in graphics
Parts:
- moved H1 6.10 mm to (154.5, 30.0)
- moved H2 3.00 mm to (81.5, 29.0)
Other:
- board size 83.5 x 59.5 mm -> 83.5 x 57 mm
- board text added: "12"
- board text added: "3.3"
- board text added: "gnd"
- board text added: "l1"
- board text added: "l2"
- board text added: "ma"
- board text added: "mb"
- board text added: "mdr1"
- board text added: "mdr2"
- board text added: "mdr3"
- board text added: "mdr4"
- board text added: "s1"
- board text added: "s2"
- board text added: "s3"
- board text added: "s4"

Commit message: done
Routing:
- net +3.3V: track 189.5 -> 189.2 mm, vias 0 -> 2
- net sda: track 27.7 -> 28.0 mm, vias 0 -> 1
- net scl: vias 0 -> 1
Changed lines of the file:
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@@
+	)
+	(segment
+		(start 94.87 41.48)
+		(end 97.8 38.55)
+		(width 0.2)
+		(layer "F.Cu")
+		(net 4)
 	)
 	(segment
@@
 	)
 	(segment
-		(start 125.35 65.12)
-		(end 125.35 60.65)
-		(width 0.2)
-		(layer "F.Cu")
-		(net 4)
-	)
-	(segment
 		(start 113.82 31)
 		(end 111.85 29.03)
@@
 	)
 	(segment
+		(start 109.88 31)
+		(end 111.85 29.03)
+		(width 0.2)
+		(layer "F.Cu")
+		(net 4)
+	)
+	(segment
 		(start 137.96 76.54)
 		(end 136 78.5)
@@
 	)
 	(segment
-		(start 126.1 59.9)
-		(end 135.37 59.9)
+		(start 102 34.3)
+		(end 105.3 31)
+		(width 0.2)
+		(layer "F.Cu")
+		(net 4)
+	)
+	(segment
+		(start 105.3 31)
+		(end 109.88 31)
+		(width 0.2)
+		(layer "F.Cu")
+		(net 4)
+	)
+	(segment
+		(start 118.5 29)
+		(end 116.5 31)
+		(width 0.2)
+		(layer "F.Cu")
+		(net 4)
+	)
+	(segment
+		(start 125.35 65.12)
+		(end 125.35 61.9)
+		(width 0.2)
+		(layer "F.Cu")
+		(net 4)
+	)
+	(segment
+		(start 121.445 29)
+		(end 118.5 29)
+		(width 0.2)
+		(layer "F.Cu")
+		(net 4)
+	)
+	(segment
+		(start 94.87 42.13)
+		(end 94.87 41.48)
 		(width 0.2)
 		(layer "F.Cu")
@@
 	)
 	(segment
-		(start 106 31)
-		(end 94.87 42.13)
-		(width 0.2)
-		(layer "F.Cu")
-		(net 4)
-	)
-	(segment
-		(start 125.35 60.65)
-		(end 126.1 59.9)
-		(width 0.2)
-		(layer "F.Cu")
-		(net 4)
-	)
-	(segment
-		(start 109.88 31)
-		(end 106 31)
-		(width 0.2)
-		(layer "F.Cu")
-		(net 4)
-	)
-	(segment
-		(start 118.5 29)
-		(end 116.5 31)
-		(width 0.2)
-		(layer "F.Cu")
-		(net 4)
-	)
-	(segment
-		(start 111.85 29.03)
-		(end 109.88 31)
-		(width 0.2)
-		(layer "F.Cu")
-		(net 4)
-	)
-	(segment
-		(start 121.445 29)
-		(end 118.5 29)
-		(width 0.2)
-		(layer "F.Cu")
+		(start 125.35 61.9)
+		(end 127.35 59.9)
+		(width 0.2)
+		(layer "F.Cu")
+		(net 4)
+	)
+	(segment
+		(start 127.35 59.9)
+		(end 135.37 59.9)
+		(width 0.2)
+		(layer "F.Cu")
+		(net 4)
+	)
+	(via
+		(at 102 34.3)
+		(size 0.6)
+		(drill 0.3)
+		(layers "F.Cu" "B.Cu")
+		(net 4)
+	)
+	(via
+		(at 97.8 38.55)
+		(size 0.6)
+		(drill 0.3)
+		(layers "F.Cu" "B.Cu")
 		(net 4)
 	)
@@
 	)
 	(segment
+		(start 97.8 38.55)
+		(end 102 34.35)
+		(width 0.2)
+		(layer "B.Cu")
+		(net 4)
+	)
+	(segment
 		(start 134.17 58.7)
 		(end 135.51 60.04)
@@
 		(start 134.17 43.7)
 		(end 134.17 58.7)
+		(width 0.2)
+		(layer "B.Cu")
+		(net 4)
+	)
+	(segment
+		(start 102 34.35)
+		(end 102 34.3)
 		(width 0.2)
 		(layer "B.Cu")
@@
 	)
 	(segment
-		(start 137.04 36.873916)
-		(end 137 36.913916)
-		(width 0.2)
-		(layer "F.Cu")
-		(net 69)
-	)
-	(segment
-		(start 137.04 31)
-		(end 137.04 36.873916)
-		(width 0.2)
-		(layer "F.Cu")
-		(net 69)
-	)
-	(segment
 		(start 137 36.913916)
 		(end 137 38.833916)
@@
 	)
 	(segment
+		(start 137 36.913916)
+		(end 137 35.4)
+		(width 0.2)
+		(layer "F.Cu")
+		(net 69)
+	)
+	(segment
 		(start 137.5 46.5)
 		(end 131.27 46.5)
@@
 		(net 69)
 	)
-	(segment
-		(start 138 33.42)
-		(end 138 38.5)
-		(width 0.2)
-		(layer "F.Cu")
-		(net 70)
+	(via
+		(at 137 35.4)
+		(size 0.6)
+		(drill 0.3)
+		(layers "F.Cu" "B.Cu")
+		(net 69)
+	)
+	(segment
+		(start 137 35.4)
+		(end 137.04 35.36)
+		(width 0.2)
+		(layer "B.Cu")
+		(net 69)
+	)
+	(segment
+		(start 137.04 35.36)
+		(end 137.04 31)
+		(width 0.2)
+		(layer "B.Cu")
+		(net 69)
 	)
 	(segment
@@
 	)
 	(segment
-		(start 140 31.42)
-		(end 138 33.42)
-		(width 0.2)
-		(layer "F.Cu")
-		(net 70)
-	)
-	(segment
 		(start 140 40.5)
 		(end 140 45.5)
@@
 	)
 	(segment
+		(start 138 38.5)
+		(end 138 35.7)
+		(width 0.2)
+		(layer "F.Cu")
+		(net 70)
+	)
+	(segment
 		(start 138 47.5)
 		(end 132.81 47.5)
@@
 		(net 70)
 	)
+	(via
+		(at 138 35.7)
+		(size 0.6)
+		(drill 0.3)
+		(layers "F.Cu" "B.Cu")
+		(net 70)
+	)
+	(segment
+		(start 138 32.58)
+		(end 139.58 31)
+		(width 0.2)
+		(layer "B.Cu")
+		(net 70)
+	)
+	(segment
+		(start 138 35.7)
+		(end 138 32.58)
+		(width 0.2)
+		(layer "B.Cu")
+		(net 70)
+	)

Commit message: done???????
yeah
Parts:
- added G***: LOGO, LOGO, F.Cu at (82.5, 50.5)
- added G***: LOGO, LOGO, F.Cu at (83.5, 37.5)
- added G***: LOGO, LOGO, F.Cu at (84.0, 68.0)
- added G***: LOGO, LOGO, F.Cu at (86.5, 76.5)
