File: 500g/Rata2i2.0/pcbn't/Schematic/Schematic.kicad_pcb (KiCad board)
At the start: 2 copper layers, 83.5 x 57 mm, 36 parts, among them J1 Screw_Terminal_01x03, J10 Conn_01x03_Pin, J11 Screw_Terminal_01x02, J12 Screw_Terminal_01x02, J2 Screw_Terminal_01x03, J3 Screw_Terminal_01x03, J4 Screw_Terminal_01x03, J5 Screw_Terminal_01x03, J6 Screw_Terminal_01x03, J7 Battery, J8 Conn_01x08_Pin, SW1 SW_SPDT, U1 DEV-16771, U3 R-78K5.0-0.5, U4 R-78K5.0-0.5, U5 ROB-14450

Commit message: done!!
no more drawings i pinky promise nonemore
Parts:
- added G***: LOGO, LOGO, F.Cu at (91.5, 32.5)
Changed lines of the file:
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@@
 			(outputformat 1)
 			(mirror no)
-			(drillshape 1)
+			(drillshape 0)
 			(scaleselection 1)
-			(outputdirectory "")
+			(outputdirectory "../../../../../../../Desktop/pcb pcb pcb pcb rat rat rat/")
 		)
 	)
@@
 			)
 			(stroke
+				(width 0)
+				(type solid)
+			)
+			(fill solid)
+			(layer "F.SilkS")
+		)
+	)
+	(footprint "LOGO"
+		(layer "F.Cu")
+		(at 91.5 32.5)
+		(property "Reference" "G***"
+			(at 0 0 0)
+			(layer "F.SilkS")
+			(hide yes)
+			(effects
+				(font
+					(size 1.5 1.5)
+					(thickness 0.3)
+				)
+			)
+		)
+		(property "Value" "LOGO"
+			(at 0.75 0 0)
+			(layer "F.SilkS")
+			(hide yes)
+			(effects
+				(font
+					(size 1.5 1.5)
+					(thickness 0.3)
+				)
+			)
+		)
+		(property "Footprint" ""
+			(at 0 0 0)
+			(layer "F.Fab")
+			(hide yes)
+			(effects
+				(font
+					(size 1.27 1.27)
+					(thickness 0.15)
+				)
+			)
+		)
+		(property "Datasheet" ""
+			(at 0 0 0)
+			(layer "F.Fab")
+			(hide yes)
+			(effects
+				(font
+					(size 1.27 1.27)
+					(thickness 0.15)
+				)
+			)
+		)
+		(property "Description" ""
+			(at 0 0 0)
+			(layer "F.Fab")
+			(hide yes)
+			(effects
+				(font
+					(size 1.27 1.27)
+					(thickness 0.15)
+				)
+			)
+		)
+		(attr board_only exclude_from_pos_files exclude_from_bom)
+		(fp_poly
+			(pts
+				(xy -0.931333 -0.896056) (xy -0.999503 -0.779424) (xy -1.065389 -0.762) (xy -1.164135 -0.811229)
+				(xy -1.165931 -0.862542) (xy -1.081658 -0.97435) (xy -0.980205 -0.988566)
+			)
+			(stroke
+				(width 0)
+				(type solid)
+			)
+			(fill solid)
+			(layer "F.SilkS")
+		)
+		(fp_poly
+			(pts
+				(xy -1.454027 -0.950788) (xy -1.439333 -0.893997) (xy -1.486205 -0.755414) (xy -1.586233 -0.708309)
+				(xy -1.639191 -0.73608) (xy -1.694223 -0.870683) (xy -1.64362 -0.988332) (xy -1.566333 -1.016)
+			)
+			(stroke
+				(width 0)
+				(type solid)
+			)
+			(fill solid)
+			(layer "F.SilkS")
+		)
+		(fp_poly
+			(pts
+				(xy -1.261769 -0.639518) (xy -1.196209 -0.484906) (xy -1.1836 -0.449533) (xy -1.064053 -0.243016)
+				(xy -0.921452 -0.1532) (xy -0.797012 -0.096776) (xy -0.779813 -0.042333) (xy -0.875406 0.018746)
+				(xy -1.077414 0.047036) (xy -1.326424 0.044007) (xy -1.56302 0.011129) (xy -1.727786 -0.05013) (xy -1.74751 -0.066272)
+				(xy -1.835601 -0.222092) (xy -1.798094 -0.344245) (xy -1.686278 -0.381) (xy -1.544458 -0.440731)
+				(xy -1.422961 -0.550333) (xy -1.322713 -0.655162)
+			)
+			(stroke
+				(width 0)
+				(type solid)
+			)
+			(fill solid)
+			(layer "F.SilkS")
+		)
+		(fp_poly
+			(pts
+				(xy -0.484122 -2.211492) (xy -0.356949 -2.022125) (xy -0.240722 -1.769132) (xy -0.157394 -1.503751)
+				(xy -0.12892 -1.277215) (xy -0.13818 -1.207529) (xy -0.1336 -1.030219) (xy -0.055315 -0.966933)
+				(xy 0.027192 -0.889021) (xy 0.056075 -0.714833) (xy 0.04882 -0.508111) (xy 0.011746 -0.185004) (xy -0.051372 -0.000196)
+				(xy -0.154535 0.076918) (xy -0.222369 0.084667) (xy -0.310523 0.033757) (xy -0.296333 -0.084667)
+				(xy -0.289101 -0.217303) (xy -0.41107 -0.253944) (xy -0.420285 -0.254) (xy -0.565625 -0.303407)
+				(xy -0.658193 -0.413252) (xy -0.664944 -0.525973) (xy -0.604365 -0.574656) (xy -0.545063 -0.636533)
+				(xy -0.596422 -0.724192) (xy -0.645273 -0.878226) (xy -0.62359 -0.948791) (xy -0.579282 -1.083432)
+				(xy -0.550666 -1.280656) (xy -0.542592 -1.473502) (xy -0.55991 -1.595012) (xy -0.575796 -1.608667)
+				(xy -0.652012 -1.549343) (xy -0.7258 -1.4605) (xy -0.843251 -1.365753) (xy -0.926104 -1.401704)
+				(xy -0.96338 -1.539512) (xy -0.929483 -1.755801) (xy -0.846222 -1.991385) (xy -0.735404 -2.187076)
+				(xy -0.618835 -2.283687) (xy -0.600288 -2.286)
+			)
+			(stroke
+				(width 0)
+				(type solid)
+			)
+			(fill solid)
+			(layer "F.SilkS")
+		)
+		(fp_poly
+			(pts
+				(xy -1.890838 -2.082013) (xy -1.783469 -1.919385) (xy -1.691246 -1.740496) (xy -1.613889 -1.654228)
+				(xy -1.531087 -1.528402) (xy -1.524 -1.47667) (xy -1.588135 -1.378914) (xy -1.734968 -1.361115)
+				(xy -1.896141 -1.426702) (xy -1.9304 -1.456267) (xy -2.00446 -1.495845) (xy -2.030848 -1.394063)
+				(xy -2.032 -1.335314) (xy -2.079 -1.116134) (xy -2.15965 -0.985113) (xy -2.230534 -0.866131) (xy -2.210358 -0.809911)
+				(xy -2.159893 -0.700685) (xy -2.141041 -0.499288) (xy -2.1414 -0.480722) (xy -2.089521 -0.187868)
+				(xy -1.967367 0.056532) (xy -1.85285 0.259634) (xy -1.862102 0.38615) (xy -1.87691 0.40371) (xy -1.920028 0.539945)
+				(xy -1.92108 0.769009) (xy -1.88817 1.022002) (xy -1.829403 1.230023) (xy -1.7694 1.317649) (xy -1.63337 1.316164)
+				(xy -1.49222 1.167618) (xy -1.362951 0.89283) (xy -1.324128 0.772295) (xy -1.212478 0.484102) (xy -1.100031 0.357957)
+				(xy -0.998112 0.394699) (xy -0.918046 0.595164) (xy -0.891981 0.740325) (xy -0.82071 1.104858) (xy -0.734035 1.304102)
+				(xy -0.63828 1.337193) (xy -0.539765 1.203268) (xy -0.444811 0.901463) (xy -0.423333 0.804333) (xy -0.356514 0.540484)
+				(xy -0.286037 0.350437) (xy -0.244595 0.290521) (xy -0.116401 0.29421) (xy 0.014359 0.401277) (xy 0.086519 0.558217)
+				(xy 0.088485 0.581867) (xy 0.125785 0.753119) (xy 0.210199 0.972325) (xy 0.210824 0.973667) (xy 0.272024 1.095573)
+				(xy 0.306426 1.11874) (xy 0.320436 1.022689) (xy 0.320463 0.786939) (xy 0.317667 0.632184) (xy 0.328272 0.21611)
+				(xy 0.376531 -0.054614) (xy 0.458463 -0.174404) (xy 0.57009 -0.137676) (xy 0.70743 0.061154) (xy 0.714716 0.075094)
+				(xy 0.841114 0.319521) (xy 1.476163 -0.013246) (xy 1.854567 -0.218277) (xy 2.080076 -0.36152) (xy 2.154083 -0.450956)
+				(xy 2.077987 -0.494567) (xy 1.853181 -0.500335) (xy 1.558192 -0.482373) (xy 1.213141 -0.450659)
+				(xy 0.913787 -0.414085) (xy 0.717096 -0.379777) (xy 0.6985 -0.37484) (xy 0.549578 -0.374898) (xy 0.502703 -0.458723)
+				(xy 0.557159 -0.575494) (xy 0.702665 -0.670869) (xy 0.974369 -0.741951) (xy 1.324287 -0.791214)
+				(xy 1.691061 -0.814658) (xy 2.013331 -0.808283) (xy 2.224669 -0.770096) (xy 2.455469 -0.634481)
+				(xy 2.52005 -0.469217) (xy 2.41879 -0.274985) (xy 2.152065 -0.052466) (xy 1.720253 0.197656) (xy 1.678466 0.218899)
+				(xy 1.334505 0.401322) (xy 1.129757 0.538579) (xy 1.046788 0.649811) (xy 1.068163 0.754157) (xy 1.126834 0.824453)
+				(xy 1.216957 0.891455) (xy 1.286912 0.85213) (xy 1.371844 0.681751) (xy 1.389647 0.639538) (xy 1.494832 0.449889)
+				(xy 1.597802 0.358677) (xy 1.624871 0.358179) (xy 1.715789 0.446178) (xy 1.843697 0.631374) (xy 1.975321 0.856901)
+				(xy 2.077384 1.06589) (xy 2.116667 1.19865) (xy 2.054101 1.264397) (xy 1.91644 1.263148) (xy 1.778734 1.206194)
+				(xy 1.722548 1.139345) (xy 1.669468 1.056209) (xy 1.582101 1.093113) (xy 1.51695 1.149379) (xy 1.299933 1.248298)
+				(xy 1.062997 1.195809) (xy 0.837387 1.001921) (xy 0.772097 0.91073) (xy 0.595519 0.635) (xy 0.594093 1.0268)
+				(xy 0.556626 1.353621) (xy 0.450758 1.536724) (xy 0.281956 1.569458) (xy 0.180479 1.529965) (xy 0.017131 1.376798)
+				(xy -0.047511 1.253685) (xy -0.091067 1.149969) (xy -0.141618 1.161408) (xy -0.227388 1.304326)
+				(xy -0.266935 1.380596) (xy -0.44966 1.618924) (xy -0.659235 1.695666) (xy -0.877594 1.608242) (xy -0.998241 1.485014)
+				(xy -1.162105 1.276694) (xy -1.357811 1.485014) (xy -1.58601 1.647893) (xy -1.819352 1.686269) (xy -2.008944 1.593208)
+				(xy -2.021403 1.579102) (xy -2.099234 1.414049) (xy -2.172229 1.146831) (xy -2.227807 0.844438)
+				(xy -2.253386 0.573861) (xy -2.240404 0.413054) (xy -2.244865 0.226042) (xy -2.297449 0.097796)
+				(xy -2.413176 -0.015404) (xy -2.59544 -0.034533) (xy -2.691085 -0.022024) (xy -2.883545 -0.002843)
+				(xy -2.953873 -0.044354) (xy -2.949913 -0.135692) (xy -2.850312 -0.274847) (xy -2.729635 -0.323389)
+				(xy -2.581186 -0.375924) (xy -2.54 -0.433059) (xy -2.614015 -0.475819) (xy -2.80878 -0.464793) (xy -2.844657 -0.458519)
+				(xy -3.043686 -0.431537) (xy -3.120672 -0.463659) (xy -3.1191 -0.560516) (xy -3.012598 -0.699433)
+				(xy -2.852381 -0.746881) (xy -2.729639 -0.772253) (xy -2.633709 -0.83509) (xy -2.546312 -0.964574)
+				(xy -2.44917 -1.189889) (xy -2.324006 -1.540218) (xy -2.28611 -1.651) (xy -2.155929 -1.941254) (xy -2.019664 -2.087332)
+			)
+			(stroke
