File: Skibidi/Skibid-i/Skibidi-ControlBoard/Skibidi2.0/Skibidi2.0.kicad_pcb (KiCad board)
At the start: 2 copper layers, 86.2 x 49 mm, 70 parts, among them IC1 TEENSY_4.1, J1 Screw_Terminal_01x03, J10 Screw_Terminal_01x03, J11 Screw_Terminal_01x03, J12 12V, J13 Conn_01x03_Pin, J15 Conn_02x05_Odd_Even, J16 P78E05-1000, J2 Screw_Terminal_01x03, J3 Screw_Terminal_01x03, J4 Screw_Terminal_01x03, J5 Screw_Terminal_01x03, J6 Screw_Terminal_01x03, J7 Screw_Terminal_01x03, J8 Screw_Terminal_01x03, J9 Screw_Terminal_01x03, SW1 SW_Nidec_CAS-120A1, SW2 210-4MS

Commit message: skibidi 2.0 done
Parts:
- removed J15: Conn_02x05_Odd_Even, Connector_PinSocket_2.54mm:PinSocket_2x05_P2.54mm_Vertical
- added +: Conn_01x08_Pin, Connector_PinHeader_2.54mm:PinHeader_1x08_P2.54mm_Vertical, F.Cu at (148.2, 60.6)
- added G***: LOGO, askibidi:turtwig, F.Cu at (197.7, 53.1)
- added G***: LOGO, askibidi:turtwig, F.Cu at (231.7, 32.0)
- added J17: Conn_02x05_Odd_Even, Connector_PinSocket_2.54mm:PinSocket_2x05_P2.54mm_Vertical, F.Cu at (179.3, 68.7)
- R16, R17: moved to B.Cu
- moved C4 8.16 mm to (152.0, 37.3), turned to -90 degrees
- moved D8 7.33 mm to (233.9, 52.9)
- moved R15 7.32 mm to (233.9, 58.8)
- moved G*** 6.13 mm to (229.2, 58.0)
- moved G*** 4.23 mm to (190.3, 53.2)
- moved C11 3.99 mm to (148.7, 36.6)
- moved J13 3.67 mm to (148.3, 25.4)
- moved C7 3.13 mm to (148.2, 66.2)
- moved H1 1.33 mm to (155.6, 26.6)
- moved 10uF 1.00 mm to (186.1, 65.3)
- moved 10uF 0.95 mm to (186.1, 68.9)
- moved H3 0.50 mm to (162.5, 67.4)
- moved H2 0.40 mm to (232.3, 26.1)
- renumbered R3 to 1, R13 to 1, R7 to 1, R1 to 1, R11 to 1, R5 to 1, R9 to 1, C6 to 10uF, C14 to 10uF, R4 to 2, R6 to 2, R12 to 2, R14 to 2, R10 to 2, R2 to 2, R8 to 2, C9 to C, C15 to C, C3 to C, C5 to C, C2 to C, SW1 to ON, R23 to R
Connections:
- IC1 pad 24: DIP1 -> PWMB
- IC1 pad 25: DIP2 -> PWMA
Routing:
- net PWMA: track 0.00 -> 48.1 mm, vias 0 -> 1
- net SDA: track 0.00 -> 35.0 mm, vias 0 -> 2
- net PWMB: track 0.00 -> 34.1 mm, vias 0 -> 1
- net SCL: track 0.00 -> 33.2 mm, vias 0 -> 2
- net +5V: track 76.7 -> 66.4 mm
- net +3.3V: track 203.2 -> 209.6 mm
- net Start: track 63.1 -> 65.6 mm
- net BDC11: track 33.3 -> 35.0 mm
- net BDC22: track 4.49 -> 5.68 mm
- net BDC2: track 4.49 -> 5.60 mm
- net LN1: track 43.6 -> 42.6 mm
- net +12V: track 167.2 -> 168.1 mm
- net Net-(D8-A): track 2.72 -> 3.60 mm
Other:
- board size 86.2 x 49 mm -> 90 x 49 mm
- board text added: "15"
- board text added: "USB!"
