File: Joe-i/Joe-i.kicad_sch (KiCad schematic)
At the start: 41 parts, among them J1 Screw3, J10 Screw_Terminal_01x02, J12 xt30, J2 Screw3, J3 Screw3, J4 Screw3, J5 Screw_Terminal_01x02, J6 Conn_01x03_Pin, J7 Screw3, J8 Screw3, J9 Conn_01x03_Pin, SW1 SW_DIP_x04, SW2 SW_DPDT_x2, U1 DRV8874PWPR, U2 DRV8874PWPR

Commit message: more work
Parts:
- removed C1: 0.1uF, Capacitor_SMD:C_0805_2012Metric, symbol Device:C
Connections:
- net DIP1: now also R6.2, SW1.8; no longer R7.2, SW1.7
- net DIP2: now also R7.2, SW1.7; no longer R6.2, SW1.8
Changed lines of the file:
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@@
 	)
 	(junction
-		(at 30.48 39.37)
-		(diameter 0)
-		(color 0 0 0 0)
-	)
-	(junction
 		(at 96.52 149.86)
 		(diameter 0)
@@
 		)
 	)
-	(global_label "DIP2"
+	(global_label "DIP1"
 		(shape input)
 		(at 238.76 33.02 0)
@@
 		)
 	)
-	(global_label "DIP1"
+	(global_label "DIP2"
 		(shape input)
 		(at 238.76 35.56 0)
@@
 	)
 	(symbol
-		(lib_id "power:GND")
-		(at 30.48 31.75 180)
-		(unit 1)
-		(exclude_from_sim no)
-		(in_bom yes)
-		(on_board yes)
-		(dnp no)
-		(fields_autoplaced yes)
-		(property "Reference" "#PWR02"
-			(at 30.48 25.4 0)
-			(effects
-				(font
-					(size 1.27 1.27)
-				)
-				(hide yes)
-			)
-		)
-		(property "Value" "GND"
-			(at 30.48 26.67 0)
-			(effects
-				(font
-					(size 1.27 1.27)
-				)
-			)
-		)
-		(property "Footprint" ""
-			(at 30.48 31.75 0)
-			(effects
-				(font
-					(size 1.27 1.27)
-				)
-				(hide yes)
-			)
-		)
-		(property "Datasheet" ""
-			(at 30.48 31.75 0)
-			(effects
-				(font
-					(size 1.27 1.27)
-				)
-				(hide yes)
-			)
-		)
-		(property "Description" "Power symbol creates a global label with name \"GND\" , ground"
-			(at 30.48 31.75 0)
-			(effects
-				(font
-					(size 1.27 1.27)
-				)
-				(hide yes)
-			)
-		)
-		(pin "1"
-		)
-		(instances
-			(project "Joe-i"
-				(path "/f79ffdde-4cd4-4bae-9efe-36cb5fedd80b"
-					(reference "#PWR02")
-					(unit 1)
-				)
-			)
-		)
-	)
-	(symbol
 		(lib_id "Mechanical:MountingHole")
 		(at 218.44 172.72 0)
@@
 					(unit 1)
 				)
-			)
-		)
-	)
-	(symbol
-		(lib_id "Device:C")
-		(at 30.48 35.56 180)
-		(unit 1)
-		(exclude_from_sim no)
-		(in_bom yes)
-		(on_board yes)
-		(dnp no)
-		(fields_autoplaced yes)
-		(property "Reference" "C1"
-			(at 26.67 36.8301 0)
-			(effects
-				(font
-					(size 1.27 1.27)
-				)
-				(justify left)
-			)
-		)
-		(property "Value" "0.1uF"
-			(at 26.67 34.2901 0)
-			(effects
-				(font
-					(size 1.27 1.27)
-				)
-				(justify left)
-			)
-		)
-		(property "Footprint" "Capacitor_SMD:C_0805_2012Metric"
-			(at 29.5148 31.75 0)
-			(effects
-				(font
-					(size 1.27 1.27)
-				)
-				(hide yes)
-			)
-		)
-		(property "Datasheet" "~"
-			(at 30.48 35.56 0)
-			(effects
-				(font
-					(size 1.27 1.27)
-				)
-				(hide yes)
-			)
-		)
-		(property "Description" "Unpolarized capacitor"
-			(at 30.48 35.56 0)
-			(effects
-				(font
-					(size 1.27 1.27)
-				)
-				(hide yes)
-			)
-		)
-		(pin "2"
-		)
-		(pin "1"
-		)
-		(instances
-			(project "Joe-i"
-				(path "/f79ffdde-4cd4-4bae-9efe-36cb5fedd80b"
-					(reference "C1")
-					(unit 1)
-				)

Commit message: almost done
Parts:
- removed SW1: SW_DIP_x04, JOEJOE:dip, symbol Switch:SW_DIP_x04
- added SW3: SW_DIP_x02, JOEJOE:Dipswitch2, symbol Switch:SW_DIP_x02
- SW2: footprint JOEJOE:realswitch -> Connector_PinHeader_2.54mm:PinHeader_1x03_P2.54mm_Vertical
Connections:
- net 5v: now also SW3.1, SW3.2
- net DIP1: now also SW3.4
- net DIP2: now also SW3.3
- no-connect marks 18 -> 14
Changed lines of the file:
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@@
 	)
 	(no_connect
-		(at 228.6 40.64)
-	)
-	(no_connect
 		(at 30.48 72.39)
 	)
@@
 	)
 	(no_connect
-		(at 213.36 40.64)
-	)
-	(no_connect
 		(at 160.02 119.38)
 	)
@@
 	)
 	(no_connect
-		(at 228.6 38.1)
-	)
-	(no_connect
 		(at 228.6 135.89)
 	)
@@
 	)
 	(no_connect
-		(at 213.36 38.1)
-	)
-	(no_connect
 		(at 30.48 52.07)
 	)
@@
 	)
 	(symbol
+		(lib_id "Switch:SW_DIP_x02")
+		(at 220.98 35.56 0)
+		(unit 1)
+		(exclude_from_sim no)
+		(in_bom yes)
+		(on_board yes)
+		(dnp no)
+		(fields_autoplaced yes)
+		(property "Reference" "SW3"
+			(at 220.98 25.4 0)
+			(effects
+				(font
+					(size 1.27 1.27)
+				)
+			)
+		)
+		(property "Value" "SW_DIP_x02"
+			(at 220.98 27.94 0)
+			(effects
+				(font
+					(size 1.27 1.27)
+				)
+			)
+		)
+		(property "Footprint" "JOEJOE:Dipswitch2"
+			(at 220.98 35.56 0)
+			(effects
+				(font
+					(size 1.27 1.27)
+				)
+				(hide yes)
+			)
+		)
+		(property "Datasheet" "~"
+			(at 220.98 35.56 0)
+			(effects
+				(font
+					(size 1.27 1.27)
+				)
+				(hide yes)
+			)
+		)
+		(property "Description" "2x DIP Switch, Single Pole Single Throw (SPST) switch, small symbol"
+			(at 220.98 35.56 0)
+			(effects
+				(font
+					(size 1.27 1.27)
+				)
+				(hide yes)
+			)
+		)
+		(pin "2"
+		)
+		(pin "1"
+		)
+		(pin "4"
+		)
+		(pin "3"
+		)
+		(instances
+			(project ""
+				(path "/f79ffdde-4cd4-4bae-9efe-36cb5fedd80b"
+					(reference "SW3")
+					(unit 1)
+				)
+			)
+		)
+	)
+	(symbol
 		(lib_id "Switch:SW_DPDT_x2")
 		(at 111.76 175.26 0)
@@
 			)
 		)
-		(property "Footprint" "JOEJOE:realswitch"
+		(property "Footprint" "Connector_PinHeader_2.54mm:PinHeader_1x03_P2.54mm_Vertical"
 			(at 111.76 175.26 0)
 			(effects
@@
 					(unit 1)
 				)
-			)
-		)
-	)
-	(symbol
-		(lib_id "Switch:SW_DIP_x04")
-		(at 220.98 38.1 0)
-		(unit 1)
-		(exclude_from_sim no)
-		(in_bom yes)
-		(on_board yes)
-		(dnp no)
-		(fields_autoplaced yes)
-		(property "Reference" "SW1"
-			(at 220.98 25.4 0)
-			(effects
-				(font
-					(size 1.27 1.27)
-				)
-			)
-		)
-		(property "Value" "SW_DIP_x04"
-			(at 220.98 27.94 0)
-			(effects
-				(font
-					(size 1.27 1.27)
-				)
-			)
-		)
-		(property "Footprint" "JOEJOE:dip"
-			(at 220.98 38.1 0)
-			(effects
-				(font
-					(size 1.27 1.27)
-				)
-				(hide yes)
-			)
-		)
-		(property "Datasheet" "~"
-			(at 220.98 38.1 0)
-			(effects
-				(font
-					(size 1.27 1.27)
-				)
-				(hide yes)
-			)
-		)
-		(property "Description" "4x DIP Switch, Single Pole Single Throw (SPST) switch, small symbol"
-			(at 220.98 38.1 0)
-			(effects
-				(font
-					(size 1.27 1.27)
-				)
-				(hide yes)
-			)
-		)
-		(pin "6"
-		)
-		(pin "3"
-		)
-		(pin "4"
-		)
-		(pin "1"
-		)
-		(pin "5"
-		)
-		(pin "8"
-		)
-		(pin "7"
-		)
-		(pin "2"
-		)
-		(instances
-			(project "Joe-i"
-				(path "/f79ffdde-4cd4-4bae-9efe-36cb5fedd80b"
-					(reference "SW1")
-					(unit 1)
-				)

Commit message: DONE BUT IDK
Connections:
- net +5V: no longer U1.3 (SLEEP_N), U1.5 (VREF), U2.3 (SLEEP_N), U2.5 (VREF)
- net 5v: now also U1.3 (SLEEP_N), U1.5 (VREF), U2.3 (SLEEP_N), U2.5 (VREF)
- net DIP1: now also R7.2, SW3.3; no longer R6.2, SW3.4
- net DIP2: now also R6.2, SW3.4; no longer R7.2, SW3.3

Commit message: uwefhiqdanjkshbgvqrevfad
Parts:
- added U3: DRV8874PWPR, DRV8874PWPR:SOP65P640X120-17N, symbol 8874[1]:DRV8874PWPR
Changed lines of the file:
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@@
+	)
+	(symbol
+		(lib_id "8874[1]:DRV8874PWPR")
+		(at 105.41 69.85 0)
+		(unit 1)
+		(exclude_from_sim no)
+		(in_bom yes)
+		(on_board yes)
+		(dnp no)
+		(fields_autoplaced yes)
+		(property "Reference" "U3"
+			(at 105.41 41.91 0)
+			(effects
+				(font
+					(size 1.27 1.27)
+				)
+			)
+		)
+		(property "Value" "DRV8874PWPR"
+			(at 105.41 44.45 0)
+			(effects
+				(font
+					(size 1.27 1.27)
+				)
+			)
+		)
+		(property "Footprint" "DRV8874PWPR:SOP65P640X120-17N"
+			(at 105.41 69.85 0)
+			(effects
+				(font
+					(size 1.27 1.27)
+				)
+				(justify bottom)
+				(hide yes)
+			)
+		)
+		(property "Datasheet" ""
+			(at 105.41 69.85 0)
+			(effects
+				(font
+					(size 1.27 1.27)
+				)
+				(hide yes)
+			)
+		)
+		(property "Description" ""
+			(at 105.41 69.85 0)
+			(effects
+				(font
+					(size 1.27 1.27)
+				)
+				(hide yes)
+			)
+		)
+		(property "MF" "Texas Instruments"
+			(at 105.41 69.85 0)
+			(effects
+				(font
+					(size 1.27 1.27)
+				)
+				(justify bottom)
+				(hide yes)
+			)
+		)
+		(property "Description_1" "\n                        \n                            40-V, 6-A H-bridge motor driver with integrated current sensing feedback\n                        \n"
+			(at 105.41 69.85 0)
+			(effects
+				(font
+					(size 1.27 1.27)
+				)
+				(justify bottom)
+				(hide yes)
+			)
+		)
+		(property "Package" "HTSSOP-16 Texas Instruments"
+			(at 105.41 69.85 0)
+			(effects
+				(font
+					(size 1.27 1.27)
+				)
+				(justify bottom)
+				(hide yes)
+			)
+		)
+		(property "Price" "None"
+			(at 105.41 69.85 0)
+			(effects
+				(font
+					(size 1.27 1.27)
+				)
+				(justify bottom)
+				(hide yes)
+			)
+		)
+		(property "SnapEDA_Link" "https://www.snapeda.com/parts/DRV8874PWPR/Texas+Instruments/view-part/?ref=snap"
+			(at 105.41 69.85 0)
+			(effects
+				(font
+					(size 1.27 1.27)
+				)
+				(justify bottom)
+				(hide yes)
+			)
+		)
+		(property "MP" "DRV8874PWPR"
+			(at 105.41 69.85 0)
+			(effects
+				(font
+					(size 1.27 1.27)
+				)
+				(justify bottom)
+				(hide yes)
+			)
+		)
+		(property "Availability" "In Stock"
+			(at 105.41 69.85 0)
+			(effects
+				(font
+					(size 1.27 1.27)
+				)
+				(justify bottom)
+				(hide yes)
+			)
+		)
+		(property "Check_prices" "https://www.snapeda.com/parts/DRV8874PWPR/Texas+Instruments/view-part/?ref=eda"
+			(at 105.41 69.85 0)
+			(effects
+				(font
+					(size 1.27 1.27)
+				)
+				(justify bottom)
+				(hide yes)
+			)
+		)
+		(pin "13"
+		)
+		(pin "10"
+		)
+		(pin "1"
+		)
+		(pin "11"
+		)
+		(pin "12"
+		)
+		(pin "14"
+		)
+		(pin "15"
+		)
+		(pin "16"
+		)
+		(pin "9"
+		)
+		(pin "2"
+		)
+		(pin "3"
+		)
+		(pin "6"
+		)
+		(pin "5"
+		)
+		(pin "4"
+		)
+		(pin "7"
+		)
+		(pin "8"
+		)
+		(instances
+			(project ""
+				(path "/f79ffdde-4cd4-4bae-9efe-36cb5fedd80b"
+					(reference "U3")
+					(unit 1)
+				)
+			)
+		)
 	)
 	(symbol

Commit message: almost done
Parts:
- removed C10, C11, C8, C9: 0.1uF, Capacitor_SMD:C_0805_2012Metric, symbol Device:C
- removed C12: 0.022uF, Capacitor_SMD:C_0805_2012Metric, symbol Device:C
- removed U1, U2: DRV8874PWPR, JOEJOE:DRV8874, symbol DRV8874:DRV8874PWPR
- removed U3: DRV8874PWPR, DRV8874PWPR:SOP65P640X120-17N, symbol 8874[1]:DRV8874PWPR
- added C1: 10uF, Capacitor_SMD:C_0805_2012Metric, symbol Device:C
- added R5, R8: R_US, Resistor_SMD:R_0805_2012Metric, symbol Device:R_US
- added U1, U2: DRV8871DDAR, Joe-ifootprints:DRV8871, symbol DRV8871:DRV8871DDAR
- C5: value 0.022uF -> 10uF
- C6, C7: value 0.1uF -> 10uF
Connections:
- net +12V: now also C5.1, C1.1, U1.5 (VM), U2.5 (VM)
- net DIP1: now also R6.2, SW3.4; no longer R7.2, SW3.3
- net DIP2: now also R7.2, SW3.3; no longer R6.2, SW3.4
- net GND: now also C5.2, C7.2, C1.2, R5.2, R8.2, U1.1 (GND), U1.7 (PGND), U1.9 (PAD), U2.1 (GND), U2.7 (PGND), U2.9 (PAD)
- net MOTOR1A: now also U1.3 (IN1)
- net MOTOR1B: now also U1.2 (IN2)
- net MOTOR2A: now also U2.2 (IN2)
- net MOTOR2B: now also U2.3 (IN1)
- net at J10.2 (Pin_2): now also U2.8 (OUT2)
- net at J10.1 (Pin_1): now also U2.6 (OUT1)
- net at J5.2 (Pin_2): now also U1.8 (OUT2)
- net at J5.1 (Pin_1): now also U1.6 (OUT1)
- new net: R5.1, U1.4 (ILIM)
- new net: R8.1, U2.4 (ILIM)
- no-connect marks 14 -> 8
