File: Joe-i/Joe-i.kicad_pcb (KiCad board)
At the start: 2 copper layers, 67.1 x 52.3 mm, 39 parts, among them J1 Screw3, J10 Screw_Terminal_01x02, J12 xt30, J2 Screw3, J3 Screw3, J4 Screw3, J5 Screw_Terminal_01x02, J6 Conn_01x03_Pin, J7 Screw3, J8 Screw3, J9 Conn_01x03_Pin, SW1 SW_DIP_x04, SW2 SW_DPDT_x2, U1 DRV8874PWPR, U2 DRV8874PWPR

Commit message: more work
Parts:
- removed C1: 0.1uF, Capacitor_SMD:C_0805_2012Metric
- added H1: MountingHole, MountingHole:MountingHole_2.5mm, F.Cu at (254.1, 66.8)
- added H2: MountingHole, MountingHole:MountingHole_2.5mm, F.Cu at (254.1, 73.4)
- C10, C2, C3, C4, C6, C8, C9, R6, R7: moved to B.Cu
- moved SW1 96.0 mm to (240.4, 103.1), turned to -90 degrees
- moved R6 93.6 mm to (240.4, 107.0), turned to -90 degrees
- moved R7 91.0 mm to (237.0, 113.6)
- moved C2 81.2 mm to (226.6, 88.2), turned to -90 degrees
- moved C6 75.1 mm to (214.8, 108.6), turned to -90 degrees
- moved C7 74.8 mm to (213.3, 113.2)
- moved C4 72.2 mm to (215.8, 98.1)
- moved J10 72.1 mm to (192.9, 66.3), turned to 180 degrees
- moved C9 70.6 mm to (211.3, 108.5), turned to -90 degrees
- moved C3 68.6 mm to (207.4, 104.1), turned to -90 degrees
- moved C8 55.1 mm to (192.9, 109.8), turned to 90 degrees
- moved C10 54.2 mm to (189.2, 109.8), turned to 90 degrees
- moved C11 45.1 mm to (194.3, 113.7)
- moved J6 40.1 mm to (226.3, 70.3), turned to 180 degrees
- moved J9 28.0 mm to (226.5, 78.8)
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- renumbered D to D1, D to D2, D to D3, D to D4
Connections:
- R6 pad 2: DIP2 -> DIP1
- R7 pad 2: DIP1 -> DIP2
- SW1 pad 7: DIP1 -> DIP2
- SW1 pad 8: DIP2 -> DIP1
Routing:
- net 5v: track 0.00 -> 77.0 mm, vias 0 -> 3
- net +12V: track 19.3 -> 83.5 mm, vias 0 -> 3
- net DIP1: track 0.00 -> 50.1 mm
- net DIP2: track 0.00 -> 46.5 mm
- net +5V: track 0.00 -> 26.5 mm
- net MOTOR1A: track 21.5 -> 33.2 mm
- net ST: track 0.00 -> 10.4 mm
- net Net-(U2-VCP): track 0.00 -> 10.1 mm
- net MOTOR1B: track 29.1 -> 37.4 mm
- net Net-(U1-VCP): track 0.00 -> 7.75 mm
- net Net-(D2-A): track 8.11 -> 2.35 mm
- net Net-(U1-CPL): track 8.11 -> 3.76 mm
- net Net-(J12-Pin_2): track 65.6 -> 61.6 mm
- net S1: track 18.9 -> 22.6 mm
- net S2: track 29.1 -> 32.6 mm
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
Commit message: almost done
Parts:
- removed SW1: SW_DIP_x04, JOEJOE:dip
- added SW3: SW_DIP_x02, JOEJOE:Dipswitch2, F.Cu at (233.9, 108.2)
- SW2: footprint JOEJOE:realswitch -> Connector_PinHeader_2.54mm:PinHeader_1x03_P2.54mm_Vertical
- moved J5 70.0 mm to (239.9, 107.2), turned to 0 degrees
- moved J10 41.6 mm to (190.8, 107.9)
- moved SW2 24.1 mm to (203.6, 87.1), turned to 180 degrees
- moved R6 23.0 mm to (225.0, 124.1)
- moved R7 12.0 mm to (226.6, 119.6)
- moved C8 10.0 mm to (201.6, 104.8), turned to -90 degrees
- moved C10 9.84 mm to (197.6, 104.7), turned to -90 degrees
Routing:
- net DIP1: track 50.1 -> 0.00 mm
- net DIP2: track 46.5 -> 0.00 mm
- net Net-(J5-Pin_2): track 0.00 -> 29.5 mm, vias 0 -> 1
- net Net-(J12-Pin_2): track 61.6 -> 36.2 mm
- net Net-(J10-Pin_1): track 0.00 -> 20.4 mm
- net Net-(J10-Pin_2): track 0.00 -> 16.9 mm
- net Net-(J5-Pin_1): track 0.00 -> 13.8 mm, vias 0 -> 1
- net +12V: track 83.5 -> 79.7 mm, vias 3 -> 2
- net MOTOR1B: track 37.4 -> 39.5 mm
- net MOTOR1A: track 33.2 -> 35.1 mm
- net S4: track 76.7 -> 75.3 mm
- net unconnected-(SW2A-C-Pad3): track 1.10 -> 0.00 mm
- net S3: track 67.1 -> 66.4 mm
- net 5v: track 77.0 -> 76.4 mm
- net Net-(D1-A): track 15.4 -> 15.2 mm, vias 0 -> 2

Commit message: DONE BUT IDK
Parts:
- moved R 15.9 mm to (232.8, 110.2), turned to 90 degrees
- moved ON 13.2 mm to (203.9, 73.8)
- moved R 12.8 mm to (235.3, 110.2), turned to 90 degrees
- moved J2 11.5 mm to (196.7, 98.2)
- moved J4 11.2 mm to (185.3, 98.2)
- moved R 10.9 mm to (183.2, 112.2), turned to -90 degrees
- moved R 9.86 mm to (184.1, 102.2), turned to 0 degrees
- moved D 8.77 mm to (188.8, 113.5), turned to 180 degrees
- moved D 8.71 mm to (183.3, 106.5), turned to 90 degrees
- moved C4 6.31 mm to (214.8, 104.3), turned to -90 degrees
- moved R 1.10 mm to (240.0, 102.1)
- moved R 0.95 mm to (245.9, 101.9)
- moved C7 0.43 mm to (212.9, 113.2)
- moved C5 0.28 mm to (217.4, 113.3)
- moved C9 0.06 mm to (211.4, 108.6)
- renumbered D4 to D, D1 to D, D2 to D, D3 to D, SW2 to ON, R2 to R, R4 to R, R3 to R, R1 to R, R7 to R, R6 to R
Connections:
- R pad 2: DIP2 -> DIP1
- R pad 2: DIP1 -> DIP2
- SW3 pad 3: DIP2 -> DIP1
- SW3 pad 4: DIP1 -> DIP2
- U1 pad 3: +5V -> 5v
- U1 pad 5: +5V -> 5v
- U2 pad 3: +5V -> 5v
- U2 pad 5: +5V -> 5v
Routing:
- net 5v: track 76.4 -> 152.9 mm, vias 3 -> 5
- net DIP1: track 0.00 -> 41.2 mm, vias 0 -> 2
- net DIP2: track 0.00 -> 36.7 mm, vias 0 -> 2
- net GND: track 1.37 -> 21.2 mm, vias 0 -> 2
- net Net-(J12-Pin_2): track 36.2 -> 16.6 mm
- net +12V: track 79.7 -> 95.3 mm
- net S4: track 75.3 -> 60.9 mm, vias 1 -> 0
- net +5V: track 26.5 -> 37.1 mm, vias 0 -> 2
- net MOTOR1B: track 39.5 -> 41.2 mm
- net MOTOR1A: track 35.1 -> 36.8 mm
- net S3: track 66.4 -> 64.7 mm, vias 0 -> 3
- net Net-(J10-Pin_1): track 20.4 -> 21.5 mm
- net Net-(J5-Pin_1): track 13.8 -> 14.7 mm
- net Net-(D3-A): track 3.82 -> 4.68 mm
- net Net-(D4-A): track 4.31 -> 3.50 mm
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Other:
- board text added: "+"
- board text added: "-"
- board text added: "0.022uF"
- board text added: "0.1uF"
- board text added: "D2"
- board text added: "D4"
- board text added: "D7"
- board text added: "D8"
- board text added: "Joe-i"
- board text added: "OFF"

Commit message: uwefhiqdanjkshbgvqrevfad
Parts:
- moved J6 1.70 mm to (226.2, 72.0)
Routing:
- net 5v: track 152.9 -> 151.2 mm
Changed lines of the file:
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@@
 		)
 		(property "Value" "180"
-			(at 0 1.65 360)
+			(at 0 1.65 0)
 			(layer "F.Fab")
 			(effects
@@
 		)
 		(fp_text user "${REFERENCE}"
-			(at 0 0 360)
+			(at 0 0 0)
 			(layer "F.Fab")
 			(effects
@@
 	(footprint "Connector_PinHeader_2.54mm:PinHeader_1x03_P2.54mm_Vertical"
 		(layer "F.Cu")
-		(at 226.35 70.275 180)
+		(at 226.225 71.975 180)
 		(descr "Through hole straight pin header, 1x03, 2.54mm pitch, single row")
 		(tags "Through hole pin header THT 1x03 2.54mm single row")
@@
 		)
 		(property "Value" "LED"
-			(at 0 1.82 360)
+			(at 0 1.82 0)
 			(layer "F.Fab")
 			(effects
@@
 		)
 		(fp_text user "${REFERENCE}"
-			(at 0 0 360)
+			(at 0 0 0)
 			(layer "F.Fab")
 			(effects
@@
 	)
 	(segment
+		(start 227.85 73.425)
+		(end 227.85 71.06)
+		(width 0.2)
+		(layer "F.Cu")
+		(net 4)
+	)
+	(segment
 		(start 227.65 110.075001)
 		(end 227.65 110.649999)
@@
 	)
 	(segment
-		(start 227.85 69.235)
-		(end 226.35 67.735)
+		(start 209.499999 109.674999)
+		(end 210.3 109.674999)
 		(width 0.2)
 		(layer "F.Cu")
@@
 	)
 	(segment
-		(start 209.499999 109.674999)
-		(end 210.3 109.674999)
+		(start 228.55 110.15)
+		(end 228.1 109.7)
 		(width 0.2)
 		(layer "F.Cu")
@@
 	)
 	(segment
-		(start 228.55 110.15)
-		(end 228.1 109.7)
+		(start 227.85 92.4)
+		(end 227.85 73.425)
 		(width 0.2)
 		(layer "F.Cu")
@@
 	)
 	(segment
+		(start 227.85 71.06)
+		(end 226.225 69.435)
+		(width 0.2)
+		(layer "F.Cu")
+		(net 4)
+	)
+	(segment
 		(start 227.65 92.6)
 		(end 227.85 92.4)
@@
 	)
 	(segment
-		(start 227.85 92.4)
-		(end 227.85 69.235)
-		(width 0.2)
-		(layer "F.Cu")
-		(net 4)
-	)
-	(segment
 		(start 232.68 112.8998)
 		(end 235.22 112.8998)
@@
 	)
 	(segment
-		(start 226.5 73.74)
+		(start 222.74 69.98)
+		(end 224.75 71.99)
+		(width 0.2)
+		(layer "F.Cu")
+		(net 24)
+	)
+	(segment
+		(start 224.75 77.025)
 		(end 226.5 78.775)
 		(width 0.2)
@@
 	)
 	(segment
-		(start 222.74 69.98)
-		(end 226.5 73.74)
+		(start 224.75 71.99)
+		(end 224.75 77.025)
 		(width 0.2)
 		(layer "F.Cu")

Commit message: almost done
Parts:
- removed C10, C11, C8, C9: 0.1uF, Capacitor_SMD:C_0805_2012Metric
- removed C12: 0.022uF, Capacitor_SMD:C_0805_2012Metric
- added C1: 10uF, Capacitor_SMD:C_0805_2012Metric, F.Cu at (221.6, 112.5)
- added R5: R_US, Resistor_SMD:R_0805_2012Metric, F.Cu at (207.7, 112.8)
- added R8: R_US, Resistor_SMD:R_0805_2012Metric, F.Cu at (202.1, 105.5)
- C5: value 0.022uF -> 10uF
- C6: value 0.1uF -> 10uF; moved to F.Cu
- C7: value 0.1uF -> 10uF
- R6, R7: renamed from R; moved to F.Cu
- U1, U2: value DRV8874PWPR -> DRV8871DDAR; footprint JOEJOE:DRV8874 -> Joe-ifootprints:DRV8871
- moved C7 19.4 mm to (194.4, 107.2), turned to 90 degrees
- moved C6 17.5 mm to (197.3, 107.2), turned to 90 degrees
- moved U1 10.4 mm to (213.1, 110.9), turned to 0 degrees
- moved R6 9.72 mm to (223.9, 106.1), turned to 0 degrees
- moved R1 7.48 mm to (246.1, 106.5), turned to -90 degrees
- moved R2 7.09 mm to (241.1, 96.7)
- moved R4 4.98 mm to (184.4, 97.3), turned to 180 degrees
- moved D2 4.93 mm to (247.3, 111.2)
- moved R7 4.30 mm to (236.2, 106.0)
- moved U2 4.28 mm to (202.4, 110.7)
- moved C4 3.58 mm to (214.7, 100.8)
- moved J1 2.98 mm to (228.7, 100.7)
- moved J3 2.90 mm to (240.0, 100.7)
- moved SW3 2.58 mm to (231.4, 108.8)
- moved J2 2.50 mm to (196.6, 100.7)
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- renumbered D to D1, D to D2, D to D3, D to D4, R to R1, R to R2, R to R3, R to R4, ON to SW2
Connections:
- C5 pad 1: Net-(U1-CPH) -> +12V
- C5 pad 2: Net-(U1-CPL) -> GND
- C7 pad 2: Net-(U1-VCP) -> GND
- R6 pad 2: DIP2 -> DIP1
- R7 pad 2: DIP1 -> DIP2
- SW3 pad 3: DIP1 -> DIP2
- SW3 pad 4: DIP2 -> DIP1
- U1 pad 1: MOTOR1A -> GND
- U1 pad 3: 5v -> MOTOR1A
- U1 pad 4: unconnected-(U1-FAULT_N-Pad4) -> Net-(U1-ILIM)
- U1 pad 5: 5v -> +12V
- U1 pad 6: unconnected-(U1-IPROPI-Pad6) -> Net-(J5-Pin_1)
- U1 pad 7: unconnected-(U1-IMODE-Pad7) -> GND
- U1 pad 8: Net-(J5-Pin_1) -> Net-(J5-Pin_2)
- U2 pad 1: MOTOR2A -> GND
- U2 pad 2: MOTOR2B -> MOTOR2A
- U2 pad 3: 5v -> MOTOR2B
- U2 pad 4: unconnected-(U2-FAULT_N-Pad4) -> Net-(U2-ILIM)
- U2 pad 5: 5v -> +12V
- U2 pad 6: unconnected-(U2-IPROPI-Pad6) -> Net-(J10-Pin_1)
- U2 pad 7: unconnected-(U2-IMODE-Pad7) -> GND
- U2 pad 8: Net-(J10-Pin_1) -> Net-(J10-Pin_2)
Routing:
- net 5v: track 151.2 -> 83.7 mm, vias 5 -> 1
- net +12V: track 95.3 -> 69.6 mm, vias 2 -> 0
- net Net-(J5-Pin_1): track 14.7 -> 28.2 mm, vias 1 -> 0
- net Net-(D2-A): track 2.98 -> 16.0 mm
- net Net-(J10-Pin_1): track 21.5 -> 10.9 mm
- net Net-(U2-VCP): track 10.1 -> 0.00 mm
- net S1: track 23.1 -> 32.7 mm
- net Net-(U1-VCP): track 8.20 -> 0.00 mm
- net Net-(U2-CPH): track 7.74 -> 0.00 mm
- net Net-(D1-A): track 14.7 -> 7.25 mm, vias 2 -> 0
- net GND: track 21.2 -> 14.6 mm, vias 2 -> 1
- net Net-(U2-CPL): track 5.89 -> 0.00 mm
- net Net-(U1-CPH): track 5.87 -> 0.00 mm
- net MOTOR2A: track 38.5 -> 43.9 mm
- net MOTOR2B: track 45.4 -> 50.4 mm
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Other:
- board text removed: "0.022uF"
- board text removed: "0.1uF"

Commit message: dicki
Parts:
- removed R7: 1k, Resistor_SMD:R_0805_2012Metric
- added D: LED, LED_SMD:LED_1206_3216Metric, F.Cu at (236.6, 102.1)
- added D: LED, LED_SMD:LED_1206_3216Metric, F.Cu at (225.7, 102.0)
- added D: LED, LED_SMD:LED_1206_3216Metric, F.Cu at (203.8, 82.9)
- added D: LED, LED_SMD:LED_1206_3216Metric, F.Cu at (204.0, 92.9)
- added R: 180, Resistor_SMD:R_0805_2012Metric, F.Cu at (203.8, 78.1)
- added R: 180, Resistor_SMD:R_0805_2012Metric, F.Cu at (203.9, 88.2)
- added R11: 180, Resistor_SMD:R_0805_2012Metric, F.Cu at (236.6, 106.8)
- R5: moved to B.Cu
- R6: value 1k -> 180
- moved R 5.57 mm to (246.6, 97.5), turned to -90 degrees
- moved R 5.42 mm to (246.7, 111.8)
- moved D 4.70 mm to (246.8, 106.5)
- moved R5 2.33 mm to (205.4, 113.2), turned to 180 degrees
- moved D 1.82 mm to (240.5, 113.5)
- moved R6 1.81 mm to (225.8, 106.1), turned to 90 degrees
- moved R 1.21 mm to (183.2, 97.6), turned to -90 degrees
- moved J12 0.83 mm to (214.7, 78.5)
- moved D 0.58 mm to (189.3, 113.5)
- moved D 0.30 mm to (183.7, 106.5)
- moved J5 0.29 mm to (242.3, 107.9)
- moved SW2 0.22 mm to (203.7, 73.8)
- renumbered D4 to D, D1 to D, D2 to D, D3 to D, R2 to R, R4 to R, R3 to R, R1 to R
Connections:
- R6 pad 1: GND -> DIP1
- R6 pad 2: DIP1 -> Net-(D8-A)
- TB1 pad 22: unconnected-(TB1-A3-Pad22) -> Led1
- TB1 pad 23: unconnected-(TB1-A4-Pad23) -> Led2
- U1 pad 2: MOTOR1B -> MOTOR1A
- U1 pad 3: MOTOR1A -> MOTOR1B
Routing:
- net GND: track 14.6 -> 95.0 mm, vias 1 -> 10
- net 5v: track 83.7 -> 133.9 mm, vias 1 -> 2
- net +12V: track 69.6 -> 90.6 mm, vias 0 -> 1
- net Net-(D2-A): track 16.0 -> 7.26 mm
- net DIP2: track 36.7 -> 43.7 mm
- net Led2: track 0.00 -> 6.15 mm
- net Led1: track 0.00 -> 5.61 mm
- net DIP1: track 38.0 -> 33.2 mm
- net S1: track 32.7 -> 37.2 mm
- net S2: track 31.6 -> 35.9 mm
- net Net-(D6-A): track 0.00 -> 2.53 mm
- net Net-(D5-A): track 0.00 -> 2.51 mm
- net Net-(D7-A): track 0.00 -> 2.40 mm
- net Net-(D1-A): track 7.25 -> 5.09 mm
- net S4: track 60.4 -> 62.3 mm
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Other:
- board text added: "0.1uF"
- board text added: "10uF"
- board text added: "30k"
- board text added: "47uF"
- board text added: "Dick-i"
- board text removed: "Joe-i"

Commit message: done with joei
Parts:
- added ?: , , F.Cu at (214.9, 66.5)
- added ?: , , F.Cu at (237.0, 96.7)
- added J11: Conn_01x04_Pin, Connector_PinHeader_2.54mm:PinHeader_1x04_P2.54mm_Vertical, F.Cu at (189.8, 97.3)
- C1, C5: moved to B.Cu
- C4: moved to F.Cu
- moved H1 74.7 mm to (195.2, 112.8)
- moved H2 49.1 mm to (224.9, 112.9)
- moved C1 3.80 mm to (218.8, 109.9), turned to 180 degrees
- moved D 0.97 mm to (203.0, 92.9)
- moved R 0.97 mm to (202.9, 88.2)
- moved R5 0.83 mm to (205.6, 112.4)
- moved D 0.50 mm to (203.3, 82.9)
- moved R 0.47 mm to (203.3, 78.1)
- moved D 0.43 mm to (225.8, 101.6)
- moved J6 0.33 mm to (226.3, 72.3)
- moved C5 0.31 mm to (218.8, 112.4), turned to 180 degrees
Connections:
- TB1 pad 12: MOTOR2B -> Servo
- TB1 pad 14: unconnected-(TB1-D11/MOSI-Pad14) -> MOTOR2B
- TB1 pad 21: unconnected-(TB1-A2-Pad21) -> Led1
- TB1 pad 22: Led1 -> Led2
- TB1 pad 23: Led2 -> SDA
- TB1 pad 24: unconnected-(TB1-A5-Pad24) -> SCL
Routing:
- net SDA: track 0.00 -> 22.8 mm, vias 0 -> 1
- net SCL: track 0.00 -> 19.0 mm, vias 0 -> 1
- net +5V: track 37.0 -> 55.0 mm, vias 2 -> 3
- net +12V: track 90.6 -> 85.3 mm, vias 1 -> 2
- net Led2: track 6.15 -> 11.2 mm
- net MOTOR2B: track 51.1 -> 55.5 mm, vias 1 -> 2
- net Servo: track 0.00 -> 3.65 mm
- net Led1: track 5.61 -> 4.38 mm
- net GND: track 95.0 -> 95.8 mm, vias 10 -> 9
- net Net-(J10-Pin_2): track 14.4 -> 15.0 mm
- net 5v: track 133.9 -> 133.3 mm, vias 2 -> 3
- net Net-(D8-A): track 1.88 -> 2.40 mm
Other:
- board text added: "-Joe Sung"
- board text added: "-Rudra Goel"
- board text added: "A"
- board text added: "B"
- board text added: "Joe-i"
- board text added: "O"
- board text removed: "Dick-i"

Commit message: added mounting hole measurements
Other:
- board text added: "Mounting Hole diameter 2.5mm"
