File: 500g/Ballsi/ballsi/ballsi.kicad_sch (KiCad schematic)
At the start: 4 parts, among them J1 Conn_01x03, J2 Conn_01x03, J3 Conn_01x03

Commit message: added microcontroller sensors and motordriver
Parts:
- added J1, J2: Conn_01x02, symbol Connector_Generic:Conn_01x02
- added L_LINE, R_IR1, R_LINE: Conn_01x03, Connector_JST:JST_PH_B3B-PH-K_1x03_P2.00mm_Vertical, symbol Connector_Generic:Conn_01x03
- added L_MOTOR_DRIVER, L_MOTOR_DRIVER1: DRV8871DDARQ1, DDA0008H_N_TEX, symbol DRV8871:DRV8871DDARQ1
- added R2, R3: 32kΩ, symbol Device:R
- renumbered J1 to L_IR, J2 to M_IR, J3 to R_IR
Connections:
- net R_IN1: now reaches A1.12 (D9)
- net R_IN1: now also L_MOTOR_DRIVER1.3 (IN1)
- net R_IN2: now reaches A1.13 (D10)
- net R_IN2: now also L_MOTOR_DRIVER1.2 (IN2)
- net START_MOD: now reaches A1.15 (D12)
- net START_MOD: now also R_IR1.3 (Pin_3)
- net +3V3: now reaches A1.17 (3V3)
- net L_LINE: now reaches A1.19 (A0)
- net L_LINE: now also L_LINE.1 (Pin_1)
- net R_LINE: now reaches A1.20 (A1)
- net R_LINE: now also R_LINE.1 (Pin_1)
- net +5V: now reaches A1.27 (+5V)
- net +5V: now also L_IR.2 (Pin_2), M_IR.2 (Pin_2), R_IR.2 (Pin_2), L_LINE.2 (Pin_2), R_IR1.1 (Pin_1), R_LINE.2 (Pin_2)
- net GND: now reaches A1.29 (GND)
- net GND: now also A1.4 (GND), L_IR.3 (Pin_3), M_IR.3 (Pin_3), R_IR.3 (Pin_3), L_LINE.3 (Pin_3), L_MOTOR_DRIVER.1 (GND), L_MOTOR_DRIVER.7 (PGND), L_MOTOR_DRIVER.9 (PAD), L_MOTOR_DRIVER1.1 (GND), L_MOTOR_DRIVER1.7 (PGND), L_MOTOR_DRIVER1.9 (PAD), R2.2, R3.2, R_IR1.2 (Pin_2), R_LINE.3 (Pin_3)
- net +12V: now reaches A1.30 (VIN)
- net +12V: now also L_MOTOR_DRIVER.5 (VM), L_MOTOR_DRIVER1.5 (VM)
- net M_IR: now reaches A1.5 (D2)
- net M_IR: now also M_IR.1 (Pin_1)
- net L_IR: now reaches A1.6 (D3)
- net L_IR: now also L_IR.1 (Pin_1)
- net R_IR: now reaches A1.7 (D4)
- net R_IR: now also R_IR.1 (Pin_1)
- net L_IN1: now reaches A1.8 (D5)
- net L_IN1: now also L_MOTOR_DRIVER.3 (IN1)
- net L_IN2: now reaches A1.9 (D6)
- net L_IN2: now also L_MOTOR_DRIVER.2 (IN2)
- new net: L_MOTOR_DRIVER1.4 (ILIM), R2.1
- new net: J2.2 (Pin_2), L_MOTOR_DRIVER1.6 (OUT1)
- new net: J2.1 (Pin_1), L_MOTOR_DRIVER1.8 (OUT2)
- new net: L_MOTOR_DRIVER.4 (ILIM), R3.1
- new net: J1.1 (Pin_1), L_MOTOR_DRIVER.8 (OUT2)
- new net: J1.2 (Pin_2), L_MOTOR_DRIVER.6 (OUT1)
Other:
- moved on the sheet: A1, L_IR, M_IR, R_IR

Commit message: finished schematic
Parts:
- removed R_IR1: Conn_01x03, Connector_JST:JST_PH_B3B-PH-K_1x03_P2.00mm_Vertical, symbol Connector_Generic:Conn_01x03
- added C1: 0.1uF, symbol Device:C
- added F1: 5A, symbol Device:Fuse
- added K1: G6DN-1A-SL DC12, RELAY_G6DN-1A_OMR, symbol G6DN-1A-SL-DC12:G6DN-1A-SL_DC12
- added Power: Conn_01x02, symbol Connector_Generic:Conn_01x02
- added R4, R5: 10kΩ, symbol Device:R
- added START_MOD: Conn_01x04, symbol Connector_Generic:Conn_01x04
- added SW: SW_SPST, symbol Switch:SW_SPST
- added SW_DIP: SW_DIP_x02, symbol Switch:SW_DIP_x02
Connections:
- net +12V: now also C1.1, F1.1, K1.5; no longer L_MOTOR_DRIVER.5 (VM), L_MOTOR_DRIVER1.5 (VM)
- net +5V: now also R4.1, R5.1, START_MOD.1 (Pin_1)
- net GND: now also C1.2, K1.2, Power.2 (Pin_2), START_MOD.2 (Pin_2), SW_DIP.1, SW_DIP.2
- net START_MOD: now also K1.1, START_MOD.3 (Pin_3)
- net DIP1: now reaches A1.10 (D7)
- net DIP1: now also R4.2, SW_DIP.4
- net DIP2: now reaches A1.11 (D8)
- net DIP2: now also R5.2, SW_DIP.3
- new net: F1.2, SW.1 (A)
- new net: Power.1 (Pin_1), SW.2 (B)
- new net MOTOR_PWR: K1.8, L_MOTOR_DRIVER.5 (VM), L_MOTOR_DRIVER1.5 (VM)
Other:
- moved on the sheet: L_IR, L_LINE, M_IR, R_IR, R_LINE

Commit message: updated everything
Parts:
- removed SW: SW_SPST, symbol Switch:SW_SPST
- added C2, C3, C4, C5: 10uF, Capacitor_SMD:C_1206_3216Metric_Pad1.33x1.80mm_HandSolder, symbol Device:C
- added SW1: 1101M2S3CQE2, 1101M2S3CQE2:SW_1101M2S3CQE2, symbol 1101M2S3CQE2:1101M2S3CQE2
- C1: footprint (none) -> Capacitor_SMD:C_1206_3216Metric_Pad1.33x1.80mm_HandSolder
- F1: footprint (none) -> Fuse:Fuse_1206_3216Metric_Pad1.42x1.75mm_HandSolder
- J1, J2: footprint (none) -> Connector_PinSocket_2.54mm:PinSocket_1x02_P2.54mm_Vertical
- K1: footprint RELAY_G6DN-1A_OMR -> G6DN-1A-SL:RELAY_G6DN-1A_OMR
- L_IR1: renamed from L_IR; footprint Connector_JST:JST_PH_B3B-PH-K_1x03_P2.00mm_Vertical -> Connector_PinSocket_2.54mm:PinSocket_1x03_P2.54mm_Vertical
- L_LINE1: renamed from L_LINE; footprint Connector_JST:JST_PH_B3B-PH-K_1x03_P2.00mm_Vertical -> Connector_PinSocket_2.54mm:PinSocket_1x03_P2.54mm_Vertical
- L_MOTOR_DRIVER1: renamed from L_MOTOR_DRIVER; footprint DDA0008H_N_TEX -> DRV8871:DDA0008H_N_TEX
- M_IR1: renamed from M_IR; footprint Connector_JST:JST_PH_B3B-PH-K_1x03_P2.00mm_Vertical -> Connector_PinSocket_2.54mm:PinSocket_1x03_P2.54mm_Vertical
- Power1: renamed from Power; footprint (none) -> Connector_AMASS:AMASS_XT30U-F_1x02_P5.0mm_Vertical
- R2, R3, R4, R5: footprint (none) -> Resistor_SMD:R_1206_3216Metric_Pad1.30x1.75mm_HandSolder
- R_IR1: renamed from R_IR; footprint Connector_JST:JST_PH_B3B-PH-K_1x03_P2.00mm_Vertical -> Connector_PinSocket_2.54mm:PinSocket_1x03_P2.54mm_Vertical
- R_LINE1: renamed from R_LINE; footprint Connector_JST:JST_PH_B3B-PH-K_1x03_P2.00mm_Vertical -> Connector_PinSocket_2.54mm:PinSocket_1x03_P2.54mm_Vertical
- R_MOTOR_DRIVER1: renamed from L_MOTOR_DRIVER1; footprint DDA0008H_N_TEX -> DRV8871:DDA0008H_N_TEX
- START_MOD1: renamed from START_MOD; footprint (none) -> Connector_PinHeader_2.54mm:PinHeader_1x04_P2.54mm_Vertical
- SW_DIP1: renamed from SW_DIP; footprint (none) -> 418117270902:418117270902
Connections:
- net +5V: now also SW_DIP1.1, SW_DIP1.2; no longer R4.1, R5.1
- net GND: now also Power1.1 (Pin_1), R4.1, R5.1, C2.2, C3.2, C4.2, C5.2; no longer Power1.2 (Pin_2), SW_DIP1.1, SW_DIP1.2
- net L_IR: now also A1.5 (D2); no longer A1.6 (D3)
- net MOTOR_PWR: now also C2.1, C3.1, C4.1, C5.1
- net M_IR: now also A1.6 (D3); no longer A1.5 (D2)
- net at F1.2: now also SW1.2
- new net: Power1.2 (Pin_2), SW1.1
- no-connect marks 0 -> 14
Other:
- note added: "Dipswitch"
- note added: "IR Sensors"
- note added: "Line Sensors"
- note added: "MicroController"
- note added: "Motor Drivers"
- note added: "Power Input"
- note added: "Relay"
- note added: "Start Module"
- moved on the sheet: F1, Power1

Commit message: finished v2s
Parts:
- added D1: D, Diode_SMD:D_1206_3216Metric_Pad1.42x1.75mm_HandSolder, symbol Device:D
- added Q1: BC549, Package_TO_SOT_THT:TO-92_Inline, symbol Transistor_BJT:BC549
- added R1, R6: R, Resistor_SMD:R_1206_3216Metric_Pad1.30x1.75mm_HandSolder, symbol Device:R
- C2, C4: value 10uF -> 50uF
- R2, R3: value 32kΩ -> 24kΩ
Connections:
- net +5V: now also R6.1
- net GND: now also Q1.3 (E); no longer K1.2
- net START_MOD: no longer K1.1
- net Kill_Switch: now reaches START_MOD1.4 (Pin_4)
- net Kill_Switch: now also A1.14 (D11), R1.1
- new net: D1.2 (A), K1.2, Q1.1 (C)
- new net: Q1.2 (B), R1.2
- new net: D1.1 (K), K1.1, R6.2
- no-connect marks 14 -> 13
Other:
- moved on the sheet: K1
