File: 500g/Sp-I/Sp-I.kicad_pcb (KiCad board)
At the start: 2 copper layers, 95 x 30 mm, 14 parts, among them IC1 TEENSY_4.1, J1 Left IR, J2 Middle IR, J3 Right IR, J4 Conn_01x04, J5 Left Line Sensor, J6 Right Line Sensor, J7 Right Motor Driver, J8 Left Motor Driver, J9 Conn_01x02, U1 TSR 1-2450

Commit message: wired pcb
Parts:
- moved IC1 137.6 mm to (184.8, 127.0), turned to 180 degrees
- moved J7 66.6 mm to (157.5, 144.0), turned to 180 degrees
- moved F1 56.9 mm to (111.5, 139.0)
- moved C6 54.1 mm to (111.5, 144.0), turned to 180 degrees
- moved J9 52.4 mm to (106.0, 144.0), turned to 90 degrees
- moved J1 49.9 mm to (144.9, 125.5), turned to -90 degrees
- moved J2 49.2 mm to (140.1, 138.5), turned to 90 degrees
- moved J4 48.3 mm to (115.9, 145.5), turned to 90 degrees
- moved U1 44.9 mm to (108.5, 131.5), turned to 90 degrees
- moved J3 44.3 mm to (149.5, 129.5), turned to 90 degrees
- moved MT1 43.4 mm to (170.5, 134.5), turned to 180 degrees
- moved J5 42.5 mm to (145.0, 143.1)
- moved J6 40.6 mm to (149.5, 138.5), turned to 90 degrees
- moved J8 38.7 mm to (137.0, 126.1)
Connections:
- IC1 pad 1: unconnected-(IC1-TX1-Pad1) -> Kill_Switch
- IC1 pad 22: unconnected-(IC1-A8-Pad22) -> Left_Line
- IC1 pad 23: unconnected-(IC1-A9-Pad23) -> Right_Line
- IC1 pad 5: Start_Module -> DIR_L
- IC1 pad 53: unconnected-(IC1-3.3V_(250_M_A_MAX)-Pad53) -> +3.3V
- IC1 pad 57: unconnected-(IC1-RX1-Pad57) -> Start_Module
- IC1 pad 6: Kill_Switch -> PWM_L
- IC1 pad 7: DIR_L -> DIR_R
- IC1 pad 70: unconnected-(IC1-GND_5-Pad70) -> GND
- IC1 pad 8: PWM_L -> PWM_R
Routing:
- net +3.3V: track 0.00 -> 132.5 mm
- net 5V: track 0.00 -> 101.4 mm
- net Start_Module: track 0.00 -> 81.9 mm
- net Kill_Switch: track 0.00 -> 78.5 mm
- net Middle_IR: track 0.00 -> 49.4 mm
- net Left_IR: track 0.00 -> 44.5 mm
- net DIR_L: track 0.00 -> 42.0 mm
- net Right_Line: track 0.00 -> 41.3 mm
- net PWM_L: track 0.00 -> 40.1 mm
- net Left_Line: track 0.00 -> 33.5 mm
- net Right_IR: track 0.00 -> 31.2 mm
- net DIR_R: track 0.00 -> 19.4 mm
- net PWM_R: track 0.00 -> 15.9 mm
- net Net-(U1-+VIN): track 0.00 -> 9.02 mm
- net SDA: track 0.00 -> 7.63 mm, vias 0 -> 1
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
Commit message: finished?
Parts:
- moved J2 6.72 mm to (145.4, 134.5), turned to -90 degrees
- moved J1 0.55 mm to (145.5, 125.5)
Routing:
- net GND: track 0.00 -> 21.5 mm, vias 0 -> 1
- net Middle_IR: track 49.4 -> 50.0 mm
- net +3.3V: track 132.5 -> 132.0 mm
- added copper zone on B.Cu, net GND
- added copper zone on F.Cu, net GND
Other:
- board text added: "Xander Riddle"

Commit message: idk changes
Parts:
- added REF**: MountingHole_3mm_Pad, MountingHole:MountingHole_3mm_Pad, F.Cu at (121.5, 124.5)
- added REF**: MountingHole_3mm_Pad, MountingHole:MountingHole_3mm_Pad, F.Cu at (190.5, 134.5)
- moved J1 3.21 mm to (142.4, 124.5)
- moved J2 2.95 mm to (142.5, 134.5)
- moved J3 2.74 mm to (152.1, 128.5)
- moved J6 2.55 mm to (152.1, 138.5)
- moved J5 1.50 mm to (145.0, 144.6)
Routing:
- net +3.3V: track 132.0 -> 89.6 mm
- net Middle_IR: track 50.0 -> 30.5 mm
- net Right_Line: track 41.3 -> 27.6 mm
- net PWM_L: track 40.1 -> 28.5 mm
- net Left_IR: track 44.2 -> 33.3 mm
- net DIR_L: track 42.0 -> 33.4 mm
- net Right_IR: track 31.2 -> 26.2 mm
- net Left_Line: track 33.5 -> 29.3 mm
- removed copper zone on B.Cu, net GND
- removed copper zone on F.Cu, net GND

Commit message: finished v2s
Parts:
- removed C6: 0.1uF, Capacitor_SMD:C_0805_2012Metric_Pad1.18x1.45mm_HandSolder
- removed F1: Fuse, MFU0603FF01000P500:FUS_VISHAY_MFU0603_VIS
- removed J1: Left IR, Connector_JST:JST_PH_S3B-PH-K_1x03_P2.00mm_Horizontal
- removed J2: Middle IR, Connector_JST:JST_PH_S3B-PH-K_1x03_P2.00mm_Horizontal
- removed J3: Right IR, Connector_JST:JST_PH_S3B-PH-K_1x03_P2.00mm_Horizontal
- removed J5: Left Line Sensor, Connector_JST:JST_PH_S3B-PH-K_1x03_P2.00mm_Horizontal
- removed J6: Right Line Sensor, Connector_JST:JST_PH_S3B-PH-K_1x03_P2.00mm_Horizontal
- removed J8: Left Motor Driver, Connector_PinHeader_2.54mm:PinHeader_1x08_P2.54mm_Vertical
- removed J9: Conn_01x02, Connector_AMASS:AMASS_XT30U-F_1x02_P5.0mm_Vertical
- removed MT1: ICM-42670-P, ICM_42670_P:XDCR_ICM-42670-P
- removed the REF** at (121.5, 124.5)
- removed the REF** at (190.5, 134.5)
- added 0.1uF: 0.1uF, Capacitor_SMD:C_1206_3216Metric_Pad1.33x1.80mm_HandSolder, F.Cu at (151.0, 135.8)
- added 0.1uF: 0.1uF, Capacitor_SMD:C_1206_3216Metric_Pad1.33x1.80mm_HandSolder, F.Cu at (136.8, 135.8)
- added 0.1uF: 0.1uF, Capacitor_SMD:C_1206_3216Metric_Pad1.33x1.80mm_HandSolder, F.Cu at (134.2, 135.8)
- added 10kΩ: 10kΩ, Resistor_SMD:R_1206_3216Metric_Pad1.30x1.75mm_HandSolder, F.Cu at (115.2, 124.2)
- added 10kΩ: 10kΩ, Resistor_SMD:R_1206_3216Metric_Pad1.30x1.75mm_HandSolder, F.Cu at (115.2, 126.8)
- added 18kΩ: 18kΩ, Resistor_SMD:R_1206_3216Metric_Pad1.30x1.75mm_HandSolder, F.Cu at (151.0, 142.8)
- added 18kΩ: 18kΩ, Resistor_SMD:R_1206_3216Metric_Pad1.30x1.75mm_HandSolder, F.Cu at (148.5, 142.8)
- added 1A: Fuse, Fuse:Fuse_1206_3216Metric_Pad1.42x1.75mm_HandSolder, F.Cu at (149.8, 122.2)
- added 1kΩ: R, Resistor_SMD:R_1206_3216Metric_Pad1.30x1.75mm_HandSolder, F.Cu at (148.5, 135.8)
- added 50uF: 50uF, Capacitor_SMD:C_1206_3216Metric_Pad1.33x1.80mm_HandSolder, F.Cu at (141.8, 135.8)
- added 50uF: 50uF, Capacitor_SMD:C_1206_3216Metric_Pad1.33x1.80mm_HandSolder, F.Cu at (139.2, 135.8)
- added <: D, Diode_SMD:D_1206_3216Metric_Pad1.42x1.75mm_HandSolder, F.Cu at (146.0, 135.8)
- added G***: LOGO, spy:spy23inverted, F.Cu at (112.8, 137.9)
- added K1: G6DN-1A-SL DC12, ul_G6DN-1A-SL-DC12:RELAY_G6DN-1A_OMR, F.Cu at (160.3, 127.7)
- added L_IR: Left IR, Connector_PinSocket_2.54mm:PinSocket_1x03_P2.54mm_Vertical, F.Cu at (115.8, 140.8)
- added L_Line: Left Line Sensor, Connector_PinSocket_2.54mm:PinSocket_1x03_P2.54mm_Vertical, F.Cu at (106.8, 140.8)
- added L_MTR: Left Motor, Connector_PinSocket_2.54mm:PinSocket_1x02_P2.54mm_Vertical, F.Cu at (124.8, 140.7)
- added L_MTR_DRV: DRV8871DDARQ1, DRV8871DDARQ1:DDA0008H_N_TEX, F.Cu at (156.8, 139.1)
- added M_IR: Middle IR, Connector_PinSocket_2.54mm:PinSocket_1x03_P2.54mm_Vertical, F.Cu at (131.2, 140.8)
- added Q2: BC549, Package_TO_SOT_THT:TO-92_Inline, F.Cu at (138.5, 127.8)
- added R6: R, Resistor_SMD:R_1206_3216Metric_Pad1.30x1.75mm_HandSolder, F.Cu at (146.0, 142.8)
- added REF**: MountingHole_3mm, MountingHole:MountingHole_3mm, F.Cu at (105.2, 125.2)
- added REF**: MountingHole_3mm, MountingHole:MountingHole_3mm, F.Cu at (189.8, 125.2)
- added R_IR: Right IR, Connector_PinSocket_2.54mm:PinSocket_1x03_P2.54mm_Vertical, F.Cu at (174.2, 140.8)
- added R_Line: Right Line Sensor, Connector_PinSocket_2.54mm:PinSocket_1x03_P2.54mm_Vertical, F.Cu at (183.2, 140.8)
- added R_MTR: Right Motor, Connector_PinSocket_2.54mm:PinSocket_1x02_P2.54mm_Vertical, F.Cu at (167.7, 140.7)
- added R_MTR_DRV: DRV8871DDARQ1, DRV8871DDARQ1:DDA0008H_N_TEX, F.Cu at (162.8, 139.1)
- added SW3: 1101M2S3CQE2, 1101M2S3CQE2:SW_1101M2S3CQE2, F.Cu at (124.5, 124.2)
- added SW_DIP1: SW_DIP_x02, 418117270902:418117270902, F.Cu at (127.6, 133.5)
- IC1: footprint TEENSY_4.1:TEENSY41 -> Teensy4:TEENSY41
- J4: value Conn_01x04 -> Start Module
- J7: value Right Motor Driver -> Conn_01x02; footprint Connector_PinHeader_2.54mm:PinHeader_1x08_P2.54mm_Vertical -> Connector_AMASS:AMASS_XT30U-F_1x02_P5.0mm_Vertical
- U1: footprint footprints:TSR1-SINGLE_TRP -> TSR_1_2450:TSR1-SINGLE_TRP
- moved U1 57.0 mm to (165.3, 127.0), turned to 0 degrees
- moved J7 31.5 mm to (182.2, 124.5)
- moved J4 18.1 mm to (104.4, 131.5)
- moved IC1 5.27 mm to (187.0, 131.8)
Connections:
- net 5V renamed +5V
- IC1 pad 18: SDA -> unconnected-(IC1-A4-Pad18)
- IC1 pad 19: SCL -> unconnected-(IC1-A5-Pad19)
- IC1 pad 20: unconnected-(IC1-A6-Pad20) -> DIP1
- IC1 pad 21: unconnected-(IC1-A7-Pad21) -> DIP2
- IC1 pad 5: DIR_L -> L_IN2
- IC1 pad 6: PWM_L -> L_IN1
- IC1 pad 7: DIR_R -> R_IN1
- IC1 pad 71: unconnected-(IC1-GND_6-Pad71) -> GND
- IC1 pad 8: PWM_R -> R_IN2
- J7 pad 2: DIR_R -> Net-(J7-Pin_2)
Routing:
- net DIP2: track 0.00 -> 117.8 mm
- net DIP1: track 0.00 -> 111.8 mm
- net +3.3V: track 89.6 -> 154.0 mm, vias 0 -> 1
- net Net-(J7-Pin_2): track 0.00 -> 60.8 mm
- net MOTOR_PWR: track 0.00 -> 47.6 mm
- net Net-(D1-A): track 0.00 -> 45.8 mm
- net Left_Line: track 29.3 -> 73.7 mm
- net Left_IR: track 33.3 -> 73.0 mm
- net Net-(J9-Pin_1): track 0.00 -> 38.3 mm, vias 0 -> 1
- net +12V: track 0.00 -> 34.4 mm
- net +5V: track 101.4 -> 67.5 mm, vias 0 -> 2
- net DIR_L: track 33.4 -> 0.00 mm
- net Net-(J9-Pin_2): track 4.82 -> 37.7 mm, vias 0 -> 1
- net Net-(Q2-B): track 0.00 -> 30.6 mm
- net L_IN2: track 0.00 -> 28.6 mm, vias 0 -> 1
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- added copper zone on B.Cu, net GND
- added copper zone on F.Cu, net GND
Other:
- board text added: "+"
- board text added: "-"
- board text added: "1kΩ"
- board text added: "D"
- board text added: "Xander Riddle 5/12/2025"
- board text added: "k"
- board text added: "s"
- board text removed: "Xander Riddle"
