File: 3kg/Ferrarii/CustomML2/CustomML2.kicad_pcb (KiCad board)
At the start: 2 copper layers, 10 x 22 mm, 9 parts, among them J1 some 4 hole connector idk, U1 QRE1113GR, U2 QRE1113GR

Commit message: ml2 push for xandie wandie
Other:
- board text added: "HUH"
Changed lines of the file:
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@@
 		(layer "Edge.Cuts")
+	)
+	(gr_text "HUH"
+		(at 79.5 40 0)
+		(layer "F.SilkS")
+		(effects
+			(font
+				(size 1 1)
+				(thickness 0.1)
+			)
+			(justify left bottom)
+		)
 	)
 	(gr_text "bruh moment"

Commit message: custom ml2 update for xandie wandie, moved resistors to same side as sensor and removed notches from screw hole
Parts:
- removed REF** (x2): MountingHole_3.2mm_M3, MountingHole:MountingHole_3.2mm_M3
- J1: footprint Connector:FanPinHeader_1x04_P2.54mm_Vertical -> Connector_PinHeader_2.54mm:PinHeader_1x04_P2.54mm_Vertical
- R1, R2, R3, R4: footprint Resistor_SMD:R_0805_2012Metric_Pad1.20x1.40mm_HandSolder -> Resistor_SMD:R_0201_0603Metric_Pad0.64x0.40mm_HandSolder; moved to F.Cu
- moved U2 23.9 mm to (46.0, 43.0), turned to -90 degrees
- moved U1 23.2 mm to (46.0, 36.5), turned to -90 degrees
- moved J1 23.0 mm to (41.0, 35.9), turned to 0 degrees
- moved R2 22.3 mm to (43.4, 39.7), turned to 90 degrees
- moved R4 20.6 mm to (45.0, 39.8)
- moved R3 18.9 mm to (46.8, 39.8), turned to -90 degrees
- moved R1 17.5 mm to (48.5, 39.8)
Routing:
- net 3.3V: track 17.6 -> 10.2 mm
- net Net-(R1-Pad1): track 4.93 -> 2.16 mm, vias 1 -> 0
- net Net-(R3-Pad1): track 4.45 -> 6.85 mm, vias 1 -> 0
- net Signal2: track 8.75 -> 6.96 mm, vias 1 -> 0
- net Signal1: track 5.44 -> 5.81 mm, vias 1 -> 0
- net GND: vias 0 -> 3
Other:
- outline, holes or cut-outs redrawn
- board text added: "220"
- board text added: "3.3V"
- board text added: "47k"
- board text added: "GND"
- board text added: "Signal 1"
- board text added: "Signal 2"
- board text added: "When opportunity doesn't knock, build a door."
- board text removed: "HUH"
- board text removed: "bruh moment"
