File: 3kg/Ferrarii/Ferrarii/Ferrarii.kicad_pcb (KiCad board)
At the start: 2 copper layers, 101 parts, among them J1 Encoder_Left, J10 MD, J11 LCD_Screen, J12 DS_45R, J13 DS_60R, J14 DS_90R, J15 DS_FR, J16 LS_LF1, J17 LS_RF1, J18 LS_BL1, J19 LS_BR1, J2 Encoder_Right, J20 LS_PlowLeft, J21 LS_PlowMid, J22 12v, J23 LS_LF2, J24 LS_RF2, J25 LS_BL2, J26 LS_BR2, J27 LS_PlowRight, J28 12v, J3 DS_FL, J4 Start Module, J5 12vPower, J6 DS_45L, J7 DS_60L, J8 DS_90L, J9 DS_Mid, Q1 LTV-826S, Q2 LTV-826S, Q3 LTV-826S, Q4 LTV-826S, Q5 LTV-826S, SW1 219-3LPSTR, SW2 SW_SPST, U1 DEV-16771

Commit message: ferrarii stuff placed, not wired
Parts:
- removed SW2: SW_SPST, GF-123-0054:SW_GF-123-0054
- C1, C13, C14, C15, C16, C17, C18, C19, C2, C20, C21, C22, C23, C24, C25, C26, C4, C5, C9, Q1, Q2, Q3, Q4, Q5, R21, R22, R23, R24, R25, R27, R28, R29, R30, R32: moved to B.Cu
- J16, J17, J18, J19, J20, J21, J23, J24, J25, J26, J27: footprint Connector_JST:JST_PH_S3B-PH-K_1x03_P2.00mm_Horizontal -> Connector_PinHeader_2.54mm:PinHeader_1x03_P2.54mm_Vertical
- moved J13 214.6 mm to (222.5, 74.0), turned to -90 degrees
- moved J14 214.4 mm to (222.4, 83.2), turned to -90 degrees
- moved J4 210.7 mm to (189.2, 128.4), turned to 180 degrees
- moved J12 210.1 mm to (218.0, 64.3)
- moved J19 200.9 mm to (198.0, 128.5), turned to 180 degrees
- moved J17 197.3 mm to (209.5, 69.2), turned to 180 degrees
- moved J26 195.5 mm to (201.8, 128.5), turned to 180 degrees
- moved J24 191.3 mm to (213.5, 69.2), turned to 180 degrees
- moved J9 189.6 mm to (191.8, 64.3)
- moved J2 189.5 mm to (214.5, 128.4), turned to 180 degrees
- moved J15 189.3 mm to (201.0, 64.3)
- moved J3 185.2 mm to (182.5, 64.3)
- moved U1 180.2 mm to (181.5, 108.6)
- moved J18 178.6 mm to (165.2, 128.5), turned to 180 degrees
- moved F1 175.7 mm to (221.5, 115.0)
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- renumbered SW1 to dip
Connections:
- F1 pad 2: Net-(SW2-B) -> +12V
Routing:
- net +3.3V: track 0.00 -> 10.2 mm
Other:
- board outline added: 75 x 71 mm

Commit message: added footprints, fixed schematic
Parts:
- removed C1, C10, C11, C12, C13, C14, C15, C16, C17, C18, C19, C2, C20, C21, C22, C23, C24, C25, C26, C3, C4, C5, C6, C7, C8, C9: 0.1uF, Capacitor_SMD:C_0805_2012Metric_Pad1.18x1.45mm_HandSolder
- removed D1, D2, D3, D4, D5, D6, D7, D8, D9: LED, LED_SMD:LED_0805_2012Metric_Pad1.15x1.40mm_HandSolder
- removed F1: Fuse, C1F-1:FUSC3215X83N
- removed J1: Encoder_Left, Connector_JST:JST_PH_S5B-PH-K_1x05_P2.00mm_Horizontal
- removed J10: MD, Connector_PinHeader_2.54mm:PinHeader_1x02_P2.54mm_Vertical
- removed J11: LCD_Screen, Connector_JST:JST_PH_S4B-PH-K_1x04_P2.00mm_Horizontal
- removed J12: DS_45R, Connector_JST:JST_PH_S3B-PH-K_1x03_P2.00mm_Horizontal
- removed J13: DS_60R, Connector_JST:JST_PH_S3B-PH-K_1x03_P2.00mm_Horizontal
- removed J14: DS_90R, Connector_JST:JST_PH_S3B-PH-K_1x03_P2.00mm_Horizontal
- removed J15: DS_FR, Connector_JST:JST_PH_S3B-PH-K_1x03_P2.00mm_Horizontal
- removed J16: LS_LF1, Connector_PinHeader_2.54mm:PinHeader_1x03_P2.54mm_Vertical
- removed J17: LS_RF1, Connector_PinHeader_2.54mm:PinHeader_1x03_P2.54mm_Vertical
- removed J18: LS_BL1, Connector_PinHeader_2.54mm:PinHeader_1x03_P2.54mm_Vertical
- removed J19: LS_BR1, Connector_PinHeader_2.54mm:PinHeader_1x03_P2.54mm_Vertical
- removed J2: Encoder_Right, Connector_JST:JST_PH_S5B-PH-K_1x05_P2.00mm_Horizontal
- removed J20: LS_PlowLeft, Connector_PinHeader_2.54mm:PinHeader_1x03_P2.54mm_Vertical
- removed J21: LS_PlowMid, Connector_PinHeader_2.54mm:PinHeader_1x03_P2.54mm_Vertical
- removed J22, J28: 12v, Connector_AMASS:AMASS_XT30U-F_1x02_P5.0mm_Vertical
- removed J23: LS_LF2, Connector_PinHeader_2.54mm:PinHeader_1x03_P2.54mm_Vertical
- removed J24: LS_RF2, Connector_PinHeader_2.54mm:PinHeader_1x03_P2.54mm_Vertical
- removed J25: LS_BL2, Connector_PinHeader_2.54mm:PinHeader_1x03_P2.54mm_Vertical
- removed J26: LS_BR2, Connector_PinHeader_2.54mm:PinHeader_1x03_P2.54mm_Vertical
- removed J27: LS_PlowRight, Connector_PinHeader_2.54mm:PinHeader_1x03_P2.54mm_Vertical
- removed J3: DS_FL, Connector_JST:JST_PH_S3B-PH-K_1x03_P2.00mm_Horizontal
- removed J4: Start Module, Connector_JST:JST_PH_S3B-PH-K_1x03_P2.00mm_Horizontal
- removed J5: 12vPower, Connector_AMASS:AMASS_XT30U-F_1x02_P5.0mm_Vertical
- removed J6: DS_45L, Connector_JST:JST_PH_S3B-PH-K_1x03_P2.00mm_Horizontal
- removed J7: DS_60L, Connector_JST:JST_PH_S3B-PH-K_1x03_P2.00mm_Horizontal
- removed J8: DS_90L, Connector_JST:JST_PH_S3B-PH-K_1x03_P2.00mm_Horizontal
- removed J9: DS_Mid, Connector_JST:JST_PH_S3B-PH-K_1x03_P2.00mm_Horizontal
- removed PS1: TSR_1-2450, TSR_1-2450:CONV_TSR_1-2450
- removed Q1, Q2, Q3, Q4, Q5: LTV-826S, LTV826:DIL8-SMD
- removed R1, R2, R4, R5, R6, R7: 2.7k, Resistor_SMD:R_0805_2012Metric_Pad1.20x1.40mm_HandSolder
- removed R12, R13, R14, R15, R16, R17, R18, R19, R20, R23, R24, R25, R26, R27, R28, R29, R30, R32: 500, Resistor_SMD:R_0805_2012Metric_Pad1.20x1.40mm_HandSolder
- removed R21, R22, R3: 10k, Resistor_SMD:R_0805_2012Metric_Pad1.20x1.40mm_HandSolder
- removed U1: DEV-16771, DEV-16771:MODULE_DEV-16771
- removed U4: ~, BMI323:SEN-21325
- removed dip: 219-3LPSTR, 219-3LPSTR:SW_219-3LPSTR
Routing:
- net +3.3V: track 10.2 -> 0.00 mm
Other:
- board outline removed

Commit message: initial pcb layout, improvements needed and no wiring and no xander waifu
Parts:
- added C1: 0.1uF, Capacitor_SMD:C_0805_2012Metric_Pad1.18x1.45mm_HandSolder, F.Cu at (165.5, 90.5)
- added C2: 0.1uF, Capacitor_SMD:C_0805_2012Metric_Pad1.18x1.45mm_HandSolder, F.Cu at (169.0, 90.5)
- added C24: 0.1uF, Capacitor_SMD:C_0805_2012Metric_Pad1.18x1.45mm_HandSolder, F.Cu at (185.0, 127.0)
- added C25: 0.1uF, Capacitor_SMD:C_0805_2012Metric_Pad1.18x1.45mm_HandSolder, F.Cu at (185.5, 106.0)
- added C4: 0.1uF, Capacitor_SMD:C_0805_2012Metric_Pad1.18x1.45mm_HandSolder, F.Cu at (241.0, 73.5)
- added D1: LED, LED_SMD:LED_0805_2012Metric_Pad1.15x1.40mm_HandSolder, F.Cu at (190.5, 127.0)
- added D2: LED, LED_SMD:LED_0805_2012Metric_Pad1.15x1.40mm_HandSolder, F.Cu at (195.5, 127.0)
- added D3: LED, LED_SMD:LED_0805_2012Metric_Pad1.15x1.40mm_HandSolder, F.Cu at (204.0, 127.0)
- added D4: LED, LED_SMD:LED_0805_2012Metric_Pad1.15x1.40mm_HandSolder, F.Cu at (209.0, 127.0)
- added D5: LED, LED_SMD:LED_0805_2012Metric_Pad1.15x1.40mm_HandSolder, F.Cu at (217.5, 127.0)
- added D6: LED, LED_SMD:LED_0805_2012Metric_Pad1.15x1.40mm_HandSolder, F.Cu at (222.5, 127.0)
- added D7: LED, LED_SMD:LED_0805_2012Metric_Pad1.15x1.40mm_HandSolder, F.Cu at (230.5, 127.0)
- added D8: LED, LED_SMD:LED_0805_2012Metric_Pad1.15x1.40mm_HandSolder, F.Cu at (235.5, 127.0)
- added F2: 3544-2, 3544_2:FUSE_3544-2, F.Cu at (172.5, 117.9)
- added J1: distance sensors signals, Connector_PinSocket_2.54mm:PinSocket_1x08_P2.54mm_Vertical, F.Cu at (183.3, 133.5)
- added J10: MD, Connector_PinHeader_2.54mm:PinHeader_1x02_P2.54mm_Vertical, F.Cu at (243.0, 125.2)
- added J11: LCD_Screen, Connector_JST:JST_PH_S4B-PH-K_1x04_P2.00mm_Horizontal, F.Cu at (178.0, 64.0)
- added J2: distance sensor power, Connector_PinHeader_2.54mm:PinHeader_1x02_P2.54mm_Vertical, F.Cu at (172.2, 133.5)
- added J3: line sensor power, Connector_PinHeader_2.54mm:PinHeader_1x02_P2.54mm_Vertical, F.Cu at (234.7, 133.5)
- added J4: Start Module, Connector_JST:JST_PH_S3B-PH-K_1x03_P2.00mm_Horizontal, F.Cu at (237.5, 64.0)
- added J5: 12vPower, Connector_AMASS:AMASS_XT30U-F_1x02_P5.0mm_Vertical, F.Cu at (169.5, 126.1)
- added J6: line sensor jst, Connector_PinSocket_2.54mm:PinSocket_1x08_P2.54mm_Vertical, F.Cu at (226.0, 133.5)
- added PS1: TSR_1-2450, TSR_1-2450:CONV_TSR_1-2450, F.Cu at (172.6, 104.8)
- added Q1: LTV-826S, LTV826:DIL8-SMD, F.Cu at (191.5, 116.0)
- added Q2: LTV-826S, LTV826:DIL8-SMD, F.Cu at (205.0, 116.0)
- added Q3: LTV-826S, LTV826:DIL8-SMD, F.Cu at (218.5, 116.0)
- added Q4: LTV-826S, LTV826:DIL8-SMD, F.Cu at (231.5, 115.8)
- added R1: 1k, Resistor_SMD:R_0805_2012Metric_Pad1.20x1.40mm_HandSolder, F.Cu at (243.4, 87.1)
- added R12: 500, Resistor_SMD:R_0805_2012Metric_Pad1.20x1.40mm_HandSolder, F.Cu at (188.0, 127.0)
- added R13: 500, Resistor_SMD:R_0805_2012Metric_Pad1.20x1.40mm_HandSolder, F.Cu at (193.0, 127.0)
- added R14: 500, Resistor_SMD:R_0805_2012Metric_Pad1.20x1.40mm_HandSolder, F.Cu at (201.5, 127.0)
- added R15: 500, Resistor_SMD:R_0805_2012Metric_Pad1.20x1.40mm_HandSolder, F.Cu at (206.5, 127.0)
- added R16: 500, Resistor_SMD:R_0805_2012Metric_Pad1.20x1.40mm_HandSolder, F.Cu at (215.0, 127.0)
- added R17: 500, Resistor_SMD:R_0805_2012Metric_Pad1.20x1.40mm_HandSolder, F.Cu at (220.0, 127.0)
- added R18: 500, Resistor_SMD:R_0805_2012Metric_Pad1.20x1.40mm_HandSolder, F.Cu at (228.0, 127.0)
- added R19: 500, Resistor_SMD:R_0805_2012Metric_Pad1.20x1.40mm_HandSolder, F.Cu at (233.0, 127.0)
- added R2: 1k, Resistor_SMD:R_0805_2012Metric_Pad1.20x1.40mm_HandSolder, F.Cu at (243.4, 97.6)
- added R23: 500, Resistor_SMD:R_0805_2012Metric_Pad1.20x1.40mm_HandSolder, F.Cu at (195.5, 106.0)
- added R24: 500, Resistor_SMD:R_0805_2012Metric_Pad1.20x1.40mm_HandSolder, F.Cu at (190.5, 106.0)
- added R25: 500, Resistor_SMD:R_0805_2012Metric_Pad1.20x1.40mm_HandSolder, F.Cu at (204.0, 106.0)
- added R26: 500, Resistor_SMD:R_0805_2012Metric_Pad1.20x1.40mm_HandSolder, F.Cu at (209.0, 106.0)
- added R27: 500, Resistor_SMD:R_0805_2012Metric_Pad1.20x1.40mm_HandSolder, F.Cu at (217.5, 106.0)
- added R28: 500, Resistor_SMD:R_0805_2012Metric_Pad1.20x1.40mm_HandSolder, F.Cu at (222.5, 106.0)
- added R29: 500, Resistor_SMD:R_0805_2012Metric_Pad1.20x1.40mm_HandSolder, F.Cu at (230.5, 106.0)
- added R30: 500, Resistor_SMD:R_0805_2012Metric_Pad1.20x1.40mm_HandSolder, F.Cu at (235.5, 106.0)
- added REF**: MountingHole_2.5mm, MountingHole:MountingHole_2.5mm, F.Cu at (208.2, 64.0)
- added REF**: MountingHole_3mm, MountingHole:MountingHole_3mm, F.Cu at (242.5, 139.5)
- added REF**: MountingHole_2.5mm, MountingHole:MountingHole_2.5mm, F.Cu at (201.8, 64.0)
- added REF**: MountingHole_3mm, MountingHole:MountingHole_3mm, F.Cu at (167.5, 139.5)
- added SW1: SW_Push, Button_Switch_THT:SW_PUSH_6mm_H5mm, F.Cu at (231.1, 82.6)
- added SW2: SW_Push, Button_Switch_THT:SW_PUSH_6mm_H5mm, F.Cu at (230.9, 92.9)
- added SW3: SW_SPST, Connector_PinHeader_2.54mm:PinHeader_1x02_P2.54mm_Vertical, F.Cu at (171.2, 112.0)
- added U1: DEV-16771, DEV-16771:MODULE_DEV-16771, F.Cu at (194.5, 90.0)
Other:
- board outline added: 85 x 83 mm

Commit message: pcb layout and wiring is done! still need to add silkscreen and xander waifu
Parts:
- removed SW3: SW_SPST, Connector_PinHeader_2.54mm:PinHeader_1x02_P2.54mm_Vertical
- added S1: 1101M2S3CQE2, 1101M2S3CQE2:SW_1101M2S3CQE2, F.Cu at (172.3, 118.0)
- C1, C2, C24, C25, C4, PS1, Q1, Q2, Q3, Q4, R1, R12, R13, R14, R15, R16, R17, R18, R19, R2, R23, R24, R25, R26, R27, R28, R29, R30: moved to B.Cu
- J11: footprint Connector_JST:JST_PH_S4B-PH-K_1x04_P2.00mm_Horizontal -> Connector_PinHeader_2.54mm:PinHeader_1x04_P2.54mm_Vertical
- J4: footprint Connector_JST:JST_PH_S3B-PH-K_1x03_P2.00mm_Horizontal -> Connector_PinHeader_2.54mm:PinHeader_1x03_P2.54mm_Vertical
- moved R2 48.2 mm to (202.0, 73.0)
- moved R1 34.4 mm to (212.0, 73.0)
- moved SW2 34.2 mm to (205.2, 70.2), turned to -90 degrees
- moved SW1 20.1 mm to (215.3, 70.3), turned to -90 degrees
- moved R24 18.4 mm to (208.1, 100.5)
- moved PS1 16.8 mm to (188.0, 111.5)
- moved R30 15.6 mm to (220.9, 100.5)
- moved C24 11.6 mm to (174.0, 130.5), turned to 180 degrees
- moved R18 11.1 mm to (238.5, 123.5)
- moved R25 10.7 mm to (213.2, 100.5)
- moved D2 10.6 mm to (185.5, 123.5)
- moved R13 10.6 mm to (183.0, 123.5)
- moved D4 9.66 mm to (200.0, 123.5)
- moved R15 9.66 mm to (197.5, 123.5)
- moved R16 9.66 mm to (224.0, 123.5)
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Connections:
- C4 pad 1: +3.3V -> GND
- C4 pad 2: GND -> +3.3V
- D1 pad 1: Net-(D1-K) -> GND
- D2 pad 1: Net-(D2-K) -> GND
- D3 pad 1: Net-(D3-K) -> GND
- D4 pad 1: Net-(D4-K) -> GND
- D5 pad 1: Net-(D5-K) -> GND
- D6 pad 1: Net-(D6-K) -> GND
- D7 pad 1: Net-(D7-K) -> GND
- D8 pad 1: Net-(D8-K) -> GND
- F2 pad 1_1: Net-(SW3-B) -> +12V
- F2 pad 1_2: Net-(SW3-B) -> +12V
- F2 pad 2_1: Net-(J5-Pin_2) -> Net-(F2-Pad2_1)
- F2 pad 2_2: Net-(J5-Pin_2) -> Net-(F2-Pad2_1)
- J11 pad 1: GND -> LCD_SDA
- J11 pad 2: +5V -> LCD_SCL
- J11 pad 3: LCD_SDA -> +3.3V
- J11 pad 4: LCD_SCL -> GND
- J4 pad 1: JSUMOStartMod -> +3.3V
- J4 pad 3: +3.3V -> JSUMOStartMod
- Q1 pad 1: OCT_F -> OCT_30L
- Q1 pad 2: Net-(D1-A) -> Net-(Q1-Pad2)
- Q1 pad 3: OCT_30L -> OCT_F
- Q1 pad 4: Net-(D2-A) -> Net-(Q1-Pad4)
- Q1 pad 5: DS_30L -> DS_F
- Q1 pad 7: DS_F -> DS_30L
- Q2 pad 1: OCT_60L -> OCT_90L
- Q2 pad 2: Net-(D3-A) -> Net-(Q2-Pad2)
- Q2 pad 3: OCT_90L -> OCT_60L
- Q2 pad 4: Net-(D4-A) -> Net-(Q2-Pad4)
- Q2 pad 5: DS_90L -> DS_60L
- Q2 pad 7: DS_60L -> DS_90L
- Q3 pad 1: OCT_30R -> OCT_60R
- Q3 pad 2: Net-(D5-A) -> Net-(Q3-Pad2)
- Q3 pad 3: OCT_60R -> OCT_30R
- Q3 pad 4: Net-(D6-A) -> Net-(Q3-Pad4)
- Q3 pad 5: DS_60R -> DS_30R
- Q3 pad 7: DS_30R -> DS_60R
- Q4 pad 1: OCT_90R -> OCT_B
- Q4 pad 2: Net-(D7-A) -> Net-(Q4-Pad2)
- Q4 pad 3: OCT_B -> OCT_90R
- Q4 pad 4: Net-(D8-A) -> Net-(Q4-Pad4)
- Q4 pad 5: DS_B -> DS_90R
- Q4 pad 7: DS_90R -> DS_B
- R12 pad 1: GND -> Net-(D1-A)
- R12 pad 2: Net-(D1-K) -> Net-(Q1-Pad2)
- R13 pad 1: GND -> Net-(D2-A)
- R13 pad 2: Net-(D2-K) -> Net-(Q1-Pad4)
- R14 pad 1: GND -> Net-(D3-A)
- R14 pad 2: Net-(D3-K) -> Net-(Q2-Pad2)
- R15 pad 1: GND -> Net-(D4-A)
- R15 pad 2: Net-(D4-K) -> Net-(Q2-Pad4)
- R16 pad 1: GND -> Net-(D5-A)
- R16 pad 2: Net-(D5-K) -> Net-(Q3-Pad2)
- R17 pad 1: GND -> Net-(D6-A)
- R17 pad 2: Net-(D6-K) -> Net-(Q3-Pad4)
- R18 pad 1: GND -> Net-(D7-A)
- R18 pad 2: Net-(D7-K) -> Net-(Q4-Pad2)
- R19 pad 1: GND -> Net-(D8-A)
- R19 pad 2: Net-(D8-K) -> Net-(Q4-Pad4)
- R23 pad 2: DS_30L -> DS_F
- R24 pad 2: DS_F -> DS_30L
- R25 pad 2: DS_60L -> DS_90L
- R26 pad 2: DS_90L -> DS_60L
- R27 pad 2: DS_30R -> DS_60R
- R28 pad 2: DS_60R -> DS_30R
- R29 pad 2: DS_90R -> DS_B
- R30 pad 2: DS_B -> DS_90R
- U1 pad 13: JSUMOStartMod -> unconnected-(U1-SCK-Pad13)
- U1 pad 33: unconnected-(U1-MCLK2-Pad33) -> JSUMOStartMod
Routing:
- net +3.3V: track 0.00 -> 251.5 mm
- net LS_RB2: track 0.00 -> 60.8 mm
- net LS_RB1: track 0.00 -> 59.5 mm
- net LS_LB1: track 0.00 -> 59.4 mm
- net LS_LF1: track 0.00 -> 59.0 mm
- net LS_LF2: track 0.00 -> 58.7 mm
- net LS_LB2: track 0.00 -> 58.7 mm
- net LS_RF2: track 0.00 -> 58.7 mm
- net LS_RF1: track 0.00 -> 58.7 mm
- net +12V: track 0.00 -> 58.0 mm
- net LCD_SCL: track 0.00 -> 51.5 mm
- net MD_TX: track 0.00 -> 50.7 mm
- net +5V: track 0.00 -> 49.8 mm
- net LCD_SDA: track 0.00 -> 49.7 mm
- net MD_RX: track 0.00 -> 46.1 mm
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- added copper zone on B.Cu, net GND
- added copper zone on F.Cu, net GND

Commit message: added necessary silkscreen to control pcb, still need to put the less necessary silkscreen
Parts:
- added D10: LED, LED_SMD:LED_0805_2012Metric_Pad1.15x1.40mm_HandSolder, F.Cu at (203.6, 81.3)
- added D9: LED, LED_SMD:LED_0805_2012Metric_Pad1.15x1.40mm_HandSolder, F.Cu at (213.2, 81.2)
- added R3: 500, Resistor_SMD:R_0805_2012Metric_Pad1.20x1.40mm_HandSolder, B.Cu at (213.2, 84.2)
- added R4: 500, Resistor_SMD:R_0805_2012Metric_Pad1.20x1.40mm_HandSolder, B.Cu at (203.8, 84.2)
Routing:
- net Button2: track 22.0 -> 27.4 mm
- net Button1: track 23.2 -> 28.2 mm
- net Net-(D10-K): track 0.00 -> 3.35 mm, vias 0 -> 1
- net Net-(D9-K): track 0.00 -> 3.01 mm, vias 0 -> 1
- removed copper zone on B.Cu, net GND
- removed copper zone on F.Cu, net GND
Other:
- board text added: "0.1uF"
- board text added: "12V"
- board text added: "3.3V"
- board text added: "30L"
- board text added: "30R"
- board text added: "5V"
- board text added: "60L"
- board text added: "60R"
- board text added: "90L"
- board text added: "90R"
- board text added: "<- 1Kohm resistors"
- board text added: "<- 500 ohm resistors"
- board text added: "<- this row is all 500 ohm"
- board text added: "B"
- board text added: "Butt1"
- board text added: "Butt2"
- board text added: "DDS"
- board text added: "F"
- board text added: "GND"
- board text added: "LB1"
- board text added: "LB2"
- board text added: "LCD_SCL"
- board text added: "LCD_SDA"
- board text added: "LF1"
- board text added: "LF2"
- board text added: "Line"
- board text added: "RB1"
- board text added: "RB2"
- board text added: "RF1"
- board text added: "RF2"
- board text added: "RX"
- board text added: "SCL"
- board text added: "SDA"
- board text added: "StartMod"
- board text added: "TX"
- board text added: "This row is all 500 ohms"

Commit message: i think ferarrii pcb is done
Parts:
- added G***: LOGO, LOGO, F.Cu at (226.8, 70.5)
- moved R4 5.41 mm to (208.2, 81.2), turned to 180 degrees
Routing:
- net Net-(D10-K): track 3.35 -> 2.61 mm
- added copper zone on B.Cu, net GND
- added copper zone on F.Cu, net GND
Other:
- board text added: "Ferrarii"
- board text added: "{dblquote}What's wrong with Gura?{dblquote} - Xander Riddle"
