File: RCSummer25/Controller_Simple/Controller_Simple.kicad_pcb (KiCad board)
At the start: 2 copper layers, 140 x 80 mm, 29 parts, among them J1 Conn_02x04_Odd_Even, J2 Conn_01x05_Pin, J3 Conn_01x05_Pin, J4 Conn_01x02_Pin, SW1 SW_Push, SW2 SW_Push, SW3 SW_Push, SW4 SW_Push, SW5 SW_Push, SW6 SW_Push, SW7 SW_Push, SW8 SW_Push, SW9 SW_Nidec_CAS-120A1, U2 YAAJ_BluePill

Commit message: Fixed issues with Simple_Controller
Parts:
- moved C2 2.69 mm to (105.0, 66.5), turned to 0 degrees
Connections:
- D1 pad 1: +12V -> GND
- F1 pad 1: Net-(F1-Pad1) -> +12V
- R9 pad 2: Net-(F1-Pad1) -> +12V
- U2 pad 20: unconnected-(U2-3V3-Pad20) -> +3.3V
Routing:
- net +12V: track 22.1 -> 34.1 mm
- net Net-(F1-Pad1): track 4.69 -> 0.00 mm
Changed lines of the file:
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@@
 	(net 41 "unconnected-(U2-PB9-Pad17)")
 	(net 42 "Net-(D1-A)")
-	(net 43 "Net-(F1-Pad1)")
-	(net 44 "Net-(J4-Pin_2)")
-	(net 45 "unconnected-(U2-3V3-Pad20)")
+	(net 43 "Net-(J4-Pin_2)")
 	(footprint "Resistor_SMD:R_0805_2012Metric"
 		(layer "F.Cu")
@@
 	(footprint "Capacitor_SMD:C_0805_2012Metric_Pad1.18x1.45mm_HandSolder"
 		(layer "F.Cu")
-		(at 102.5 67.5 -90)
+		(at 105 66.5)
 		(descr "Capacitor SMD 0805 (2012 Metric), square (rectangular) end terminal, IPC-7351 nominal with elongated pad for handsoldering. (Body size source: IPC-SM-782 page 76, https://www.pcb-3d.com/wordpress/wp-content/uploads/ipc-sm-782a_amendment_1_and_2.pdf, https://docs.google.com/spreadsheets/d/1BsfQQcO9C6DZCsRaXUlFlo91Tg2WpOkGARC1WS5S8t0/edit?usp=sharing), generated with kicad-footprint-generator")
 		(tags "capacitor handsolder")
 		(property "Reference" "C2"
-			(at 0 -1.68 90)
+			(at 0 -1.68 0)
 			(layer "F.SilkS")
 			(effects
@@
 		)
 		(property "Value" "10uF"
-			(at 0 1.68 90)
+			(at 0 1.68 0)
 			(layer "F.Fab")
 			(effects
@@
 		)
 		(property "Datasheet" ""
-			(at 0 0 90)
+			(at 0 0 0)
 			(layer "F.Fab")
 			(hide yes)
@@
 		)
 		(property "Description" "Unpolarized capacitor"
-			(at 0 0 90)
+			(at 0 0 0)
 			(layer "F.Fab")
 			(hide yes)
@@
 		(attr smd)
 		(fp_line
-			(start -0.261252 0.735)
-			(end 0.261252 0.735)
+			(start -0.261252 -0.735)
+			(end 0.261252 -0.735)
 			(stroke
 				(width 0.12)
@@
 		)
 		(fp_line
-			(start -0.261252 -0.735)
-			(end 0.261252 -0.735)
+			(start -0.261252 0.735)
+			(end 0.261252 0.735)
 			(stroke
 				(width 0.12)
@@
 		)
 		(fp_line
-			(start -1.88 0.98)
-			(end -1.88 -0.98)
+			(start -1.88 -0.98)
+			(end 1.88 -0.98)
 			(stroke
 				(width 0.05)
@@
 		)
 		(fp_line
-			(start 1.88 0.98)
-			(end -1.88 0.98)
+			(start -1.88 0.98)
+			(end -1.88 -0.98)
 			(stroke
 				(width 0.05)
@@
 		)
 		(fp_line
-			(start -1.88 -0.98)
-			(end 1.88 -0.98)
+			(start 1.88 -0.98)
+			(end 1.88 0.98)
 			(stroke
 				(width 0.05)
@@
 		)
 		(fp_line
-			(start 1.88 -0.98)
-			(end 1.88 0.98)
+			(start 1.88 0.98)
+			(end -1.88 0.98)
 			(stroke
 				(width 0.05)
@@
 		)
 		(fp_line
-			(start -1 0.625)
-			(end -1 -0.625)
+			(start -1 -0.625)
+			(end 1 -0.625)
 			(stroke
 				(width 0.1)
@@
 		)
 		(fp_line
-			(start 1 0.625)
-			(end -1 0.625)
+			(start -1 0.625)
+			(end -1 -0.625)
 			(stroke
 				(width 0.1)
@@
 		)
 		(fp_line
-			(start -1 -0.625)
-			(end 1 -0.625)
+			(start 1 -0.625)
+			(end 1 0.625)
 			(stroke
 				(width 0.1)
@@
 		)
 		(fp_line
-			(start 1 -0.625)
-			(end 1 0.625)
+			(start 1 0.625)
+			(end -1 0.625)
 			(stroke
 				(width 0.1)
@@
 		)
 		(fp_text user "${REFERENCE}"
-			(at 0 0 90)
+			(at 0 0 0)
 			(layer "F.Fab")
 			(effects
@@
 		)
 		(pad "1" smd roundrect
-			(at -1.0375 0 270)
+			(at -1.0375 0)
 			(size 1.175 1.45)
 			(layers "F.Cu" "F.Mask" "F.Paste")
@@
 		)
 		(pad "2" smd roundrect
-			(at 1.0375 0 270)
+			(at 1.0375 0)
 			(size 1.175 1.45)
 			(layers "F.Cu" "F.Mask" "F.Paste")
@@
 			(layers "*.Cu" "*.Mask")
 			(remove_unused_layers no)
-			(net 44 "Net-(J4-Pin_2)")
+			(net 43 "Net-(J4-Pin_2)")
 			(pinfunction "Pin_2")
 			(pintype "passive")
@@
 			(layers "F.Cu" "F.Mask" "F.Paste")
 			(roundrect_rratio 0.25)
-			(net 3 "+12V")
+			(net 1 "GND")
 			(pinfunction "K")
 			(pintype "passive")
@@
 			(layers "F.Cu" "F.Mask" "F.Paste")
 			(roundrect_rratio 0.217391)
-			(net 43 "Net-(F1-Pad1)")
+			(net 3 "+12V")
 			(pintype "passive")
 		)
@@
 			(layers "F.Cu" "F.Mask" "F.Paste")
 			(roundrect_rratio 0.243902)
-			(net 43 "Net-(F1-Pad1)")
+			(net 3 "+12V")
 			(pintype "passive")
 		)
@@
 			(layers "*.Cu" "*.Mask")
 			(remove_unused_layers no)
-			(net 44 "Net-(J4-Pin_2)")
+			(net 43 "Net-(J4-Pin_2)")
 			(pinfunction "B")
 			(pintype "passive")
@@
 			(layers "*.Cu" "*.Mask")
 			(remove_unused_layers no)
-			(net 45 "unconnected-(U2-3V3-Pad20)")
+			(net 2 "+3.3V")
 			(pinfunction "3V3")
-			(pintype "power_in+no_connect")
+			(pintype "power_in")
 		)
 		(pad "21" thru_hole circle
@@
 	)
 	(segment
-		(start 104.9625 66.4625)
-		(end 110 71.5)
+		(start 106 81)
+		(end 106 68.5375)
+		(width 0.2)
+		(layer "F.Cu")
+		(net 3)
+	)
+	(segment
+		(start 103.9225 66.54)
+		(end 103.9625 66.5)
 		(width 0.2)
 		(layer "F.Cu")
@@
 	)
 	(segment
-		(start 102.5 66.4625)
-		(end 90.0775 66.4625)
+		(start 90 66.54)
+		(end 103.9225 66.54)
+		(width 0.2)
+		(layer "F.Cu")
+		(net 3)
+	)
+	(segment
+		(start 108.325 81)
+		(end 110 79.325)
+		(width 0.2)
+		(layer "F.Cu")
+		(net 3)
+	)
+	(segment
+		(start 106 81)
+		(end 108.325 81)
 		(width 0.2)
 		(layer "F.Cu")
@@
 	)
 	(segment
-		(start 102.5 66.4625)
-		(end 104.9625 66.4625)
+		(start 106 68.5375)
+		(end 103.9625 66.5)
 		(width 0.2)
 		(layer "F.Cu")
@@
 	)
 	(segment
-		(start 108.325 81)
-		(end 110 79.325)
-		(width 0.2)
-		(layer "F.Cu")
-		(net 43)
-	)
-	(segment
-		(start 106 81)
-		(end 108.325 81)
-		(width 0.2)
-		(layer "F.Cu")
-		(net 43)
-	)
-	(segment
 		(start 110 87.5)
 		(end 119.5 78)
 		(width 0.2)
 		(layer "F.Cu")
-		(net 44)
+		(net 43)
 	)
 	(segment
@@
 		(width 0.2)
 		(layer "F.Cu")
-		(net 44)
+		(net 43)
 	)
 	(segment
@@
 		(width 0.2)
 		(layer "F.Cu")
-		(net 44)
+		(net 43)
 	)
 	(segment
@@
 		(width 0.2)
 		(layer "F.Cu")
-		(net 44)
+		(net 43)
 	)
 	(zone
