File: RCSummer25/Controller_Simple/Controller_Simple.kicad_sch (KiCad schematic)
At the start: 29 parts, among them J1 Conn_02x04_Odd_Even, J2 Conn_01x05_Pin, J3 Conn_01x05_Pin, J4 Conn_01x02_Pin, SW1 SW_Push, SW2 SW_Push, SW3 SW_Push, SW4 SW_Push, SW5 SW_Push, SW6 SW_Push, SW7 SW_Push, SW8 SW_Push, SW9 SW_Nidec_CAS-120A1, U2 YAAJ_BluePill

Commit message: Fixed issues with Simple_Controller
Connections:
- net +12V: now also F1.1, R9.2; no longer D1.1 (K)
- net GND: now also D1.1 (K)
Changed lines of the file:
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@@
 	)
 	(junction
+		(at 193.04 40.64)
+		(diameter 0)
+		(color 0 0 0 0)
+	)
+	(junction
 		(at 196.85 74.93)
 		(diameter 0)
@@
 	(wire
 		(pts
+			(xy 187.96 40.64) (xy 193.04 40.64)
+		)
+		(stroke
+			(width 0)
+			(type default)
+		)
+	)
+	(wire
+		(pts
 			(xy 72.39 87.63) (xy 68.58 87.63)
 		)
@@
 	(symbol
 		(lib_id "power:GND")
+		(at 193.04 24.13 180)
+		(unit 1)
+		(exclude_from_sim no)
+		(in_bom yes)
+		(on_board yes)
+		(dnp no)
+		(fields_autoplaced yes)
+		(property "Reference" "#PWR036"
+			(at 193.04 17.78 0)
+			(effects
+				(font
+					(size 1.27 1.27)
+				)
+				(hide yes)
+			)
+		)
+		(property "Value" "GND"
+			(at 193.04 19.05 0)
+			(effects
+				(font
+					(size 1.27 1.27)
+				)
+			)
+		)
+		(property "Footprint" ""
+			(at 193.04 24.13 0)
+			(effects
+				(font
+					(size 1.27 1.27)
+				)
+				(hide yes)
+			)
+		)
+		(property "Datasheet" ""
+			(at 193.04 24.13 0)
+			(effects
+				(font
+					(size 1.27 1.27)
+				)
+				(hide yes)
+			)
+		)
+		(property "Description" "Power symbol creates a global label with name \"GND\" , ground"
+			(at 193.04 24.13 0)
+			(effects
+				(font
+					(size 1.27 1.27)
+				)
+				(hide yes)
+			)
+		)
+		(pin "1"
+		)
+		(instances
+			(project ""
+				(path "/6c578a11-c7c4-4e4b-b372-f2769ce1c845"
+					(reference "#PWR036")
+					(unit 1)
+				)
+			)
+		)
+	)
+	(symbol
+		(lib_id "power:GND")
 		(at 100.33 69.85 0)
 		(unit 1)
@@
 	(symbol
 		(lib_id "power:+12V")
-		(at 193.04 24.13 0)
+		(at 187.96 40.64 90)
 		(unit 1)
 		(exclude_from_sim no)
@@
 		(fields_autoplaced yes)
 		(property "Reference" "#PWR018"
-			(at 193.04 27.94 0)
+			(at 191.77 40.64 0)
 			(effects
 				(font
@@
 		)
 		(property "Value" "+12V"
-			(at 193.04 19.05 0)
+			(at 186.69 38.1 90)
 			(effects
 				(font
@@
 		)
 		(property "Footprint" ""
-			(at 193.04 24.13 0)
+			(at 187.96 40.64 0)
 			(effects
 				(font
@@
 		)
 		(property "Datasheet" ""
-			(at 193.04 24.13 0)
+			(at 187.96 40.64 0)
 			(effects
 				(font
@@
 		)
 		(property "Description" "Power symbol creates a global label with name \"+12V\""
-			(at 193.04 24.13 0)
+			(at 187.96 40.64 0)
 			(effects
 				(font
@@
 		)
 		(instances
-			(project ""
+			(project "Controller_Simple"
 				(path "/6c578a11-c7c4-4e4b-b372-f2769ce1c845"
 					(reference "#PWR018")
