File: 500g/Rata2i2.0/pcbn't/Schematic - Copy/Schematic.kicad_pcb (KiCad board)
At the start: 2 copper layers, 83.5 x 57 mm, 37 parts, among them J1 Screw_Terminal_01x03, J10 Conn_01x03_Pin, J11 Screw_Terminal_01x02, J12 Screw_Terminal_01x02, J2 Screw_Terminal_01x03, J3 Screw_Terminal_01x03, J4 Screw_Terminal_01x03, J5 Screw_Terminal_01x03, J6 Screw_Terminal_01x03, J7 Battery, J8 Conn_01x08_Pin, SW1 SW_SPDT, U1 DEV-16771, U3 R-78K5.0-0.5, U4 R-78K5.0-0.5, U5 ROB-14450

Commit message: updated rata2i schematic
blah blah blah
Parts:
- added D1: LED, LED_SMD:LED_1206_3216Metric, F.Cu at (86.2, 73.3)
- added J13: Screw_Terminal_01x03, TerminalBlock:TerminalBlock_Xinya_XY308-2.54-3P_1x03_P2.54mm_Horizontal, F.Cu at (81.7, 57.0)
- added J14: Screw_Terminal_01x03, TerminalBlock:TerminalBlock_Xinya_XY308-2.54-3P_1x03_P2.54mm_Horizontal, F.Cu at (82.0, 68.6)
- added J15: Screw_Terminal_01x03, TerminalBlock:TerminalBlock_Xinya_XY308-2.54-3P_1x03_P2.54mm_Horizontal, F.Cu at (92.7, 77.5)
- added J9: Screw_Terminal_01x03, TerminalBlock:TerminalBlock_Xinya_XY308-2.54-3P_1x03_P2.54mm_Horizontal, F.Cu at (82.2, 40.6)
- added R1: R_US, Resistor_SMD:R_0805_2012Metric, F.Cu at (85.6, 76.5)
- added U2: NRF24L01_Breakout, RF_Module:nRF24L01_Breakout, F.Cu at (71.0, 45.1)
- moved G*** 44.3 mm to (56.0, 86.0)
- moved G*** 39.3 mm to (55.0, 64.5)
- moved G*** 38.3 mm to (56.0, 47.0)
- moved G*** 23.5 mm to (74.5, 89.5)
- moved G*** 13.6 mm to (88.0, 90.0)
- moved J11 11.2 mm to (102.8, 79.3), turned to 90 degrees
- moved J12 2.50 mm to (103.0, 70.0), turned to -90 degrees
Connections:
- J1 pad 1: +3.3V -> +5V
- J2 pad 1: +3.3V -> +5V
- J3 pad 1: +3.3V -> +5V
- J4 pad 1: +3.3V -> +5V
- U1 pad 16: unconnected-(U1-A2-Pad16) -> L3
- U1 pad 18: unconnected-(U1-A4-Pad18) -> L4
- U1 pad 23: unconnected-(U1-A9-Pad23) -> s6
- U1 pad 24: unconnected-(U1-A10-Pad24) -> s5
- U1 pad 25: unconnected-(U1-A11-Pad25) -> mode 3
- U1 pad 26: unconnected-(U1-A12-Pad26) -> mode 2
- U1 pad 27: unconnected-(U1-A13-Pad27) -> mode 1
- U1 pad 38: unconnected-(U1-A14-Pad38) -> mode 0
Routing:
- net Net-(J11-Pin_1): track 79.9 -> 0.00 mm
- net Net-(J11-Pin_2): track 74.4 -> 0.00 mm
- net Net-(J12-Pin_2): track 71.5 -> 0.00 mm
- net Net-(J12-Pin_1): track 67.5 -> 1.74 mm
- net s5: track 0.00 -> 31.8 mm, vias 0 -> 1
- net GND: track 139.8 -> 140.3 mm, vias 0 -> 1

Commit message: IT WORKS!!!!!
yippee
Parts:
- added C6: 10 uF, Capacitor_SMD:C_0805_2012Metric, F.Cu at (173.1, 43.0)
- added C7: 10 uF, Capacitor_SMD:C_0805_2012Metric, F.Cu at (173.1, 46.0)
- added J11: Screw_Terminal_01x02, TerminalBlock:TerminalBlock_Xinya_XY308-2.54-2P_1x02_P2.54mm_Horizontal, F.Cu at (164.4, 36.8)
- added J12: Screw_Terminal_01x02, TerminalBlock:TerminalBlock_Xinya_XY308-2.54-2P_1x02_P2.54mm_Horizontal, F.Cu at (172.0, 36.8)
- added R6: R_US, Resistor_SMD:R_0805_2012Metric, F.Cu at (173.1, 49.0)
- added U5: DRV8871DDAR, DRV8871DDAR:VREG_LM5017MR_NOPB, F.Cu at (166.6, 44.7)
Connections:
- C1 pad 2: GND -> +12V
- C2 pad 2: GND -> +12V
- C3 pad 1: GND -> +12V
- C4 pad 2: GND -> +12V
- C5 pad 1: +3.3V -> +12V
- C5 pad 2: GND -> +12V
- D1 pad 1: GND -> +12V
- D2 pad 1: GND -> +12V
- D3 pad 1: GND -> +12V
- D4 pad 1: GND -> +12V
- D6 pad 1: GND -> +12V
- J1 pad 1: +5V -> +12V
- J1 pad 2: GND -> +12V
- J10 pad 2: GND -> +12V
- J10 pad 3: +3.3V -> +12V
- J13 pad 1: +5V -> +12V
- J13 pad 2: GND -> +12V
- J14 pad 1: GND -> +12V
- J14 pad 2: +3.3V -> +12V
- J15 pad 1: GND -> +12V
- J15 pad 2: +3.3V -> +12V
- J2 pad 1: +5V -> +12V
- J2 pad 2: GND -> +12V
- J3 pad 1: +5V -> +12V
- J3 pad 2: GND -> +12V
- J4 pad 1: +5V -> +12V
- J4 pad 2: GND -> +12V
- J5 pad 1: GND -> +12V
- J5 pad 2: +3.3V -> +12V
- J6 pad 1: GND -> +12V
- J6 pad 2: +3.3V -> +12V
- J7 pad 1: GND -> +12V
- J8 pad 1: +3.3V -> +12V
- J8 pad 2: GND -> +12V
- J9 pad 1: +5V -> +12V
- J9 pad 2: GND -> +12V
- U1 pad 1: unconnected-(U1-TX1-Pad1) -> CE
- U1 pad 11: unconnected-(U1-MOSI-Pad11) -> MOSI
- U1 pad 12: unconnected-(U1-MISO-Pad12) -> MISO
- U1 pad 13: unconnected-(U1-SCK-Pad13) -> SCK
- U1 pad 3.3V_1: +3.3V -> +12V
- U1 pad 3.3V_2: +3.3V -> +12V
- U1 pad 3.3V_3: +3.3V -> +12V
- U1 pad 7: unconnected-(U1-RX2-Pad7) -> ~CSN
- U1 pad GND1: GND -> +12V
- U1 pad GND2: GND -> +12V
- U1 pad GND3: GND -> +12V
- U1 pad GND4: GND -> +12V
- U1 pad GND5: GND -> +12V
- U1 pad USB_GND1: GND -> +12V
- U1 pad USB_GND2: GND -> +12V
- U2 pad 1: unconnected-(U2-GND-Pad1) -> +12V
- U2 pad 2: unconnected-(U2-VCC-Pad2) -> +12V
- U2 pad 3: unconnected-(U2-CE-Pad3) -> CE
- U2 pad 4: unconnected-(U2-~{CSN}-Pad4) -> ~CSN
- U2 pad 5: unconnected-(U2-SCK-Pad5) -> SCK
- U2 pad 6: unconnected-(U2-MOSI-Pad6) -> MOSI
- U2 pad 7: unconnected-(U2-MISO-Pad7) -> MISO
- U3 pad 2: GND -> +12V
- U4 pad 2: GND -> +12V
- U4 pad 3: +3.3V -> +12V
Routing:
- net GND: track 140.3 -> 67.0 mm, vias 1 -> 0
- net +12V: track 116.9 -> 190.2 mm, vias 0 -> 3
- net +3.3V: vias 2 -> 0
- added copper zone on F.Cu, net +12V
- removed copper zone on F.Cu, net GND

Commit message: All parts done!
Need to wire :(
Parts:
- removed the U5 at (105.5, 36.6)
- added J16: Screw_Terminal_01x07, TerminalBlock:TerminalBlock_Xinya_XY308-2.54-7P_1x07_P2.54mm_Horizontal, F.Cu at (94.8, 30.5)
- C6, C7, R6, U5: moved to B.Cu
- moved J11 67.4 mm to (97.2, 42.3), turned to 180 degrees
- moved J12 61.2 mm to (111.0, 41.0)
- moved U5 55.1 mm to (112.8, 56.9), turned to 180 degrees
- moved R6 49.0 mm to (125.0, 58.0), turned to 90 degrees
- moved C7 46.7 mm to (127.9, 58.0), turned to 90 degrees
- moved C6 44.7 mm to (130.9, 58.0), turned to 90 degrees
- moved U2 10.0 mm to (63.0, 39.1)
Connections:
- C1 pad 2: +12V -> +3.3V
- C2 pad 2: +12V -> +3.3V
- C3 pad 1: +12V -> +3.3V
- C4 pad 2: +12V -> +3.3V
- C5 pad 1: +12V -> +3.3V
- C5 pad 2: +12V -> +3.3V
- C6 pad 2: +12V -> +3.3V
- C7 pad 2: +12V -> +3.3V
- D1 pad 1: +12V -> +3.3V
- D2 pad 1: +12V -> +3.3V
- D3 pad 1: +12V -> +3.3V
- D4 pad 1: +12V -> +3.3V
- D6 pad 1: +12V -> +3.3V
- J1 pad 1: +12V -> +3.3V
- J1 pad 2: +12V -> +3.3V
- J10 pad 2: +12V -> +3.3V
- J10 pad 3: +12V -> +3.3V
- J11 pad 2: +12V -> +3.3V
- J12 pad 2: +12V -> +3.3V
- J13 pad 1: +12V -> +3.3V
- J13 pad 2: +12V -> +3.3V
- J14 pad 1: +12V -> +3.3V
- J14 pad 2: +12V -> +3.3V
- J15 pad 1: +12V -> +3.3V
- J15 pad 2: +12V -> +3.3V
- J2 pad 1: +12V -> +3.3V
- J2 pad 2: +12V -> +3.3V
- J3 pad 1: +12V -> +3.3V
- J3 pad 2: +12V -> +3.3V
- J4 pad 1: +12V -> +3.3V
- J4 pad 2: +12V -> +3.3V
- J5 pad 1: +12V -> +3.3V
- J5 pad 2: +12V -> +3.3V
- J6 pad 1: +12V -> +3.3V
- J6 pad 2: +12V -> +3.3V
- J7 pad 1: +12V -> +3.3V
- J8 pad 1: +12V -> +3.3V
- J8 pad 2: +12V -> +3.3V
- J9 pad 1: +12V -> +3.3V
- J9 pad 2: +12V -> +3.3V
- R6 pad 1: +12V -> +3.3V
- U1 pad 3.3V_1: +12V -> +3.3V
- U1 pad 3.3V_2: +12V -> +3.3V
- U1 pad 3.3V_3: +12V -> +3.3V
- U1 pad GND1: +12V -> +3.3V
- U1 pad GND2: +12V -> +3.3V
- U1 pad GND3: +12V -> +3.3V
- U1 pad GND4: +12V -> +3.3V
- U1 pad GND5: +12V -> +3.3V
- U1 pad USB_GND1: +12V -> +3.3V
- U1 pad USB_GND2: +12V -> +3.3V
- U2 pad 1: +12V -> +3.3V
- U2 pad 2: +12V -> +3.3V
- U3 pad 2: +12V -> +3.3V
- U4 pad 2: +12V -> +3.3V
- U4 pad 3: +12V -> +3.3V
- U5 pad 1: +12V -> +3.3V
- U5 pad 7: +12V -> +3.3V
Routing:
- net +12V: track 190.2 -> 53.0 mm, vias 3 -> 1
- net GND: track 67.0 -> 0.00 mm
- net motorbpwm: track 44.4 -> 0.00 mm
- net +5V: track 109.4 -> 76.1 mm, vias 5 -> 3
- net motorapwm: track 24.1 -> 0.00 mm
- net +3.3V: track 189.2 -> 201.7 mm
- net mdr2: track 9.14 -> 0.59 mm
- net mdr3: track 6.33 -> 0.00 mm
- net mdr1: track 6.33 -> 0.00 mm
- net mdr4: track 6.33 -> 0.00 mm
- net CE: track 0.00 -> 5.72 mm, vias 0 -> 1
- net start: track 29.0 -> 23.3 mm, vias 2 -> 1
- net Net-(J12-Pin_1): track 1.74 -> 0.00 mm

Commit message: 2 motor drivers, 2 less sensors :D
mostly connected but it REALLY doesn't like the motor drivers, maybe moving to the normal side will make it better?
Parts:
- removed the J12 at (111.0, 41.0)
- removed J8: Conn_01x08_Pin, Connector_PinHeader_2.54mm:PinHeader_1x08_P2.54mm_Vertical
- added C8: 10 uF, Capacitor_SMD:C_0805_2012Metric, B.Cu at (98.0, 79.0)
- added C9: 10 uF, Capacitor_SMD:C_0805_2012Metric, B.Cu at (98.0, 76.5)
- added J19: motor 2, TerminalBlock:TerminalBlock_Xinya_XY308-2.54-2P_1x02_P2.54mm_Horizontal, F.Cu at (92.5, 70.5)
- added R7: R_US, Resistor_SMD:R_0805_2012Metric, B.Cu at (98.0, 85.5)
- added U6: motor driver 2, DRV8871DDAR:VREG_LM5017MR_NOPB, B.Cu at (103.5, 83.8)
- J1: value Screw_Terminal_01x03 -> distance 1
- J10: value Conn_01x03_Pin -> start; footprint Connector_PinHeader_2.54mm:PinHeader_1x03_P2.54mm_Vertical -> TerminalBlock:TerminalBlock_Xinya_XY308-2.54-3P_1x03_P2.54mm_Horizontal
- J11: value Screw_Terminal_01x02 -> motor 1
- J13: value Screw_Terminal_01x03 -> distance 6
- J14: value Screw_Terminal_01x03 -> line 4
- J15: value Screw_Terminal_01x03 -> line 3
- J2: value Screw_Terminal_01x03 -> distance 2
- J3: value Screw_Terminal_01x03 -> distance 3
- J4: value Screw_Terminal_01x03 -> distance 4
- J5: value Screw_Terminal_01x03 -> line 1
- J6: value Screw_Terminal_01x03 -> line 2
- J9: value Screw_Terminal_01x03 -> distance 5
- U3: value R-78K5.0-0.5 -> R-78K5.0-0.5 (vr 5v)
- U4: value R-78K5.0-0.5 -> R-78K5.0-0.5 (vr 3.3v)
- U5: value DRV8871DDAR -> motor driver 1
- moved U2 69.4 mm to (128.9, 61.0), turned to 90 degrees
- moved J11 56.3 mm to (146.5, 69.5), turned to 0 degrees
- moved J16 48.6 mm to (123.8, 69.5)
- moved J10 47.8 mm to (102.0, 70.0), turned to 0 degrees
- moved R1 41.6 mm to (83.1, 118.0)
- moved D1 40.1 mm to (83.4, 113.3)
- moved C1 40.0 mm to (153.5, 105.5)
- moved C2 40.0 mm to (160.5, 103.5)
- moved C3 40.0 mm to (91.0, 85.0)
- moved C4 40.0 mm to (161.0, 85.5)
- moved C5 40.0 mm to (137.1, 118.5)
- moved D2 40.0 mm to (119.0, 117.5)
- moved D3 40.0 mm to (129.4, 77.5)
- moved D4 40.0 mm to (142.9, 77.0)
- moved D6 40.0 mm to (130.1, 118.0)
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Connections:
- C1 pad 2: +3.3V -> GND
- C2 pad 2: +3.3V -> GND
- C3 pad 1: +3.3V -> GND
- C4 pad 2: +3.3V -> GND
- C5 pad 2: +3.3V -> GND
- C6 pad 2: +3.3V -> GND
- C7 pad 2: +3.3V -> GND
- D1 pad 1: +3.3V -> GND
- D2 pad 1: +3.3V -> GND
- D3 pad 1: +3.3V -> GND
- D4 pad 1: +3.3V -> GND
- D6 pad 1: +3.3V -> GND
- J1 pad 2: +3.3V -> GND
- J10 pad 2: +3.3V -> GND
- J11 pad 2: +3.3V -> Net-(J11-Pin_2)
- J13 pad 2: +3.3V -> GND
- J14 pad 1: +3.3V -> GND
- J15 pad 1: +3.3V -> GND
- J16 pad 1: +3.3V -> GND
- J2 pad 2: +3.3V -> GND
- J3 pad 2: +3.3V -> GND
- J4 pad 2: +3.3V -> GND
- J5 pad 1: +3.3V -> GND
- J6 pad 1: +3.3V -> GND
- J7 pad 1: +3.3V -> GND
- J9 pad 2: +3.3V -> GND
- R6 pad 1: +3.3V -> GND
- U1 pad 18: L4 -> unconnected-(U1-A4-Pad18)
- U1 pad 19: mdr1 -> unconnected-(U1-A5-Pad19)
- U1 pad 20: mdr2 -> L4
- U1 pad 25: mode 3 -> unconnected-(U1-A11-Pad25)
- U1 pad 26: mode 2 -> unconnected-(U1-A12-Pad26)
- U1 pad 27: mode 1 -> unconnected-(U1-A13-Pad27)
- U1 pad 38: mode 0 -> unconnected-(U1-A14-Pad38)
- U1 pad 39: int -> unconnected-(U1-A15-Pad39)
- U1 pad 40: sda -> mdr2
- U1 pad 41: scl -> mdr1
- U1 pad 6: motorapwm -> unconnected-(U1-OUT1D-Pad6)
- U1 pad 9: motorbpwm -> unconnected-(U1-OUT1C-Pad9)
- U1 pad GND1: +3.3V -> GND
- U1 pad GND2: +3.3V -> GND
- U1 pad GND3: +3.3V -> GND
- U2 pad 1: +3.3V -> GND
- U3 pad 2: +3.3V -> GND
- U4 pad 2: +3.3V -> GND
- U5 pad 1: +3.3V -> GND
- U5 pad 7: +3.3V -> GND
- U5 pad 8: Net-(J12-Pin_1) -> Net-(J11-Pin_2)
Routing:
- net GND: track 0.00 -> 53.2 mm
- net Net-(J11-Pin_1): track 0.00 -> 36.0 mm
- net Net-(J11-Pin_2): track 0.00 -> 35.9 mm
- net s5: track 31.8 -> 66.8 mm, vias 1 -> 2
- net int: track 29.5 -> 0.00 mm
- net L4: track 0.00 -> 28.7 mm
- net scl: track 28.0 -> 0.00 mm, vias 1 -> 0
- net sda: track 28.0 -> 0.00 mm, vias 1 -> 0
- net +5V: track 76.1 -> 55.9 mm, vias 3 -> 2
- net s6: track 0.00 -> 18.7 mm
- net Net-(J19-Pin_2): track 0.00 -> 18.1 mm
- net Net-(J19-Pin_1): track 0.00 -> 17.6 mm
- net +12V: track 53.0 -> 65.1 mm, vias 1 -> 0
- net +3.3V: track 201.7 -> 191.4 mm
- net CE: track 5.72 -> 0.00 mm, vias 1 -> 0
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Other:
- board size 83.5 x 57 mm -> 90.5 x 58 mm
- board text removed: "12"
- board text removed: "ma"
- board text removed: "mb"
- board text removed: "mdr1"
- board text removed: "mdr2"

Commit message: connected NRF
Routing:
- net MISO: track 0.00 -> 80.1 mm
- net CE: track 0.00 -> 47.7 mm, vias 0 -> 2
- net ~CSN: track 0.00 -> 44.6 mm, vias 0 -> 5
- net MOSI: track 0.00 -> 41.6 mm, vias 0 -> 2
- net SCK: track 0.00 -> 24.4 mm, vias 0 -> 1
- net +3.3V: track 191.4 -> 206.8 mm
- net GND: track 53.2 -> 64.1 mm
