File: 500g/Rata2i2.0/pcbn't/Schematic - Copy/Schematic.kicad_sch (KiCad schematic)
At the start: 39 parts, among them J1 Screw_Terminal_01x03, J10 Conn_01x03_Pin, J11 Screw_Terminal_01x02, J12 Screw_Terminal_01x02, J13 Screw_Terminal_01x03, J14 Screw_Terminal_01x03, J15 Screw_Terminal_01x03, J2 Screw_Terminal_01x03, J3 Screw_Terminal_01x03, J4 Screw_Terminal_01x03, J5 Screw_Terminal_01x03, J6 Screw_Terminal_01x03, J7 Battery, J8 Conn_01x08_Pin, J9 Screw_Terminal_01x03, SW1 SW_SPDT, SW2 SW_DIP_x04, U1 DEV-16771, U3 R-78K5.0-0.5, U4 R-78K5.0-0.5, U5 ROB-14450

Commit message: updated rata2i schematic
blah blah blah
Parts:
- added U2: NRF24L01_Breakout, RF_Module:nRF24L01_Breakout, symbol RF:NRF24L01_Breakout
Connections:
- net GND is gone; now on net +5V: C1.2, C2.2, C3.1, C4.2, C5.2, D1.1 (K), D2.1 (K), D3.1 (K), D4.1 (K), D6.1 (K), J1.2 (Pin_2), J10.2 (Pin_2), J13.2 (Pin_2), J14.1 (Pin_1), J15.1 (Pin_1), J2.2 (Pin_2), J3.2 (Pin_2), J4.2 (Pin_2), J5.1 (Pin_1), J6.1 (Pin_1), J7.1 (Pin_1), J8.2 (Pin_2), J9.2 (Pin_2), U1.GND1 (GND), U1.GND2 (GND), U1.GND3 (GND), U1.GND4 (GND), U1.GND5 (GND), U1.USB_GND1 (USB_GND), U1.USB_GND2 (USB_GND), U3.2 (GND), U4.2 (GND), U5.3 (GND), U5.8 (GND), U5.9 (GND)
- net +3.3V: now also J14.2 (Pin_2), J15.2 (Pin_2), J5.2 (Pin_2), J6.2 (Pin_2)
- net +5V: no longer J14.2 (Pin_2), J15.2 (Pin_2), J5.2 (Pin_2), J6.2 (Pin_2)
- net L2: no longer J14.3 (Pin_3), J15.3 (Pin_3)
- net s4: no longer J13.3 (Pin_3), J9.3 (Pin_3)
- net L3: now reaches U1.16 (A2)
- net L3: now also J15.3 (Pin_3)
- net L4: now reaches U1.18 (A4)
- net L4: now also J14.3 (Pin_3)
- net s6: now reaches U1.23 (A9)
- net s6: now also J13.3 (Pin_3)
- net s5: now reaches U1.24 (A10)
- net s5: now also J9.3 (Pin_3)
- no-connect marks 36 -> 32
Other:
- moved on the sheet: J9

Commit message: updated rata2i again
asdf
Parts:
- removed SW2: SW_DIP_x04, symbol Switch:SW_DIP_x04
- removed U5: ROB-14450, pleseowrk:driver, symbol motor driver:ROB-14450
- added C6, C7: 10 uF, Capacitor_SMD:C_0805_2012Metric, symbol Device:C
- added R6: R_US, Resistor_SMD:R_0805_2012Metric, symbol Device:R_US
- added U5: DRV8871DDAR, DRV8871DDAR:VREG_LM5017MR_NOPB, symbol DRV8871DDAR:DRV8871DDAR
- J11, J12: footprint TerminalBlock:TerminalBlock_Xinya_XY308-2.54-2P_1x02_P2.54mm_Horizontal -> (none)
Connections:
- net +3.3V is gone; now on net +12V: C5.1, J10.3 (Pin_3), J14.2 (Pin_2), J15.2 (Pin_2), J5.2 (Pin_2), J6.2 (Pin_2), J8.1 (Pin_1), U1.3.3V_1 (3.3V), U1.3.3V_2 (3.3V), U1.3.3V_3 (3.3V), U4.3 (+VOUT)
- net +12V: now also C1.2, C2.2, C3.1, C4.2, C5.2, D1.1 (K), D2.1 (K), D3.1 (K), D4.1 (K), D6.1 (K), J1.1 (Pin_1), J1.2 (Pin_2), J10.2 (Pin_2), J11.2 (Pin_2), J12.2 (Pin_2), J13.1 (Pin_1), J13.2 (Pin_2), J14.1 (Pin_1), J15.1 (Pin_1), J2.1 (Pin_1), J2.2 (Pin_2), J3.1 (Pin_1), J3.2 (Pin_2), J4.1 (Pin_1), J4.2 (Pin_2), J5.1 (Pin_1), J6.1 (Pin_1), J7.1 (Pin_1), J8.2 (Pin_2), J9.1 (Pin_1), J9.2 (Pin_2), U1.GND1 (GND), U1.GND2 (GND), U1.GND3 (GND), U1.GND4 (GND), U1.GND5 (GND), U1.USB_GND1 (USB_GND), U1.USB_GND2 (USB_GND), U2.1 (GND), U2.2 (VCC), U3.2 (GND), U4.2 (GND), C6.1, C6.2, C7.1, C7.2, R6.1, U5.1 (GND), U5.5 (VM), U5.7 (PGND)
- net +5V: no longer C1.2, C2.2, C3.1, C4.2, C5.2, D1.1 (K), D2.1 (K), D3.1 (K), D4.1 (K), D6.1 (K), J1.1 (Pin_1), J1.2 (Pin_2), J10.2 (Pin_2), J13.1 (Pin_1), J13.2 (Pin_2), J14.1 (Pin_1), J15.1 (Pin_1), J2.1 (Pin_1), J2.2 (Pin_2), J3.1 (Pin_1), J3.2 (Pin_2), J4.1 (Pin_1), J4.2 (Pin_2), J5.1 (Pin_1), J6.1 (Pin_1), J7.1 (Pin_1), J8.2 (Pin_2), J9.1 (Pin_1), J9.2 (Pin_2), U1.GND1 (GND), U1.GND2 (GND), U1.GND3 (GND), U1.GND4 (GND), U1.GND5 (GND), U1.USB_GND1 (USB_GND), U1.USB_GND2 (USB_GND), U3.2 (GND), U4.2 (GND)
- net mdr1: now also U5.2 (IN2)
- net mdr2: now also U5.3 (IN1)
- net at J11.1 (Pin_1): now also U5.6 (OUT1)
- net at J12.1 (Pin_1): now also U5.8 (OUT2)
- net CE: now reaches U2.3 (CE)
- net CE: now also U1.1 (TX1)
- net ~CSN: now reaches U2.4 (~{CSN})
- net ~CSN: now also U1.7 (RX2)
- net SCK: now reaches U2.5 (SCK)
- net SCK: now also U1.13 (SCK)
- net MOSI: now reaches U2.6 (MOSI)
- net MOSI: now also U1.11 (MOSI)
- net MISO: now reaches U2.7 (MISO)
- net MISO: now also U1.12 (MISO)
- new net: R6.2, U5.4 (ILIM)
- no-connect marks 32 -> 30
Other:
- moved on the sheet: J8, R4, U2

Commit message: IT WORKS!!!!!
yippee
Parts:
- J11, J12: footprint (none) -> TerminalBlock:TerminalBlock_Xinya_XY308-2.54-2P_1x02_P2.54mm_Horizontal
Connections:
- no-connect marks 30 -> 31
Changed lines of the file:
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@@
 	)
 	(no_connect
+		(at 255.27 135.89)
+	)
+	(no_connect
 		(at 60.96 72.39)
 	)
@@
 	(wire
 		(pts
-			(xy 234.95 96.52) (xy 237.49 96.52)
-		)
-		(stroke
-			(width 0)
-			(type default)
-		)
-	)
-	(wire
-		(pts
 			(xy 236.22 58.42) (xy 236.22 59.69)
 		)
@@
 	(wire
 		(pts
+			(xy 234.95 96.52) (xy 237.49 96.52)
+		)
+		(stroke
+			(width 0)
+			(type default)
+		)
+	)
+	(wire
+		(pts
 			(xy 58.42 46.99) (xy 60.96 46.99)
 		)
@@
 	)
 	(label "10 µF"
-		(at 63.5 184.15 0)
-		(effects
-			(font
-				(size 1.27 1.27)
-			)
-			(justify left bottom)
-		)
-	)
-	(label "10 µF"
 		(at 124.46 172.72 0)
 		(effects
@@
 		)
 	)
-	(label "10 µF"
-		(at 63.5 158.75 0)
-		(effects
-			(font
-				(size 1.27 1.27)
-			)
-			(justify left bottom)
-		)
-	)
 	(label "200 Ω"
 		(at 46.99 78.74 180)
@@
 			)
 		)
-		(property "Footprint" ""
+		(property "Footprint" "TerminalBlock:TerminalBlock_Xinya_XY308-2.54-2P_1x02_P2.54mm_Horizontal"
 			(at 267.97 140.97 0)
 			(effects
@@
 			)
 		)
-		(property "Footprint" ""
+		(property "Footprint" "TerminalBlock:TerminalBlock_Xinya_XY308-2.54-2P_1x02_P2.54mm_Horizontal"
 			(at 273.05 148.59 0)
 			(effects
@@
 	(symbol
 		(lib_id "power:+3.3V")
-		(at 231.14 91.44 180)
+		(at 231.14 91.44 90)
 		(unit 1)
 		(exclude_from_sim no)
@@
 		(dnp no)
 		(property "Reference" "#PWR060"
-			(at 231.14 87.63 0)
+			(at 234.95 91.44 0)
 			(effects
 				(font
@@
 		)
 		(property "Value" "+3.3V"
-			(at 231.394 96.774 0)
+			(at 225.806 91.694 0)
 			(effects
 				(font

Commit message: All parts done!
Need to wire :(
Parts:
- added J16: Screw_Terminal_01x07, TerminalBlock:TerminalBlock_Xinya_XY308-2.54-7P_1x07_P2.54mm_Horizontal, symbol Connector:Screw_Terminal_01x07
Connections:
- net +12V: no longer C1.2, C2.2, C3.1, C4.2, C5.1, C5.2, C6.2, C7.2, D1.1 (K), D2.1 (K), D3.1 (K), D4.1 (K), D6.1 (K), J1.1 (Pin_1), J1.2 (Pin_2), J10.2 (Pin_2), J10.3 (Pin_3), J11.2 (Pin_2), J12.2 (Pin_2), J13.1 (Pin_1), J13.2 (Pin_2), J14.1 (Pin_1), J14.2 (Pin_2), J15.1 (Pin_1), J15.2 (Pin_2), J2.1 (Pin_1), J2.2 (Pin_2), J3.1 (Pin_1), J3.2 (Pin_2), J4.1 (Pin_1), J4.2 (Pin_2), J5.1 (Pin_1), J5.2 (Pin_2), J6.1 (Pin_1), J6.2 (Pin_2), J7.1 (Pin_1), J8.1 (Pin_1), J8.2 (Pin_2), J9.1 (Pin_1), J9.2 (Pin_2), R6.1, U1.3.3V_1 (3.3V), U1.3.3V_2 (3.3V), U1.3.3V_3 (3.3V), U1.GND1 (GND), U1.GND2 (GND), U1.GND3 (GND), U1.GND4 (GND), U1.GND5 (GND), U1.USB_GND1 (USB_GND), U1.USB_GND2 (USB_GND), U2.1 (GND), U2.2 (VCC), U3.2 (GND), U4.2 (GND), U4.3 (+VOUT), U5.1 (GND), U5.7 (PGND)
- net CE: now also J16.2 (Pin_2)
- net MISO: now also J16.5 (Pin_5)
- net MOSI: now also J16.6 (Pin_6)
- net SCK: now also J16.4 (Pin_4)
- net ~CSN: now also J16.3 (Pin_3)
- new net +3.3V: C1.2, C2.2, C3.1, C4.2, C5.1, C5.2, C6.2, C7.2, D1.1 (K), D2.1 (K), D3.1 (K), D4.1 (K), D6.1 (K), J1.1 (Pin_1), J1.2 (Pin_2), J10.2 (Pin_2), J10.3 (Pin_3), J11.2 (Pin_2), J12.2 (Pin_2), J13.1 (Pin_1), J13.2 (Pin_2), J14.1 (Pin_1), J14.2 (Pin_2), J15.1 (Pin_1), J15.2 (Pin_2), J16.1 (Pin_1), J16.7 (Pin_7), J2.1 (Pin_1), J2.2 (Pin_2), J3.1 (Pin_1), J3.2 (Pin_2), J4.1 (Pin_1), J4.2 (Pin_2), J5.1 (Pin_1), J5.2 (Pin_2), J6.1 (Pin_1), J6.2 (Pin_2), J7.1 (Pin_1), J8.1 (Pin_1), J8.2 (Pin_2), J9.1 (Pin_1), J9.2 (Pin_2), R6.1, U1.3.3V_1 (3.3V), U1.3.3V_2 (3.3V), U1.3.3V_3 (3.3V), U1.GND1 (GND), U1.GND2 (GND), U1.GND3 (GND), U1.GND4 (GND), U1.GND5 (GND), U1.USB_GND1 (USB_GND), U1.USB_GND2 (USB_GND), U2.1 (GND), U2.2 (VCC), U3.2 (GND), U4.2 (GND), U4.3 (+VOUT), U5.1 (GND), U5.7 (PGND)

Commit message: 2 motor drivers, 2 less sensors :D
mostly connected but it REALLY doesn't like the motor drivers, maybe moving to the normal side will make it better?
Parts:
- removed J12: Screw_Terminal_01x02, TerminalBlock:TerminalBlock_Xinya_XY308-2.54-2P_1x02_P2.54mm_Horizontal, symbol Connector:Screw_Terminal_01x02
- removed J8: Conn_01x08_Pin, Connector_PinHeader_2.54mm:PinHeader_1x08_P2.54mm_Vertical, symbol Connector:Conn_01x08_Pin
- added C8, C9: 10 uF, Capacitor_SMD:C_0805_2012Metric, symbol Device:C
- added J19: motor 2, TerminalBlock:TerminalBlock_Xinya_XY308-2.54-2P_1x02_P2.54mm_Horizontal, symbol Connector:Screw_Terminal_01x02
- added R7: R_US, Resistor_SMD:R_0805_2012Metric, symbol Device:R_US
- added U6: motor driver 2, DRV8871DDAR:VREG_LM5017MR_NOPB, symbol DRV8871DDAR:DRV8871DDAR
- J1: value Screw_Terminal_01x03 -> distance 1
- J10: value Conn_01x03_Pin -> start; footprint Connector_PinHeader_2.54mm:PinHeader_1x03_P2.54mm_Vertical -> TerminalBlock:TerminalBlock_Xinya_XY308-2.54-3P_1x03_P2.54mm_Horizontal
- J11: value Screw_Terminal_01x02 -> motor 1
- J13: value Screw_Terminal_01x03 -> distance 6
- J14: value Screw_Terminal_01x03 -> line 4
- J15: value Screw_Terminal_01x03 -> line 3
- J2: value Screw_Terminal_01x03 -> distance 2
- J3: value Screw_Terminal_01x03 -> distance 3
- J4: value Screw_Terminal_01x03 -> distance 4
- J5: value Screw_Terminal_01x03 -> line 1
- J6: value Screw_Terminal_01x03 -> line 2
- J9: value Screw_Terminal_01x03 -> distance 5
- U3: value R-78K5.0-0.5 -> R-78K5.0-0.5 (vr 5v)
- U4: value R-78K5.0-0.5 -> R-78K5.0-0.5 (vr 3.3v)
- U5: value DRV8871DDAR -> motor driver 1
Connections:
- net scl is gone; now on net mdr1: U1.41 (A17)
- net sda is gone; now on net mdr2: U1.40 (A16)
- net +12V: now also C8.1, C9.1, U6.5 (VM)
- net +3.3V: no longer C1.2, C2.2, C3.1, C4.2, C5.2, C6.2, C7.2, D1.1 (K), D2.1 (K), D3.1 (K), D4.1 (K), D6.1 (K), J1.2 (Pin_2), J10.2 (Pin_2), J11.2 (Pin_2), J13.2 (Pin_2), J14.1 (Pin_1), J15.1 (Pin_1), J16.1 (Pin_1), J2.2 (Pin_2), J3.2 (Pin_2), J4.2 (Pin_2), J5.1 (Pin_1), J6.1 (Pin_1), J7.1 (Pin_1), J9.2 (Pin_2), R6.1, U1.GND1 (GND), U1.GND2 (GND), U1.GND3 (GND), U1.GND4 (GND), U1.GND5 (GND), U1.USB_GND1 (USB_GND), U1.USB_GND2 (USB_GND), U2.1 (GND), U3.2 (GND), U4.2 (GND), U5.1 (GND), U5.7 (PGND)
- net L4: now also U1.20 (A6); no longer U1.18 (A4)
- net mdr1: no longer U1.19 (A5)
- net mdr2: no longer U1.20 (A6)
- net mdr3: now also U6.2 (IN2)
- net mdr4: now also U6.3 (IN1)
- net at U5.8 (OUT2): now also J11.2 (Pin_2)
- net int: no longer names the net of U1.39 (A15)
- net mode 0: no longer names the net of U1.38 (A14)
- net mode 1: no longer names the net of U1.27 (A13)
- net mode 2: no longer names the net of U1.26 (A12)
- net mode 3: no longer names the net of U1.25 (A11)
- net motorapwm: no longer names the net of U1.6 (OUT1D)
- net motorbpwm: no longer names the net of U1.9 (OUT1C)
- new net: R7.2, U6.4 (ILIM)
- new net: J19.1 (Pin_1), U6.6 (OUT1)
- new net: J19.2 (Pin_2), U6.8 (OUT2)
- new net GND: C1.2, C2.2, C3.1, C4.2, C5.2, C6.2, C7.2, C8.2, C9.2, D1.1 (K), D2.1 (K), D3.1 (K), D4.1 (K), D6.1 (K), J1.2 (Pin_2), J10.2 (Pin_2), J13.2 (Pin_2), J14.1 (Pin_1), J15.1 (Pin_1), J16.1 (Pin_1), J2.2 (Pin_2), J3.2 (Pin_2), J4.2 (Pin_2), J5.1 (Pin_1), J6.1 (Pin_1), J7.1 (Pin_1), J9.2 (Pin_2), R6.1, R7.1, U1.GND1 (GND), U1.GND2 (GND), U1.GND3 (GND), U1.GND4 (GND), U1.GND5 (GND), U1.USB_GND1 (USB_GND), U1.USB_GND2 (USB_GND), U2.1 (GND), U3.2 (GND), U4.2 (GND), U5.1 (GND), U5.7 (PGND), U6.1 (GND), U6.7 (PGND)
- no-connect marks 31 -> 38
Other:
- note added: "<- motor drivers ->"
- note added: "note: joe and cody said the footprint and symbol don't look right?"
- note removed: "imu"
- note removed: "led (just 1 lmao)"
- note removed: "motor driver"
- moved on the sheet: C6, C7, D1, D4, J10, J11, J13, J14, J15, J16, J4, J5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

Commit message: connected everything that wasn't connected
please someone check if this is sussy
Parts:
- removed J15: line 3, TerminalBlock:TerminalBlock_Xinya_XY308-2.54-3P_1x03_P2.54mm_Horizontal, symbol Connector:Screw_Terminal_01x03
- added R8: R_US, Resistor_SMD:R_0805_2012Metric, symbol Device:R_US
- added SW2: SW_Push, Button_Switch_THT:SW_PUSH_6mm, symbol Switch:SW_Push
Connections:
- net +3.3V: now also SW2.1
- net GND: now also R8.2
- net GPIO pin: now reaches U1.25 (A11)
- net GPIO pin: now also R8.1, SW2.2
- no-connect marks 38 -> 37

Commit message: Changed motor driver pins
mdr1 - 28
mdr2 - 29
mdr3 - 18
mdr4 - 22
Connections:
- net mdr1: now also U1.28 (RX7); no longer U1.41 (A17)
- net mdr2: now also U1.29 (TX7); no longer U1.40 (A16)
- net mdr3: now also U1.18 (A4); no longer U1.21 (A7)

Commit message: Working on making power traces lorge
Parts:
- C6, C8: value 10 uF -> .1 uF
- C7, C9: value 10 uF -> 47 uF
- renumbered R6 to R6(30k)1, R7 to R7(30k)1
Changed lines of the file:
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@@
 	)
 	(label "200 Ω"
-		(at 46.99 78.74 180)
+		(at 44.45 80.01 180)
 		(effects
 			(font
@@
 		(dnp no)
 		(fields_autoplaced yes)
-		(property "Reference" "R7"
+		(property "Reference" "R7(30k)1"
 			(at 160.02 100.3299 0)
 			(effects
@@
 			(project "Schematic"
 				(path "/68c7ddae-445d-49f5-81ac-f496a7c86e74"
-					(reference "R7")
+					(reference "R7(30k)1")
 					(unit 1)
 				)
@@
 			)
 		)
-		(property "Value" "10 uF"
+		(property "Value" "47 uF"
 			(at 274.32 95.2499 0)
 			(effects
@@
 			)
 		)
-		(property "Value" "10 uF"
+		(property "Value" ".1 uF"
 			(at 189.992 94.996 0)
 			(effects
@@
 			)
 		)
-		(property "Value" "10 uF"
+		(property "Value" "47 uF"
 			(at 207.01 95.2499 0)
 			(effects
@@
 			)
 		)
-		(property "Value" "10 uF"
+		(property "Value" ".1 uF"
 			(at 256.794 93.472 0)
 			(effects
@@
 		(dnp no)
 		(fields_autoplaced yes)
-		(property "Reference" "R6"
+		(property "Reference" "R6(30k)1"
 			(at 224.79 100.3299 0)
 			(effects
@@
 			(project ""
 				(path "/68c7ddae-445d-49f5-81ac-f496a7c86e74"
-					(reference "R6")
+					(reference "R6(30k)1")
 					(unit 1)
 				)
