File: 500g/Spi-v3/Spii_v3/Spii_v3.kicad_pcb (KiCad board)
At the start: 2 copper layers, 45 parts, among them J10 Right Motor, J7 Conn_01x02, J9 Left Motor, SW1 SW_Push, SW2 1101M2S3CQE2, SW3 1101M2S3CQE2, U2 TSR 1-2450

Commit message: made some pcb
Parts:
- moved Teensy 4.0 186.6 mm to (208.5, 139.1), turned to -90 degrees
- moved F1 183.7 mm to (210.3, 142.5), turned to 180 degrees
- moved U2 162.1 mm to (224.2, 137.0), turned to 90 degrees
- moved D5 153.7 mm to (203.5, 122.0), turned to 90 degrees
- moved H1 146.6 mm to (222.2, 123.8)
- moved TV1 143.8 mm to (179.4, 127.5), turned to 90 degrees
- moved J7 142.3 mm to (209.0, 126.0)
- moved D4 136.8 mm to (183.5, 122.0), turned to 90 degrees
- moved D3 135.2 mm to (180.0, 122.0), turned to 90 degrees
- moved SIGNAL1 135.1 mm to (174.9, 143.5), turned to 90 degrees
- moved D2 133.9 mm to (176.5, 122.0), turned to 90 degrees
- moved C2 128.0 mm to (191.6, 100.1)
- moved C3 128.0 mm to (191.6, 103.5)
- moved C4 128.0 mm to (191.6, 106.8)
- moved C5 128.0 mm to (191.6, 110.2)
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Other:
- board outline added: 95 x 30 mm

Commit message: added spi and more pcb progress
Parts:
- moved LN_PWR1 71.0 mm to (172.0, 143.5), turned to 90 degrees
- moved IR_PWR1 67.8 mm to (165.8, 143.5), turned to 90 degrees
- moved J10 58.5 mm to (160.5, 123.5), turned to 90 degrees
- moved J9 43.0 mm to (196.8, 123.5), turned to 90 degrees
- moved START_MOD1 6.73 mm to (171.5, 128.9), turned to 0 degrees
- moved TV1 6.18 mm to (185.5, 127.0), turned to -90 degrees
- moved SIGNAL1 3.39 mm to (178.3, 143.5)
- moved D6 1.25 mm to (148.0, 130.2)
- moved SW1 1.25 mm to (144.8, 122.2)

Commit message: added some gerbs
Parts:
- added G***: LOGO, spy:spy23inverted, F.Cu at (170.1, 136.9)
- -       +: renamed from D4
- -       +: renamed from D6
- -       +: renamed from D5
- -       +: renamed from D3
- -       +: renamed from D2
- -       +: renamed from J10
- 0.1uF: renamed from C3; moved to B.Cu
- 0.1uF: renamed from C6; moved to B.Cu
- 18kΩ: renamed from R_L_MTR1; moved to B.Cu
- 18kΩ: renamed from R_R_MTR1; moved to B.Cu
- 1kΩ: renamed from R3; footprint Resistor_SMD:R_0805_2012Metric_Pad1.20x1.40mm_HandSolder -> Resistor_SMD:R_1206_3216Metric_Pad1.30x1.75mm_HandSolder
- 500Ω: renamed from R_BUTTON1; footprint Resistor_SMD:R_0805_2012Metric_Pad1.20x1.40mm_HandSolder -> Resistor_SMD:R_1206_3216Metric_Pad1.30x1.75mm_HandSolder
- 50uF: renamed from C4; moved to B.Cu
- 50uF: renamed from C5; moved to B.Cu
- L_IR: renamed from LS_L_IR1; moved to B.Cu
- M_IR: renamed from LS_M_IR1; moved to B.Cu
- R_IR: renamed from LS_R_IR1; moved to B.Cu
- R_LN  L_LN  R_IR  M_IR  L_IR: renamed from SIGNAL1
- S_MOD: renamed from LS_START_MOD1; moved to B.Cu
- moved L_IR 69.1 mm to (213.2, 133.8), turned to 180 degrees
- moved M_IR 64.9 mm to (208.2, 133.8), turned to 180 degrees
- moved R_IR 61.1 mm to (203.2, 133.8), turned to 180 degrees
- moved 500Ω 58.9 mm to (156.5, 122.9), turned to -90 degrees
- moved S_MOD 57.6 mm to (198.2, 133.8), turned to 180 degrees
- moved 10kΩ 55.0 mm to (161.5, 137.2), turned to -90 degrees
- moved 10kΩ 52.8 mm to (159.0, 137.2), turned to -90 degrees
- moved 500Ω 51.0 mm to (176.5, 123.0), turned to -90 degrees
- moved L_MOTOR_DRIVER1 48.3 mm to (183.8, 135.8), turned to 90 degrees
- moved 18kΩ 47.9 mm to (164.0, 137.2), turned to -90 degrees
- moved 500Ω 47.6 mm to (180.0, 123.0), turned to -90 degrees
- moved 500Ω 47.4 mm to (203.5, 123.0), turned to -90 degrees
- moved 0.1uF 45.9 mm to (156.5, 129.8), turned to 90 degrees
- moved 0.1uF 45.9 mm to (154.0, 129.8), turned to -90 degrees
- moved 500Ω 44.4 mm to (183.5, 122.9), turned to -90 degrees
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- renumbered D1 to -+, C2 to 0.1uF, R2 to 10kΩ, R1 to 10kΩ, LED_R3 to 500Ω, LED_R4 to 500Ω, LED_R5 to 500Ω, LED_R1 to 500Ω, LED_R2 to 500Ω, IR_PWR1 to IR_PWR, LN_PWR1 to LN_PWR
Routing:
- net +3.3V: track 0.00 -> 194.0 mm, vias 0 -> 4
- net +5V: track 0.00 -> 135.7 mm, vias 0 -> 2
- net LED4: track 0.00 -> 103.5 mm, vias 0 -> 3
- net LED5: track 0.00 -> 87.8 mm, vias 0 -> 1
- net +3.3|5: track 0.00 -> 86.2 mm, vias 0 -> 1
- net +12V: track 0.00 -> 82.0 mm, vias 0 -> 3
- net Net-(J7-Pin_2): track 0.00 -> 78.4 mm
- net Button: track 0.00 -> 67.4 mm, vias 0 -> 1
- net GND: track 0.00 -> 64.6 mm, vias 0 -> 14
- net LED1: track 0.00 -> 59.9 mm
- net LCD_SCL: track 0.00 -> 48.5 mm, vias 0 -> 2
- net LED2: track 0.00 -> 46.9 mm, vias 0 -> 1
- net DIP1: track 0.00 -> 46.9 mm, vias 0 -> 1
- net LED3: track 0.00 -> 46.2 mm, vias 0 -> 1
- net LCD_SDA: track 0.00 -> 46.0 mm, vias 0 -> 1
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- added copper zone on B.Cu, net GND
- added copper zone on F.Cu, net GND
Other:
- board text added: "+ -"
- board text added: "+ - S"
- board text added: "+5V"
- board text added: "- + SCL SDA"
- board text added: "3.3V"
- board text added: "DIP2 DIP1 PUSH"
- board text added: "IR_PWR"
- board text added: "LED5 LED4 LED3 LED2 LED1"
- board text added: "OFF"
- board text added: "ON"
- board text added: "R_IR M_IR L_IR R_IN2 R_IN1 L_IN2 L_IN1 GND"
- board text added: "R_LN L_LN 3V3 GND 5V"
- board text added: "SDA SCL"
- board text added: "START"
- board text added: "Xander Riddle 10/2/2025"

Commit message: finishing touches
Parts:
- removed 1kΩ: 1kΩ, Resistor_SMD:R_1206_3216Metric_Pad1.30x1.75mm_HandSolder
- D2, D3, D4, D5, D6, J10: renamed from -       +
- SIGNAL1: renamed from R_LN  L_LN  R_IR  M_IR  L_IR
- moved LS_M_IR1 0.25 mm to (208.2, 134.0)
- moved LS_R_IR1 0.25 mm to (203.2, 134.0)
- moved LS_START_MOD1 0.25 mm to (198.2, 134.0)
- moved LS_L_IR1 0.10 mm to (213.2, 133.8)
- renumbered 0.1uF to C2, 0.1uF to C3, 50uF to C4, 50uF to C5, 0.1uF to C6, -+ to D1, IR_PWR to IR_PWR1, 500Ω to LED_R1, 500Ω to LED_R2, 500Ω to LED_R3, 500Ω to LED_R4, 500Ω to LED_R5, LN_PWR to LN_PWR1, L_IR to LS_L_IR1, M_IR to LS_M_IR1, R_IR to LS_R_IR1, S_MOD to LS_START_MOD1, 10kΩ to R1, 10kΩ to R2, 500Ω to R_BUTTON1, 18kΩ to R_L_MTR1, 18kΩ to R_R_MTR1
Connections:
- LS_START_MOD1 pad 1: +3.3|5 -> +5V
- LS_START_MOD1 pad 5: +3.3|5 -> +5V
Routing:
- net +5V: track 135.7 -> 165.6 mm
- net GND: track 64.6 -> 81.2 mm, vias 14 -> 16
- net Net-(J9-Pin_2): track 41.1 -> 27.3 mm, vias 4 -> 5
- net +3.3V: track 194.0 -> 200.1 mm
- net M_IR: track 5.16 -> 7.35 mm
- net +3.3|5: track 86.2 -> 84.7 mm
- net Button: track 67.4 -> 66.5 mm, vias 1 -> 0
- net DIP2: track 38.5 -> 39.3 mm
- net Net-(J9-Pin_1): track 26.7 -> 25.9 mm
- net R_IN2: track 42.6 -> 41.8 mm
Other:
- board text added: "- +"
- board text added: "0.1uF"
- board text added: "10kΩ"
- board text added: "18kΩ"
- board text added: "500Ω"
- board text added: "50uF"
- board text added: "LN_PWR"
- board text added: "L_IR"
- board text added: "M_IR"
- board text added: "R_IR"
- board text added: "R_LN L_LN R_IR M_IR L_IR"
- board text added: "S_MOD"
