File: 500g/Luigi/Luigi.kicad_sch (KiCad schematic)
At the start: 28 parts, among them J3 Motor 2, J4 Motor 1, SW1 SW_DIP_x02, SW2 SW_Push, U1 DRV8871DDA, U2 DRV8871DDA, U3 L78L05_TO92

Commit message: Fixed the switches
Parts:
- removed BT_SW1: SW_SPST, Button_Switch_THT:SW_DIP_SPSTx01_Slide_6.7x4.1mm_W7.62mm_P2.54mm_LowProfile, symbol Switch:SW_SPST
- added S1: 500SSP1S2M2QEA, Luigi:SW_500SSP1S2M2QEA, symbol SPDT_slide_switch:500SSP1S2M2QEA
Connections:
- net BV: now also U1.5 (VM), U2.5 (VM); no longer SW1.1, SW1.2
- net Reg5: now also SW1.1, SW1.2
- net dip4: now reaches SW1.4
- net dip4: now also A1.19 (A0); no longer U2.5 (VM)
- net dip3: now reaches SW1.3
- net dip3: now also A1.20 (A1); no longer U1.5 (VM)
- net at F1.2: now also S1.1
- net at BT1.2 (-): now also S1.2
- net at lineSensor1.3 (Pin_3): now also A1.21 (A2); no longer A1.19 (A0)
- net at L_dis1.3 (Pin_3): now also A1.22 (A3); no longer A1.20 (A1)
- no-connect marks 0 -> 1
Other:
- moved on the sheet: F1, SW1
