File: 500g/Luigi/Luigi.kicad_sch (KiCad schematic)
At the start: 28 parts, among them J3 Motor 2, J4 Motor 1, SW1 SW_DIP_x02, SW2 SW_Push, U1 DRV8871DDA, U2 DRV8871DDA, U3 L78L05_TO92

Commit message: Levi v1
Parts:
- added R3, R4, R5: R_Small_US, Resistor_SMD:R_0805_2012Metric, symbol Device:R_Small_US
Connections:
- net GND: now also R3.1, R4.1, R5.2
- net at A1.25 (A6), SW2.1: now also R5.1
- net dip3 renamed dip13
- net dip13: now also R3.2
- net dip4 renamed dip14
- net dip14: now also R4.2
