File: 500g/Luigi/Luigi.kicad_pcb (KiCad board)
At the start: 2 copper layers, 99 x 40 mm, 33 parts, among them J3 Motor 2, J4 Motor 1, SW1 SW_DIP_x02, SW2 SW_Push, U1 DRV8871DDA, U2 DRV8871DDA, U3 L78L05_TO92

Commit message: Levi v1
Parts:
- added R3: R_Small_US, Resistor_SMD:R_0805_2012Metric, F.Cu at (103.0, 98.5)
- added R4: R_Small_US, Resistor_SMD:R_0805_2012Metric, F.Cu at (109.5, 98.5)
- added R5: R_Small_US, Resistor_SMD:R_0805_2012Metric, B.Cu at (174.0, 86.0)
- 0.1uF1, 10uF2: moved to B.Cu
- moved 0.1uF1 4.23 mm to (121.0, 105.0), turned to 180 degrees
- moved 10uF2 1.50 mm to (121.0, 109.5), turned to 180 degrees
- moved G*** 1.50 mm to (187.5, 104.0)
- moved SW1 1.23 mm to (107.3, 86.5)
- moved L_dis1 0.50 mm to (130.0, 80.5)
- moved FL_dis1 0.28 mm to (141.0, 80.5)
- moved FC_dis1 0.25 mm to (152.0, 80.5)
Connections:
- net dip3 renamed dip13
- net dip4 renamed dip14
Routing:
- net Reg5: track 162.4 -> 155.9 mm
- net BV: track 70.1 -> 75.7 mm
- net Net-(A1-A6): track 28.9 -> 33.4 mm
- net dip13: track 44.2 -> 47.1 mm
- net dip14: track 39.2 -> 42.0 mm
