File: Skibidi-Second-Edition/Skibidi-Second_Edition/Skibidi-Second_Edition.kicad_pcb (KiCad board)
At the start: 2 copper layers, 93.2 x 58.4 mm, 68 parts, among them IC1 TEENSY_4.1, J1 Screw_Terminal_01x03, J10 Screw_Terminal_01x03, J12 12V, J13 Conn_01x03_Pin, J14 Conn_01x08_Pin, J15 Conn_02x05_Odd_Even, J16 P78E05-1000, J17 Conn_01x04_Pin, J2 Screw_Terminal_01x03, J3 Screw_Terminal_01x03, J4 Screw_Terminal_01x03, J5 Screw_Terminal_01x03, J6 Screw_Terminal_01x03, J8 Screw_Terminal_01x03, J9 Screw_Terminal_01x03, SW1 SW_Nidec_CAS-120A1, SW2 210-4MS

Commit message: bobbi
Parts:
- removed C11, C9: 0.1uF, Capacitor_SMD:C_0805_2012Metric
- removed J9: Screw_Terminal_01x03, Connector_JST:JST_EH_B3B-EH-A_1x03_P2.50mm_Vertical
- added C10: 0.1uF, Capacitor_SMD:C_0805_2012Metric, B.Cu at (105.4, 29.3)
- added C4: 0.1uF, Capacitor_SMD:C_0805_2012Metric, F.Cu at (114.8, 27.6)
- added J7: Screw_Terminal_01x03, Connector_JST:JST_PH_B3B-PH-K_1x03_P2.00mm_Vertical, F.Cu at (111.8, 33.1)
- added R25: 10k, Capacitor_SMD:C_1206_3216Metric, B.Cu at (50.0, 68.4)
- C1, C2, C3, C5, C6, C8: moved to B.Cu
- J1, J10, J2, J3, J4, J5, J6, J8: footprint Connector_JST:JST_EH_B3B-EH-A_1x03_P2.50mm_Vertical -> Connector_JST:JST_PH_B3B-PH-K_1x03_P2.00mm_Vertical
- moved C7 108.0 mm to (36.8, 27.6)
- moved C12 76.1 mm to (51.5, 60.2), turned to 90 degrees
- moved J1 73.1 mm to (33.9, 33.1)
- moved J10 72.4 mm to (102.3, 33.2)
- moved J14 56.5 mm to (87.6, 55.9), turned to 90 degrees
- moved J13 55.0 mm to (79.1, 76.2), turned to 90 degrees
- moved J5 34.6 mm to (64.1, 33.2)
- moved C5 30.6 mm to (67.2, 29.6)
- moved J6 19.6 mm to (54.1, 33.1)
- moved J2 18.1 mm to (92.8, 33.1)
- moved C3 16.8 mm to (77.0, 29.7)
- moved R15 14.9 mm to (100.9, 27.9)
- moved C6 13.6 mm to (86.4, 29.5)
- moved C1 13.1 mm to (47.4, 30.0)
- moved J4 12.8 mm to (73.9, 33.1)
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Connections:
- IC1 pad 18: unconnected-(IC1-A4-Pad18) -> SDA1
- IC1 pad 19: unconnected-(IC1-A5-Pad19) -> SCL1
- IC1 pad 33: unconnected-(IC1-MCLK2-Pad33) -> DIP2
- J1 pad 1: GND -> LN1
- J1 pad 2: +3.3V -> GND
- J1 pad 3: LN1 -> +3.3V
- J10 pad 1: GND -> OM1
- J10 pad 2: +3.3V -> GND
- J10 pad 3: LN3 -> +12V
- J14 pad 3: SDA -> SDA1
- J14 pad 4: SCL -> SCL1
- J15 pad 3: PWMA -> PWMB
- J15 pad 4: PWMB -> PWMA
- J15 pad 5: BDC1 -> BDC11
- J15 pad 7: BDC11 -> BDC1
- J2 pad 1: +12V -> OM2
- J2 pad 3: OM1 -> +12V
- J3 pad 1: +12V -> OM3
- J3 pad 3: OM3 -> +12V
- J4 pad 1: +12V -> OM4
- J4 pad 3: OM5 -> +12V
- J5 pad 1: +12V -> OM5
- J5 pad 3: OM2 -> +12V
- J6 pad 1: +12V -> OM6
- J6 pad 3: OM4 -> +12V
- J8 pad 1: +12V -> OM7
- J8 pad 3: OM7 -> +12V
- SW2 pad 3: unconnected-(SW2-Pad3) -> +3.3V
- SW2 pad 6: unconnected-(SW2-Pad6) -> DIP2
Routing:
- net +3.3V: track 0.00 -> 218.0 mm
- net LN1: track 0.00 -> 70.4 mm, vias 0 -> 2
- net +5V: track 11.2 -> 67.3 mm
- net LN2: track 0.00 -> 47.1 mm
- net +12V: track 125.1 -> 147.2 mm
- net DIP2: track 0.00 -> 21.5 mm
- net Start: track 0.00 -> 16.4 mm
- net BDC1: track 32.4 -> 48.4 mm
- net BDC11: track 32.4 -> 42.8 mm, vias 0 -> 1
- net BDC22: track 10.2 -> 20.3 mm
- net BDC2: track 9.37 -> 18.0 mm
- net SDA1: track 0.00 -> 7.49 mm
- net SCL1: track 0.00 -> 7.49 mm
- net Dis7: track 58.9 -> 52.1 mm
- net Dis2: track 13.6 -> 18.8 mm
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- added copper zone on B.Cu, net GND
- added copper zone on F.Cu, net GND
Other:
- board size 93.2 x 58.4 mm -> 90 x 55 mm
- board text added: "${REFERENCE}"

Commit message: wf
Parts:
- added H2: MountingHole, MountingHole:MountingHole_2.5mm, F.Cu at (47.2, 78.0)
- added H4: MountingHole, MountingHole:MountingHole_2.5mm, F.Cu at (92.1, 78.6)
- added H4: MountingHole, MountingHole:MountingHole_2.5mm, F.Cu at (33.0, 77.8)
- moved H3 121.9 mm to (115.8, 27.2)
- moved H1 85.0 mm to (33.3, 27.4)
- moved H5 69.9 mm to (33.2, 47.0)
- moved H2 58.4 mm to (33.3, 57.0)
- moved H4 57.1 mm to (71.3, 78.2)
- moved C4 4.92 mm to (110.2, 29.3)
- moved C7 2.68 mm to (39.5, 27.4), turned to -90 degrees
- moved SW2 1.26 mm to (35.0, 73.6)
Connections:
- J14 pad 3: SDA1 -> SCL1
- J14 pad 4: SCL1 -> SDA1
Routing:
- net SCL1: track 7.49 -> 10.1 mm, vias 0 -> 1
- net +5V: track 67.3 -> 69.7 mm
- net +3.3V: track 218.0 -> 220.0 mm, vias 0 -> 1
- net DIP3: track 58.7 -> 60.2 mm
- net DIP4: track 52.2 -> 53.5 mm
- net SDA1: track 7.49 -> 6.44 mm
Other:
- board size 90 x 55 mm -> 90 x 57.4 mm
- board text added: "+"
- board text added: "-"
- board text added: "Designed by Joe Sung"
- board text added: "S"
