File: 500g/Rata2i2.0/pcbn't/500Updated/500Updated.kicad_sch (KiCad schematic)
At the start: 48 parts, among them J1 distance 1, J10 start, J11 motor 1, J13 distance 6, J14 line 4, J16 Screw_Terminal_01x07, J19 motor 2, J2 distance 2, J3 distance 3, J4 distance 4, J5 line 1, J6 line 2, J7 Battery, J8 line 3, J9 distance 5, SW1 SW_SPDT, SW2 SW_Push, U1 DEV-16771, U2 NRF24L01_Breakout, U3 R-78K5.0-0.5 (vr 5v), U4 R-78K5.0-0.5 (vr 3.3v), U5 motor driver 1, U6 motor driver 2

Commit message: Redid rata2i
drc hates me
Connections:
- net GPIO pin: now also U1.40 (A16); no longer U1.25 (A11)
- net L1: now also U1.37 (CS3); no longer U1.14 (A0)
- net L2: now also U1.2 (OUT2); no longer U1.15 (A1)
- net L3: now also U1.30 (CRX3); no longer U1.16 (A2)
- net L4: now also U1.15 (A1); no longer U1.20 (A6)
- net mdr1: now also U1.29 (TX7); no longer U1.28 (RX7)
- net mdr2: now also U1.28 (RX7); no longer U1.29 (TX7)
- net mdr3: now also U1.22 (A8); no longer U1.18 (A4)
- net mdr4: now also U1.18 (A4); no longer U1.22 (A8)
- net s1: now also U1.21 (A7); no longer U1.5 (IN2)
- net s2: now also U1.19 (A5); no longer U1.2 (OUT2)
- net s3: now also U1.23 (A9); no longer U1.3 (LRCLK2)
- net s4: now also U1.38 (A14); no longer U1.4 (BCLK2)
- net s5: now also U1.33 (MCLK2); no longer U1.24 (A10)
- net s6: now also U1.41 (A17); no longer U1.23 (A9)
- net start: now also U1.34 (RX8); no longer U1.17 (A3)

Commit message: ONE ERROR REMAINS...
RAHGHHHHHHHH
Connections:
- net GND: now also U5.9 (PAD), U6.9 (PAD)
- no-connect marks 37 -> 35
Changed lines of the file:
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@@
 	)
 	(no_connect
-		(at 260.35 100.33)
-	)
-	(no_connect
 		(at 59.69 77.47)
 	)
@@
 	)
 	(no_connect
-		(at 194.31 100.33)
-	)
-	(no_connect
 		(at 100.33 72.39)
 	)
@@
 	(wire
 		(pts
+			(xy 195.58 100.33) (xy 194.31 100.33)
+		)
+		(stroke
+			(width 0)
+			(type default)
+		)
+	)
+	(wire
+		(pts
 			(xy 264.16 97.79) (xy 269.24 97.79)
 		)
@@
 	(wire
 		(pts
+			(xy 260.35 100.33) (xy 264.16 100.33)
+		)
+		(stroke
+			(width 0)
+			(type default)
+		)
+	)
+	(wire
+		(pts
 			(xy 101.6 92.71) (xy 100.33 92.71)
 		)
@@
 	)
 	(symbol
+		(lib_id "power:GND")
+		(at 195.58 100.33 90)
+		(unit 1)
+		(exclude_from_sim no)
+		(in_bom yes)
+		(on_board yes)
+		(dnp no)
+		(fields_autoplaced yes)
+		(property "Reference" "#PWR045"
+			(at 201.93 100.33 0)
+			(effects
+				(font
+					(size 1.27 1.27)
+				)
+				(hide yes)
+			)
+		)
+		(property "Value" "GND"
+			(at 199.39 100.3299 90)
+			(effects
+				(font
+					(size 1.27 1.27)
+				)
+				(justify right)
+			)
+		)
+		(property "Footprint" ""
+			(at 195.58 100.33 0)
+			(effects
+				(font
+					(size 1.27 1.27)
+				)
+				(hide yes)
+			)
+		)
+		(property "Datasheet" ""
+			(at 195.58 100.33 0)
+			(effects
+				(font
+					(size 1.27 1.27)
+				)
+				(hide yes)
+			)
+		)
+		(property "Description" "Power symbol creates a global label with name \"GND\" , ground"
+			(at 195.58 100.33 0)
+			(effects
+				(font
+					(size 1.27 1.27)
+				)
+				(hide yes)
+			)
+		)
+		(pin "1"
+		)
+		(instances
+			(project ""
+				(path "/12510c2b-b621-44d9-ad20-a826d0bba445"
+					(reference "#PWR045")
+					(unit 1)
+				)
+			)
+		)
+	)
+	(symbol
 		(lib_id "Device:C")
 		(at 196.85 93.98 180)
@@
 					(unit 1)
 				)
+			)
+		)
+	)
+	(symbol
+		(lib_id "power:GND")
+		(at 264.16 100.33 90)
+		(unit 1)
+		(exclude_from_sim no)
+		(in_bom yes)
+		(on_board yes)
+		(dnp no)
+		(fields_autoplaced yes)
+		(property "Reference" "#PWR047"
+			(at 270.51 100.33 0)
+			(effects
+				(font
+					(size 1.27 1.27)
+				)
+				(hide yes)
+			)
+		)
+		(property "Value" "GND"
+			(at 267.97 100.3299 90)
+			(effects
+				(font
+					(size 1.27 1.27)
+				)
+				(justify right)
+			)
+		)
+		(property "Footprint" ""
+			(at 264.16 100.33 0)
+			(effects
+				(font
+					(size 1.27 1.27)
+				)
+				(hide yes)
+			)
+		)
+		(property "Datasheet" ""
+			(at 264.16 100.33 0)
+			(effects
+				(font
+					(size 1.27 1.27)
+				)
+				(hide yes)
+			)
+		)
+		(property "Description" "Power symbol creates a global label with name \"GND\" , ground"
+			(at 264.16 100.33 0)
+			(effects
+				(font
+					(size 1.27 1.27)
+				)
+				(hide yes)
+			)
+		)
+		(pin "1"
+		)
+		(instances
+			(project ""
+				(path "/12510c2b-b621-44d9-ad20-a826d0bba445"
+					(reference "#PWR047")
+					(unit 1)
+				)

Commit message: Last error fixed
Connections:
- net s5: now also U1.25 (A11); no longer U1.33 (MCLK2)
Changed lines of the file:
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@@
-	)
-	(no_connect
-		(at 100.33 115.57)
 	)
 	(no_connect
@@
 	)
 	(no_connect
+		(at 59.69 92.71)
+	)
+	(no_connect
 		(at 100.33 46.99)
 	)
@@
 	(wire
 		(pts
+			(xy 100.33 115.57) (xy 101.6 115.57)
+		)
+		(stroke
+			(width 0)
+			(type default)
+		)
+	)
+	(wire
+		(pts
 			(xy 254 46.99) (xy 259.08 46.99)
 		)
@@
 	(wire
 		(pts
-			(xy 58.42 64.77) (xy 59.69 64.77)
+			(xy 48.26 64.77) (xy 59.69 64.77)
 		)
 		(stroke
@@
 		(pts
 			(xy 256.54 44.45) (xy 259.08 44.45)
-		)
-		(stroke
-			(width 0)
-			(type default)
-		)
-	)
-	(wire
-		(pts
-			(xy 57.15 92.71) (xy 59.69 92.71)
 		)
 		(stroke
@@
 	(global_label "~CSN"
 		(shape input)
-		(at 58.42 64.77 180)
+		(at 48.26 64.77 180)
 		(fields_autoplaced yes)
 		(effects
@@
 		)
 		(property "Intersheetrefs" "${INTERSHEET_REFS}"
-			(at 50.7177 64.77 0)
+			(at 40.5577 64.77 0)
 			(effects
 				(font
@@
 		)
 	)
+	(global_label "s5"
+		(shape input)
+		(at 101.6 115.57 0)
+		(fields_autoplaced yes)
+		(effects
+			(font
+				(size 1.27 1.27)
+			)
+			(justify left)
+		)
+		(property "Intersheetrefs" "${INTERSHEET_REFS}"
+			(at 106.8228 115.57 0)
+			(effects
+				(font
+					(size 1.27 1.27)
+				)
+				(justify left)
+				(hide yes)
+			)
+		)
+	)
 	(global_label "mdr2"
 		(shape input)
@@
 			(effects
 				(font
-					(size 1.27 1.27)
-				)
-				(justify right)
-				(hide yes)
-			)
-		)
-	)
-	(global_label "s5"
-		(shape input)
-		(at 57.15 92.71 180)
-		(fields_autoplaced yes)
-		(effects
-			(font
-				(size 1.27 1.27)
-			)
-			(justify right)
-		)
-		(property "Intersheetrefs" "${INTERSHEET_REFS}"
-			(at 51.9272 92.71 0)
-			(effects
-				(font

Commit message: Working on making power traces lorge
Parts:
- C6, C8: value 10 uF -> .1 uF
- C7, C9: value 10 uF -> 47 uF
- renumbered R8 to R8(10k?)
Changed lines of the file:
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@@
 	(wire
 		(pts
+			(xy 222.25 148.59) (xy 224.79 148.59)
+		)
+		(stroke
+			(width 0)
+			(type default)
+		)
+	)
+	(wire
+		(pts
 			(xy 54.61 74.93) (xy 59.69 74.93)
 		)
@@
 		(dnp no)
 		(fields_autoplaced yes)
-		(property "Reference" "R8"
+		(property "Reference" "R8(10k?)"
 			(at 241.3 151.1299 0)
 			(effects
@@
 			(project "500Updated"
 				(path "/12510c2b-b621-44d9-ad20-a826d0bba445"
-					(reference "R8")
+					(reference "R8(10k?)")
 					(unit 1)
 				)
@@
 			)
 		)
-		(property "Value" "10 uF"
+		(property "Value" "47 uF"
 			(at 273.05 95.2499 0)
 			(effects
@@
 			)
 		)
-		(property "Value" "10 uF"
+		(property "Value" ".1 uF"
 			(at 188.722 94.996 0)
 			(effects
@@
 			)
 		)
-		(property "Value" "10 uF"
+		(property "Value" "47 uF"
 			(at 205.74 95.2499 0)
 			(effects
@@
 			)
 		)
-		(property "Value" "10 uF"
+		(property "Value" ".1 uF"
 			(at 255.524 93.472 0)
 			(effects
@@
 	(symbol
 		(lib_id "power:+3.3V")
-		(at 224.79 148.59 0)
+		(at 222.25 148.59 0)
 		(unit 1)
 		(exclude_from_sim no)
@@
 		(fields_autoplaced yes)
 		(property "Reference" "#PWR014"
-			(at 224.79 152.4 0)
+			(at 222.25 152.4 0)
 			(effects
 				(font
@@
 		)
 		(property "Value" "+3.3V"
-			(at 224.79 143.51 0)
+			(at 222.25 143.51 0)
 			(effects
 				(font
@@
 		)
 		(property "Footprint" ""
-			(at 224.79 148.59 0)
+			(at 222.25 148.59 0)
 			(effects
 				(font
@@
 		)
 		(property "Datasheet" ""
-			(at 224.79 148.59 0)
+			(at 222.25 148.59 0)
 			(effects
 				(font
@@
 		)
 		(property "Description" "Power symbol creates a global label with name \"+3.3V\""
-			(at 224.79 148.59 0)
+			(at 222.25 148.59 0)
 			(effects
 				(font
