File: 500g/Rata2i2.0/pcbn't/500Updated/500Updated.kicad_pcb (KiCad board)
At the start: 2 copper layers, 48 parts, among them J1 distance 1, J10 start, J11 motor 1, J13 distance 6, J14 line 4, J16 Screw_Terminal_01x07, J19 motor 2, J2 distance 2, J3 distance 3, J4 distance 4, J5 line 1, J6 line 2, J7 Battery, J8 line 3, J9 distance 5, SW1 SW_SPDT, SW2 SW_Push, U1 DEV-16771, U2 NRF24L01_Breakout, U3 R-78K5.0-0.5 (vr 5v), U4 R-78K5.0-0.5 (vr 3.3v), U5 motor driver 1, U6 motor driver 2

Commit message: Redid rata2i
drc hates me
Parts:
- moved R1 128.4 mm to (83.6, 50.0), turned to -90 degrees
- moved C5 122.8 mm to (88.5, 44.5), turned to 180 degrees
- moved C1 120.8 mm to (88.5, 38.0), turned to 90 degrees
- moved C3 119.3 mm to (88.5, 47.0)
- moved J10 118.9 mm to (159.2, 46.5), turned to 90 degrees
- moved R3 115.9 mm to (106.0, 38.0), turned to 180 degrees
- moved R5 114.1 mm to (94.0, 76.5), turned to 180 degrees
- moved R7 112.9 mm to (117.5, 39.0), turned to 180 degrees
- moved C2 112.4 mm to (87.0, 62.0), turned to 180 degrees
- moved C4 111.7 mm to (91.0, 62.0)
- moved C9 109.2 mm to (117.5, 36.5)
- moved C8 108.9 mm to (117.5, 34.0)
- moved R8 99.0 mm to (146.0, 34.0), turned to 90 degrees
- moved R2 92.5 mm to (114.0, 77.0), turned to 180 degrees
- moved R4 81.9 mm to (153.0, 38.5), turned to 180 degrees
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Connections:
- U1 pad 14: L1 -> unconnected-(U1-A0-Pad14)
- U1 pad 15: L2 -> L4
- U1 pad 16: L3 -> unconnected-(U1-A2-Pad16)
- U1 pad 17: start -> unconnected-(U1-A3-Pad17)
- U1 pad 18: mdr3 -> mdr4
- U1 pad 19: unconnected-(U1-A5-Pad19) -> s2
- U1 pad 2: s2 -> L2
- U1 pad 20: L4 -> unconnected-(U1-A6-Pad20)
- U1 pad 21: unconnected-(U1-A7-Pad21) -> s1
- U1 pad 22: mdr4 -> mdr3
- U1 pad 23: s6 -> s3
- U1 pad 24: s5 -> unconnected-(U1-A10-Pad24)
- U1 pad 25: GPIO pin -> unconnected-(U1-A11-Pad25)
- U1 pad 28: mdr1 -> mdr2
- U1 pad 29: mdr2 -> mdr1
- U1 pad 3: s3 -> unconnected-(U1-LRCLK2-Pad3)
- U1 pad 30: unconnected-(U1-CRX3-Pad30) -> L3
- U1 pad 33: unconnected-(U1-MCLK2-Pad33) -> s5
- U1 pad 34: unconnected-(U1-RX8-Pad34) -> start
- U1 pad 37: unconnected-(U1-CS3-Pad37) -> L1
- U1 pad 38: unconnected-(U1-A14-Pad38) -> s4
- U1 pad 4: s4 -> unconnected-(U1-BCLK2-Pad4)
- U1 pad 40: unconnected-(U1-A16-Pad40) -> GPIO pin
- U1 pad 41: unconnected-(U1-A17-Pad41) -> s6
- U1 pad 5: s1 -> unconnected-(U1-IN2-Pad5)
Routing:
- net +3.3V: track 0.00 -> 223.6 mm
- net +12V: track 0.00 -> 160.0 mm
- net +5V: track 0.00 -> 33.8 mm
- net s1: track 0.00 -> 32.1 mm
- net CE: track 24.6 -> 0.00 mm
- net GPIO pin: track 0.00 -> 23.7 mm
- net s5: track 0.00 -> 22.8 mm
- net s4: track 0.00 -> 22.2 mm
- net s2: track 5.86 -> 28.0 mm
- net s3: track 0.00 -> 13.5 mm
- net Net-(J7-Pin_2): track 0.00 -> 11.9 mm
- net Net-(J11-Pin_1): track 0.00 -> 9.79 mm
- net Net-(U5-ILIM): track 0.00 -> 9.60 mm
- net Net-(U6-ILIM): track 0.00 -> 9.35 mm
- net Net-(J11-Pin_2): track 0.00 -> 9.33 mm
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
Commit message: updated 500g
Routing:
- added copper zone on F.Cu, net GND
Changed lines of the file:
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@@
 		(pad "10" thru_hole circle
 			(at -0.65 -1.95 270)
-			(size 0.3 0.3)
-			(drill 0.2)
+			(size 0.45 0.45)
+			(drill 0.25)
 			(layers "*.Cu" "*.Mask")
 			(remove_unused_layers no)
@@
 		(pad "11" thru_hole circle
 			(at 0.65 -1.95 270)
-			(size 0.3 0.3)
-			(drill 0.2)
+			(size 0.45 0.45)
+			(drill 0.25)
 			(layers "*.Cu" "*.Mask")
 			(remove_unused_layers no)
@@
 		(pad "12" thru_hole circle
 			(at -0.65 -0.65 270)
-			(size 0.3 0.3)
-			(drill 0.2)
+			(size 0.45 0.45)
+			(drill 0.25)
 			(layers "*.Cu" "*.Mask")
 			(remove_unused_layers no)
@@
 		(pad "13" thru_hole circle
 			(at 0.65 -0.65 270)
-			(size 0.3 0.3)
-			(drill 0.2)
+			(size 0.45 0.45)
+			(drill 0.25)
 			(layers "*.Cu" "*.Mask")
 			(remove_unused_layers no)
@@
 		(pad "14" thru_hole circle
 			(at -0.65 0.65 270)
-			(size 0.3 0.3)
-			(drill 0.2)
+			(size 0.45 0.45)
+			(drill 0.25)
 			(layers "*.Cu" "*.Mask")
 			(remove_unused_layers no)
@@
 		(pad "15" thru_hole circle
 			(at 0.65 0.65 270)
-			(size 0.3 0.3)
-			(drill 0.2)
+			(size 0.45 0.45)
+			(drill 0.25)
 			(layers "*.Cu" "*.Mask")
 			(remove_unused_layers no)
@@
 		(pad "16" thru_hole circle
 			(at -0.65 1.95 270)
-			(size 0.3 0.3)
-			(drill 0.2)
+			(size 0.45 0.45)
+			(drill 0.25)
 			(layers "*.Cu" "*.Mask")
 			(remove_unused_layers no)
@@
 		(pad "17" thru_hole circle
 			(at 0.65 1.95 270)
-			(size 0.3 0.3)
-			(drill 0.2)
+			(size 0.45 0.45)
+			(drill 0.25)
 			(layers "*.Cu" "*.Mask")
 			(remove_unused_layers no)
@@
 			(pinfunction "PGND")
 			(pintype "power_in")
+			(zone_connect 2)
 		)
 		(pad "8" smd roundrect
@@
 		(pad "10" thru_hole circle
 			(at -0.65 -1.95 90)
-			(size 0.3 0.3)
-			(drill 0.2)
+			(size 0.45 0.45)
+			(drill 0.25)
 			(layers "*.Cu" "*.Mask")
 			(remove_unused_layers no)
@@
 		(pad "11" thru_hole circle
 			(at 0.65 -1.95 90)
-			(size 0.3 0.3)
-			(drill 0.2)
+			(size 0.45 0.45)
+			(drill 0.25)
 			(layers "*.Cu" "*.Mask")
 			(remove_unused_layers no)
@@
 		(pad "12" thru_hole circle
 			(at -0.65 -0.65 90)
-			(size 0.3 0.3)
-			(drill 0.2)
+			(size 0.45 0.45)
+			(drill 0.25)
 			(layers "*.Cu" "*.Mask")
 			(remove_unused_layers no)
@@
 		(pad "13" thru_hole circle
 			(at 0.65 -0.65 90)
-			(size 0.3 0.3)
-			(drill 0.2)
+			(size 0.45 0.45)
+			(drill 0.25)
 			(layers "*.Cu" "*.Mask")
 			(remove_unused_layers no)
@@
 		(pad "14" thru_hole circle
 			(at -0.65 0.65 90)
-			(size 0.3 0.3)
-			(drill 0.2)
+			(size 0.45 0.45)
+			(drill 0.25)
 			(layers "*.Cu" "*.Mask")
 			(remove_unused_layers no)
@@
 		(pad "15" thru_hole circle
 			(at 0.65 0.65 90)
-			(size 0.3 0.3)
-			(drill 0.2)
+			(size 0.45 0.45)
+			(drill 0.25)
 			(layers "*.Cu" "*.Mask")
 			(remove_unused_layers no)
@@
 		(pad "16" thru_hole circle
 			(at -0.65 1.95 90)
-			(size 0.3 0.3)
-			(drill 0.2)
+			(size 0.45 0.45)
+			(drill 0.25)
 			(layers "*.Cu" "*.Mask")
 			(remove_unused_layers no)
@@
 		(pad "17" thru_hole circle
 			(at 0.65 1.95 90)
-			(size 0.3 0.3)
-			(drill 0.2)
+			(size 0.45 0.45)
+			(drill 0.25)
 			(layers "*.Cu" "*.Mask")
 			(remove_unused_layers no)
@@
 	)
 	(gr_rect
-		(start 68.5 25)
-		(end 169.5 90)
+		(start 72.5 30)
+		(end 167 85)
 		(stroke
 			(width 0.2)
@@
 		(net 53)
 	)
+	(zone
+		(net 2)
+		(net_name "GND")
+		(layer "F.Cu")
+		(hatch edge 0.5)
+		(connect_pads
+			(clearance 0.5)
+		)
+		(min_thickness 0.25)
+		(filled_areas_thickness no)
+		(fill
+			(thermal_gap 0.5)
+			(thermal_bridge_width 0.5)
+		)
+		(polygon
+			(pts
+				(xy 72.5 30) (xy 169.5 30) (xy 169.5 85) (xy 72.5 85)
+			)
+		)
+	)
 	(embedded_fonts no)

Commit message: ONE ERROR REMAINS...
RAHGHHHHHHHH
Parts:
- removed U2: NRF24L01_Breakout, RF_Module:nRF24L01_Breakout
- moved H1 2.06 mm to (78.5, 34.0)
- moved H2 1.58 mm to (160.5, 34.0)
Connections:
- U5 pad 9: unconnected-(U5-PAD-Pad9) -> GND
- U6 pad 9: unconnected-(U6-PAD-Pad9) -> GND
Routing:
- net GND: track 0.00 -> 63.0 mm
- net CE: track 0.00 -> 22.8 mm
- net Net-(D6-A): track 0.00 -> 2.19 mm
- net +3.3V: track 223.6 -> 224.8 mm
- net mdr3: track 6.60 -> 7.16 mm
- added copper zone on B.Cu, net GND
Other:
- board outline added: 94 x 57 mm

Commit message: Last error fixed
Parts:
- moved H1 1.58 mm to (77.0, 33.5)
- moved H2 0.50 mm to (160.5, 33.5)
Connections:
- U1 pad 25: unconnected-(U1-A11-Pad25) -> s5
- U1 pad 33: s5 -> unconnected-(U1-MCLK2-Pad33)
Routing:
- net s5: track 22.8 -> 30.6 mm
- net GND: track 63.0 -> 70.7 mm, vias 0 -> 1
- net mdr1: track 8.22 -> 8.85 mm
Other:
- board size 94 x 57 mm -> 90.5 x 54.5 mm
- board text added: "rata2i :D"
Changed lines of the file:
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@@
 	(net 57 "unconnected-(U1-A2-Pad16)")
 	(net 58 "unconnected-(U1-A6-Pad20)")
-	(net 59 "unconnected-(U1-A11-Pad25)")
+	(net 59 "unconnected-(U1-MCLK2-Pad33)")
 	(net 60 "unconnected-(U1-A3-Pad17)")
 	(footprint "DRV8871DDAR:VREG_LM5017MR_NOPB"
@@
 			(at 2.54 -4.22 0)
 			(layer "F.SilkS")
+			(hide yes)
 			(effects
 				(font
@@
 		)
 		(property "Value" "line 3"
-			(at 2.54 4.52 0)
+			(at 2.5 -4 0)
 			(layer "F.Fab")
 			(effects
@@
 		)
 		(property "Value" "distance 2"
-			(at 2.54 4.52 0)
+			(at 2.54 -2.5 0)
 			(layer "F.Fab")
 			(effects
@@
 		(tags "THT Terminal Block Xinya XY308-2.54-3P pitch 2.54mm size 8.12x6.5mm drill 1.2mm pad 2mm")
 		(property "Reference" "J9"
-			(at 2.54 -4.22 0)
+			(at 2.54 4.5 0)
 			(layer "F.SilkS")
+			(hide yes)
 			(effects
 				(font
@@
 		)
 		(property "Value" "distance 5"
-			(at 2.54 4.52 0)
+			(at 2.54 -4.5 0)
 			(layer "F.Fab")
 			(effects
@@
 	(footprint "MountingHole:MountingHole_2.5mm"
 		(layer "F.Cu")
-		(at 78.5 34)
+		(at 77 33.5)
 		(descr "Mounting Hole 2.5mm, no annular, generated by kicad-footprint-generator mountinghole.py")
 		(tags "mountinghole")
@@
 			(at 1.27 -4.22 0)
 			(layer "F.SilkS")
+			(hide yes)
 			(effects
 				(font
@@
 		)
 		(property "Value" "motor 1"
-			(at 1.27 4.52 0)
+			(at 7.5 2.5 0)
 			(layer "F.Fab")
 			(effects
@@
 	(footprint "MountingHole:MountingHole_2.5mm"
 		(layer "F.Cu")
-		(at 160.5 34)
+		(at 160.5 33.5)
 		(descr "Mounting Hole 2.5mm, no annular, generated by kicad-footprint-generator mountinghole.py")
 		(tags "mountinghole")
@@
 		)
 		(fp_text user "Teensy 4.1"
-			(at -0.25 -0.34 0)
+			(at 25.595 -4.805 0)
 			(layer "F.Fab")
 			(effects
@@
 			(layers "*.Cu" "*.Mask")
 			(remove_unused_layers no)
-			(net 59 "unconnected-(U1-A11-Pad25)")
+			(net 18 "s5")
 			(pinfunction "A11")
-			(pintype "bidirectional+no_connect")
+			(pintype "bidirectional")
 			(solder_mask_margin 0.102)
 		)
@@
 			(layers "*.Cu" "*.Mask")
 			(remove_unused_layers no)
-			(net 18 "s5")
+			(net 59 "unconnected-(U1-MCLK2-Pad33)")
 			(pinfunction "MCLK2")
-			(pintype "bidirectional")
+			(pintype "bidirectional+no_connect")
 			(solder_mask_margin 0.102)
 		)
@@
 	)
 	(gr_rect
-		(start 72.5 29)
-		(end 166.5 86)
+		(start 73.5 30)
+		(end 164 84.5)
 		(stroke
 			(width 0.05)
@@
 		(layer "Edge.Cuts")
 	)
+	(gr_text "rata2i :D"
+		(at 75 83 0)
+		(layer "F.SilkS")
+		(effects
+			(font
+				(size 1.5 1.5)
+				(thickness 0.3)
+				(bold yes)
+			)
+			(justify left bottom)
+		)
+	)
 	(segment
 		(start 112.78616 33)
@@
 	)
 	(segment
+		(start 85.75 55.75)
+		(end 85.6 55.9)
+		(width 0.2)
+		(layer "F.Cu")
+		(net 2)
+	)
+	(segment
 		(start 141.755 69.245)
 		(end 139.85 71.15)
@@
 	)
 	(segment
+		(start 85.6 55.9)
+		(end 83.5875 55.9)
+		(width 0.2)
+		(layer "F.Cu")
+		(net 2)
+	)
+	(segment
 		(start 111.55 43.65)
 		(end 111.55 41.585)
@@
 		(net 2)
 	)
+	(via
+		(at 85.75 55.75)
+		(size 0.6)
+		(drill 0.3)
+		(layers "F.Cu" "B.Cu")
+		(net 2)
+	)
 	(segment
 		(start 90.54 68.5)
@@
 	)
 	(segment
+		(start 90.75 54.5)
+		(end 87 54.5)
+		(width 0.2)
+		(layer "B.Cu")
+		(net 2)
+	)
+	(segment
 		(start 119.26 71)
 		(end 116.76 73.5)
@@
 	)
 	(segment
+		(start 87 54.5)
+		(end 85.75 55.75)
+		(width 0.2)
+		(layer "B.Cu")
+		(net 2)
+	)
+	(segment
 		(start 116.42 45.5)
 		(end 117.92 44)
@@
 	)
 	(segment
-		(start 154.92 72)
-		(end 155.92 71)
+		(start 156.5 70.42)
+		(end 156.5 64)
+		(width 0.2)
+		(layer "F.Cu")
+		(net 18)
+	)
+	(segment
+		(start 140.26 62)
+		(end 136.835 65.425)
 		(width 0.2)
 		(layer "F.Cu")
@@
 	)
 	(segment
-		(start 155.92 71)
-		(end 155.92 51.49)
+		(start 156.5 64)
+		(end 154.5 62)
 		(width 0.2)
 		(layer "F.Cu")
@@
 	)
 	(segment
-		(start 155.92 51.49)
-		(end 154.615 50.185)
+		(start 154.5 62)
+		(end 140.26 62)
+		(width 0.2)
+		(layer "F.Cu")
+		(net 18)
+	)
+	(segment
+		(start 154.92 72)
+		(end 156.5 70.42)
 		(width 0.2)
 		(layer "F.Cu")
@@
 	)
 	(segment
-		(start 141.16 67)
-		(end 145.42 67)
+		(start 146.5 67)
+		(end 146.995 66.505)
 		(width 0.2)
 		(layer "F.Cu")
@@
 	)
 	(segment
+		(start 146.995 66.505)
+		(end 146.995 65.425)
+		(width 0.2)
+		(layer "F.Cu")
+		(net 46)
+	)
+	(segment
 		(start 140.485 67.675)
 		(end 141.16 67)
@@
 	)
 	(segment
-		(start 145.42 67)
-		(end 146.995 65.425)
+		(start 141.16 67)
+		(end 146.5 67)
 		(width 0.2)
 		(layer "F.Cu")
@@
 		(polygon
 			(pts
-				(xy 166.5 29) (xy 166.5 86) (xy 72.5 86) (xy 72.5 29)
+				(xy 164 30) (xy 164 84.5) (xy 73.5 84.5) (xy 73.5 30)
 			)
 		)

Commit message: Working on making power traces lorge
Routing:
- net +12V: track 160.3 -> 161.3 mm
- net +3.3V: track 224.8 -> 225.8 mm

Commit message: Finished making power traces lorge
sequel
Routing:
- net GND: track 70.7 -> 36.6 mm
- net +3.3V: track 225.8 -> 240.6 mm

Commit message: changed voltage regulator footprint
so this is what we forgot to change from last year -_-
Routing:
- net GND: track 36.6 -> 29.6 mm, vias 1 -> 0
- net +3.3V: track 240.6 -> 242.6 mm
- net +5V: track 33.8 -> 32.6 mm
Changed lines of the file:
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@@
 		)
 		(pad "2" thru_hole circle
-			(at 0 1.75 90)
+			(at 2.5 1.75 90)
 			(size 1.358 1.358)
 			(drill 0.85)
@@
 		)
 		(pad "3" thru_hole circle
-			(at 2.54 1.75 90)
+			(at 0 1.75 90)
 			(size 1.358 1.358)
 			(drill 0.85)
@@
 		)
 		(pad "2" thru_hole circle
-			(at 0 1.75 270)
+			(at 2.5 1.75 270)
 			(size 1.358 1.358)
 			(drill 0.85)
@@
 		)
 		(pad "3" thru_hole circle
-			(at 2.54 1.75 270)
+			(at 0 1.75 270)
 			(size 1.358 1.358)
 			(drill 0.85)
@@
 	)
 	(segment
-		(start 85.75 55.75)
-		(end 85.6 55.9)
+		(start 92.04 44.54)
+		(end 92 44.5)
 		(width 0.2)
 		(layer "F.Cu")
@@
 	)
 	(segment
-		(start 85.6 55.9)
-		(end 83.5875 55.9)
-		(width 0.2)
-		(layer "F.Cu")
-		(net 2)
-	)
-	(segment
 		(start 111.55 43.65)
 		(end 111.55 41.585)
@@
 	)
 	(segment
+		(start 92.75 44.54)
+		(end 92.04 44.54)
+		(width 0.2)
+		(layer "F.Cu")
+		(net 2)
+	)
+	(segment
 		(start 140.485 71.785)
 		(end 139.85 71.15)
@@
 		(net 2)
 	)
-	(via
-		(at 85.75 55.75)
-		(size 0.6)
-		(drill 0.3)
-		(layers "F.Cu" "B.Cu")
-		(net 2)
-	)
 	(segment
 		(start 103.46 43.5)
@@
 	)
 	(segment
-		(start 90.75 54.5)
-		(end 87 54.5)
-		(width 0.2)
-		(layer "B.Cu")
-		(net 2)
-	)
-	(segment
 		(start 105.46 45.5)
 		(end 116.42 45.5)
@@
 	)
 	(segment
-		(start 87 54.5)
-		(end 85.75 55.75)
-		(width 0.2)
-		(layer "B.Cu")
-		(net 2)
-	)
-	(segment
 		(start 116.42 45.5)
 		(end 117.92 44)
@@
 	)
 	(segment
-		(start 87.8775 49.0875)
-		(end 90.75 51.96)
+		(start 87.95 55.55)
+		(end 87.95 62)
 		(width 0.5)
 		(layer "F.Cu")
@@
 	)
 	(segment
-		(start 90.75 51.96)
-		(end 87.95 54.76)
+		(start 89 54.5)
+		(end 83.5875 49.0875)
 		(width 0.5)
 		(layer "F.Cu")
@@
 	)
 	(segment
-		(start 87.95 54.76)
-		(end 87.95 62)
+		(start 96.195 50.185)
+		(end 91.88 54.5)
 		(width 0.5)
 		(layer "F.Cu")
@@
 	)
 	(segment
-		(start 83.5875 49.0875)
-		(end 87.8775 49.0875)
+		(start 89 54.5)
+		(end 87.95 55.55)
 		(width 0.5)
 		(layer "F.Cu")
@@
 	)
 	(segment
-		(start 94.42 51.96)
-		(end 90.75 51.96)
+		(start 90.75 54.5)
+		(end 89 54.5)
 		(width 0.5)
 		(layer "F.Cu")
@@
 	)
 	(segment
-		(start 96.195 50.185)
-		(end 94.42 51.96)
+		(start 91.88 54.5)
+		(end 90.75 54.5)
 		(width 0.5)
 		(layer "F.Cu")
@@
 	)
 	(segment
-		(start 101.275 50.185)
-		(end 95.63 44.54)
+		(start 95.29 44.54)
+		(end 92.75 42)
 		(width 0.5)
 		(layer "F.Cu")
@@
 	)
 	(segment
-		(start 92.04 44.54)
-		(end 92 44.5)
-		(width 0.2)
-		(layer "F.Cu")
-		(net 4)
-	)
-	(segment
 		(start 134.5 71)
 		(end 131.755 68.255)
@@
 	)
 	(segment
-		(start 143 34)
-		(end 145.5 31.5)
+		(start 95.63 44.54)
+		(end 95.29 44.54)
 		(width 0.5)
 		(layer "F.Cu")
@@
 	)
 	(segment
-		(start 92 44.5)
-		(end 89.45 44.5)
+		(start 101.275 50.185)
+		(end 95.63 44.54)
+		(width 0.5)
+		(layer "F.Cu")
+		(net 4)
+	)
+	(segment
+		(start 143 34)
+		(end 145.5 31.5)
 		(width 0.5)
 		(layer "F.Cu")
@@
 	)
 	(segment
-		(start 95.63 44.54)
-		(end 92.75 44.54)
-		(width 0.5)
-		(layer "F.Cu")
-		(net 4)
-	)
-	(segment
 		(start 127.42 43.08)
 		(end 127.42 44)
@@
 	)
 	(segment
+		(start 92.75 42)
+		(end 91.95 42)
+		(width 0.5)
+		(layer "F.Cu")
+		(net 4)
+	)
+	(segment
 		(start 109.42 71)
 		(end 107.42 73)
@@
 	)
 	(segment
-		(start 92.75 44.54)
-		(end 92.04 44.54)
-		(width 0.2)
+		(start 91.95 42)
+		(end 89.45 44.5)
+		(width 0.5)
 		(layer "F.Cu")
 		(net 4)
