File: 500g/Yippi/Yippi.kicad_sch (KiCad schematic)
At the start: 24 parts, among them J1 distance 1, J10 start, J13 analog distance 6, J14 line 3, J2 distance 2, J3 distance 3, J4 distance 4, J5 line 1, J6 line 2, J7 Battery, J9 distance 5, SW1 SW_SPDT, U1 DEV-16771, U2 R-78K5.0-0.5 (vr 3.3v), U3 R-78K5.0-0.5 (vr 5v), U5 R-78K5.0-0.5 (vr 5v)

Commit message: yippi update
added most of the parts
need to change to jst stuff
Parts:
- added C10, C12, C15, C8: .1 uF, Capacitor_SMD:C_0805_2012Metric, symbol Device:C
- added C11, C13, C7, C9: 47 uF, Capacitor_SMD:C_0805_2012Metric, symbol Device:C
- added C14: .1, Capacitor_SMD:C_0805_2012Metric, symbol Device:C
- added D1, D2, D3: LED, LED_SMD:LED_1206_3216Metric, symbol Device:LED
- added J11: servo motor 2, TerminalBlock:TerminalBlock_Xinya_XY308-2.54-3P_1x03_P2.54mm_Horizontal, symbol Connector:Screw_Terminal_01x03
- added J12: motor 1, TerminalBlock:TerminalBlock_Xinya_XY308-2.54-2P_1x02_P2.54mm_Horizontal, symbol Connector:Screw_Terminal_01x02
- added J15: motor 3, TerminalBlock:TerminalBlock_Xinya_XY308-2.54-2P_1x02_P2.54mm_Horizontal, symbol Connector:Screw_Terminal_01x02
- added J16: motor 4, TerminalBlock:TerminalBlock_Xinya_XY308-2.54-2P_1x02_P2.54mm_Horizontal, symbol Connector:Screw_Terminal_01x02
- added J19: motor 2, TerminalBlock:TerminalBlock_Xinya_XY308-2.54-2P_1x02_P2.54mm_Horizontal, symbol Connector:Screw_Terminal_01x02
- added J8: servo motor 1, TerminalBlock:TerminalBlock_Xinya_XY308-2.54-3P_1x03_P2.54mm_Horizontal, symbol Connector:Screw_Terminal_01x03
- added R1, R2, R3: 200, Resistor_SMD:R_0805_2012Metric, symbol Device:R_US
- added R6(30k)1, R6(30k)2, R7(30k)1, R7(30k)2: R_US, Resistor_SMD:R_0805_2012Metric, symbol Device:R_US
- added U4, U8: motor driver 1, DRV8871DDAR:VREG_LM5017MR_NOPB, symbol DRV8871DDAR:DRV8871DDAR
- added U6, U7: motor driver 2, DRV8871DDAR:VREG_LM5017MR_NOPB, symbol DRV8871DDAR:DRV8871DDAR
- J13: value analog distance 6 -> ANALOG distance 6
Connections:
- net +12V: now also C10.1, C11.1, C12.1, C13.1, C15.1, C7.1, C8.1, C9.1, U4.5 (VM), U6.5 (VM), U7.5 (VM), U8.5 (VM)
- net +3.3V: now also U1.3.3V_1 (3.3V), U1.3.3V_2 (3.3V), U1.3.3V_3 (3.3V), C14.2
- net +5V: now also J11.1 (Pin_1), J8.1 (Pin_1)
- net GND: now also U1.GND1 (GND), U1.GND2 (GND), U1.GND3 (GND), U1.GND4 (GND), U1.GND5 (GND), U1.USB_GND1 (USB_GND), U1.USB_GND2 (USB_GND), C10.2, C11.2, C12.2, C13.2, C15.2, C7.2, C8.2, C9.2, D1.1 (K), D2.1 (K), D3.1 (K), J11.3 (Pin_3), J8.3 (Pin_3), R6(30k)1.1, R6(30k)2.1, R7(30k)1.1, R7(30k)2.1, U4.1 (GND), U4.7 (PGND), U6.1 (GND), U6.7 (PGND), U7.1 (GND), U7.7 (PGND), U8.1 (GND), U8.7 (PGND)
- net L1: now also U1.41 (A17), R3.1
- net L2: now also U1.40 (A16)
- net L3: now also U1.39 (A15)
- net s1: now also U1.14 (A0), R2.1
- net s2: now also U1.15 (A1)
- net s3: now also U1.16 (A2)
- net s4: now also U1.17 (A3)
- net s5: now also U1.18 (A4)
- net s6: now also U1.19 (A5), R1.1
- net start: now also U1.38 (A14)
- net at U1.VIN: now also C14.1
- new net: D3.2 (A), R3.2
- new net: R7(30k)1.2, U6.4 (ILIM)
- new net: R6(30k)2.2, U8.4 (ILIM)
- new net: R6(30k)1.2, U4.4 (ILIM)
- new net: J12.1 (Pin_1), U4.6 (OUT1)
- new net: J12.2 (Pin_2), U4.8 (OUT2)
- new net: R7(30k)2.2, U7.4 (ILIM)
- new net: J16.1 (Pin_1), U8.6 (OUT1)
- new net: J16.2 (Pin_2), U8.8 (OUT2)
- new net: D2.2 (A), R2.2
- new net: D1.2 (A), R1.2
- new net: J15.1 (Pin_1), U7.6 (OUT1)
- new net: J15.2 (Pin_2), U7.8 (OUT2)
- new net: J19.1 (Pin_1), U6.6 (OUT1)
- new net: J19.2 (Pin_2), U6.8 (OUT2)
- new net mdr1: U4.2 (IN2)
- new net mdr2: U4.3 (IN1)
- new net mdr3: U6.2 (IN2)
- new net mdr4: U6.3 (IN1)
- new net mdr5: U7.3 (IN1)
- new net mdr6: U7.2 (IN2)
- new net mdr7: U8.3 (IN1)
- new net mdr8: U8.2 (IN2)
- new net servo1: J8.2 (Pin_2)
- new net servo2: J11.2 (Pin_2)
- no-connect marks 1 -> 46
Other:
- note added: "extra 5v voltage regulator so that we have 1 per servo motor <3"
- note added: "note: servo1 and servo2 need to be pwm"
- note added: "todo: assign sensor footprints to JST CONNECTORS"
- moved on the sheet: C1, C2, C3, C4, C6, H1, H2, J1, J10, J13, J14, J2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
