File: 500g/Sp-I/Sp-ii-top-board/Sp-ii-top-board/Sp-ii-top-board.kicad_sch (KiCad schematic)
At the start: 46 parts, among them J7 Conn_01x02

Commit message: finished spi top board
Parts:
- removed D1, D6: LED, LED_SMD:LED_1206_3216Metric_Pad1.42x1.75mm_HandSolder, symbol Device:LED
- removed J7: Conn_01x02, Connector_AMASS:AMASS_XT30U-F_1x02_P5.0mm_Vertical, symbol Connector_Generic:Conn_01x02
- removed TV_1: Conn_01x04, Connector_PinSocket_2.54mm:PinSocket_1x04_P2.54mm_Vertical, symbol Connector_Generic:Conn_01x04
- added H_1, H_2: MountingHole, MountingHole:MountingHole_3.2mm_M3, symbol Mechanical:MountingHole
- added J1: XT30PW-M, XT30PW-M:AMASS_XT30PW-M, symbol XT30PW-M:XT30PW-M
- added LOW_PWR_1, SRT_TMR_1: LED, LED_SMD:LED_1206_3216Metric_Pad1.42x1.75mm_HandSolder, symbol Device:LED
- added R12, R_500_9: 500Ω, Resistor_SMD:R_1206_3216Metric_Pad1.30x1.75mm_HandSolder, symbol Device:R_US
- added START_MOD_1: Conn_01x03, Connector_PinSocket_2.54mm:PinSocket_1x03_P2.54mm_Vertical, symbol Connector_Generic:Conn_01x03
- added TV_H_1, TV_H_2, TV_H_3, TV_H_4: MountingHole, MountingHole:MountingHole_2.2mm_M2_DIN965_Pad_TopOnly, symbol Mechanical:MountingHole
- added U1: DM-OLED096-636, DM-OLED096-636:MODULE_DM-OLED096-636, symbol DM-OLED096-636:DM-OLED096-636
- D_BLN_1: renamed from D8; footprint (none) -> LED_SMD:LED_1206_3216Metric_Pad1.42x1.75mm_HandSolder
- D_L50_1: renamed from D7; footprint (none) -> LED_SMD:LED_1206_3216Metric_Pad1.42x1.75mm_HandSolder
- D_L90_1: renamed from D5; footprint (none) -> LED_SMD:LED_1206_3216Metric_Pad1.42x1.75mm_HandSolder
- D_LLN_1: renamed from D9; footprint (none) -> LED_SMD:LED_1206_3216Metric_Pad1.42x1.75mm_HandSolder
- D_M_1: renamed from D3; footprint (none) -> LED_SMD:LED_1206_3216Metric_Pad1.42x1.75mm_HandSolder
- D_R50_1: renamed from D2; footprint (none) -> LED_SMD:LED_1206_3216Metric_Pad1.42x1.75mm_HandSolder
- D_R90_1: renamed from D4; footprint (none) -> LED_SMD:LED_1206_3216Metric_Pad1.42x1.75mm_HandSolder
- D_RLN_1: renamed from D10; footprint (none) -> LED_SMD:LED_1206_3216Metric_Pad1.42x1.75mm_HandSolder
- F1: footprint (none) -> Fuse:Fuse_1206_3216Metric_Pad1.42x1.75mm_HandSolder
- IR_SW_1, PWR_SW_1: footprint 1101M2S3CQE2:1101M2S3CQE2 -> 1101:1101M2S3CQE2
- L_MOTOR_DRIVER_1, R_MOTOR_DRIVER_1: footprint DRV8871DDARQ1:DDA0008H_N_TEX -> DRV8871:DDA0008H_N_TEX
- R_3.3k_1, R_500_1, R_500_2, R_8.9k_1: footprint Resistor_SMD:R_0805_2012Metric_Pad1.20x1.40mm_HandSolder -> Resistor_SMD:R_1206_3216Metric_Pad1.30x1.75mm_HandSolder
- R_500_10: renamed from R5; value R_US -> 500Ω; footprint (none) -> Resistor_SMD:R_1206_3216Metric_Pad1.30x1.75mm_HandSolder
- R_500_11: renamed from R7; value R_US -> 500Ω; footprint (none) -> Resistor_SMD:R_1206_3216Metric_Pad1.30x1.75mm_HandSolder
- R_500_3: renamed from R6; value R_US -> 500Ω; footprint (none) -> Resistor_SMD:R_1206_3216Metric_Pad1.30x1.75mm_HandSolder
- R_500_4: renamed from R8; value R_US -> 500Ω; footprint (none) -> Resistor_SMD:R_1206_3216Metric_Pad1.30x1.75mm_HandSolder
- R_500_5: renamed from R3; value R_US -> 500Ω; footprint (none) -> Resistor_SMD:R_1206_3216Metric_Pad1.30x1.75mm_HandSolder
- R_500_6: renamed from R9; value R_US -> 500Ω; footprint (none) -> Resistor_SMD:R_1206_3216Metric_Pad1.30x1.75mm_HandSolder
- R_500_7: renamed from R4; value R_US -> 500Ω; footprint (none) -> Resistor_SMD:R_1206_3216Metric_Pad1.30x1.75mm_HandSolder
- R_500_8: renamed from R10; value R_US -> 500Ω; footprint (none) -> Resistor_SMD:R_1206_3216Metric_Pad1.30x1.75mm_HandSolder
- SW_DIP_1: renamed from SW_DIP1; footprint 4181172270902:418117270902 -> 4181:418117270902
- renumbered C2 to C_0.1uF_1, C3 to C_0.1uF_2, C4 to C_50uF_1, C5 to C_50uF_2, R1 to R_10k_1, R2 to R_10k_2, R_L_MTR1 to R_18k_1, R_R_MTR1 to R_18k_2
Connections:
- net +3.3V: now also U1.2 (VCC_IN)
- net +5V: now also START_MOD_1.1 (Pin_1)
- net Button_1: now also R_500_2.1
- net Button_2: now also R_500_1.1
- net GND: now also R_500_8.2, J1.N, R12.1, R_500_9.2, START_MOD_1.2 (Pin_2), U1.1 (GND); no longer R_500_8.1
- net LCD_SCL: now also U1.3 (SCL)
- net LCD_SDA: now also U1.4 (SDA)
- net Start_Mod: now also START_MOD_1.3 (Pin_3)
- net at D_RLN_1.1 (K): now also R_500_8.1; no longer R_500_8.2
- net at PWR_SW_1.1: now also J1.P
- net LED_1: now reaches Teensy 4.0.11
- net LED_1: now also LOW_PWR_1.2 (A)
- net LED_2: now reaches Teensy 4.0.12
- net LED_2: now also SRT_TMR_1.2 (A)
- new net: LOW_PWR_1.1 (K), R_500_9.1
- new net: R12.2, SRT_TMR_1.1 (K)
- no-connect marks 13 -> 11
Other:
- note added: "Start Module"
- moved on the sheet: C_50uF_1, C_50uF_2, PUSH_1, PUSH_2, R_10k_1, R_500_1, R_500_2, R_500_8, SW_DIP_1
