File: 500g/Sp-I/Sp-ii-top-board/Sp-ii-top-board/Sp-ii-top-board.kicad_pcb (KiCad board)
At the start: 2 copper layers, 85 x 37 mm, 80 parts, among them J7 Conn_01x02, U1 DM-OLED096-636

Commit message: finished and ordered
Parts:
- added G***: LOGO, RoboBuzz:RoboBuzz, F.Cu at (166.0, 111.0)
