File: 3kg/Kitti/Kitti_PCB_layout/Kitti_PCB_layout.kicad_sch (KiCad schematic)
At the start: 9 parts, among them IC1 TEENSY_4.1, J1 JS17250, J2 JS17250, J3 JS17250, J4 JS17250, J5 TF_mini, J6 TF_mini, J7 TF_mini, J8 TF_mini

Commit message: updated schematics
Parts:
- added J10, J11, J12, J13, J9: JS17250, symbol Line_Sensors:JS17250
Other:
- moved on the sheet: J1, J2, J3, J4, J5, J6, J7, J8

Commit message: added IR to schematic
Parts:
- removed J10, J11, J12, J13, J9: JS17250, symbol Line_Sensors:JS17250
- added J10, J11, J12, J13, J14, J15, J16, J17, J9: Omron E3Z-D82, symbol IRsensor:Omron E3Z-D82
Other:
- moved on the sheet: J5, J6, J7, J8

Commit message: motor driver and labels
Parts:
- added J18: Conn_02x05_Odd_Even, symbol Connector_Generic:Conn_02x05_Odd_Even
Other:
- note added: "Lidar Sensors"
- note added: "Line Sensors"
- note added: "Motor Driver"
- note added: "Omron IR sensors"
Changed lines of the file:
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@@
 	(generator_version "9.0")
 	(paper "A4")
+	(text "Motor Driver"
+		(exclude_from_sim no)
+		(at 258.572 151.13 0)
+		(effects
+			(font
+				(size 2.54 2.54)
+			)
+		)
+	)
+	(text "Omron IR sensors"
+		(exclude_from_sim no)
+		(at 245.618 96.266 0)
+		(effects
+			(font
+				(size 2.54 2.54)
+			)
+		)
+	)
+	(text "Lidar Sensors"
+		(exclude_from_sim no)
+		(at 31.242 189.23 0)
+		(effects
+			(font
+				(size 2.54 2.54)
+			)
+		)
+	)
+	(text "Line Sensors"
+		(exclude_from_sim no)
+		(at 88.138 189.23 0)
+		(effects
+			(font
+				(size 2.54 2.54)
+			)
+		)
+	)
+	(polyline
+		(pts
+			(xy 12.7 134.62) (xy 127 134.62)
+		)
+		(stroke
+			(width 0)
+			(type default)
+		)
+	)
+	(polyline
+		(pts
+			(xy 127 196.85) (xy 127 198.12)
+		)
+		(stroke
+			(width 0)
+			(type default)
+		)
+	)
+	(polyline
+		(pts
+			(xy 73.66 134.62) (xy 73.66 198.12)
+		)
+		(stroke
+			(width 0)
+			(type default)
+		)
+	)
+	(polyline
+		(pts
+			(xy 224.79 12.7) (xy 224.79 99.06)
+		)
+		(stroke
+			(width 0)
+			(type default)
+		)
+	)
+	(polyline
+		(pts
+			(xy 127 134.62) (xy 127 196.85)
+		)
+		(stroke
+			(width 0)
+			(type default)
+		)
+	)
+	(polyline
+		(pts
+			(xy 284.48 99.06) (xy 224.79 99.06)
+		)
+		(stroke
+			(width 0)
+			(type default)
+		)
+	)
 	(symbol
 		(lib_id "IRsensor:Omron E3Z-D82")
@@
 					(unit 1)
 				)
+			)
+		)
+	)
+	(symbol
+		(lib_id "Connector_Generic:Conn_02x05_Odd_Even")
+		(at 259.08 139.7 0)
+		(unit 1)
+		(exclude_from_sim no)
+		(in_bom yes)
+		(on_board yes)
+		(dnp no)
+		(fields_autoplaced yes)
+		(property "Reference" "J18"
+			(at 260.35 128.27 0)
+			(effects
+				(font
+					(size 1.27 1.27)
+				)
+			)
+		)
+		(property "Value" "Conn_02x05_Odd_Even"
+			(at 260.35 130.81 0)
+			(effects
+				(font
+					(size 1.27 1.27)
+				)
+			)
+		)
+		(property "Footprint" ""
+			(at 259.08 139.7 0)
+			(effects
+				(font
+					(size 1.27 1.27)
+				)
+				(hide yes)
+			)
+		)
+		(property "Datasheet" "~"
+			(at 259.08 139.7 0)
+			(effects
+				(font
+					(size 1.27 1.27)
+				)
+				(hide yes)
+			)
+		)
+		(property "Description" "Generic connector, double row, 02x05, odd/even pin numbering scheme (row 1 odd numbers, row 2 even numbers), script generated (kicad-library-utils/schlib/autogen/connector/)"
+			(at 259.08 139.7 0)
+			(effects
+				(font
+					(size 1.27 1.27)
+				)
+				(hide yes)
+			)
+		)
+		(pin "8"
+		)
+		(pin "1"
+		)
+		(pin "6"
+		)
+		(pin "10"
+		)
+		(pin "5"
+		)
+		(pin "4"
+		)
+		(pin "3"
+		)
+		(pin "7"
+		)
+		(pin "9"
+		)
+		(pin "2"
+		)
+		(instances
+			(project ""
+				(path "/7546ba49-78f3-4d70-aac0-ddd551a614da"
+					(reference "J18")
+					(unit 1)
+				)

Commit message: updated sensors
Parts:
- added C1, C10, C11, C12, C13, C14, C15, C16, C17, C18, C2, C3, C4, C5, C6, C7, C8, C9: 0.1uF, symbol Device:C
- added J19: Conn_01x03_Pin, symbol Connector:Conn_01x03_Pin
- added U1: AMS1117-5.0, Package_TO_SOT_SMD:SOT-223-3_TabPin2, symbol Regulator_Linear:AMS1117-5.0
Connections:
- net +5V: now reaches J13.5V (Pin_1)
- net +5V: now also J1.5V (Pin_4), J10.5V (Pin_1), J11.5V (Pin_1), J12.5V (Pin_1), J14.5V (Pin_1), J15.5V (Pin_1), J16.5V (Pin_1), J17.5V (Pin_1), J2.5V (Pin_4), J3.5V (Pin_4), J4.5V (Pin_4), J5.5V (Pin_1), J6.5V (Pin_1), J7.5V (Pin_1), J8.5V (Pin_1), J9.5V (Pin_1), C10.2, C11.2, C12.2, C13.2, C14.2, C15.2, C16.2, C17.2, C18.2, C2.2, C3.2, C4.2, C5.2, C6.2, C7.2, C8.2, C9.2
- net GND: now reaches J13.GND (Pin_2)
- net GND: now also J1.GND (Pin_5), J10.GND (Pin_2), J11.GND (Pin_2), J12.GND (Pin_2), J14.GND (Pin_2), J15.GND (Pin_2), J16.GND (Pin_2), J17.GND (Pin_2), J18.1 (Pin_1), J2.GND (Pin_5), J3.GND (Pin_5), J4.GND (Pin_5), J5.GND (Pin_4), J6.GND (Pin_4), J7.GND (Pin_4), J8.GND (Pin_4), J9.GND (Pin_2), C1.2, C10.1, C11.1, C12.1, C13.1, C14.1, C15.1, C16.1, C17.1, C18.1, C2.1, C3.1, C4.1, C5.1, C6.1, C7.1, C8.1, C9.1, J19.2 (Pin_2)
- net IR_1: now reaches J13.Out (Pin_3)
- net IR_1: now also IC1.1 (TX1)
- net IR_4: now reaches J14.Out (Pin_3)
- net IR_4: now also IC1.4 (BCLK2)
- net IR_5: now reaches J11.Out (Pin_3)
- net IR_5: now also IC1.5 (IN2)
- net L_3: now reaches J2.Signal_NOR (Pin_3)
- net L_3: now also IC1.12 (MISO)
- net IR_3: now reaches J10.Out (Pin_3)
- net IR_3: now also IC1.3 (LRCLK2)
- net Lid_3_RX: now reaches J7.RXD (Pin_2)
- net Lid_3_RX: now also IC1.34 (RX8)
- net Lid_3_TX: now reaches J7.TXD (Pin_3)
- net Lid_3_TX: now also IC1.35 (TX8)
- net Lid_1_RX: now reaches J5.RXD (Pin_2)
- net Lid_1_RX: now also IC1.21 (A7)
- net Lid_1_TX: now reaches J5.TXD (Pin_3)
- net Lid_1_TX: now also IC1.20 (A6)
- net L_2: now reaches J3.Signal_NOR (Pin_3)
- net L_2: now also IC1.11 (MOSI)
- net L_4: now reaches J4.Signal_NOR (Pin_3)
- net L_4: now also IC1.24 (A10)
- net Lid_4_RX: now reaches J6.RXD (Pin_2)
- net Lid_4_RX: now also IC1.28 (RX7)
- net Lid_4_TX: now reaches J6.TXD (Pin_3)
- net Lid_4_TX: now also IC1.29 (TX7)
- net IR_7: now reaches J15.Out (Pin_3)
- net IR_7: now also IC1.7 (RX2)
- net Lid_2_RX: now reaches J8.RXD (Pin_2)
- net Lid_2_RX: now also IC1.16 (A2)
- net Lid_2_TX: now reaches J8.TXD (Pin_3)
- net Lid_2_TX: now also IC1.17 (A3)
- net L_1: now reaches IC1.10 (CS_1)
- net L_1: now also J1.Signal_NOR (Pin_3)
- net IR_2: now reaches IC1.2 (OUT2)
- net IR_2: now also J9.Out (Pin_3)
- net IR_6: now reaches IC1.6 (OUT1D)
- net IR_6: now also J12.Out (Pin_3)
- net IR_8: now reaches IC1.8 (TX2)
- net IR_8: now also J16.Out (Pin_3)
- net IR_9: now reaches IC1.9 (OUT1C)
- net IR_9: now also J17.Out (Pin_3)
- new net +3.3V: C1.1, J19.3 (Pin_3)
- new net Start: J19.1 (Pin_1)
- no-connect marks 0 -> 8
Other:
- note added: "Start Module"
- moved on the sheet: J1, J2, J3, J4, J5, J6, J7, J9

Commit message: updated schematics
Connections:
- net +5V: now also U1.2 (VO); no longer C10.2, C2.2, C3.2, C4.2, C5.2, C6.2, C7.2, C8.2, C9.2, J10.5V (Pin_1), J11.5V (Pin_1), J12.5V (Pin_1), J13.5V (Pin_1), J14.5V (Pin_1), J15.5V (Pin_1), J16.5V (Pin_1), J17.5V (Pin_1), J9.5V (Pin_1)
- net GND: now also IC1.48 (GND_2), IC1.49 (GND_3), IC1.69 (GND_4), IC1.70 (GND_5), IC1.71 (GND_6), U1.1 (GND)
- net +6.5V: now reaches U1.3 (VI)
- new net +12V: C10.2, C2.2, C3.2, C4.2, C5.2, C6.2, C7.2, C8.2, C9.2, J10.5V (Pin_1), J11.5V (Pin_1), J12.5V (Pin_1), J13.5V (Pin_1), J14.5V (Pin_1), J15.5V (Pin_1), J16.5V (Pin_1), J17.5V (Pin_1), J9.5V (Pin_1)
Other:
- note added: "Voltage Regulator"
- moved on the sheet: U1

Commit message: resistor and motor driver
Parts:
- added R1, R3, R5, R7: 2 kOHm, symbol Device:R_US
- added R2, R4, R6, R8: 1 kOhm, symbol Device:R_US
Connections:
- net +5V: now also J18.9 (Pin_9)
- net GND: now also R1.1, R3.1, R5.1, R7.1
- net L_1: now also R2.2; no longer IC1.10 (CS_1)
- net L_2: now also R4.2; no longer IC1.11 (MOSI)
- net L_3: now also R6.2; no longer IC1.12 (MISO)
- net L_4: now also R8.2; no longer IC1.24 (A10)
- net A2: now reaches J18.3 (Pin_3)
- net A2: now also IC1.19 (A5)
- net B2: now reaches J18.4 (Pin_4)
- net B2: now also IC1.15 (A1)
- net A1: now reaches J18.5 (Pin_5)
- net A1: now also IC1.18 (A4)
- net B1: now reaches J18.6 (Pin_6)
- net B1: now also IC1.14 (A0)
- net PWMA: now reaches J18.7 (Pin_7)
- net PWMB: now reaches J18.8 (Pin_8)
- new net L_1T: IC1.10 (CS_1), R1.2, R2.1
- new net L_2T: IC1.11 (MOSI), R3.2, R4.1
- new net L_3T: IC1.12 (MISO), R5.2, R6.1
- new net L_4T: IC1.24 (A10), R7.2, R8.1
- no-connect marks 8 -> 10
Other:
- note added: "Convert 5V to 3.3V"

Commit message: kitti
Parts:
- removed C10, C5, C9: 0.1uF, symbol Device:C
- removed J12, J16, J17: Omron E3Z-D82, symbol IRsensor:Omron E3Z-D82
- removed U1: AMS1117-5.0, Package_TO_SOT_SMD:SOT-223-3_TabPin2, symbol Regulator_Linear:AMS1117-5.0
- added C19, C20, C21: 0.1uF, Capacitor_SMD:C_0805_2012Metric_Pad1.18x1.45mm_HandSolder, symbol Device:C
- added D1, D2, D3, D4, D5, D7, D8, D9: LED, LED_SMD:LED_1206_3216Metric_Pad1.42x1.75mm_HandSolder, symbol Device:LED
- added D10, D11, D12, D13: BZV55B47, Diode_SMD:D_MiniMELF, symbol Diode:BZV55B47
- added F1: Fuse, Fuse:Fuse_0805_2012Metric_Pad1.15x1.40mm_HandSolder, symbol Device:Fuse
- added J16: Conn_01x02_Pin, TerminalBlock_TE-Connectivity:TerminalBlock_TE_282834-2_1x02_P2.54mm_Horizontal, symbol Connector:Conn_01x02_Pin
- added J20: Screw_Terminal_01x03, TerminalBlock_TE-Connectivity:TerminalBlock_TE_282834-3_1x03_P2.54mm_Horizontal, symbol Connector:Screw_Terminal_01x03
- added J21: Screw_Terminal_01x07, TerminalBlock_TE-Connectivity:TerminalBlock_TE_282834-7_1x07_P2.54mm_Horizontal, symbol Connector:Screw_Terminal_01x07
- added J22, J23: Omron E3Z-D82, TerminalBlock_TE-Connectivity:TerminalBlock_TE_282834-3_1x03_P2.54mm_Horizontal, symbol IRsensor:Omron E3Z-D82
- added R10, R11, R12, R13, R15, R16, R17, R9: 1 kOhm, Resistor_SMD:R_0805_2012Metric_Pad1.20x1.40mm_HandSolder, symbol Device:R_US
- added SW1: SW_Nidec_CAS-120A1, Button_Switch_SMD:Nidec_Copal_CAS-120A, symbol Switch:SW_Nidec_CAS-120A1
- C1, C11, C12, C13, C14, C15, C16, C17, C18, C2, C3, C4, C6, C7, C8: footprint (none) -> Capacitor_SMD:C_0805_2012Metric_Pad1.18x1.45mm_HandSolder
- J1, J10, J11, J13, J14, J15, J19, J2, J3, J4, J9: footprint (none) -> TerminalBlock_TE-Connectivity:TerminalBlock_TE_282834-3_1x03_P2.54mm_Horizontal
- J18: footprint (none) -> Connector_PinHeader_2.54mm:PinHeader_2x05_P2.54mm_Horizontal
- J5, J6, J7, J8: footprint (none) -> TerminalBlock_TE-Connectivity:TerminalBlock_TE_282834-4_1x04_P2.54mm_Horizontal
- R1, R2, R3, R4, R5, R6, R7, R8: footprint (none) -> Resistor_SMD:R_0805_2012Metric_Pad1.20x1.40mm_HandSolder
Connections:
- net +12V: now also C20.2, C21.2, F1.1, J20.1 (Pin_1), J22.5V (Pin_1), J23.5V (Pin_1)
- net +3.3V: now also C19.2, J21.1 (Pin_1); no longer C1.1, J19.3 (Pin_3)
- net +5V: now also C1.1, J19.3 (Pin_3), J20.3 (Pin_3)
- net A1: now also D11.1 (K)
- net A2: now also D12.1 (K)
- net B1: now also D10.1 (K)
- net B2: now also D13.1 (K)
- net GND: now also C19.1, C20.1, C21.1, D1.1 (K), D10.2 (A), D11.2 (A), D12.2 (A), D13.2 (A), D2.1 (K), D3.1 (K), D4.1 (K), D5.1 (K), D7.1 (K), D8.1 (K), D9.1 (K), J16.1 (Pin_1), J20.2 (Pin_2), J21.2 (Pin_2), J22.GND (Pin_2), J23.GND (Pin_2), SW1.3 (A)
- net IR_1: now also J15.Out (Pin_3), R15.2; no longer J13.Out (Pin_3)
- net IR_2: now also J10.Out (Pin_3), R12.2; no longer J9.Out (Pin_3)
- net IR_3: now also J13.Out (Pin_3), R16.2; no longer J10.Out (Pin_3)
- net IR_4: now also J22.Out (Pin_3), R9.2; no longer J14.Out (Pin_3)
- net IR_5: now also R13.2
- net IR_6: now also J14.Out (Pin_3), R17.2
- net IR_7: now also J23.Out (Pin_3), R10.2; no longer J15.Out (Pin_3)
- net IR_8: now also J9.Out (Pin_3), R11.2
- net L_4T: now also IC1.26 (A12); no longer IC1.24 (A10)
- net PWMA: now also IC1.33 (MCLK2)
- net PWMB: now also IC1.37 (CS_3)
- net Start: now also IC1.13 (SCK)
- net SDA: now reaches IC1.25 (A11)
- net SDA: now also J21.4 (Pin_4)
- new net: D4.2 (A), R12.1
- new net: D3.2 (A), R11.1
- new net: D9.2 (A), R17.1
- new net: D7.2 (A), R15.1
- new net: D2.2 (A), R10.1
- new net: D1.2 (A), R9.1
- new net: D8.2 (A), R16.1
- new net: J16.2 (Pin_2), SW1.2 (B)
- new net: F1.2, SW1.1 (C)
- new net: D5.2 (A), R13.1
- new net SCL: IC1.24 (A10), J21.3 (Pin_3)
- no-connect marks 10 -> 37
Other:
- moved on the sheet: C8, J15, J18

Commit message: Kitti to Strawberri
Parts:
- removed C14, C16, C17, C18: 0.1uF, Capacitor_SMD:C_0805_2012Metric_Pad1.18x1.45mm_HandSolder, symbol Device:C
- removed J1, J2, J3, J4: JS17250, TerminalBlock_TE-Connectivity:TerminalBlock_TE_282834-3_1x03_P2.54mm_Horizontal, symbol Line_Sensors:JS17250
- removed J6, J7, J8: TF_mini, TerminalBlock_TE-Connectivity:TerminalBlock_TE_282834-4_1x04_P2.54mm_Horizontal, symbol LidarSensor:TF_mini
- removed R1, R3, R5, R7: 2 kOHm, Resistor_SMD:R_0805_2012Metric_Pad1.20x1.40mm_HandSolder, symbol Device:R_US
- removed R2, R4, R6, R8: 1 kOhm, Resistor_SMD:R_0805_2012Metric_Pad1.20x1.40mm_HandSolder, symbol Device:R_US
- added C10, C5, C9: 0.1uF, symbol Device:C
- added J1, J2, J3, J4, J6, J7: Screw_Terminal_01x03, TerminalBlock_TE-Connectivity:TerminalBlock_TE_282834-3_1x03_P2.54mm_Horizontal, symbol Connector:Screw_Terminal_01x03
- C11, C12, C13: footprint Capacitor_SMD:C_0805_2012Metric_Pad1.18x1.45mm_HandSolder -> (none)
Connections:
- net +5V: now also C11.1, C12.1, C13.1, C10.1, C5.1, C9.1, J1.2 (Pin_2), J2.2 (Pin_2), J3.2 (Pin_2), J4.2 (Pin_2), J6.2 (Pin_2), J7.2 (Pin_2); no longer C11.2, C12.2, C13.2
- net GND: now also C11.2, C12.2, C13.2, C10.2, C5.2, C9.2, J1.3 (Pin_3), J2.3 (Pin_3), J3.3 (Pin_3), J4.3 (Pin_3), J6.3 (Pin_3), J7.3 (Pin_3); no longer C11.1, C12.1, C13.1
- net L_1T: now also J1.1 (Pin_1), J2.1 (Pin_1), J3.1 (Pin_1), J4.1 (Pin_1), J6.1 (Pin_1), J7.1 (Pin_1)
- no-connect marks 37 -> 29
Other:
- note removed: "Convert 5V to 3.3V"
- note removed: "Line Sensors"
