File: 3kg/Kitti/Kitti_PCB_layout/Kitti_PCB_layout.kicad_pcb (KiCad board)
At the start: 2 copper layers, 170 x 30 mm, 62 parts, among them IC1 TEENSY_4.1, J1 Screw_Terminal_01x03, J10 Screw_Terminal_01x03, J11 Screw_Terminal_01x03, J12 Screw_Terminal_01x03, J16 Conn_01x02_Pin, J18 Conn_02x05_Odd_Even, J19 Conn_01x03_Pin, J2 Screw_Terminal_01x03, J20 Screw_Terminal_01x03, J21 Screw_Terminal_01x07, J3 Screw_Terminal_01x03, J4 Screw_Terminal_01x04, J5 Screw_Terminal_01x03, J6 Screw_Terminal_01x03, J7 Screw_Terminal_01x03, J8 Screw_Terminal_01x03, J9 Screw_Terminal_01x03, Q1 BF244C, Q2 BF244C, Q3 BF244C, Q4 BF244C, Q5 BF244C, Q6 BF244C, Q7 BF244C, SW1 SW_Nidec_CAS-120A1, SW2 219-3LPSTR

Commit message: layout
Parts:
- moved J16 261.5 mm to (-1046.1, -461.0)
- moved C10 254.5 mm to (-1039.0, -441.5), turned to -90 degrees
- moved C9 254.3 mm to (-1039.0, -434.0), turned to 90 degrees
- moved C4 252.3 mm to (-1041.0, -454.0), turned to -90 degrees
- moved C7 243.3 mm to (-1028.0, -439.0)
- moved Q6 240.5 mm to (-1034.4, -446.3), turned to -90 degrees
- moved R17 239.9 mm to (-1041.0, -449.0), turned to -90 degrees
- moved SW1 236.6 mm to (-1031.4, -460.0), turned to 180 degrees
- moved SW2 232.2 mm to (-1014.5, -434.5), turned to 90 degrees
- moved Q7 230.5 mm to (-1024.3, -440.1)
- moved D9 227.8 mm to (-1038.5, -451.5), turned to -90 degrees
- moved F1 222.8 mm to (-1027.5, -455.0), turned to 90 degrees
- moved D2 218.3 mm to (-1026.5, -435.5)
- moved J7 216.7 mm to (-1046.1, -440.0), turned to 90 degrees
- moved R10 215.5 mm to (-1022.0, -435.5)
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Connections:
- J1 pad 1: L_1T -> L_2T
- J2 pad 1: L_1T -> L_4T
- J3 pad 1: L_1T -> L_3T
- Q2 pad 2: IR_1 -> IR_2
- Q3 pad 2: IR_1 -> IR_3
- Q4 pad 2: IR_1 -> IR_4
- Q5 pad 2: IR_1 -> IR_5
- Q6 pad 2: IR_1 -> IR_6
- Q7 pad 2: IR_1 -> IR_7
Other:
- board size 170 x 30 mm -> 170 x 35 mm

Commit message: layout and wiring done!!! check and add details. I'm so Tired.
Parts:
- moved Q5 5.99 mm to (-923.2, -450.9)
- moved C19 5.99 mm to (-919.0, -449.0)
- moved C6 5.99 mm to (-919.0, -452.5)
- moved D5 5.99 mm to (-921.5, -455.0)
- moved J10 5.99 mm to (-925.9, -460.0)
- moved R13 5.99 mm to (-926.0, -455.0)
- moved C5 3.46 mm to (-889.5, -456.0), turned to -90 degrees
- turned R2 to -90 degrees
Routing:
- net GND: track 0.00 -> 370.1 mm, vias 0 -> 5
- net +5V: track 0.00 -> 265.6 mm, vias 0 -> 18
- net +3.3V: track 0.00 -> 230.2 mm, vias 0 -> 22
- net +12V: track 0.00 -> 229.0 mm, vias 0 -> 21
- net IR_1T: track 0.00 -> 111.6 mm, vias 0 -> 6
- net Algo1: track 0.00 -> 98.2 mm, vias 0 -> 14
- net L_1T: track 0.00 -> 97.3 mm, vias 0 -> 8
- net L_2T: track 0.00 -> 94.2 mm, vias 0 -> 6
- net L_3T: track 0.00 -> 88.2 mm
- net L_4T: track 0.00 -> 77.2 mm
- net Start: track 0.00 -> 75.8 mm, vias 0 -> 8
- net Algo2: track 0.00 -> 73.4 mm, vias 0 -> 10
- net IR_6T: track 0.00 -> 66.5 mm, vias 0 -> 1
- net Algo3: track 0.00 -> 65.6 mm, vias 0 -> 8
- net IR_5T: track 0.00 -> 65.0 mm, vias 0 -> 2
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
Commit message: wiring fix. Please Check it Out.
Routing:
- net GND: track 370.1 -> 1.04 mm, vias 5 -> 0
- net +12V: track 229.0 -> 297.7 mm, vias 21 -> 4
- net L_1T: track 97.3 -> 95.8 mm, vias 8 -> 2
- net Algo2: track 73.4 -> 72.1 mm, vias 10 -> 8
- net IR_5T: track 65.0 -> 66.0 mm
- net Algo1: track 98.2 -> 97.5 mm, vias 14 -> 10
- net IR_1T: track 111.6 -> 112.0 mm, vias 6 -> 4
- net +3.3V: track 230.2 -> 230.0 mm, vias 22 -> 16
- net Algo3: vias 8 -> 6
- net +5V: vias 18 -> 14
- added copper zone on B.Cu, net (none)
- added copper zone on F.Cu, net (none)
Other:
- board size 170 x 35 mm -> 173.5 x 37 mm
