File: 3kg/Strawberri/Strawberri/Strawberri.kicad_sch (KiCad schematic)
At the start: 70 parts, among them J1 Screw_Terminal_01x08, J13 Screw_Terminal_01x03, J14 Screw_Terminal_01x03, J15 Conn_02x05_Odd_Even, J17 Screw_Terminal_01x03, J18 Screw_Terminal_01x03, J19 Screw_Terminal_01x03, J20 Screw_Terminal_01x03, J21 Screw_Terminal_01x03, J7 Battery, J9 Conn_01x03, SW1 SW_SPDT, SW2 SW_DIP_x03, U1 DEV-16771, U9 R-78K5.0-0.5 (vr 5v)

Commit message: 0 errors
doesnt have servos
Parts:
- removed C18: .1 µF, Capacitor_SMD:C_0805_2012Metric, symbol Device:C
- removed D1, D2, D3, D4, D5, D6, D7: LED, LED_SMD:LED_1206_3216Metric, symbol Device:LED
- removed J1: Screw_Terminal_01x08, Connector_JST:JST_PH_B8B-PH-K_1x08_P2.00mm_Vertical, symbol Connector:Screw_Terminal_01x08
- removed J13: Screw_Terminal_01x03, Connector_JST:JST_PH_B3B-PH-K_1x03_P2.00mm_Vertical, symbol Connector:Screw_Terminal_01x03
- removed R1, R10, R12, R14, R4, R6, R8: R_Small_US, Resistor_SMD:R_0805_2012Metric_Pad1.20x1.40mm_HandSolder, symbol Device:R_Small_US
- removed octo1, octo2, octo3, octo4, octo5, octo6, octo7: PC817, Connector_Molex:Molex_Pico-EZmate_Slim_202656-0021_1x02-1MP_P1.20mm_Vertical, symbol 2026-01-23_00-22-03:PC817
- added C7: .1 µF, Capacitor_SMD:C_0805_2012Metric, symbol Device:C
- added H3, H4: MountingHole, MountingHole:MountingHole_2.5mm, symbol Mechanical:MountingHole
- added J2: Screw_Terminal_01x04, Connector_JST:JST_PH_B4B-PH-K_1x04_P2.00mm_Vertical, symbol Connector:Screw_Terminal_01x04
- added J3: Screw_Terminal_01x06, Connector_JST:JST_PH_B6B-PH-K_1x06_P2.00mm_Vertical, symbol Connector:Screw_Terminal_01x06
- added R1: 27000, Resistor_SMD:R_0805_2012Metric, symbol Device:R_US
- added R10, R12, R14, R4, R6, R8: 10000, Resistor_SMD:R_0805_2012Metric, symbol Device:R_US
- J15: footprint Connector:Tag-Connect_TC2050-IDC-FP_2x05_P1.27mm_Vertical -> Connector_PinSocket_2.54mm:PinSocket_2x05_P2.54mm_Vertical
- J7: footprint Connector_JST:JST_PH_B3B-PH-K_1x03_P2.00mm_Vertical -> Connector_AMASS:AMASS_XT30U-F_1x02_P5.0mm_Vertical
- R11, R13, R3, R5, R7, R9: value R_US -> 27000
- R2: value R_US -> 10000
- SW1: footprint pleseowrk:switch -> work:switch
- SW2: footprint switch:SW_219-3LPSTR -> 3switch:219-3LPSTR
- U9: footprint pleseowrk:voltageregulator -> voltage_regulator:CONV_TSR_1-2450
Connections:
- net dis5 is gone; now on net l1: U1.26 (A12)
- net dis6 is gone; now on net PWMA: U1.27 (A13)
- net dis7 is gone; now on net switch2: U1.20 (A6)
- net dis8 is gone; now on net switch1: U1.21 (A7)
- net +12V: now also C7.1
- net +5V: now also J2.4 (Pin_4), J3.1 (Pin_1)
- net GND: now also R2.2, C7.2, J2.1 (Pin_1), J3.2 (Pin_2), R10.2, R12.2, R14.2, R4.2, R6.2, R8.2
- net OM1: now also U1.23 (A9), R1.2; no longer om1.3 (Pin_3)
- net OM2: now also R3.2, U1.22 (A8), R4.1; no longer R3.1, om2.3 (Pin_3)
- net OM3: now also R5.2, U1.0 (RX1), R6.1; no longer R5.1, om3.3 (Pin_3)
- net OM4: now also R7.2, U1.3 (LRCLK2), R8.1; no longer R7.1, om4.3 (Pin_3)
- net OM5: now also R9.2, U1.33 (MCLK2), R10.1; no longer R9.1, om5.3 (Pin_3)
- net OM6: now also R11.2, U1.34 (RX8), R12.1; no longer R11.1, om6.3 (Pin_3)
- net OM7: now also R13.2, U1.32 (OUT1B), R14.1; no longer R13.1, om7.3 (Pin_3)
- net PWMB: now also U1.28 (RX7)
- net ado: now also U1.39 (A15), J3.5 (Pin_5)
- net dis3: no longer U1.24 (A10)
- net dis4: no longer U1.25 (A11)
- net int: now also U1.38 (A14), J3.6 (Pin_6)
- net l1: no longer U1.41 (A17)
- net l2: now also U1.1 (TX1); no longer U1.40 (A16)
- net l3: now also U1.2 (OUT2); no longer U1.39 (A15)
- net l4: now also U1.8 (TX2); no longer U1.38 (A14)
- net scl: now also U1.41 (A17), J3.3 (Pin_3)
- net sda: now also U1.40 (A16), J3.4 (Pin_4)
- net start: now also U1.10 (CS1); no longer U1.13 (SCK)
- net switch3: now also U1.19 (A5)
- net dis1: no longer names the net of U1.14 (A0)
- net dis2: no longer names the net of U1.15 (A1)
- new net: R13.1, om7.3 (Pin_3)
- new net: R9.1, om5.3 (Pin_3)
- new net: R7.1, om4.3 (Pin_3)
- new net: R3.1, om2.3 (Pin_3)
- new net: R5.1, om3.3 (Pin_3)
- new net: R11.1, om6.3 (Pin_3)
- new net: R1.1, om1.3 (Pin_3)
- new net receiver: J2.3 (Pin_3), U1.25 (A11)
- new net transmitter: J2.2 (Pin_2), U1.24 (A10)
- no-connect marks 39 -> 29
Other:
- note added: "note: omron, line - digital analog - analog"
- note added: "to do: add labels to microcontroller finalize motor driver connection"
- note removed: "to do: add labels to microcontroller"
- moved on the sheet: C1, C12, C13, H1, H2, J14, J15, J21, om1
