File: 3kg/Ferrarii-2026/Control_Board/Control_Board.kicad_pcb (KiCad board)
At the start: 2 copper layers, 24 parts, among them J1 Left Signal Bus, J2 Start Module, J3 Optional Back Diffusion, J4 Right Signal Bus, J5 Screw_Terminal_01x10, U1 AMS1117-5.0

Commit message: added edge cuts
Parts:
- moved BT1 169.5 mm to (-69.3, 80.4)
- moved J1 169.5 mm to (-17.9, 107.4)
- moved J2 169.5 mm to (-18.4, 158.6)
- moved J3 169.5 mm to (-7.76, 157.2)
- moved J4 169.5 mm to (-17.9, 113.9)
- moved J5 169.5 mm to (-71.2, 104.3)
- moved R1 169.5 mm to (-18.1, 119.4)
- moved R10 169.5 mm to (-12.5, 129.3)
- moved R11 169.5 mm to (-12.5, 132.7)
- moved R12 169.5 mm to (-12.5, 136.0)
- moved R13 169.5 mm to (-6.89, 119.4)
- moved R14 169.5 mm to (-6.89, 122.7)
- moved R15 169.5 mm to (-6.89, 126.0)
- moved R16 169.5 mm to (-6.89, 129.3)
- moved R2 169.5 mm to (-18.1, 122.7)
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Other:
- board outline added: 174 x 109 mm
- board text added: "Motor Driver"

Commit message: new dxf (screw holes) for pcb edge cuts
Parts:
- J5: value Screw_Terminal_01x10 -> uLCD Screen
- moved J4 223.6 mm to (197.5, 54.0), turned to 90 degrees
- moved R11 214.1 mm to (181.0, 41.0)
- moved R15 212.1 mm to (187.0, 40.2)
- moved R10 210.6 mm to (175.0, 33.5)
- moved R13 208.8 mm to (194.0, 62.5)
- moved R14 208.0 mm to (181.0, 33.5)
- moved R12 205.4 mm to (173.5, 49.0)
- moved R9 204.3 mm to (181.5, 62.0)
- moved R16 203.1 mm to (179.5, 48.5)
- moved BT1 171.8 mm to (102.0, 94.0)
- moved J2 168.4 mm to (119.5, 62.0), turned to 180 degrees
- moved J3 146.9 mm to (136.5, 129.4)
- moved J5 132.9 mm to (61.5, 97.5)
- moved R1 116.6 mm to (64.0, 36.7)
- moved R2 116.6 mm to (64.0, 40.0)
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Other:
- outline, holes or cut-outs redrawn

Commit message: added some stuff
Parts:
- added U2: 1101M2S3CQE2, 1101:1101M2S3CQE2, F.Cu at (151.0, 114.0)
- BT1: footprint Connector_AMASS:AMASS_XT30PW-M_1x02_P2.50mm_Horizontal -> Connector_AMASS:AMASS_XT30U-M_1x02_P5.0mm_Vertical
- J1, J3, J4: moved to B.Cu
- J5: value uLCD Screen -> Screw_Terminal_01x10
- moved U1 66.9 mm to (50.0, 76.0)
- moved BT1 56.4 mm to (157.0, 106.5), turned to 90 degrees
- moved J2 47.4 mm to (130.9, 108.0), turned to 0 degrees
- moved J3 19.7 mm to (119.0, 120.5), turned to 180 degrees

Commit message: changes
Parts:
- removed U1: AMS1117-5.0, Package_TO_SOT_SMD:SOT-223-3_TabPin2
- added J6: Conn_01x04, Connector_PinHeader_2.54mm:PinHeader_1x04_P2.54mm_Vertical, F.Cu at (65.3, 75.7)
- added J7: Conn_01x04, Connector_PinHeader_2.54mm:PinHeader_1x04_P2.54mm_Vertical, F.Cu at (158.3, 99.7)
- added J8: Conn_02x05_Top_Bottom, Connector_PinHeader_2.54mm:PinHeader_2x05_P2.54mm_Vertical, F.Cu at (213.8, 41.6)
- added U3: TSR1-2450E, Converter_DCDC:Converter_DCDC_TRACO_TSR1-xxxxE_THT, F.Cu at (24.4, 115.2)
- moved R1 39.1 mm to (25.2, 32.0)
- moved R2 39.1 mm to (25.2, 35.3)
- moved R3 39.1 mm to (24.2, 43.0)
- moved R4 39.1 mm to (24.2, 46.3)
- moved R5 39.1 mm to (21.2, 55.5)
- moved R6 39.1 mm to (21.2, 58.8)
- moved R13 31.4 mm to (168.0, 45.0)
- moved J5 29.5 mm to (32.4, 92.8)
- moved R7 29.5 mm to (35.4, 70.8)
- moved R8 29.5 mm to (35.4, 75.8)
- moved R9 23.2 mm to (163.0, 48.0)
- moved BT1 5.67 mm to (151.3, 106.0)
- moved U2 2.95 mm to (152.8, 116.3)
- moved J2 2.46 mm to (133.3, 107.3)
Connections:
- U2 pad 1: unconnected-(U2-Pad1) -> +12V
- U2 pad 2: unconnected-(U2-Pad2) -> +12V
Other:
- outline, holes or cut-outs redrawn
- board text added: "LED's here???"

Commit message: basic routing, gnd planes
Parts:
- J5: value Screw_Terminal_01x10 -> LCD Screen
- J6: value Conn_01x04 -> Left Encoder
- J7: value Conn_01x04 -> Right Encoder
- J8: value Conn_02x05_Top_Bottom -> Motor Control Pins
- R10, R11, R12, R13, R14, R15, R16, R9: moved to B.Cu
- moved U3 118.9 mm to (142.3, 100.7)
- moved J8 98.9 mm to (115.8, 55.2)
- moved R5 98.3 mm to (118.4, 40.8)
- moved R3 94.2 mm to (118.4, 44.8)
- moved R2 94.1 mm to (118.3, 48.8)
- moved R6 91.4 mm to (110.9, 40.8)
- moved R7 89.7 mm to (118.4, 36.8)
- moved R1 87.2 mm to (110.8, 48.8)
- moved R4 86.7 mm to (111.0, 44.8)
- moved R8 85.0 mm to (110.9, 36.8)
- moved J5 32.1 mm to (64.3, 95.8)
- moved R9 19.5 mm to (175.8, 33.3), turned to 180 degrees
- moved R13 19.4 mm to (183.4, 33.3), turned to 180 degrees
- moved J4 17.7 mm to (196.8, 36.3), turned to -90 degrees
- moved J1 17.2 mm to (73.8, 40.3), turned to -90 degrees
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Connections:
- A1 pad D0: ULCD Tx -> Teensy Rx -> R_EN_B
- A1 pad D1: ULCD Rx -> Teensy Tx -> R_EN_A
- A1 pad D10: unconnected-(A1-(CS)D10-PadD10) -> MOTOR_B_PWM
- A1 pad D11: unconnected-(A1-(SDO)D11-PadD11) -> MOTOR_B_IN1
- A1 pad D12: unconnected-(A1-(SDI)D12-PadD12) -> MOTOR_B_IN2
- A1 pad D13: unconnected-(A1-(CLK)D13-PadD13) -> L_EN_A
- A1 pad D14: unconnected-(A1-A0-PadD14) -> L_EN_B
- A1 pad D16: R_Diffusion_90_MCU -> MOTOR_A_IN2
- A1 pad D17: R_Diffusion_60_MCU -> MOTOR_A_IN1
- A1 pad D18: R_Diffusion_30_MCU -> MOTOR_A_PWM
- A1 pad D19: Back Diffusion MCU -> ULCD RST
- A1 pad D2: ULCD RST -> unconnected-(A1-PadD2)
- A1 pad D20: TR_LN_2 -> ULCD Rx -> Teensy Tx
- A1 pad D21: TR_LN_1 -> ULCD Tx -> Teensy Rx
- A1 pad D22: BR_LN_2 -> unconnected-(A1-A8-PadD22)
- A1 pad D23: BR_LN_1 -> unconnected-(A1-A9-PadD23)
- A1 pad D24: BL_LN_1 -> BR_LN_1
- A1 pad D25: BL_LN_2 -> BR_LN_2
- A1 pad D26: TL_LN_1 -> TR_LN_1
- A1 pad D27: TL_LN_2 -> TR_LN_2
- A1 pad D28: Front Diffusion MCU -> Back Diffusion MCU
- A1 pad D29: L_Diffusion_30_MCU -> R_Diffusion_30_MCU
- A1 pad D30: L_Diffusion_60_MCU -> R_Diffusion_60_MCU
- A1 pad D31: L_Diffusion_90_MCU -> R_Diffusion_90_MCU
- A1 pad D33: Start_Module_Signal -> Front Diffusion MCU
- A1 pad D34: unconnected-(A1-PadD34) -> L_Diffusion_30_MCU
- A1 pad D35: unconnected-(A1-PadD35) -> L_Diffusion_60_MCU
- A1 pad D36: unconnected-(A1-PadD36) -> L_Diffusion_90_MCU
- A1 pad D38: unconnected-(A1-A14-PadD38) -> TL_LN_2
- A1 pad D39: unconnected-(A1-A15-PadD39) -> TL_LN_1
- A1 pad D40: unconnected-(A1-A16-PadD40) -> BL_LN_2
- A1 pad D41: unconnected-(A1-A17-PadD41) -> BL_LN_1
- A1 pad D9: unconnected-(A1-PadD9) -> Start_Module_Signal
- BT1 pad 1: +12V -> +12V_BAT
- J3 pad 2: Back_Diffusion -> Back Diffusion
- J4 pad 4: Back_Diffusion -> Back Diffusion
- J8 pad 1: unconnected-(J8-Pin_1-Pad1) -> GND
- J8 pad 2: unconnected-(J8-Pin_2-Pad2) -> MOTOR_A_IN2
- J8 pad 3: unconnected-(J8-Pin_3-Pad3) -> MOTOR_A_IN1
- J8 pad 4: unconnected-(J8-Pin_4-Pad4) -> MOTOR_A_PWM
- J8 pad 5: unconnected-(J8-Pin_5-Pad5) -> +5V
- J8 pad 7: unconnected-(J8-Pin_7-Pad7) -> MOTOR_B_IN2
- J8 pad 8: unconnected-(J8-Pin_8-Pad8) -> MOTOR_B_IN1
- J8 pad 9: unconnected-(J8-Pin_9-Pad9) -> MOTOR_B_PWM
- U2 pad 2: +12V -> +12V_BAT
Routing:
- net +12V: track 0.00 -> 330.8 mm
- net +5V: track 0.00 -> 236.8 mm
- net Back Diffusion: track 0.00 -> 152.5 mm
- net BL_LN_1: track 0.00 -> 138.2 mm
- net BL_LN_2: track 0.00 -> 129.2 mm
- net TL_LN_1: track 0.00 -> 119.4 mm
- net TL_LN_2: track 0.00 -> 109.9 mm
- net BR_LN_2: track 0.00 -> 91.3 mm
- net BR_LN_1: track 0.00 -> 90.8 mm
- net TR_LN_1: track 0.00 -> 89.9 mm
- net TR_LN_2: track 0.00 -> 89.7 mm
- net R_Diffusion_90_MCU: track 0.00 -> 81.4 mm
- net R_Diffusion_60_MCU: track 0.00 -> 80.7 mm
- net Back Diffusion MCU: track 0.00 -> 80.0 mm
- net R_Diffusion_30_MCU: track 0.00 -> 79.8 mm
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- added copper zone on B.Cu, net GND
- added copper zone on F.Cu, net GND
Other:
- outline, holes or cut-outs redrawn
- board text removed: "LED's here???"

Commit message: changed some things
Routing:
- removed copper zone on B.Cu, net GND
- removed copper zone on F.Cu, net GND
Other:
- outline, holes or cut-outs redrawn
Changed lines of the file:
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@@
 		(allow_soldermask_bridges_in_footprints no)
 		(tenting front back)
-		(grid_origin 177.85 75.76571)
+		(grid_origin 90.300006 127.542594)
 		(pcbplotparams
 			(layerselection 0x00000000_00000000_55555555_5755f5ff)
@@
 		(layer "Edge.Cuts")
 	)
+	(gr_circle
+		(center 90.275 86.125)
+		(end 90.275 84.525)
+		(stroke
+			(width 0.2)
+			(type solid)
+		)
+		(fill no)
+		(layer "Edge.Cuts")
+	)
 	(gr_line
 		(start 177.85 75.76571)
@@
 		(layer "Edge.Cuts")
 	)
+	(gr_circle
+		(center 90.300006 127.542594)
+		(end 90.300006 125.942594)
+		(stroke
+			(width 0.2)
+			(type solid)
+		)
+		(fill no)
+		(layer "Edge.Cuts")
+	)
+	(gr_circle
+		(center 174.725006 33.542594)
+		(end 174.725006 31.942594)
+		(stroke
+			(width 0.2)
+			(type solid)
+		)
+		(fill no)
+		(layer "Edge.Cuts")
+	)
 	(gr_arc
 		(start 79.7 63.499999)
@@
 		(layer "Edge.Cuts")
 	)
-	(gr_circle
-		(center 90.325 89.5)
-		(end 92.075 89.5)
-		(stroke
-			(width 0.2)
-			(type default)
-		)
-		(fill no)
-		(layer "Edge.Cuts")
-	)
 	(gr_line
 		(start 85.649999 104.042589)
@@
 		(layer "Edge.Cuts")
 	)
-	(gr_circle
-		(center 174.675 73.5)
-		(end 176.425 73.5)
-		(stroke
-			(width 0.2)
-			(type default)
-		)
-		(fill no)
-		(layer "Edge.Cuts")
-	)
 	(gr_arc
 		(start 162 133.542589)
@@
 	)
 	(gr_line
-		(start 101.499999 78)
-		(end 88.650001 78)
+		(start 101.499998 83)
+		(end 88.65 83)
 		(stroke
 			(width 0.2)
@@
 		(layer "Edge.Cuts")
 	)
-	(gr_circle
-		(center 90.325 127.770593)
-		(end 92.075 127.770593)
-		(stroke
-			(width 0.2)
-			(type default)
-		)
-		(fill no)
-		(layer "Edge.Cuts")
-	)
 	(gr_line
 		(start 162 133.542589)
@@
 	)
 	(gr_arc
-		(start 87.15 79.500001)
-		(mid 87.58934 78.43934)
-		(end 88.650001 78)
-		(stroke
-			(width 0.2)
-			(type default)
-		)
-		(layer "Edge.Cuts")
-	)
-	(gr_arc
 		(start 79.7 37.54259)
 		(mid 80.139344 36.481936)
@@
 	)
 	(gr_line
-		(start 87.15 79.500001)
+		(start 87.150001 84.5)
 		(end 87.15 92.542588)
 		(stroke
@@
 	(gr_line
 		(start 103 37.54259)
-		(end 103 76.499999)
+		(end 103 81.5)
 		(stroke
 			(width 0.2)
@@
 		(layer "Edge.Cuts")
 	)
+	(gr_circle
+		(center 174.725 74.14071)
+		(end 174.725 72.54071)
+		(stroke
+			(width 0.2)
+			(type solid)
+		)
+		(fill no)
+		(layer "Edge.Cuts")
+	)
+	(gr_arc
+		(start 87.150001 84.5)
+		(mid 87.589341 83.43934)
+		(end 88.650001 83)
+		(stroke
+			(width 0.2)
+			(type solid)
+		)
+		(layer "Edge.Cuts")
+	)
 	(gr_line
 		(start 85.649999 94.042589)
@@
 	)
 	(gr_arc
-		(start 103 76.499999)
-		(mid 102.56066 77.56066)
-		(end 101.499999 78)
+		(start 102.999998 81.5)
+		(mid 102.560658 82.56066)
+		(end 101.499998 83)
 		(stroke
 			(width 0.2)
@@
 		(net 59)
 	)
-	(zone
-		(net 29)
-		(net_name "GND")
-		(layers "F.Cu" "B.Cu")
-		(hatch edge 0.5)
-		(connect_pads yes
-			(clearance 0.5)
-		)
-		(min_thickness 0.25)
-		(filled_areas_thickness no)
-		(fill yes
-			(thermal_gap 0.5)
-			(thermal_bridge_width 0.5)
-		)
-		(polygon
-			(pts
-				(xy 161.35 134.26571) (xy 161.35 77.26571) (xy 177.85 64.26571) (xy 217.85 64.26571) (xy 217.85 27.26571)
-				(xy 46.35 27.26571) (xy 46.35 103.26571) (xy 86.85 103.26571) (xy 87.85 104.76571) (xy 87.85 124.26571)
-				(xy 87.85 134.26571) (xy 91.85 134.26571) (xy 92.85 134.26571)
-			)
-		)
-	)
 	(embedded_fonts no)

Commit message: main routing and updates
Parts:
- added D1: ~, LED_SMD:LED_1206_3216Metric, F.Cu at (116.6, 28.7)
- added D10: ~, LED_SMD:LED_1206_3216Metric, F.Cu at (109.3, 55.1)
- added D11: ~, LED_SMD:LED_1206_3216Metric, F.Cu at (109.3, 59.6)
- added D12: ~, LED_SMD:LED_1206_3216Metric, F.Cu at (109.3, 64.0)
- added D13: ~, LED_SMD:LED_1206_3216Metric, F.Cu at (109.3, 68.5)
- added D2: ~, LED_SMD:LED_1206_3216Metric, F.Cu at (110.9, 30.0)
- added D3: ~, LED_SMD:LED_1206_3216Metric, F.Cu at (107.3, 34.1)
- added D4: ~, LED_SMD:LED_1206_3216Metric, F.Cu at (106.0, 39.5)
- added D5: ~, LED_SMD:LED_1206_3216Metric, F.Cu at (116.6, 40.8)
- added D6: ~, LED_SMD:LED_1206_3216Metric, F.Cu at (121.9, 30.0)
- added D7: ~, LED_SMD:LED_1206_3216Metric, F.Cu at (125.7, 34.1)
- added D8: ~, LED_SMD:LED_1206_3216Metric, F.Cu at (127.1, 39.3)
- added D9: ~, LED_SMD:LED_1206_3216Metric, F.Cu at (143.4, 130.3)
- added R17: 3.9K, Resistor_SMD:R_1206_3216Metric, B.Cu at (113.8, 118.0)
- added R18: 10K, Resistor_SMD:R_1206_3216Metric, B.Cu at (118.8, 118.0)
- added R19: 1K, Resistor_SMD:R_1206_3216Metric, F.Cu at (74.4, 28.8)
- added R20: 1K, Resistor_SMD:R_1206_3216Metric, F.Cu at (74.4, 31.9)
- added R21: 1K, Resistor_SMD:R_1206_3216Metric, F.Cu at (74.4, 35.0)
- added R22: 1K, Resistor_SMD:R_1206_3216Metric, F.Cu at (74.4, 38.2)
- added R23: 1K, Resistor_SMD:R_1206_3216Metric, F.Cu at (168.3, 39.0)
- added R24: 1K, Resistor_SMD:R_1206_3216Metric, F.Cu at (168.6, 29.1)
- added R25: 1K, Resistor_SMD:R_1206_3216Metric, F.Cu at (168.6, 32.6)
- added R26: 1K, Resistor_SMD:R_1206_3216Metric, F.Cu at (168.5, 35.8)
- added R27: 10K, Resistor_SMD:R_1206_3216Metric, F.Cu at (143.4, 127.2)
- added R28: 2.2K, Resistor_SMD:R_1206_3216Metric, F.Cu at (136.8, 127.3)
- added R29: 1K, Resistor_SMD:R_1206_3216Metric, F.Cu at (136.8, 130.3)
- added R30: 1K, Resistor_SMD:R_1206_3216Metric, F.Cu at (113.9, 114.5)
- added R31: 1K, Resistor_SMD:R_1206_3216Metric, F.Cu at (114.0, 111.1)
- added R32: 1K, Resistor_SMD:R_1206_3216Metric, F.Cu at (113.9, 107.7)
- added R33: 1K, Resistor_SMD:R_1206_3216Metric, F.Cu at (113.9, 104.4)
- added SW1: BTN1, Button_Switch_THT:SW_PUSH-12mm, F.Cu at (92.0, 105.0)
- added SW2: BTN1, Button_Switch_THT:SW_PUSH-12mm, F.Cu at (92.0, 119.6)
- added SW3: SW_DIP_x03, Button_Switch_THT:SW_DIP_SPSTx03_Slide_6.7x9.18mm_W7.62mm_P2.54mm_LowProfile, F.Cu at (120.1, 49.2)
- J6: footprint Connector_PinHeader_2.54mm:PinHeader_1x04_P2.54mm_Vertical -> Connector_PinHeader_1.00mm:PinHeader_1x04_P1.00mm_Vertical_SMD_Pin1Left
- moved J8 98.0 mm to (213.8, 51.0)
- moved R3 53.1 mm to (65.5, 39.3)
- moved R5 53.1 mm to (65.5, 35.6)
- moved R2 53.1 mm to (65.5, 43.0)
- moved R7 53.1 mm to (65.5, 31.9)
- moved R4 51.7 mm to (59.5, 39.3)
- moved R1 51.7 mm to (59.5, 43.0)
- moved R6 51.6 mm to (59.6, 35.6)
- moved R8 51.5 mm to (59.6, 31.9)
- moved J6 49.3 mm to (108.8, 49.9)
- moved J1 23.4 mm to (50.8, 36.3)
- moved R9 8.26 mm to (183.8, 35.2)
- moved R10 8.14 mm to (183.9, 45.5)
- moved R11 8.11 mm to (183.9, 41.7)
- moved R12 8.11 mm to (183.9, 38.2)
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Connections:
- A1 pad D10: MOTOR_B_PWM -> MOTOR_B_IN1
- A1 pad D11: MOTOR_B_IN1 -> MOTOR_A_IN2
- A1 pad D13: L_EN_A -> ULCD RST
- A1 pad D14: L_EN_B -> ULCD Rx -> Teensy Tx
- A1 pad D15: unconnected-(A1-A1-PadD15) -> ULCD Tx -> Teensy Rx
- A1 pad D16: MOTOR_A_IN2 -> L_EN_A
- A1 pad D17: MOTOR_A_IN1 -> LED_4
- A1 pad D18: MOTOR_A_PWM -> LED_3
- A1 pad D19: ULCD RST -> LED_2
- A1 pad D2: unconnected-(A1-PadD2) -> LOW_BAT
- A1 pad D20: ULCD Rx -> Teensy Tx -> LED_1
- A1 pad D21: ULCD Tx -> Teensy Rx -> BTN_1
- A1 pad D22: unconnected-(A1-A8-PadD22) -> BTN_2
- A1 pad D23: unconnected-(A1-A9-PadD23) -> +12V_BAT_MON
- A1 pad D28: Back Diffusion MCU -> R_Diffusion_90_MCU
- A1 pad D29: R_Diffusion_30_MCU -> R_Diffusion_60_MCU
- A1 pad D3: unconnected-(A1-PadD3) -> DIP_1
- A1 pad D30: R_Diffusion_60_MCU -> R_Diffusion_30_MCU
- A1 pad D31: R_Diffusion_90_MCU -> Back Diffusion MCU
- A1 pad D37: unconnected-(A1-PadD37) -> L_EN_B
- A1 pad D38: TL_LN_2 -> BL_LN_1
- A1 pad D39: TL_LN_1 -> BL_LN_2
- A1 pad D4: unconnected-(A1-PadD4) -> DIP_2
- A1 pad D40: BL_LN_2 -> TL_LN_1
- A1 pad D41: BL_LN_1 -> TL_LN_2
- A1 pad D5: unconnected-(A1-PadD5) -> DIP_3
- A1 pad D6: unconnected-(A1-PadD6) -> Start_Module_Signal
- A1 pad D7: unconnected-(A1-PadD7) -> MOTOR_A_PWM
- A1 pad D8: unconnected-(A1-PadD8) -> MOTOR_B_PWM
- A1 pad D9: Start_Module_Signal -> MOTOR_A_IN1
- J3 pad 2: Back Diffusion -> OPT_Back Diffusion
Routing:
- net Back Diffusion: track 152.5 -> 34.6 mm
- net +5V: track 236.8 -> 338.2 mm, vias 0 -> 3
- net DIP_1: track 0.00 -> 76.2 mm, vias 0 -> 1
- net Back Diffusion MCU: track 80.0 -> 152.4 mm, vias 0 -> 1
- net MOTOR_B_PWM: track 42.9 -> 113.8 mm
- net DIP_2: track 0.00 -> 70.6 mm, vias 0 -> 1
- net MOTOR_B_IN1: track 42.9 -> 112.6 mm
- net MOTOR_B_IN2: track 42.9 -> 111.9 mm
- net DIP_3: track 0.00 -> 65.6 mm, vias 0 -> 1
- net Net-(D10-A): track 0.00 -> 63.0 mm
- net MOTOR_A_PWM: track 51.0 -> 111.2 mm
- net Front Diffusion MCU: track 34.2 -> 93.5 mm
- net MOTOR_A_IN1: track 51.0 -> 110.1 mm
- net MOTOR_A_IN2: track 51.0 -> 109.1 mm
- net L_Diffusion_30_MCU: track 41.2 -> 96.9 mm
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- added copper zone on B.Cu, net GND
- added copper zone on F.Cu, net GND

Commit message: added holes fixed small issues
Parts:
- J8: moved to B.Cu
- SW1, SW2: footprint Button_Switch_THT:SW_PUSH-12mm -> Button_Switch_THT:SW_PUSH_6mm_H5mm
- moved SW2 4.88 mm to (91.5, 114.8)
- moved J8 4.76 mm to (209.0, 51.0), turned to 180 degrees
- moved SW1 1.35 mm to (91.5, 106.3)
Routing:
- net MOTOR_B_PWM: track 113.8 -> 102.8 mm
- net MOTOR_B_IN2: track 111.9 -> 101.1 mm
- net MOTOR_B_IN1: track 112.6 -> 101.8 mm
- net MOTOR_A_IN2: track 109.1 -> 104.3 mm
- net MOTOR_A_PWM: track 111.2 -> 106.4 mm
- net +5V: track 338.2 -> 333.5 mm
- net MOTOR_A_IN1: track 110.1 -> 105.5 mm
- net BTN_1: track 22.9 -> 20.7 mm
Other:
- outline, holes or cut-outs redrawn
