File: 3kg/Ferrarii-2026/Control_Board/Control_Board.kicad_sch (KiCad schematic)
At the start: 24 parts, among them J1 Left Signal Bus, J2 Start Module, J3 Optional Back Diffusion, J4 Right Signal Bus, J5 Screw_Terminal_01x10, U1 AMS1117-5.0

Commit message: added some stuff
Parts:
- added J6, J7: Conn_01x04, symbol Connector_Generic:Conn_01x04
- added U2: 1101M2S3CQE2, 1101:1101M2S3CQE2, symbol 1101:1101M2S3CQE2
- BT1: footprint Connector_AMASS:AMASS_XT30PW-M_1x02_P2.50mm_Horizontal -> Connector_AMASS:AMASS_XT30U-M_1x02_P5.0mm_Vertical
Changed lines of the file:
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@@
+	)
+	(symbol
+		(lib_id "Connector_Generic:Conn_01x04")
+		(at 207.01 81.28 0)
+		(unit 1)
+		(exclude_from_sim no)
+		(in_bom yes)
+		(on_board yes)
+		(dnp no)
+		(fields_autoplaced yes)
+		(property "Reference" "J6"
+			(at 209.55 81.2799 0)
+			(effects
+				(font
+					(size 1.27 1.27)
+				)
+				(justify left)
+			)
+		)
+		(property "Value" "Conn_01x04"
+			(at 209.55 83.8199 0)
+			(effects
+				(font
+					(size 1.27 1.27)
+				)
+				(justify left)
+			)
+		)
+		(property "Footprint" ""
+			(at 207.01 81.28 0)
+			(effects
+				(font
+					(size 1.27 1.27)
+				)
+				(hide yes)
+			)
+		)
+		(property "Datasheet" "~"
+			(at 207.01 81.28 0)
+			(effects
+				(font
+					(size 1.27 1.27)
+				)
+				(hide yes)
+			)
+		)
+		(property "Description" "Generic connector, single row, 01x04, script generated (kicad-library-utils/schlib/autogen/connector/)"
+			(at 207.01 81.28 0)
+			(effects
+				(font
+					(size 1.27 1.27)
+				)
+				(hide yes)
+			)
+		)
+		(pin "3"
+		)
+		(pin "1"
+		)
+		(pin "4"
+		)
+		(pin "2"
+		)
+		(instances
+			(project ""
+				(path "/6f2b6b32-1a1d-4cec-99d9-8e9530dcfe91"
+					(reference "J6")
+					(unit 1)
+				)
+			)
+		)
 	)
 	(symbol
@@
 			)
 		)
-		(property "Footprint" "Connector_AMASS:AMASS_XT30PW-M_1x02_P2.50mm_Horizontal"
+		(property "Footprint" "Connector_AMASS:AMASS_XT30U-M_1x02_P5.0mm_Vertical"
 			(at 34.036 190.5 90)
 			(effects
@@
 	)
 	(symbol
+		(lib_id "Connector_Generic:Conn_01x04")
+		(at 207.01 97.79 0)
+		(unit 1)
+		(exclude_from_sim no)
+		(in_bom yes)
+		(on_board yes)
+		(dnp no)
+		(fields_autoplaced yes)
+		(property "Reference" "J7"
+			(at 209.55 97.7899 0)
+			(effects
+				(font
+					(size 1.27 1.27)
+				)
+				(justify left)
+			)
+		)
+		(property "Value" "Conn_01x04"
+			(at 209.55 100.3299 0)
+			(effects
+				(font
+					(size 1.27 1.27)
+				)
+				(justify left)
+			)
+		)
+		(property "Footprint" ""
+			(at 207.01 97.79 0)
+			(effects
+				(font
+					(size 1.27 1.27)
+				)
+				(hide yes)
+			)
+		)
+		(property "Datasheet" "~"
+			(at 207.01 97.79 0)
+			(effects
+				(font
+					(size 1.27 1.27)
+				)
+				(hide yes)
+			)
+		)
+		(property "Description" "Generic connector, single row, 01x04, script generated (kicad-library-utils/schlib/autogen/connector/)"
+			(at 207.01 97.79 0)
+			(effects
+				(font
+					(size 1.27 1.27)
+				)
+				(hide yes)
+			)
+		)
+		(pin "3"
+		)
+		(pin "1"
+		)
+		(pin "4"
+		)
+		(pin "2"
+		)
+		(instances
+			(project "Control_Board"
+				(path "/6f2b6b32-1a1d-4cec-99d9-8e9530dcfe91"
+					(reference "J7")
+					(unit 1)
+				)
+			)
+		)
+	)
+	(symbol
 		(lib_id "Device:R_US")
 		(at 22.86 80.01 270)
@@
 					(unit 1)
 				)
+			)
+		)
+	)
+	(symbol
+		(lib_id "1101:1101M2S3CQE2")
+		(at 73.66 179.07 0)
+		(unit 1)
+		(exclude_from_sim no)
+		(in_bom yes)
+		(on_board yes)
+		(dnp no)
+		(fields_autoplaced yes)
+		(property "Reference" "U2"
+			(at 96.52 161.29 0)
+			(effects
+				(font
+					(size 1.524 1.524)
+				)
+			)
+		)
+		(property "Value" "1101M2S3CQE2"
+			(at 96.52 163.83 0)
+			(effects
+				(font
+					(size 1.524 1.524)
+				)
+			)
+		)
+		(property "Footprint" "1101:1101M2S3CQE2"
+			(at 73.66 179.07 0)
+			(effects
+				(font
+					(size 1.27 1.27)
+					(italic yes)
+				)
+				(hide yes)
+			)
+		)
+		(property "Datasheet" "1101M2S3CQE2"
+			(at 73.66 179.07 0)
+			(effects
+				(font
+					(size 1.27 1.27)
+					(italic yes)
+				)
+				(hide yes)
+			)
+		)
+		(property "Description" ""
+			(at 73.66 179.07 0)
+			(effects
+				(font
+					(size 1.27 1.27)
+				)
+				(hide yes)
+			)
+		)
+		(pin "3"
+		)
+		(pin "2"
+		)
+		(pin "1"
+		)
+		(instances
+			(project ""
+				(path "/6f2b6b32-1a1d-4cec-99d9-8e9530dcfe91"
+					(reference "U2")
+					(unit 1)
+				)

Commit message: changes
Parts:
- removed U1: AMS1117-5.0, Package_TO_SOT_SMD:SOT-223-3_TabPin2, symbol Regulator_Linear:AMS1117-5.0
- added J8: Conn_02x05_Top_Bottom, Connector_PinHeader_2.54mm:PinHeader_2x05_P2.54mm_Vertical, symbol Connector_Generic:Conn_02x05_Top_Bottom
- added U3: TSR1-2450E, Converter_DCDC:Converter_DCDC_TRACO_TSR1-xxxxE_THT, symbol Regulator_Switching:TSR1-2450E
- J6, J7: footprint (none) -> Connector_PinHeader_2.54mm:PinHeader_1x04_P2.54mm_Vertical
Connections:
- net +12V: now also U2.1, U2.2, U3.1 (Vin)
- net +5V: now also J6.2 (Pin_2), J7.2 (Pin_2), U3.3 (Vout)
- net GND: now also J6.4 (Pin_4), J7.4 (Pin_4), U3.2 (GND)
- net L_EN_A: now reaches J6.1 (Pin_1)
- net L_EN_B: now reaches J6.3 (Pin_3)
- net R_EN_A: now reaches J7.1 (Pin_1)
- net R_EN_B: now reaches J7.3 (Pin_3)
- no-connect marks 4 -> 5
Other:
- note added: "????"
- note added: "Encoders"
- note added: "Fuse??"
- note added: "Motor Driver"
- note added: "https://www.maxongroup.us/medias/sys_master/root/8814444412958/AV02-1046EN.pdf"
- moved on the sheet: J6, J7

Commit message: basic routing, gnd planes
Parts:
- J5: value Screw_Terminal_01x10 -> LCD Screen
- J6: value Conn_01x04 -> Left Encoder
- J7: value Conn_01x04 -> Right Encoder
- J8: value Conn_02x05_Top_Bottom -> Motor Control Pins
Connections:
- net Back_Diffusion is gone; now on net Back Diffusion: J3.2 (Pin_2), J4.4 (Pin_4)
- net +12V: no longer BT1.1 (+), U2.2
- net +5V: now also J8.5 (Pin_5)
- net BL_LN_1: now also A1.D41 (A17); no longer A1.D24 (A10)
- net BL_LN_2: now also A1.D40 (A16); no longer A1.D25 (A11)
- net BR_LN_1: now also A1.D24 (A10); no longer A1.D23 (A9)
- net BR_LN_2: now also A1.D25 (A11); no longer A1.D22 (A8)
- net Back Diffusion MCU: now also A1.D28; no longer A1.D19 (A5)
- net Front Diffusion MCU: now also A1.D33; no longer A1.D28
- net GND: now also J8.1 (Pin_1)
- net L_Diffusion_30_MCU: now also A1.D34; no longer A1.D29
- net L_Diffusion_60_MCU: now also A1.D35; no longer A1.D30
- net L_Diffusion_90_MCU: now also A1.D36; no longer A1.D31
- net L_EN_A: now also A1.D13 ((CLK)D13)
- net L_EN_B: now also A1.D14 (A0)
- net R_Diffusion_30_MCU: now also A1.D29; no longer A1.D18 (A4)
- net R_Diffusion_60_MCU: now also A1.D30; no longer A1.D17 (A3)
- net R_Diffusion_90_MCU: now also A1.D31; no longer A1.D16 (A2)
- net R_EN_A: now also A1.D1 ((CTX1)D1)
- net R_EN_B: now also A1.D0 ((CRX1)D0)
- net Start_Module_Signal: now also A1.D9; no longer A1.D33
- net TL_LN_1: now also A1.D39 (A15); no longer A1.D26 (A12)
- net TL_LN_2: now also A1.D38 (A14); no longer A1.D27 (A13)
- net TR_LN_1: now also A1.D26 (A12); no longer A1.D21 (A7)
- net TR_LN_2: now also A1.D27 (A13); no longer A1.D20 (A6)
- net ULCD RST: now also A1.D19 (A5); no longer A1.D2
- net ULCD Rx -> Teensy Tx: now also A1.D20 (A6); no longer A1.D1 ((CTX1)D1)
- net ULCD Tx -> Teensy Rx: now also A1.D21 (A7); no longer A1.D0 ((CRX1)D0)
- net MOTOR_B_PWM: now reaches A1.D10 ((CS)D10)
- net MOTOR_B_PWM: now also J8.9 (Pin_9)
- net MOTOR_B_IN1: now reaches A1.D11 ((SDO)D11)
- net MOTOR_B_IN1: now also J8.8 (Pin_8)
- net MOTOR_B_IN2: now reaches A1.D12 ((SDI)D12)
- net MOTOR_B_IN2: now also J8.7 (Pin_7)
- net MOTOR_A_IN2: now reaches J8.2 (Pin_2)
- net MOTOR_A_IN2: now also A1.D16 (A2)
- net MOTOR_A_IN1: now reaches J8.3 (Pin_3)
- net MOTOR_A_IN1: now also A1.D17 (A3)
- net MOTOR_A_PWM: now reaches J8.4 (Pin_4)
- net MOTOR_A_PWM: now also A1.D18 (A4)
- new net +12V_BAT: BT1.1 (+), U2.2
- no-connect marks 5 -> 7
Other:
- note removed: "????"
- note removed: "Motor Driver"
- moved on the sheet: J8

Commit message: changed some things
Other:
- note added: "https://www.maxongroup.us/medias/sys_master/ root/8814444412958/AV02-1046EN.pdf"
- note removed: "https://www.maxongroup.us/medias/sys_master/root/8814444412958/AV02-1046EN.pdf"
- moved on the sheet: A1, BT1, J2, J3, J4, J5, J6, J7, J8, U2, U3

Commit message: main routing and updates
Parts:
- added D1, D10, D11, D12, D13, D2, D3, D4, D5, D6, D7, D8, D9: ~, LED_SMD:LED_1206_3216Metric, symbol Device:LED
- added R17: 3.9K, Resistor_SMD:R_1206_3216Metric, symbol Device:R_US
- added R18, R27: 10K, Resistor_SMD:R_1206_3216Metric, symbol Device:R_US
- added R19, R20, R21, R22, R23, R24, R25, R26, R29, R30, R31, R32, R33: 1K, Resistor_SMD:R_1206_3216Metric, symbol Device:R_US
- added R28: 2.2K, Resistor_SMD:R_1206_3216Metric, symbol Device:R_US
- added SW1, SW2: BTN1, Button_Switch_THT:SW_PUSH-12mm, symbol Switch:SW_Push
- added SW3: SW_DIP_x03, Button_Switch_THT:SW_DIP_SPSTx03_Slide_6.7x9.18mm_W7.62mm_P2.54mm_LowProfile, symbol Switch:SW_DIP_x03
- J6: footprint Connector_PinHeader_2.54mm:PinHeader_1x04_P2.54mm_Vertical -> Connector_PinHeader_1.00mm:PinHeader_1x04_P1.00mm_Vertical_SMD_Pin1Left
Connections:
- net +12V_BAT: now also R27.2
- net BL_LN_1: now also A1.D38 (A14); no longer A1.D41 (A17)
- net BL_LN_2: now also A1.D39 (A15); no longer A1.D40 (A16)
- net Back Diffusion: now also R23.1; no longer J3.2 (Pin_2)
- net Back Diffusion MCU: now also A1.D31, R17.1, R18.2; no longer A1.D28
- net Front Diffusion: now also R19.1
- net GND: now also D1.1 (K), D10.1 (K), D11.1 (K), D12.1 (K), D13.1 (K), D2.1 (K), D3.1 (K), D4.1 (K), D5.1 (K), D6.1 (K), D7.1 (K), D8.1 (K), D9.1 (K), R17.2, R28.1, SW1.1, SW2.1, SW3.4, SW3.5, SW3.6
- net L_Diffusion_30: now also R20.1
- net L_Diffusion_60: now also R21.1
- net L_Diffusion_90: now also R22.1
- net L_EN_A: now also A1.D16 (A2); no longer A1.D13 ((CLK)D13)
- net L_EN_B: now also A1.D37; no longer A1.D14 (A0)
- net MOTOR_A_IN1: now also A1.D9; no longer A1.D17 (A3)
- net MOTOR_A_IN2: now also A1.D11 ((SDO)D11); no longer A1.D16 (A2)
- net MOTOR_A_PWM: now also A1.D7; no longer A1.D18 (A4)
- net MOTOR_B_IN1: now also A1.D10 ((CS)D10); no longer A1.D11 ((SDO)D11)
- net MOTOR_B_PWM: now also A1.D8; no longer A1.D10 ((CS)D10)
- net R_Diffusion_30: now also R24.1
- net R_Diffusion_30_MCU: now also A1.D30; no longer A1.D29
- net R_Diffusion_60: now also R25.1
- net R_Diffusion_60_MCU: now also A1.D29; no longer A1.D30
- net R_Diffusion_90: now also R26.1
- net R_Diffusion_90_MCU: now also A1.D28; no longer A1.D31
- net Start_Module_Signal: now also A1.D6; no longer A1.D9
- net TL_LN_1: now also A1.D40 (A16); no longer A1.D39 (A15)
- net TL_LN_2: now also A1.D41 (A17); no longer A1.D38 (A14)
- net ULCD RST: now also A1.D13 ((CLK)D13); no longer A1.D19 (A5)
- net ULCD Rx -> Teensy Tx: now also A1.D14 (A0); no longer A1.D20 (A6)
- net ULCD Tx -> Teensy Rx: now also A1.D15 (A1); no longer A1.D21 (A7)
- net LOW_BAT: now reaches A1.D2
- net LOW_BAT: now also R29.1
- net BTN_2: now reaches A1.D22 (A8)
- net BTN_2: now also SW2.2
- net +12V_BAT_MON: now reaches A1.D23 (A9)
- net +12V_BAT_MON: now also R27.1, R28.2
- net DIP_1: now reaches A1.D3
- net DIP_1: now also SW3.1
- net DIP_2: now reaches A1.D4
- net DIP_2: now also SW3.2
- net DIP_3: now reaches A1.D5
- net DIP_3: now also SW3.3
- new net: D5.2 (A), R23.2
- new net: D13.2 (A), R33.2
- new net: D3.2 (A), R21.2
- new net: D7.2 (A), R25.2
- new net: D4.2 (A), R22.2
- new net: D12.2 (A), R32.2
- new net: D1.2 (A), R19.2
- new net: D2.2 (A), R20.2
- new net: D9.2 (A), R29.2
- new net: D8.2 (A), R26.2
- new net: D10.2 (A), R30.2
- new net: D6.2 (A), R24.2
- new net: D11.2 (A), R31.2
- new net BTN_1: A1.D21 (A7), SW1.2
- new net LED_1: A1.D20 (A6), R30.1
- new net LED_2: A1.D19 (A5), R31.1
- new net LED_3: A1.D18 (A4), R32.1
- new net LED_4: A1.D17 (A3), R33.1
- new net OPT_Back Diffusion: J3.2 (Pin_2), R18.1
Other:
- moved on the sheet: J3

Commit message: added holes fixed small issues
Parts:
- SW1, SW2: footprint Button_Switch_THT:SW_PUSH-12mm -> Button_Switch_THT:SW_PUSH_6mm_H5mm
Changed lines of the file:
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@@
 			)
 		)
-		(property "Footprint" "Button_Switch_THT:SW_PUSH-12mm"
+		(property "Footprint" "Button_Switch_THT:SW_PUSH_6mm_H5mm"
 			(at 83.82 50.8 0)
 			(effects
@@
 			)
 		)
-		(property "Footprint" "Button_Switch_THT:SW_PUSH-12mm"
+		(property "Footprint" "Button_Switch_THT:SW_PUSH_6mm_H5mm"
 			(at 83.82 44.45 0)
 			(effects

Commit message: final wiring, silkscreen callouts, test points
Parts:
- added J10: BLTP2, Connector_PinHeader_1.27mm:PinHeader_1x01_P1.27mm_Vertical, symbol Connector:Screw_Terminal_01x01
- added J11: TLTP1, Connector_PinHeader_1.27mm:PinHeader_1x01_P1.27mm_Vertical, symbol Connector:Screw_Terminal_01x01
- added J12: TLTP2, Connector_PinHeader_1.27mm:PinHeader_1x01_P1.27mm_Vertical, symbol Connector:Screw_Terminal_01x01
- added J13: TRTP2, Connector_PinHeader_1.27mm:PinHeader_1x01_P1.27mm_Vertical, symbol Connector:Screw_Terminal_01x01
- added J14: TRTP1, Connector_PinHeader_1.27mm:PinHeader_1x01_P1.27mm_Vertical, symbol Connector:Screw_Terminal_01x01
- added J15: BRTP2, Connector_PinHeader_1.27mm:PinHeader_1x01_P1.27mm_Vertical, symbol Connector:Screw_Terminal_01x01
- added J16: BRTP1, Connector_PinHeader_1.27mm:PinHeader_1x01_P1.27mm_Vertical, symbol Connector:Screw_Terminal_01x01
- added J17: 3.3VTP, Connector_PinHeader_1.27mm:PinHeader_1x01_P1.27mm_Vertical, symbol Connector:Screw_Terminal_01x01
- added J18: 5VTP, Connector_PinHeader_1.27mm:PinHeader_1x01_P1.27mm_Vertical, symbol Connector:Screw_Terminal_01x01
- added J19: BMON_TP, Connector_PinHeader_1.27mm:PinHeader_1x01_P1.27mm_Vertical, symbol Connector:Screw_Terminal_01x01
- added J20: 12V TP, Connector_PinHeader_1.27mm:PinHeader_1x01_P1.27mm_Vertical, symbol Connector:Screw_Terminal_01x01
- added J21: 12VTP, Connector_PinHeader_1.27mm:PinHeader_1x01_P1.27mm_Vertical, symbol Connector:Screw_Terminal_01x01
- added J22: B1, Connector_PinHeader_1.27mm:PinHeader_1x01_P1.27mm_Vertical, symbol Connector:Screw_Terminal_01x01
- added J23: B2, Connector_PinHeader_1.27mm:PinHeader_1x01_P1.27mm_Vertical, symbol Connector:Screw_Terminal_01x01
- added J24: B_PWM, Connector_PinHeader_1.27mm:PinHeader_1x01_P1.27mm_Vertical, symbol Connector:Screw_Terminal_01x01
- added J25: A_PWM, Connector_PinHeader_1.27mm:PinHeader_1x01_P1.27mm_Vertical, symbol Connector:Screw_Terminal_01x01
- added J26: A1, Connector_PinHeader_1.27mm:PinHeader_1x01_P1.27mm_Vertical, symbol Connector:Screw_Terminal_01x01
- added J27: A2, Connector_PinHeader_1.27mm:PinHeader_1x01_P1.27mm_Vertical, symbol Connector:Screw_Terminal_01x01
- added J9: BLTP1, Connector_PinHeader_1.27mm:PinHeader_1x01_P1.27mm_Vertical, symbol Connector:Screw_Terminal_01x01
- J6: footprint Connector_PinHeader_1.00mm:PinHeader_1x04_P1.00mm_Vertical_SMD_Pin1Left -> Connector_PinHeader_2.54mm:PinHeader_1x04_P2.54mm_Vertical_SMD_Pin1Left
- renumbered D9 to LOW_BAT1, SW3 to MODE_SEL1
Connections:
- net +12V: now also J21.1 (Pin_1)
- net +12V_BAT: now also J20.1 (Pin_1)
- net +12V_BAT_MON: now also J19.1 (Pin_1)
- net +5V: now also J18.1 (Pin_1)
- net 3.3V: now also J17.1 (Pin_1)
- net BL_LN_1: now also J9.1 (Pin_1)
- net BL_LN_2: now also J10.1 (Pin_1)
- net BR_LN_1: now also J16.1 (Pin_1)
- net BR_LN_2: now also J15.1 (Pin_1)
- net MOTOR_A_IN1: now also J27.1 (Pin_1)
- net MOTOR_A_IN2: now also J26.1 (Pin_1)
- net MOTOR_A_PWM: now also J25.1 (Pin_1)
- net MOTOR_B_IN1: now also J22.1 (Pin_1)
- net MOTOR_B_IN2: now also J23.1 (Pin_1)
- net MOTOR_B_PWM: now also J24.1 (Pin_1)
- net TL_LN_1: now also J11.1 (Pin_1)
- net TL_LN_2: now also J12.1 (Pin_1)
- net TR_LN_1: now also J14.1 (Pin_1)
- net TR_LN_2: now also J13.1 (Pin_1)
Other:
- moved on the sheet: J8

Commit message: added buzz
Parts:
- added J28: GND_TP, Connector_PinHeader_1.27mm:PinHeader_1x01_P1.27mm_Vertical, symbol Connector:Screw_Terminal_01x01
Connections:
- net GND: now also J28.1 (Pin_1)
Changed lines of the file:
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@@
 	(wire
 		(pts
+			(xy 121.92 152.4) (xy 119.38 152.4)
+		)
+		(stroke
+			(width 0)
+			(type default)
+		)
+	)
+	(wire
+		(pts
 			(xy 260.35 36.83) (xy 248.92 36.83)
 		)
@@
 	(symbol
 		(lib_id "power:GND")
+		(at 121.92 152.4 0)
+		(unit 1)
+		(exclude_from_sim no)
+		(in_bom yes)
+		(on_board yes)
+		(dnp no)
+		(fields_autoplaced yes)
+		(property "Reference" "#PWR042"
+			(at 121.92 158.75 0)
+			(effects
+				(font
+					(size 1.27 1.27)
+				)
+				(hide yes)
+			)
+		)
+		(property "Value" "GND"
+			(at 121.92 157.48 0)
+			(effects
+				(font
+					(size 1.27 1.27)
+				)
+			)
+		)
+		(property "Footprint" ""
+			(at 121.92 152.4 0)
+			(effects
+				(font
+					(size 1.27 1.27)
+				)
+				(hide yes)
+			)
+		)
+		(property "Datasheet" ""
+			(at 121.92 152.4 0)
+			(effects
+				(font
+					(size 1.27 1.27)
+				)
+				(hide yes)
+			)
+		)
+		(property "Description" "Power symbol creates a global label with name \"GND\" , ground"
+			(at 121.92 152.4 0)
+			(effects
+				(font
+					(size 1.27 1.27)
+				)
+				(hide yes)
+			)
+		)
+		(pin "1"
+		)
+		(instances
+			(project ""
+				(path "/6f2b6b32-1a1d-4cec-99d9-8e9530dcfe91"
+					(reference "#PWR042")
+					(unit 1)
+				)
+			)
+		)
+	)
+	(symbol
+		(lib_id "power:GND")
 		(at 209.55 148.59 0)
 		(unit 1)
@@
 					(unit 1)
 				)
+			)
+		)
+	)
+	(symbol
+		(lib_id "Connector:Screw_Terminal_01x01")
+		(at 114.3 152.4 180)
+		(unit 1)
+		(exclude_from_sim no)
+		(in_bom yes)
+		(on_board yes)
+		(dnp no)
+		(property "Reference" "J28"
+			(at 114.046 154.94 0)
+			(effects
+				(font
+					(size 1.27 1.27)
+				)
+			)
+		)
+		(property "Value" "GND_TP"
+			(at 114.046 157.226 0)
+			(effects
+				(font
+					(size 1.27 1.27)
+				)
+			)
+		)
+		(property "Footprint" "Connector_PinHeader_1.27mm:PinHeader_1x01_P1.27mm_Vertical"
+			(at 114.3 152.4 0)
+			(effects
+				(font
+					(size 1.27 1.27)
+				)
+				(hide yes)
+			)
+		)
+		(property "Datasheet" "~"
+			(at 114.3 152.4 0)
+			(effects
+				(font
+					(size 1.27 1.27)
+				)
+				(hide yes)
+			)
+		)
+		(property "Description" "Generic screw terminal, single row, 01x01, script generated (kicad-library-utils/schlib/autogen/connector/)"
+			(at 114.3 152.4 0)
+			(effects
+				(font
+					(size 1.27 1.27)
+				)
+				(hide yes)
+			)
+		)
+		(pin "1"
+		)
+		(instances
+			(project "Control_Board"
+				(path "/6f2b6b32-1a1d-4cec-99d9-8e9530dcfe91"
+					(reference "J28")
+					(unit 1)
+				)
