File: juan-shi/juan-shi.kicad_pcb (KiCad board)
At the start: 2 copper layers, 63.4 x 35 mm, 43 parts, among them J1 Screw3, J10 Screw_Terminal_01x02, J12 xt30, J13 Screw3, J2 Screw3, J3 Screw3, J4 Screw3, J5 Screw_Terminal_01x02, J6 Conn_01x03_Pin, J7 Screw3, J8 Screw3, J9 Conn_01x03_Pin, SW2 SW_DPDT_x2, SW3 SW_DIP_x02, U1 DRV8871DDA, U3 DRV8871DDA

Commit message: joe
Parts:
- removed R7: 1k, Resistor_SMD:R_0603_1608Metric
- added D6: LED, LED_SMD:LED_1206_3216Metric, F.Cu at (231.9, 93.9)
- added D8: LED, LED_SMD:LED_1206_3216Metric, F.Cu at (242.5, 93.3)
- added R10: 1k, Resistor_SMD:R_0603_1608Metric, B.Cu at (239.4, 93.3)
- moved R6 4.57 mm to (235.1, 92.4), turned to 0 degrees
- moved J12 1.65 mm to (247.5, 95.0)
- moved C1 1.38 mm to (229.3, 81.2)
- moved R9 1.00 mm to (199.2, 65.6)
- moved J6 0.13 mm to (203.0, 94.9)
Connections:
- A1 pad 27: +5V -> 5v
- A1 pad 30: +12V -> unconnected-(A1-VIN-Pad30)
- J7 pad 3: +5V -> +3.3V
- J8 pad 3: +5V -> +3.3V
- J9 pad 3: +5V -> 5v
- R6 pad 1: GND -> Net-(D6-A)
- R6 pad 2: DIP2 -> DIP1
- SW3 pad 1: +5V -> 5v
- SW3 pad 2: +5V -> 5v
Routing:
- net +5V: track 74.7 -> 0.00 mm, vias 2 -> 0
- net +3.3V: track 0.00 -> 54.2 mm, vias 0 -> 1
- net 5v: track 110.2 -> 149.8 mm, vias 0 -> 2
- net +12V: track 79.4 -> 67.2 mm
- net Net-(D8-A): track 0.00 -> 2.83 mm, vias 0 -> 1
- net Net-(D6-A): track 0.00 -> 2.46 mm, vias 0 -> 1
- net DIP1: track 25.8 -> 28.2 mm, vias 2 -> 1
- net S5: track 11.4 -> 12.5 mm
- net DIP2: track 26.3 -> 27.3 mm
- net Net-(D5-A): track 2.59 -> 3.54 mm
- net Net-(J12-Pin_2): track 18.9 -> 19.5 mm
Other:
- board text added: "Mk2 Designer: Joe Sung"
- board text removed: "S"
