File: juan-shi/juan-shi.kicad_sch (KiCad schematic)
At the start: 42 parts, among them J1 Screw3, J10 Screw_Terminal_01x02, J12 xt30, J13 Screw3, J2 Screw3, J3 Screw3, J4 Screw3, J5 Screw_Terminal_01x02, J6 Conn_01x03_Pin, J7 Screw3, J8 Screw3, J9 Conn_01x03_Pin, SW2 SW_DPDT_x2, SW3 SW_DIP_x02, U1 DRV8871DDA, U3 DRV8871DDA

Commit message: joe
Parts:
- removed R7: 1k, Resistor_SMD:R_0603_1608Metric, symbol Device:R_US
- added D6, D8: LED, LED_SMD:LED_1206_3216Metric, symbol Device:LED
- added R10: 1k, Resistor_SMD:R_0603_1608Metric, symbol Device:R_US
Connections:
- net +12V: no longer A1.30 (VIN)
- net +3.3V: now also J7.3 (Pin_3), J8.3 (Pin_3)
- net 5v: now also A1.27 (+5V), J9.3 (Pin_3), SW3.1, SW3.2
- net DIP1: now also R6.2
- net DIP2: now also R10.2; no longer R6.2
- net GND: now also D6.1 (K), D8.1 (K); no longer R6.1
- removed net +5V: A1.27 (+5V), J7.3 (Pin_3), J8.3 (Pin_3), J9.3 (Pin_3), SW3.1, SW3.2
- new net: D8.2 (A), R10.1
- new net: D6.2 (A), R6.1
