File: 500g/NewMemberBoard/500gNewMemberBoard.kicad_sch (KiCad schematic)
At the start: 81 parts, among them J1 USB-C Connector, J10 Conn_01x03, J11 Conn_01x03, J12 Conn_01x03, J13 Conn_01x02, J2 ICSP, J3 M1, J4 M2, J5 Conn_01x03, J6 Conn_01x03, J7 Conn_01x03, J8 Conn_01x03, J9 Conn_01x03, SW1 Reset, SW2 Button1, SW3 Power, U1 ATmega328P-A, U2 AMS1117-5.0, U3 CH340C (USB to UART), U4 DRV8871DDA, U5 DRV8871DDA, U6 AMS1117-5.0, Y2 16MHz

Commit message: added tantalum capacitors
Parts:
- C1, C2, C4, C5: footprint Capacitor_SMD:C_1206_3216Metric -> Capacitor_Tantalum_SMD:CP_EIA-3216-18_Kemet-A; symbol Device:C -> Device:C_Polarized
Changed lines of the file:
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@@
 	)
 	(symbol
-		(lib_id "Device:C")
+		(lib_id "Device:C_Polarized")
 		(at 111.76 43.18 0)
 		(mirror y)
@@
 			)
 		)
-		(property "Footprint" "Capacitor_SMD:C_1206_3216Metric"
+		(property "Footprint" "Capacitor_Tantalum_SMD:CP_EIA-3216-18_Kemet-A"
 			(at 110.7948 46.99 0)
 			(effects
@@
 			)
 		)
-		(property "Description" "Unpolarized capacitor"
+		(property "Description" "Polarized capacitor"
 			(at 111.76 43.18 0)
 			(effects
@@
 	)
 	(symbol
-		(lib_id "Device:C")
+		(lib_id "Device:C_Polarized")
 		(at 177.8 43.18 0)
 		(unit 1)
@@
 		(fields_autoplaced yes)
 		(property "Reference" "C2"
-			(at 181.61 41.9099 0)
+			(at 181.61 41.0209 0)
 			(effects
 				(font
@@
 		)
 		(property "Value" "22uF"
-			(at 181.61 44.4499 0)
+			(at 181.61 43.5609 0)
 			(effects
 				(font
@@
 			)
 		)
-		(property "Footprint" "Capacitor_SMD:C_1206_3216Metric"
+		(property "Footprint" "Capacitor_Tantalum_SMD:CP_EIA-3216-18_Kemet-A"
 			(at 178.7652 46.99 0)
 			(effects
@@
 			)
 		)
-		(property "Description" "Unpolarized capacitor"
+		(property "Description" "Polarized capacitor"
 			(at 177.8 43.18 0)
 			(effects
@@
 	)
 	(symbol
-		(lib_id "Device:C")
+		(lib_id "Device:C_Polarized")
 		(at 154.94 43.18 0)
 		(mirror y)
@@
 			)
 		)
-		(property "Footprint" "Capacitor_SMD:C_1206_3216Metric"
+		(property "Footprint" "Capacitor_Tantalum_SMD:CP_EIA-3216-18_Kemet-A"
 			(at 153.9748 46.99 0)
 			(effects
@@
 			)
 		)
-		(property "Description" "Unpolarized capacitor"
+		(property "Description" "Polarized capacitor"
 			(at 154.94 43.18 0)
 			(effects
@@
 	)
 	(symbol
-		(lib_id "Device:C")
+		(lib_id "Device:C_Polarized")
 		(at 134.62 43.18 0)
 		(unit 1)
@@
 		(fields_autoplaced yes)
 		(property "Reference" "C4"
-			(at 138.43 41.9099 0)
+			(at 138.43 41.0209 0)
 			(effects
 				(font
@@
 		)
 		(property "Value" "22uF"
-			(at 138.43 44.4499 0)
+			(at 138.43 43.5609 0)
 			(effects
 				(font
@@
 			)
 		)
-		(property "Footprint" "Capacitor_SMD:C_1206_3216Metric"
+		(property "Footprint" "Capacitor_Tantalum_SMD:CP_EIA-3216-18_Kemet-A"
 			(at 135.5852 46.99 0)
 			(effects
@@
 			)
 		)
-		(property "Description" "Unpolarized capacitor"
+		(property "Description" "Polarized capacitor"
 			(at 134.62 43.18 0)
 			(effects

Commit message: fixed USBC, updated BOM
Parts:
- added R21, R22: 4.7k, Resistor_SMD:R_0603_1608Metric, symbol Device:R_US
- added U7: USBLC6-2P6, Package_TO_SOT_SMD:SOT-666, symbol Power_Protection:USBLC6-2P6
- R8: value 1k -> 10k
- U3: value CH340C (USB to UART) -> CH340X; footprint Package_SO:SOIC-16_3.9x9.9mm_P1.27mm -> Package_SO:MSOP-10_3x3mm_P0.5mm; symbol Interface_USB:CH340C -> Interface_USB:CH340X
Connections:
- net +5V: now also U3.7 (VCC); no longer U3.16 (VCC)
- net D+: now also U3.1 (UD+), U7.4 (I/O2); no longer J1.A6 (D+), J1.B6 (D+), U3.5 (UD+)
- net D-: now also U3.2 (UD-), U7.6 (I/O1); no longer J1.A7 (D-), J1.B7 (D-), U3.6 (UD-)
- net GND: now also U3.3 (GND), R22.2, U7.2 (GND); no longer U3.1 (GND)
- net RX: now also U3.8 (TXD); no longer U3.2 (TXD)
- net TX: now also U3.9 (RXD); no longer U3.3 (RXD)
- net at C7.1: now also U3.10 (V3); no longer U3.4 (V3)
- net at C6.1, F1.2, J1.A4 (VBUS)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: now also U7.5 (VBUS)
- net at C8.1: now also U3.6 (TNOW/~{DTR}), R21.2, R22.1; no longer U3.13 (~{DTR})
- new net: R21.1, U3.5 (~{CTS})
- new net USBC_D+: J1.A6 (D+), J1.B6 (D+), U7.3 (I/O2)
- new net USBC_D-: J1.A7 (D-), J1.B7 (D-), U7.1 (I/O1)
- no-connect marks 9 -> 4
Other:
- note added: "Open Source DTR"
- note added: "Push-Pull DTR"
- moved on the sheet: C14, C15, C16, C17, C7, C8, J2, J3, J4, R10, R9, U4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
